Commit message: temporary fix for the drawers etc inside of gazebo Bones stoped moving

File: iai_kitchen/urdf/IAI_drawers.urdf.xacro (robot description, xacro)
@@ -62,5 +62,8 @@
       <child link="${name}_main"/>
       <axis xyz="1. 0. 0.0"/>
-      <limit lower="0" upper="0.48" effort="0.0300" velocity="10"/>
+      <!--
+        <limit effort="300" lower="0" upper="0.48" velocity="10"/>
+        -->
+        <limit effort="300" lower="0" upper="0" velocity="10"/>
     </joint>
     <joint name="${name}_handle_joint" type="fixed">
@@ -107,6 +110,8 @@
       <parent link="${parent}"/>
       <child link="${name}_main"/>
-      <axis xyz="1. 0. 0.0"/>
-      <limit lower="0" upper="0.48" effort="300" velocity="10"/>
+      <axis xyz="1. 0. 0.0"/><!--
+    <limit effort="300" lower="0" upper="0.48" velocity="10"/>
+    -->
+    <limit effort="300" lower="0" upper="0" velocity="10"/>
     </joint>
     <joint name="${name}_handle_joint" type="fixed">

File: iai_kitchen/urdf/IAI_fridge.urdf.xacro (robot description, xacro)
@@ -40,5 +40,8 @@
       <child link="${name}_door"/>
       <axis xyz="0 0 1"/>
+      <!--
       <limit lower="0" upper="${0.5*pi}" effort="300" velocity="10"/>
+      -->
+      <limit lower="0" upper="0" effort="300" velocity="10"/>
     </joint>
     <joint name="${name}_door_handle_joint" type="fixed">

Commit message: Drawers are able to be opened and closed. TODO oven and dishwasher doors are fixed. There is a flag that can disable this, however the gravity will pull them down

File: iai_kitchen/urdf/IAI_drawers.urdf.xacro (robot description, xacro)
@@ -62,8 +62,8 @@
       <child link="${name}_main"/>
       <axis xyz="1. 0. 0.0"/>
-      <!--
         <limit effort="300" lower="0" upper="0.48" velocity="10"/>
-        -->
+<!--
         <limit effort="300" lower="0" upper="0" velocity="10"/>
+  -->
     </joint>
     <joint name="${name}_handle_joint" type="fixed">
@@ -110,8 +110,9 @@
       <parent link="${parent}"/>
       <child link="${name}_main"/>
-      <axis xyz="1. 0. 0.0"/><!--
+      <axis xyz="1. 0. 0.0"/>
     <limit effort="300" lower="0" upper="0.48" velocity="10"/>
-    -->
+<!--
     <limit effort="300" lower="0" upper="0" velocity="10"/>
+-->
     </joint>
     <joint name="${name}_handle_joint" type="fixed">

File: iai_kitchen/urdf/IAI_fridge.urdf.xacro (robot description, xacro)
@@ -40,8 +40,8 @@
       <child link="${name}_door"/>
       <axis xyz="0 0 1"/>
-      <!--
       <limit lower="0" upper="${0.5*pi}" effort="300" velocity="10"/>
-      -->
+<!--
       <limit lower="0" upper="0" effort="300" velocity="10"/>
+-->
     </joint>
     <joint name="${name}_door_handle_joint" type="fixed">

File: iai_kitchen/urdf/IAI_fridge_area.urdf.xacro (robot description, xacro)
@@ -11,5 +11,5 @@
       <sphere_inertia radius="0" mass="0"/>
       <visual>
-	  <origin xyz="0 0 0" rpy="0 0 0" />
+	  <origin xyz="0 0 0.01" rpy="0 0 0" />
 	  <geometry>
 	    <mesh filename="package://iai_kitchen/meshes/racks/FridgeArea.dae"/>
@@ -17,5 +17,5 @@
 	</visual>
     <collision>
-        <origin xyz="0 0 0" rpy="0 0 0" />
+        <origin xyz="0 0 0.01" rpy="0 0 0" />
         <geometry>
           <mesh filename="package://iai_kitchen/meshes/collision/kitchen_fridge.stl"/>

File: iai_kitchen/urdf/IAI_kitchen.urdf.xacro (robot description, xacro)
@@ -25,5 +25,5 @@
   </xacro:if>
   <gazebo>
-      <static>true</static>
+      <static>false</static>
   </gazebo>
   <!--- FIXME THIS should NOT be here -->

File: iai_kitchen/urdf/IAI_oven.urdf.xacro (robot description, xacro)
@@ -70,8 +70,8 @@
         <child link="${name}_door"/>
         <axis xyz="0 0 1"/>
-        <!--
         <limit lower="0" upper="${0.5*pi}" effort="300" velocity="10"/>
-        -->
+<!--
         <limit lower="0" upper="0" effort="0.03" velocity="10"/>
+   -->
       </joint>
     </xacro:unless>
