Commit message: fixes to island surface position and hot plate position

File: iai_kitchen/urdf/IAI_kitchen_island.urdf.xacro (robot description, xacro)
@@ -43,5 +43,5 @@
   </link>
   <joint name="${name}_surface_joint" type="fixed">
-    <origin xyz="0.0925 0. 0.42" rpy="0 0 0" />
+    <origin xyz="0.0 0. 0.42" rpy="0 0 0" />
     <parent link="${name}"/>
     <child link="${name}_surface"/>
@@ -57,5 +57,5 @@
   </link>
   <joint name="${name}_stove_joint" type="fixed">
-    <origin xyz="0.025 0.7658 0.4315" rpy="0 0 0" />
+    <origin xyz="0.0 0.7658 0.4315" rpy="0 0 0" />
     <parent link="${name}"/>
     <child link="${name}_stove"/>
