Commit message: spoon adapted -> spoon rounded

File: iai_kitchen/urdf/spoon_rounded.urdf (robot description, URDF)
Before this commit: robot spoon_adapted, 1 links, 0 joints
Links:
- removed link spoon_adapted_frame
- added link spoon_rounded_frame; visual mesh filename=package://iai_kitchen/meshes/racks/BoxyToolholder/Holder_Sp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
