Commit message: added collisions and bounding boxes

File: iai_kitchen/urdf/IAI_fridge_area.urdf.xacro (robot description, xacro)
@@ -16,4 +16,10 @@
 	  </geometry>
 	</visual>
+    <collision>
+        <origin xyz="0 0 0" rpy="0 0 0" />
+        <geometry>
+          <mesh filename="package://iai_kitchen/meshes/collision/kitchen_fridge.stl"/>
+        </geometry>
+      </collision>
     </link>
     <joint name="${name}_footprint_joint" type="fixed">

File: iai_kitchen/urdf/IAI_kitchen_island.urdf.xacro (robot description, xacro)
@@ -16,4 +16,10 @@
         </geometry>
       </visual>
+    <collision>
+        <origin xyz="0 0 0" rpy="0 0 0" />
+        <geometry>
+          <mesh filename="package://iai_kitchen/meshes/collision/kitchen_island.stl"/>
+        </geometry>
+      </collision>
   </link>
   <joint name="${name}_footprint_joint" type="fixed">

File: iai_kitchen/urdf/IAI_oven_area.urdf.xacro (robot description, xacro)
@@ -17,4 +17,10 @@
         </geometry>
       </visual>
+    <collision>
+        <origin xyz="0 0 0" rpy="0 0 0" />
+        <geometry>
+          <mesh filename="package://iai_kitchen/meshes/collision/kitchen_oven_area.stl"/>
+        </geometry>
+      </collision>
   </link>
   <joint name="${name}_footprint_joint" type="fixed">

File: iai_kitchen/urdf/IAI_sink_area.urdf.xacro (robot description, xacro)
@@ -17,4 +17,10 @@
         </geometry>
       </visual>
+    <collision>
+        <origin xyz="0 0 0" rpy="0 0 0" />
+        <geometry>
+          <mesh filename="package://iai_kitchen/meshes/collision/kitchen_sink.stl"/>
+        </geometry>
+      </collision>
   </link>
   <joint name="${name}_footprint_joint" type="fixed">

Commit message: The fridge has a closed-up collision model, this changes it to the visual
This might not be the final solution, but it adds the essential opening in the front to the fridge

File: iai_kitchen/urdf/IAI_fridge_area.urdf.xacro (robot description, xacro)
@@ -19,5 +19,6 @@
         <origin xyz="0 0 0.01" rpy="0 0 0" />
         <geometry>
-          <mesh filename="package://iai_kitchen/meshes/collision/kitchen_fridge.stl"/>
+	    <mesh filename="package://iai_kitchen/meshes/racks/FridgeArea.dae"/>
+          <!--mesh filename="package://iai_kitchen/meshes/collision/kitchen_fridge.stl"/-->
         </geometry>
       </collision>
