Commit message: addded gazebo version of the new kitchen environment

File: iai_kitchen/urdf/IAI_dish_washer.urdf.xacro (robot description, xacro)
@@ -30,9 +30,24 @@
       </visual>
     </link>
-    <joint name="${name}_main_joint" type="fixed">
+    <!--
+    <xacro:if value="simulated"/>
+    -->
+    <joint name="${name}_main_joint" type="revolute">
+      <limit lower="0" upper="0" effort="300" velocity="10"/>
       <xacro:insert_block name="origin" />
       <parent link="${parent}"/>
       <child link="${name}_main"/>
     </joint>
+    <xacro:if value="${simulated}">
+    <joint name="${name}_door_joint" type="revolute">
+      <origin xyz="0.27 0. -0.325" rpy="${-0.5*pi} 0 0" />
+      <parent link="${name}_main"/>
+      <child link="${name}_door"/>
+      <axis xyz="0 0 1"/>
+      <!-- FIXME make closed position stable instead of forbidding opening... -->
+      <limit lower="0" upper="0" effort="300" velocity="10"/>
+    </joint>
+    </xacro:if>
+    <xacro:unless value="${simulated}">
     <joint name="${name}_door_joint" type="revolute">
       <origin xyz="0.27 0. -0.325" rpy="${-0.5*pi} 0 0" />
@@ -42,4 +57,5 @@
       <limit lower="0" upper="${0.5*pi}" effort="300" velocity="10"/>
     </joint>
+    </xacro:unless>
     <joint name="${name}_door_handle_joint" type="fixed">
       <origin xyz="0.0625 -0.6325 0." rpy="${-0.5*pi} 0 0" />

File: iai_kitchen/urdf/IAI_drawers.urdf.xacro (robot description, xacro)
@@ -62,5 +62,5 @@
       <child link="${name}_main"/>
       <axis xyz="1. 0. 0.0"/>
-      <limit lower="0" upper="0.48" effort="300" velocity="10"/>
+      <limit lower="0" upper="0.48" effort="0.0300" velocity="10"/>
     </joint>
     <joint name="${name}_handle_joint" type="fixed">

File: iai_kitchen/urdf/IAI_kitchen.urdf.xacro (robot description, xacro)
@@ -2,6 +2,26 @@
 <robot name="iai_oven_area" xmlns:xacro="http://ros.org/wiki/xacro">
   <xacro:property name="pi" value="3.1415926535897931" />
+  <xacro:property name="simulated" value="true" />
+  <macro name="sphere_inertia" params="radius mass">
+        <inertial>
+          <origin xyz="0.0 0.0 0.0" rpy="0 0 0"/>
+          <mass value="1"/>
+          <inertia
+              ixx="1" ixy="0.0" ixz="0.0"
+              iyy="1" iyz="0.0"
+              izz="1"/>
+        </inertial>
+  </macro>
   <link name="room_link">
+      <sphere_inertia radius="0" mass="0"/>
   </link>
+  <xacro:if value="${simulated}">
+    <link name="world"/>
+    <joint name="world_room_joint" type="fixed">
+        <origin xyz="0 0 0 " rpy="0 0 0" />
+        <parent link="world"/>
+        <child link="room_link"/>
+      </joint>
+  </xacro:if>
   <!--- FIXME THIS should NOT be here -->
   <xacro:include filename="$(find iai_kitchen)/urdf/IAI_oven_area.urdf.xacro"/>

File: iai_kitchen/urdf/IAI_kitchen_island.urdf.xacro (robot description, xacro)
@@ -26,4 +26,18 @@
     <parent link="${name}_footprint"/>
     <child link="${name}"/>
+  </joint>
+  <link name="${name}_surface">
+    <sphere_inertia radius="0" mass="0"/>
+    <collision>
+        <origin xyz="0 0 0" rpy="0 0 0" />
+        <geometry>
+          <box size="0.8 2.45 0.02"/>
+        </geometry>
+      </collision>
+  </link>
+  <joint name="${name}_surface_joint" type="fixed">
+    <origin xyz="0.0925 0. 0.42" rpy="0 0 0" />
+    <parent link="${name}"/>
+    <child link="${name}_surface"/>
   </joint>
   <link name="${name}_stove">

File: iai_kitchen/urdf/IAI_oven.urdf.xacro (robot description, xacro)
@@ -46,11 +46,34 @@
       <child link="${name}_main"/>
     </joint>
-    <joint name="${name}_door_joint" type="revolute">
-      <origin xyz="0.2737 0. -0.2614" rpy="${-0.5*pi} 0 0" />
-      <parent link="${name}_main"/>
-      <child link="${name}_door"/>
-      <axis xyz="0 0 1"/>
-      <limit lower="0" upper="${0.5*pi}" effort="300" velocity="10"/>
-    </joint>
+    <xacro:if value="${simulated}">
+      <joint name="${name}_door_joint" type="revolute">
+        <origin xyz="0.2737 0. -0.2614" rpy="${-0.5*pi} 0 0" />
+        <parent link="${name}_main"/>
+        <child link="${name}_door"/>
+        <axis xyz="0 0 1"/>
+        <!--
+        <limit lower="0" upper="${0.5*pi}" effort="300" velocity="10"/>
+        -->
+        <!-- FIXME make the closed position stable -->
+        <limit lower="0" upper="0." effort="0.03" velocity="10"/>
+        <dynamics damping="100.1"/>
+      </joint>
+      <gazebo reference="${name}_door_joint">
+        <kp>1000000000</kp>
+        <kd>1000000000</kd>
+      </gazebo>
+    </xacro:if>
+    <xacro:unless value="${simulated}">
+      <joint name="${name}_door_joint" type="revolute">
+        <origin xyz="0.2737 0. -0.2614" rpy="${-0.5*pi} 0 0" />
+        <parent link="${name}_main"/>
+        <child link="${name}_door"/>
+        <axis xyz="0 0 1"/>
+        <!--
+        <limit lower="0" upper="${0.5*pi}" effort="300" velocity="10"/>
+        -->
+        <limit lower="0" upper="${0.5*pi}" effort="0.03" velocity="10"/>
+      </joint>
+    </xacro:unless>
     <joint name="${name}_door_handle_joint" type="fixed">
       <origin xyz="0.05876 -0.39803 0." rpy="${-0.5*pi} 0 0" />

File: iai_kitchen/urdf/IAI_sink_area.urdf.xacro (robot description, xacro)
@@ -27,4 +27,18 @@
     <parent link="${name}_footprint"/>
     <child link="${name}"/>
+  </joint>
+  <link name="${name}_surface">
+    <sphere_inertia radius="0" mass="0"/>
+    <collision>
+        <origin xyz="0 0 0" rpy="0 0 0" />
+        <geometry>
+          <box size="0.575 2.05 0.02"/>
+        </geometry>
+      </collision>
+  </link>
+  <joint name="${name}_surface_joint" type="fixed">
+    <origin xyz="0.0 0. 0.43" rpy="0 0 0" />
+    <parent link="${name}"/>
+    <child link="${name}_surface"/>
   </joint>
   <link name="${name}_sink">

Commit message: fixed shaking kitchen Bug for gazebo

File: iai_kitchen/urdf/IAI_dish_washer.urdf.xacro (robot description, xacro)
@@ -55,4 +55,7 @@
       <child link="${name}_door"/>
       <axis xyz="0 0 1"/>
+      <!--
+      <limit lower="0" upper="${0.5*pi}" effort="300" velocity="10"/>
+      -->
       <limit lower="0" upper="${0.5*pi}" effort="300" velocity="10"/>
     </joint>

File: iai_kitchen/urdf/IAI_drawers.urdf (robot description, URDF)
Before this commit: robot iai_drawers, 11 links, 10 joints
Joints:
- joint drawer_1_main_joint: limit lower=0 upper=0.48 effort=300 velocity=10 -> lower=0 upper=0 effort=300 velocity=10
- joint drawer_2_main_joint: limit lower=0 upper=0.48 effort=300 velocity=10 -> lower=0 upper=0 effort=300 velocity=10
- joint drawer_3_main_joint: limit lower=0 upper=0.48 effort=300 velocity=10 -> lower=0 upper=0 effort=300 velocity=10
- joint drawer_4_main_joint: limit lower=0 upper=0.48 effort=300 velocity=10 -> lower=0 upper=0 effort=300 velocity=10
- joint drawer_5_main_joint: limit lower=0 upper=0.48 effort=300 velocity=10 -> lower=0 upper=0 effort=300 velocity=10

File: iai_kitchen/urdf/IAI_kitchen.urdf.xacro (robot description, xacro)
@@ -24,4 +24,7 @@
       </joint>
   </xacro:if>
+  <gazebo>
+      <static>true</static>
+  </gazebo>
   <!--- FIXME THIS should NOT be here -->
   <xacro:include filename="$(find iai_kitchen)/urdf/IAI_oven_area.urdf.xacro"/>

File: iai_kitchen/urdf/IAI_oven.urdf.xacro (robot description, xacro)
@@ -73,5 +73,5 @@
         <limit lower="0" upper="${0.5*pi}" effort="300" velocity="10"/>
         -->
-        <limit lower="0" upper="${0.5*pi}" effort="0.03" velocity="10"/>
+        <limit lower="0" upper="0" effort="0.03" velocity="10"/>
       </joint>
     </xacro:unless>
