Commit message: Add collision objects to urdf. Add joint_state_publisher to launch file

File: iai_kitchen/urdf/IAI_dish_washer.urdf.xacro (robot description, xacro)
@@ -11,4 +11,10 @@
         </geometry>
       </visual>
+      <collision>
+        <origin xyz="0 0 0" rpy="0 0 0" />
+        <geometry>
+          <mesh filename="package://iai_kitchen/meshes/misc/DishWasher.dae"/>
+        </geometry>
+      </collision>
     </link>
     <link name="${name}_door">
@@ -20,4 +26,10 @@
         </geometry>
       </visual>
+      <collision>
+        <origin xyz="0 0 0" rpy="${0.5*pi} 0 0" />
+        <geometry>
+          <mesh filename="package://iai_kitchen/meshes/misc/DishWasherDoor.dae"/>
+        </geometry>
+      </collision>
     </link>
     <link name="${name}_door_handle">

File: iai_kitchen/urdf/IAI_drawers.urdf.xacro (robot description, xacro)
@@ -47,4 +47,10 @@
         </geometry>
       </visual>
+      <collision>
+        <origin xyz="0 0 0" rpy="0 0 0" />
+        <geometry>
+          <mesh filename="package://iai_kitchen/meshes/drawers/VDrawer.dae"/>
+        </geometry>
+      </collision>
     </link>
     <link name="${name}_handle">
@@ -56,4 +62,10 @@
         </geometry>
       </visual>
+      <collision>
+        <origin xyz="0 0 0" rpy="0 0 0" />
+        <geometry>
+          <mesh filename="package://iai_kitchen/meshes/handles/VHandle130.dae"/>
+        </geometry>
+      </collision>
     </link>
     <joint name="${name}_main_joint" type="prismatic">
@@ -96,4 +108,10 @@
         </geometry>
       </visual>
+      <collision>
+        <origin xyz="0 0 0" rpy="0 0 0" />
+        <geometry>
+          <mesh filename="package://iai_kitchen/meshes/drawers/Drawer_${width}_${height}.dae"/>
+        </geometry>
+      </collision>
     </link>
     <link name="${name}_handle">
@@ -133,4 +151,10 @@
         </geometry>
       </visual>
+      <collision>
+        <origin xyz="0 0 0" rpy="0 0 0" />
+        <geometry>
+          <mesh filename="package://iai_kitchen/meshes/drawers/Panel_${width}.dae"/>
+        </geometry>
+      </collision>
     </link>
     <joint name="${name}_joint" type="fixed">

File: iai_kitchen/urdf/IAI_fridge.urdf.xacro (robot description, xacro)
@@ -11,4 +11,10 @@
         </geometry>
       </visual>
+      <collision>
+        <origin xyz="0 0 0" rpy="0 0 0" />
+        <geometry>
+          <mesh filename="package://iai_kitchen/meshes/misc/Fridge.dae"/>
+        </geometry>
+      </collision>
     </link>
     <link name="${name}_door">
@@ -20,4 +26,10 @@
         </geometry>
       </visual>
+      <collision>
+        <origin xyz="0 0 0" rpy="0 0 0" />
+        <geometry>
+          <mesh filename="package://iai_kitchen/meshes/misc/FridgeDoor.dae"/>
+        </geometry>
+      </collision>
     </link>
     <link name="${name}_door_handle">

File: iai_kitchen/urdf/IAI_fridge_area.urdf.xacro (robot description, xacro)
@@ -11,16 +11,16 @@
       <sphere_inertia radius="0" mass="0"/>
       <visual>
-	  <origin xyz="0 0 0.01" rpy="0 0 0" />
-	  <geometry>
-	    <mesh filename="package://iai_kitchen/meshes/racks/FridgeArea.dae"/>
-	  </geometry>
-	</visual>
-    <collision>
-        <origin xyz="0 0 0.01" rpy="0 0 0" />
-        <geometry>
-	    <mesh filename="package://iai_kitchen/meshes/racks/FridgeArea.dae"/>
-          <!--mesh filename="package://iai_kitchen/meshes/collision/kitchen_fridge.stl"/-->
-        </geometry>
-      </collision>
+    	  <origin xyz="0 0 0.01" rpy="0 0 0" />
+    	  <geometry>
+    	    <mesh filename="package://iai_kitchen/meshes/racks/FridgeArea.dae"/>
+    	  </geometry>
+    	</visual>
+      <collision>
+          <origin xyz="0 0 0.01" rpy="0 0 0" />
+          <geometry>
+  	    <mesh filename="package://iai_kitchen/meshes/racks/FridgeArea.dae"/>
+            <!--mesh filename="package://iai_kitchen/meshes/collision/kitchen_fridge.stl"/-->
+          </geometry>
+        </collision>
     </link>
     <joint name="${name}_footprint_joint" type="fixed">

File: iai_kitchen/urdf/IAI_kitchen.urdf.xacro (robot description, xacro)
@@ -33,5 +33,5 @@
   <xacro:include filename="$(find iai_kitchen)/urdf/IAI_fridge_area.urdf.xacro"/>
   <xacro:include filename="$(find iai_kitchen)/urdf/IAI_tables.urdf.xacro"/>
-  <xacro:include filename="$(find iai_kitchen)/urdf/IAI_kitchen_walls.urdf.xacro"/>
+  <!--xacro:include filename="$(find iai_kitchen)/urdf/IAI_kitchen_walls.urdf.xacro"/-->
   <iai_sink_area name="sink_area" parent="room_link">
     <origin xyz="1.825 1.3 0" rpy="0 0 ${pi}" />

File: iai_kitchen/urdf/IAI_kitchen_island.urdf.xacro (robot description, xacro)
@@ -5,10 +5,10 @@
   <xacro:include filename="$(find iai_kitchen)/urdf/IAI_drawers.urdf.xacro"/>
   <macro name="iai_kitchen_island" params="parent name *origin">
-  <link name="${name}_footprint">
-    <sphere_inertia radius="0" mass="0"/>
-  </link>
-  <link name="${name}">
-    <sphere_inertia radius="0" mass="0"/>
-    <visual>
+    <link name="${name}_footprint">
+      <sphere_inertia radius="0" mass="0"/>
+    </link>
+    <link name="${name}">
+      <sphere_inertia radius="0" mass="0"/>
+      <visual>
         <origin xyz="0 0 0" rpy="0 0 0" />
         <geometry>
@@ -16,76 +16,82 @@
         </geometry>
       </visual>
-    <collision>
-        <origin xyz="0 0 0" rpy="0 0 0" />
-        <geometry>
-          <mesh filename="package://iai_kitchen/meshes/collision/kitchen_island.stl"/>
-        </geometry>
-      </collision>
-  </link>
-  <joint name="${name}_footprint_joint" type="fixed">
-      <xacro:insert_block name="origin" />
-    <child link="${name}_footprint"/>
-    <parent link="${parent}"/>
-  </joint>
-  <joint name="${name}_joint" type="fixed">
-    <origin xyz="0.2975 1.1292 0.421" rpy="0 0 0" />
-    <parent link="${name}_footprint"/>
-    <child link="${name}"/>
-  </joint>
-  <link name="${name}_surface">
-    <sphere_inertia radius="0" mass="0"/>
-    <collision>
-        <origin xyz="0 0 0" rpy="0 0 0" />
-        <geometry>
-          <box size="0.8 2.45 0.02"/>
-        </geometry>
-      </collision>
-  </link>
-  <joint name="${name}_surface_joint" type="fixed">
-    <origin xyz="0.0 0. 0.42" rpy="0 0 0" />
-    <parent link="${name}"/>
-    <child link="${name}_surface"/>
-  </joint>
-  <link name="${name}_stove">
-    <sphere_inertia radius="0" mass="0"/>
-    <visual>
-        <origin xyz="0 0 0" rpy="0 0 0" />
-        <geometry>
-          <mesh filename="package://iai_kitchen/meshes/misc/Stove.dae"/>
-        </geometry>
-      </visual>
-  </link>
-  <joint name="${name}_stove_joint" type="fixed">
-    <origin xyz="0.0 0.7658 0.4315" rpy="0 0 0" />
-    <parent link="${name}"/>
-    <child link="${name}_stove"/>
-  </joint>
-  <iai_generic_panel name="${name}_left_panel" parent="${name}" width="60">
-    <origin rpy="0 0 0" xyz="0.2725 -0.8 0.329 "/>
-  </iai_generic_panel>
-  <iai_drawer_60_29 name="${name}_left_upper_drawer" parent="${name}">
-    <origin rpy="0 0 0" xyz="0.0025 -0.8 0.114 "/>
-  </iai_drawer_60_29>
-  <iai_drawer_60_29 name="${name}_left_lower_drawer" parent="${name}">
-    <origin rpy="0 0 0" xyz="0.0025 -0.8 -0.176 "/>
-  </iai_drawer_60_29>
-  <iai_generic_panel name="${name}_middle_panel" parent="${name}" width="100">
-    <origin rpy="0 0 0" xyz="0.2725 0 0.329 "/>
-  </iai_generic_panel>
-  <iai_drawer_100_29 name="${name}_middle_upper_drawer" parent="${name}">
-    <origin rpy="0 0 0" xyz="0.0025 0 0.114 "/>
-  </iai_drawer_100_29>
-  <iai_drawer_100_29 name="${name}_middle_lower_drawer" parent="${name}">
-    <origin rpy="0 0 0" xyz="0.0025 0 -0.176 "/>
-  </iai_drawer_100_29>
-  <iai_generic_panel name="${name}_right_panel" parent="${name}" width="60">
-    <origin rpy="0 0 0" xyz="0.2725 0.8 0.329 "/>
-  </iai_generic_panel>
-  <iai_drawer_60_29 name="${name}_right_upper_drawer" parent="${name}">
-    <origin rpy="0 0 0" xyz="0.0025 0.8 0.114 "/>
-  </iai_drawer_60_29>
-  <iai_drawer_60_29 name="${name}_right_lower_drawer" parent="${name}">
-    <origin rpy="0 0 0" xyz="0.0025 0.8 -0.176 "/>
-  </iai_drawer_60_29>
+      <!--collision>
+          <origin xyz="0 0 0" rpy="0 0 0" />
+          <geometry>
+            <mesh filename="package://iai_kitchen/meshes/collision/kitchen_island.stl"/>
+          </geometry>
+        </collision-->
+    </link>
+    <joint name="${name}_footprint_joint" type="fixed">
+        <xacro:insert_block name="origin" />
+      <child link="${name}_footprint"/>
+      <parent link="${parent}"/>
+    </joint>
+    <joint name="${name}_joint" type="fixed">
+      <origin xyz="0.2975 1.1292 0.421" rpy="0 0 0" />
+      <parent link="${name}_footprint"/>
+      <child link="${name}"/>
+    </joint>
+    <link name="${name}_surface">
+      <sphere_inertia radius="0" mass="0"/>
+      <collision>
+          <origin xyz="0 0 0" rpy="0 0 0" />
+          <geometry>
+            <box size="0.8 2.45 0.02"/>
+          </geometry>
+        </collision>
+    </link>
+    <joint name="${name}_surface_joint" type="fixed">
+      <origin xyz="0.0 0. 0.42" rpy="0 0 0" />
+      <parent link="${name}"/>
+      <child link="${name}_surface"/>
+    </joint>
+    <link name="${name}_stove">
+      <sphere_inertia radius="0" mass="0"/>
+      <visual>
+          <origin xyz="0 0 0" rpy="0 0 0" />
+          <geometry>
+            <mesh filename="package://iai_kitchen/meshes/misc/Stove.dae"/>
+          </geometry>
+        </visual>
+        <collision>
+          <origin xyz="0 0 0" rpy="0 0 0" />
+          <geometry>
+            <mesh filename="package://iai_kitchen/meshes/misc/Stove.dae"/>
+          </geometry>
+        </collision>
+    </link>
+    <joint name="${name}_stove_joint" type="fixed">
+      <origin xyz="0.0 0.7658 0.4315" rpy="0 0 0" />
+      <parent link="${name}"/>
+      <child link="${name}_stove"/>
+    </joint>
+    <!--iai_generic_panel name="${name}_left_panel" parent="${name}" width="60">
+      <origin rpy="0 0 0" xyz="0.2725 -0.8 0.329 "/>
+    </iai_generic_panel-->
+    <iai_drawer_60_29 name="${name}_left_upper_drawer" parent="${name}">
+      <origin rpy="0 0 0" xyz="0.0025 -0.8 0.114 "/>
+    </iai_drawer_60_29>
+    <iai_drawer_60_29 name="${name}_left_lower_drawer" parent="${name}">
+      <origin rpy="0 0 0" xyz="0.0025 -0.8 -0.176 "/>
+    </iai_drawer_60_29>
+    <!--iai_generic_panel name="${name}_middle_panel" parent="${name}" width="100">
+      <origin rpy="0 0 0" xyz="0.2725 0 0.329 "/>
+    </iai_generic_panel-->
+    <iai_drawer_100_29 name="${name}_middle_upper_drawer" parent="${name}">
+      <origin rpy="0 0 0" xyz="0.0025 0 0.114 "/>
+    </iai_drawer_100_29>
+    <iai_drawer_100_29 name="${name}_middle_lower_drawer" parent="${name}">
+      <origin rpy="0 0 0" xyz="0.0025 0 -0.176 "/>
+    </iai_drawer_100_29>
+    <!--iai_generic_panel name="${name}_right_panel" parent="${name}" width="60">
+      <origin rpy="0 0 0" xyz="0.2725 0.8 0.329 "/>
+    </iai_generic_panel-->
+    <iai_drawer_60_29 name="${name}_right_upper_drawer" parent="${name}">
+      <origin rpy="0 0 0" xyz="0.0025 0.8 0.114 "/>
+    </iai_drawer_60_29>
+    <iai_drawer_60_29 name="${name}_right_lower_drawer" parent="${name}">
+      <origin rpy="0 0 0" xyz="0.0025 0.8 -0.176 "/>
+    </iai_drawer_60_29>
   </macro>
 </robot>

File: iai_kitchen/urdf/IAI_oven.urdf.xacro (robot description, xacro)
@@ -12,4 +12,10 @@
         </geometry>
       </visual>
+      <collision>
+        <origin xyz="0 0 0" rpy="0 0 0" />
+        <geometry>
+          <mesh filename="package://iai_kitchen/meshes/oven/OvenMain.dae"/>
+        </geometry>
+      </collision>
     </link>
     <link name="${name}_door">
@@ -21,4 +27,10 @@
         </geometry>
       </visual>
+      <collision>
+        <origin xyz="0 0 0" rpy="${0.5*pi} 0 0" />
+        <geometry>
+          <mesh filename="package://iai_kitchen/meshes/oven/OvenDoor.dae"/>
+        </geometry>
+      </collision>
     </link>
     <link name="${name}_door_handle">
@@ -30,4 +42,10 @@
         </geometry>
       </visual>
+      <collision>
+        <origin xyz="0 0 0" rpy="0 0 0" />
+        <geometry>
+          <mesh filename="package://iai_kitchen/meshes/handles/Handle60.dae"/>
+        </geometry>
+      </collision>
     </link>
     <link name="${name}_panel">
@@ -39,4 +57,10 @@
         </geometry>
       </visual>
+      <collision>
+        <origin xyz="0 0 0" rpy="0 0 0" />
+        <geometry>
+          <mesh filename="package://iai_kitchen/meshes/oven/OvenPanel.dae"/>
+        </geometry>
+      </collision>
     </link>
     <!-- JOINTS -->
@@ -104,4 +128,10 @@
         </geometry>
       </visual>
+      <collision>
+        <origin xyz="0 0 0" rpy="0 ${0.5 * pi} 0" />
+        <geometry>
+          <mesh filename="package://iai_kitchen/meshes/oven/Knob.dae"/>
+        </geometry>
+      </collision>
     </link>
     <joint name="${name}_joint" type="revolute">

File: iai_kitchen/urdf/IAI_oven_area.urdf.xacro (robot description, xacro)
@@ -43,10 +43,10 @@
     <origin rpy="0 0 0" xyz="0.0 -0. -0.315 "/>
   </iai_drawer_60_58>
-  <iai_vdrawer name="${name}_area_left_drawer" parent="${name}_area">
+  <!--iai_vdrawer name="${name}_area_left_drawer" parent="${name}_area">
     <origin rpy="0 0 0" xyz="0.0 -0.45 0.06 "/>
   </iai_vdrawer>
   <iai_vdrawer name="${name}_area_right_drawer" parent="${name}_area">
     <origin rpy="0 0 0" xyz="0.0 0.45 0.06 "/>
-  </iai_vdrawer>
+  </iai_vdrawer-->
   </macro>
 </robot>

File: iai_kitchen/urdf/IAI_sink_area.urdf.xacro (robot description, xacro)
@@ -51,9 +51,15 @@
     <sphere_inertia radius="0" mass="0"/>
     <visual>
-        <origin xyz="0 0 0" rpy="0 0 0" />
-        <geometry>
-          <mesh filename="package://iai_kitchen/meshes/misc/Sink.dae"/>
-        </geometry>
-      </visual>
+      <origin xyz="0 0 0" rpy="0 0 0" />
+      <geometry>
+        <mesh filename="package://iai_kitchen/meshes/misc/Sink.dae"/>
+      </geometry>
+    </visual>
+    <!--collision>
+      <origin xyz="0 0 0" rpy="0 0 0" />
+      <geometry>
+        <mesh filename="package://iai_kitchen/meshes/misc/Sink.dae"/>
+      </geometry>
+    </collision-->
   </link>
   <joint name="${name}_sink_joint" type="fixed">
@@ -62,7 +68,7 @@
     <child link="${name}_sink"/>
   </joint>
-  <iai_generic_panel name="${name}_right_panel" parent="${name}" width="60">
+  <!--iai_generic_panel name="${name}_right_panel" parent="${name}" width="60">
     <origin rpy="0 0 0" xyz="0.28 0.7 0.325 "/>
-  </iai_generic_panel>
+  </iai_generic_panel-->
   <iai_drawer_60_58 name="${name}_trash_drawer" parent="${name}">
     <origin rpy="0 0 0" xyz="0.01 0.7 -0.035 "/>
@@ -77,7 +83,7 @@
     <origin rpy="0 0 0" xyz="0.01 -0.6 -0.18 "/>
   </iai_drawer_80_29>
-  <iai_dish_washer name="${name}_dish_washer" parent="${name}">
+  <!--iai_dish_washer name="${name}_dish_washer" parent="${name}">
     <origin rpy="0 0 0" xyz="0.01 0.1 0.035 "/>
-  </iai_dish_washer>
+  </iai_dish_washer-->
   </macro>
 </robot>

File: iai_kitchen/urdf/sink_area.urdf.xacro (robot description, xacro)
@@ -14,4 +14,10 @@
         </geometry>
       </visual>
+      <collision>
+        <origin xyz="0 0 0" rpy="0 0 0" />
+        <geometry>
+          <box size=".1 .1 .1" />
+        </geometry>
+      </collision>
     </link>
     <link name="sink_area_main">
@@ -24,4 +30,10 @@
         </geometry>
       </visual>
+      <collision>
+        <origin xyz="0 0 0" rpy="0 0 0" />
+        <geometry>
+          <mesh filename="package://iai_kitchen/meshes/SinkArea.dae"/>
+        </geometry>
+      </collision>
     </link>
     <joint name="sink_area_joint" type="fixed">
@@ -40,4 +52,10 @@
         </geometry>
       </visual>
+      <collision>
+        <origin xyz="0 0 0" rpy="0 0 0" />
+        <geometry>
+          <mesh filename="package://iai_kitchen/meshes/SinkAreaMedDrawer.dae"/>
+        </geometry>
+      </collision>
     </link>
     <joint name="sink_area_drawer_left_bottom_joint" type="prismatic">
@@ -72,4 +90,10 @@
         </geometry>
       </visual>
+      <collision>
+        <origin xyz="0 0 0" rpy="0 0 0" />
+        <geometry>
+          <mesh filename="package://iai_kitchen/meshes/SinkAreaMedDrawer.dae"/>
+        </geometry>
+      </collision>
     </link>
     <joint name="sink_area_drawer_left_center_joint" type="prismatic">
@@ -103,4 +127,10 @@
         </geometry>
       </visual>
+      <collision>
+        <origin xyz="0 0 0" rpy="0 0 0" />
+        <geometry>
+          <mesh filename="package://iai_kitchen/meshes/SinkAreaSmallDrawer.dae"/>
+        </geometry>
+      </collision>
     </link>
     <joint name="sink_area_drawer_left_top_joint" type="prismatic">
@@ -134,4 +164,10 @@
         </geometry>
       </visual>
+      <collision>
+        <origin xyz="0 0 0" rpy="0 0 0" />
+        <geometry>
+          <mesh filename="package://iai_kitchen/meshes/SinkAreaInnerDishWasher.dae"/>
+        </geometry>
+      </collision>
     </link>
     <joint name="sink_area_dishwasher_joint" type="fixed">
@@ -148,4 +184,10 @@
         </geometry>
       </visual>
+      <collision>
+        <origin xyz="0 0 0" rpy="0 0 0" />
+        <geometry>
+          <mesh filename="package://iai_kitchen/meshes/SinkAreaDishWasherDoor.dae"/>
+        </geometry>
+      </collision>
     </link>
     <joint name="sink_area_dishwasher_door_joint" type="revolute">
@@ -179,4 +221,10 @@
         </geometry>
       </visual>
+      <collision>
+        <origin xyz="0 0 0" rpy="0 0 0" />
+        <geometry>
+          <mesh filename="package://iai_kitchen/meshes/SinkAreaPanel.dae"/>
+        </geometry>
+      </collision>
     </link>
     <joint name="sink_area_pane_joint" type="fixed">
@@ -193,4 +241,10 @@
         </geometry>
       </visual>
+      <collision>
+        <origin xyz="0 0 0" rpy="0 0 0" />
+        <geometry>
+          <mesh filename="package://iai_kitchen/meshes/SinkAreaTrash.dae"/>
+        </geometry>
+      </collision>
     </link>
     <joint name="sink_area_trash_joint" type="prismatic">
@@ -223,4 +277,10 @@
         </geometry>
       </visual>
+      <collision>
+        <origin xyz="0 0 0" rpy="0 0 0" />
+        <geometry>
+          <mesh filename="package://iai_kitchen/meshes/SinkAreaSink.dae"/>
+        </geometry>
+      </collision>
     </link>
     <joint name="sink_area_sink_joint" type="fixed">
