Commit message: Fix corrupted collision meshes.

File: iai_kitchen/urdf/IAI_dish_washer.urdf.xacro (robot description, xacro)
@@ -41,4 +41,11 @@
         </geometry>
       </visual>
+      <!--pumpernickel-->
+      <collision>
+        <origin xyz="0 0 0" rpy="0 0 0" />
+        <geometry>
+          <mesh filename="package://iai_kitchen/meshes/handles/Handle60.dae"/>
+        </geometry>
+      </collision>
     </link>
     <!--

File: iai_kitchen/urdf/IAI_drawers.urdf.xacro (robot description, xacro)
@@ -123,4 +123,11 @@
         </geometry>
       </visual>
+      <!--pumpernickel-->
+      <collision>
+        <origin xyz="0 0 0" rpy="0 0 0" />
+        <geometry>
+          <mesh filename="package://iai_kitchen/meshes/handles/Handle${width}.dae"/>
+        </geometry>
+      </collision>
     </link>
     <joint name="${name}_main_joint" type="prismatic">

File: iai_kitchen/urdf/IAI_kitchen.urdf.xacro (robot description, xacro)
@@ -52,5 +52,5 @@
     <origin xyz="-1 0.562175 0" rpy="0.0 0.0 0.0" />
   </iai_kitchen_wall_robohow>
-  <!--
+  <!-- Included above already
   <iai_sink_area name="sink_area" parent="room_link">
     <origin xyz="-5.29 -5.65 0" rpy="0 0 0" />

File: iai_kitchen/urdf/IAI_kitchen_island.urdf.xacro (robot description, xacro)
@@ -16,10 +16,10 @@
         </geometry>
       </visual>
-      <!--collision>
-          <origin xyz="0 0 0" rpy="0 0 0" />
-          <geometry>
-            <mesh filename="package://iai_kitchen/meshes/collision/kitchen_island.stl"/>
-          </geometry>
-        </collision-->
+      <collision>
+        <origin xyz="0 0 0" rpy="0 0 0" />
+        <geometry>
+          <mesh filename="package://iai_kitchen/meshes/collision/kitchen_island.stl"/>
+        </geometry>
+      </collision>
     </link>
     <joint name="${name}_footprint_joint" type="fixed">
@@ -67,7 +67,7 @@
       <child link="${name}_stove"/>
     </joint>
-    <!--iai_generic_panel name="${name}_left_panel" parent="${name}" width="60">
+    <iai_generic_panel name="${name}_left_panel" parent="${name}" width="60">
       <origin rpy="0 0 0" xyz="0.2725 -0.8 0.329 "/>
-    </iai_generic_panel-->
+    </iai_generic_panel>
     <iai_drawer_60_29 name="${name}_left_upper_drawer" parent="${name}">
       <origin rpy="0 0 0" xyz="0.0025 -0.8 0.114 "/>
@@ -76,7 +76,7 @@
       <origin rpy="0 0 0" xyz="0.0025 -0.8 -0.176 "/>
     </iai_drawer_60_29>
-    <!--iai_generic_panel name="${name}_middle_panel" parent="${name}" width="100">
+    <iai_generic_panel name="${name}_middle_panel" parent="${name}" width="100">
       <origin rpy="0 0 0" xyz="0.2725 0 0.329 "/>
-    </iai_generic_panel-->
+    </iai_generic_panel>
     <iai_drawer_100_29 name="${name}_middle_upper_drawer" parent="${name}">
       <origin rpy="0 0 0" xyz="0.0025 0 0.114 "/>
@@ -85,7 +85,7 @@
       <origin rpy="0 0 0" xyz="0.0025 0 -0.176 "/>
     </iai_drawer_100_29>
-    <!--iai_generic_panel name="${name}_right_panel" parent="${name}" width="60">
+    <iai_generic_panel name="${name}_right_panel" parent="${name}" width="60">
       <origin rpy="0 0 0" xyz="0.2725 0.8 0.329 "/>
-    </iai_generic_panel-->
+    </iai_generic_panel>
     <iai_drawer_60_29 name="${name}_right_upper_drawer" parent="${name}">
       <origin rpy="0 0 0" xyz="0.0025 0.8 0.114 "/>

File: iai_kitchen/urdf/IAI_oven_area.urdf.xacro (robot description, xacro)
@@ -43,10 +43,10 @@
     <origin rpy="0 0 0" xyz="0.0 -0. -0.315 "/>
   </iai_drawer_60_58>
-  <!--iai_vdrawer name="${name}_area_left_drawer" parent="${name}_area">
+  <iai_vdrawer name="${name}_area_left_drawer" parent="${name}_area">
     <origin rpy="0 0 0" xyz="0.0 -0.45 0.06 "/>
   </iai_vdrawer>
   <iai_vdrawer name="${name}_area_right_drawer" parent="${name}_area">
     <origin rpy="0 0 0" xyz="0.0 0.45 0.06 "/>
-  </iai_vdrawer-->
+  </iai_vdrawer>
   </macro>
 </robot>

File: iai_kitchen/urdf/IAI_sink_area.urdf.xacro (robot description, xacro)
@@ -37,9 +37,9 @@
     <sphere_inertia radius="0" mass="0"/>
     <collision>
-        <origin xyz="0 0 0" rpy="0 0 0" />
-        <geometry>
-          <box size="0.575 2.05 0.02"/>
-        </geometry>
-      </collision>
+      <origin xyz="0 0 0" rpy="0 0 0" />
+      <geometry>
+        <box size="0.575 2.05 0.02"/>
+      </geometry>
+    </collision>
   </link>
   <joint name="${name}_surface_joint" type="fixed">
@@ -56,10 +56,10 @@
       </geometry>
     </visual>
-    <!--collision>
+    <collision>
       <origin xyz="0 0 0" rpy="0 0 0" />
       <geometry>
         <mesh filename="package://iai_kitchen/meshes/misc/Sink.dae"/>
       </geometry>
-    </collision-->
+    </collision>
   </link>
   <joint name="${name}_sink_joint" type="fixed">
@@ -68,7 +68,7 @@
     <child link="${name}_sink"/>
   </joint>
-  <!--iai_generic_panel name="${name}_right_panel" parent="${name}" width="60">
+  <iai_generic_panel name="${name}_right_panel" parent="${name}" width="60">
     <origin rpy="0 0 0" xyz="0.28 0.7 0.325 "/>
-  </iai_generic_panel-->
+  </iai_generic_panel>
   <iai_drawer_60_58 name="${name}_trash_drawer" parent="${name}">
     <origin rpy="0 0 0" xyz="0.01 0.7 -0.035 "/>
@@ -83,7 +83,7 @@
     <origin rpy="0 0 0" xyz="0.01 -0.6 -0.18 "/>
   </iai_drawer_80_29>
-  <!--iai_dish_washer name="${name}_dish_washer" parent="${name}">
+  <iai_dish_washer name="${name}_dish_washer" parent="${name}">
     <origin rpy="0 0 0" xyz="0.01 0.1 0.035 "/>
-  </iai_dish_washer-->
+  </iai_dish_washer>
   </macro>
 </robot>

File: iai_kitchen/urdf/sink_area.urdf.xacro (robot description, xacro)
@@ -75,4 +75,11 @@
         </geometry>
       </visual>
+      <!--pumpernickel-->
+      <collision>
+        <origin xyz="0 0 0" rpy="0 0 0" />
+        <geometry>
+          <mesh filename="package://iai_kitchen/meshes/SinkAreaBigHandle.dae"/>
+        </geometry>
+      </collision>
     </link>
     <joint name="sink_area_drawer_left_bottom_handle_joint" type="fixed">
@@ -112,4 +119,11 @@
         </geometry>
       </visual>
+      <!--pumpernickel-->
+      <collision>
+        <origin xyz="0 0 0" rpy="0 0 0" />
+        <geometry>
+          <mesh filename="package://iai_kitchen/meshes/SinkAreaBigHandle.dae"/>
+        </geometry>
+      </collision>
     </link>
     <joint name="sink_area_drawer_left_center_handle_joint" type="fixed">
@@ -149,4 +163,11 @@
         </geometry>
       </visual>
+      <!--pumpernickel-->
+      <collision>
+        <origin xyz="0 0 0" rpy="0 0 0" />
+        <geometry>
+          <mesh filename="package://iai_kitchen/meshes/SinkAreaBigHandle.dae"/>
+        </geometry>
+      </collision>
     </link>
     <joint name="sink_area_drawer_left_bottom_top_joint" type="fixed">
@@ -206,4 +227,11 @@
         </geometry>
       </visual>
+      <!--pumpernickel-->
+      <collision>
+        <origin xyz="0 0 0" rpy="0 0 0" />
+        <geometry>
+          <mesh filename="package://iai_kitchen/meshes/SinkAreaSmallHandle.dae"/>
+        </geometry>
+      </collision>
     </link>
     <joint name="sink_area_dishwasher_handle_joint" type="fixed">
@@ -263,4 +291,11 @@
         </geometry>
       </visual>
+      <!--pumpernickel-->
+      <collision>
+        <origin xyz="0 0 0" rpy="0 0 0" />
+        <geometry>
+          <mesh filename="package://iai_kitchen/meshes/SinkAreaSmallHandle.dae"/>
+        </geometry>
+      </collision>
     </link>
     <joint name="sink_area_trash_handle_joint" type="fixed">

Commit message: Add fridge handle collision object. Remove search tags.

File: iai_kitchen/urdf/IAI_dish_washer.urdf.xacro (robot description, xacro)
@@ -41,5 +41,4 @@
         </geometry>
       </visual>
-      <!--pumpernickel-->
       <collision>
         <origin xyz="0 0 0" rpy="0 0 0" />

File: iai_kitchen/urdf/IAI_drawers.urdf.xacro (robot description, xacro)
@@ -123,5 +123,4 @@
         </geometry>
       </visual>
-      <!--pumpernickel-->
       <collision>
         <origin xyz="0 0 0" rpy="0 0 0" />

File: iai_kitchen/urdf/IAI_fridge.urdf.xacro (robot description, xacro)
@@ -41,4 +41,10 @@
         </geometry>
       </visual>
+      <collision>
+        <origin xyz="0 0 0" rpy="0 0 0" />
+        <geometry>
+          <mesh filename="package://iai_kitchen/meshes/handles/VHandle90.dae"/>
+        </geometry>
+      </collision>
     </link>
     <joint name="${name}_main_joint" type="fixed">

File: iai_kitchen/urdf/sink_area.urdf.xacro (robot description, xacro)
@@ -75,5 +75,4 @@
         </geometry>
       </visual>
-      <!--pumpernickel-->
       <collision>
         <origin xyz="0 0 0" rpy="0 0 0" />
@@ -119,5 +118,4 @@
         </geometry>
       </visual>
-      <!--pumpernickel-->
       <collision>
         <origin xyz="0 0 0" rpy="0 0 0" />
@@ -163,5 +161,4 @@
         </geometry>
       </visual>
-      <!--pumpernickel-->
       <collision>
         <origin xyz="0 0 0" rpy="0 0 0" />
@@ -227,5 +224,4 @@
         </geometry>
       </visual>
-      <!--pumpernickel-->
       <collision>
         <origin xyz="0 0 0" rpy="0 0 0" />
@@ -291,5 +287,4 @@
         </geometry>
       </visual>
-      <!--pumpernickel-->
       <collision>
         <origin xyz="0 0 0" rpy="0 0 0" />
