Commit message: added a table to the gazebo-kitchen-map

File: iai_kitchen/urdf/IAI_kitchen.urdf.xacro (robot description, xacro)
@@ -32,4 +32,5 @@
   <xacro:include filename="$(find iai_kitchen)/urdf/IAI_sink_area.urdf.xacro"/>
   <xacro:include filename="$(find iai_kitchen)/urdf/IAI_fridge_area.urdf.xacro"/>
+  <xacro:include filename="$(find iai_kitchen)/urdf/IAI_tables.urdf.xacro"/>
   <iai_sink_area name="sink_area" parent="room_link">
     <origin xyz="1.825 1.3 0" rpy="0 0 ${pi}" />
@@ -44,4 +45,7 @@
     <origin xyz="1.825 -0.76 0" rpy="0 0 ${pi}" />
   </iai_fridge_area>
+  <iai_table_1 name="table_area" parent="room_link">
+    <origin xyz="-1.4 -1.3 0" rpy="0 0 ${pi}" />
+  </iai_table_1>
   <!--
   <iai_sink_area name="sink_area" parent="room_link">

Commit message: added new method to spawn walls in gazebo versions < 3.0

File: iai_kitchen/urdf/IAI_kitchen.urdf.xacro (robot description, xacro)
@@ -33,4 +33,5 @@
   <xacro:include filename="$(find iai_kitchen)/urdf/IAI_fridge_area.urdf.xacro"/>
   <xacro:include filename="$(find iai_kitchen)/urdf/IAI_tables.urdf.xacro"/>
+  <xacro:include filename="$(find iai_kitchen)/urdf/IAI_kitchen_walls.urdf.xacro"/>
   <iai_sink_area name="sink_area" parent="room_link">
     <origin xyz="1.825 1.3 0" rpy="0 0 ${pi}" />
@@ -48,4 +49,7 @@
     <origin xyz="-1.4 -1.3 0" rpy="0 0 ${pi}" />
   </iai_table_1>
+  <iai_kitchen_wall_robohow parent="room_link">
+    <origin xyz="-1 0.562175 0" rpy="0.0 0.0 0.0" />
+  </iai_kitchen_wall_robohow>
   <!--
   <iai_sink_area name="sink_area" parent="room_link">

Commit message: Corrected position of meal table in the kitchen URDF

File: iai_kitchen/urdf/IAI_kitchen.urdf.xacro (robot description, xacro)
@@ -47,5 +47,5 @@
   </iai_fridge_area>
   <iai_table_1 name="table_area" parent="room_link">
-    <origin xyz="-1.4 -1.3 0" rpy="0 0 ${pi}" />
+    <origin xyz="-1.4 -1.15 0" rpy="0 0 ${pi}" />
   </iai_table_1>
   <iai_kitchen_wall_robohow parent="room_link">

Commit message: Correct position of meal table in URDF

File: iai_kitchen/urdf/IAI_kitchen.urdf.xacro (robot description, xacro)
@@ -47,5 +47,5 @@
   </iai_fridge_area>
   <iai_table_1 name="table_area" parent="room_link">
-    <origin xyz="-1.4 -1.15 0" rpy="0 0 ${pi}" />
+    <origin xyz="-1.4 -1.05 0" rpy="0 0 ${pi}" />
   </iai_table_1>
   <iai_kitchen_wall_robohow parent="room_link">

Commit message: Get kitchen walls back. Remove unnecessary collision.

File: iai_kitchen/urdf/IAI_kitchen.urdf.xacro (robot description, xacro)
@@ -33,5 +33,5 @@
   <xacro:include filename="$(find iai_kitchen)/urdf/IAI_fridge_area.urdf.xacro"/>
   <xacro:include filename="$(find iai_kitchen)/urdf/IAI_tables.urdf.xacro"/>
-  <!--xacro:include filename="$(find iai_kitchen)/urdf/IAI_kitchen_walls.urdf.xacro"/-->
+  <xacro:include filename="$(find iai_kitchen)/urdf/IAI_kitchen_walls.urdf.xacro"/>
   <iai_sink_area name="sink_area" parent="room_link">
     <origin xyz="1.825 1.3 0" rpy="0 0 ${pi}" />

File: iai_kitchen/urdf/sink_area.urdf.xacro (robot description, xacro)
@@ -14,10 +14,4 @@
         </geometry>
       </visual>
-      <collision>
-        <origin xyz="0 0 0" rpy="0 0 0" />
-        <geometry>
-          <box size=".1 .1 .1" />
-        </geometry>
-      </collision>
     </link>
     <link name="sink_area_main">

Commit message: calibrated offsets in old kitchen urdf

File: iai_kitchen/urdf/IAI_kitchen.urdf.xacro (robot description, xacro)
@@ -19,5 +19,5 @@
     <link name="world"/>
     <joint name="world_room_joint" type="fixed">
-        <origin xyz="0 0 0 " rpy="0 0 0" />
+        <origin xyz="0.02 -0.01 0" rpy="0 0 0" />
         <parent link="world"/>
         <child link="room_link"/>

File: iai_kitchen/urdf/IAI_sink_area.urdf.xacro (robot description, xacro)
@@ -69,14 +69,14 @@
   </joint>
   <iai_generic_panel name="${name}_right_panel" parent="${name}" width="60">
-    <origin rpy="0 0 0" xyz="0.28 0.7 0.325 "/>
+    <origin rpy="0 0 0" xyz="0.28 0.7 0.355 "/>
   </iai_generic_panel>
   <iai_drawer_60_58 name="${name}_trash_drawer" parent="${name}">
-    <origin rpy="0 0 0" xyz="0.01 0.7 -0.035 "/>
+    <origin rpy="0 0 0" xyz="0.01 0.7 -0.015 "/>
   </iai_drawer_60_58>
   <iai_drawer_80_14 name="${name}_left_upper_drawer" parent="${name}">
-    <origin rpy="0 0 0" xyz="0.01 -0.6 0.325 "/>
+    <origin rpy="0 0 0" xyz="0.01 -0.6 0.345 "/>
   </iai_drawer_80_14>
   <iai_drawer_80_29 name="${name}_left_middle_drawer" parent="${name}">
-    <origin rpy="0 0 0" xyz="0.01 -0.6 0.11 "/>
+    <origin rpy="0 0 0" xyz="0.01 -0.6 0.12 "/>
   </iai_drawer_80_29>
   <iai_drawer_80_29 name="${name}_left_bottom_drawer" parent="${name}">
@@ -84,5 +84,5 @@
   </iai_drawer_80_29>
   <iai_dish_washer name="${name}_dish_washer" parent="${name}">
-    <origin rpy="0 0 0" xyz="0.01 0.1 0.035 "/>
+    <origin rpy="0 0 0" xyz="0.01 0.1 0.044 "/>
   </iai_dish_washer>
   </macro>

Commit message: reverted some urdf offset changes and applied offset changes to old urdf

File: iai_kitchen/urdf/IAI_kitchen.urdf.xacro (robot description, xacro)
@@ -35,8 +35,8 @@
   <xacro:include filename="$(find iai_kitchen)/urdf/IAI_kitchen_walls.urdf.xacro"/>
   <iai_sink_area name="sink_area" parent="room_link">
-    <origin xyz="1.825 1.3 0" rpy="0 0 ${pi}" />
+    <origin xyz="1.825 1.32 0" rpy="0 0 ${pi}" />
   </iai_sink_area>
   <iai_oven_area name="oven_area" parent="room_link">
-    <origin xyz="1.805 2.5 0" rpy="0 0 ${pi}" />
+    <origin xyz="1.805 2.52 0" rpy="0 0 ${pi}" />
   </iai_oven_area>
   <iai_kitchen_island name="kitchen_island" parent="room_link">
@@ -44,5 +44,5 @@
   </iai_kitchen_island>
   <iai_fridge_area name="fridge_area" parent="room_link">
-    <origin xyz="1.825 -0.76 0" rpy="0 0 ${pi}" />
+    <origin xyz="1.825 -0.74 0" rpy="0 0 ${pi}" />
   </iai_fridge_area>
   <iai_table_1 name="table_area" parent="room_link">

File: iai_kitchen/urdf_obj/iai_kitchen_python.urdf.xacro (robot description, xacro)
@@ -35,14 +35,14 @@
   <xacro:include filename="$(find iai_kitchen)/urdf_obj/IAI_kitchen_walls.urdf.xacro"/>
   <iai_sink_area name="sink_area" parent="room_link">
-    <origin xyz="1.845 1.35 0" rpy="0 0 ${pi}" />
+    <origin xyz="1.825 1.32 0" rpy="0 0 ${pi}" />
   </iai_sink_area>
   <iai_oven_area name="oven_area" parent="room_link">
-    <origin xyz="1.825 2.55 0" rpy="0 0 ${pi}" />
+    <origin xyz="1.805 2.52 0" rpy="0 0 ${pi}" />
   </iai_oven_area>
   <iai_kitchen_island name="kitchen_island" parent="room_link">
-    <origin xyz="-1.355 0.58 0" rpy="0 0 0" />
+    <origin xyz="-1.365 0.59 0" rpy="0 0 0" />
   </iai_kitchen_island>
   <iai_fridge_area name="fridge_area" parent="room_link">
-    <origin xyz="1.845 -0.72 0" rpy="0 0 ${pi}" />
+    <origin xyz="1.825 -0.74 0" rpy="0 0 ${pi}" />
   </iai_fridge_area>
   <iai_table_1 name="table_area" parent="room_link">
