Commit message: Center meshes, adjust joint coordinates.

File: iai_kitchen/urdf/IAI_fridge.urdf.xacro (robot description, xacro)
@@ -54,5 +54,5 @@
     </joint>
     <joint name="${name}_door_joint" type="revolute">
-      <origin xyz="0.29 0.3 0.245" rpy="0 0 0" />
+      <origin xyz="0.29 0 0.245" rpy="0 0 0" />
       <parent link="${name}_main"/>
       <child link="${name}_door"/>
@@ -64,5 +64,5 @@
     </joint>
     <joint name="${name}_door_handle_joint" type="fixed">
-      <origin xyz="0.06 -0.57 0." rpy="0 0 0" />
+      <origin xyz="0.06 -0.27 0." rpy="0 0 0" />
       <parent link="${name}_door"/>
       <child link="${name}_door_handle"/>

File: iai_kitchen/urdf/IAI_sink_area.urdf.xacro (robot description, xacro)
@@ -64,5 +64,5 @@
   </link>
   <joint name="${name}_sink_joint" type="fixed">
-    <origin xyz="0.005 0.47 0.4414" rpy="0 0 0" />
+    <origin xyz="0.005 0.57 0.4114" rpy="0 0 0" />
     <parent link="${name}"/>
     <child link="${name}_sink"/>

Commit message: Revert change of coordinates for sink and fridgedoor in semantic map. Change coordinates of sink and fridgedoor in urdf. Set joint coordinates to original ones

File: iai_kitchen/urdf/IAI_fridge.urdf.xacro (robot description, xacro)
@@ -21,5 +21,5 @@
       <sphere_inertia radius="0" mass="0"/>
       <visual>
-        <origin xyz="0 0 0" rpy="0 0 0" />
+        <origin xyz="0 -0.3 0" rpy="0 0 0" />
         <geometry>
           <mesh filename="package://iai_kitchen/meshes/misc/FridgeDoor.dae"/>
@@ -27,5 +27,5 @@
       </visual>
       <collision>
-        <origin xyz="0 0 0" rpy="0 0 0" />
+        <origin xyz="0 -0.3 0" rpy="0 0 0" />
         <geometry>
           <mesh filename="package://iai_kitchen/meshes/misc/FridgeDoor.dae"/>
@@ -54,5 +54,5 @@
     </joint>
     <joint name="${name}_door_joint" type="revolute">
-      <origin xyz="0.29 0 0.245" rpy="0 0 0" />
+      <origin xyz="0.29 0.3 0.245" rpy="0 0 0" />
       <parent link="${name}_main"/>
       <child link="${name}_door"/>
@@ -64,5 +64,5 @@
     </joint>
     <joint name="${name}_door_handle_joint" type="fixed">
-      <origin xyz="0.06 -0.27 0." rpy="0 0 0" />
+      <origin xyz="0.06 -0.57 0." rpy="0 0 0" />
       <parent link="${name}_door"/>
       <child link="${name}_door_handle"/>

File: iai_kitchen/urdf/IAI_sink_area.urdf.xacro (robot description, xacro)
@@ -51,5 +51,5 @@
     <sphere_inertia radius="0" mass="0"/>
     <visual>
-      <origin xyz="0 0 0" rpy="0 0 0" />
+      <origin xyz="0 0.1 -0.03" rpy="0 0 0" />
       <geometry>
         <mesh filename="package://iai_kitchen/meshes/misc/Sink.dae"/>
@@ -57,5 +57,5 @@
     </visual>
     <collision>
-      <origin xyz="0 0 0" rpy="0 0 0" />
+      <origin xyz="0 0.1 -0.43" rpy="0 0 0" />
       <geometry>
         <mesh filename="package://iai_kitchen/meshes/misc/Sink.dae"/>
@@ -64,5 +64,5 @@
   </link>
   <joint name="${name}_sink_joint" type="fixed">
-    <origin xyz="0.005 0.57 0.4114" rpy="0 0 0" />
+    <origin xyz="0.005 0.47 0.4414" rpy="0 0 0" />
     <parent link="${name}"/>
     <child link="${name}_sink"/>

Commit message: fixed fridge door in urdf

File: iai_kitchen/urdf/IAI_fridge.urdf.xacro (robot description, xacro)
@@ -21,5 +21,5 @@
       <sphere_inertia radius="0" mass="0"/>
       <visual>
-        <origin xyz="0 -0.3 0" rpy="0 0 0" />
+        <origin xyz="0 0 0" rpy="0 0 0" />
         <geometry>
           <mesh filename="package://iai_kitchen/meshes/misc/FridgeDoor.dae"/>
@@ -27,5 +27,5 @@
       </visual>
       <collision>
-        <origin xyz="0 -0.3 0" rpy="0 0 0" />
+        <origin xyz="0 0 0" rpy="0 0 0" />
         <geometry>
           <mesh filename="package://iai_kitchen/meshes/misc/FridgeDoor.dae"/>

Commit message: no_json_obj.launch uses upload kitchen obj

File: iai_kitchen/urdf/IAI_fridge.urdf.xacro (robot description, xacro)
@@ -21,5 +21,5 @@
       <sphere_inertia radius="0" mass="0"/>
       <visual>
-        <origin xyz="0 0 0" rpy="0 0 0" />
+        <origin xyz="0 0.3 0" rpy="0 0 0" />
         <geometry>
           <mesh filename="package://iai_kitchen/meshes/misc/FridgeDoor.dae"/>
@@ -27,5 +27,5 @@
       </visual>
       <collision>
-        <origin xyz="0 0 0" rpy="0 0 0" />
+        <origin xyz="0 0.3 0" rpy="0 0 0" />
         <geometry>
           <mesh filename="package://iai_kitchen/meshes/misc/FridgeDoor.dae"/>
