Commit message: Adjusted table reference point to be in the center of the bounding box.

File: iai_kitchen/urdf/IAI_tables.urdf.xacro (robot description, xacro)
@@ -6,5 +6,5 @@
       <sphere_inertia radius="0" mass="0"/>
       <visual>
-        <origin xyz="0 0 0" rpy="0 0 0" />
+        <origin xyz="0 0 0.3619" rpy="0 0 0" />
         <geometry>
           <mesh filename="package://iai_kitchen/meshes/misc/big_table_1.dae"/>
@@ -12,5 +12,5 @@
       </visual>
       <collision>
-        <origin xyz="0 0 0" rpy="0 0 0" />
+        <origin xyz="0 0 0.3619" rpy="0 0 0" />
         <geometry>
           <mesh filename="package://iai_kitchen/meshes/misc/big_table_1.stl"/>

File: iai_kitchen/urdf_obj/IAI_tables.urdf.xacro (robot description, xacro)
@@ -6,5 +6,5 @@
       <sphere_inertia radius="0" mass="0"/>
       <visual>
-        <origin xyz="0 0 0" rpy="0 0 0" />
+        <origin xyz="0 0 0.3619" rpy="0 0 0" />
         <geometry>
           <mesh filename="package://iai_kitchen/meshes/misc/big_table_1.obj"/>
@@ -12,5 +12,5 @@
       </visual>
       <collision>
-        <origin xyz="0 0 0" rpy="0 0 0" />
+        <origin xyz="0 0 0.3619" rpy="0 0 0" />
         <geometry>
           <mesh filename="package://iai_kitchen/meshes/misc/big_table_1.stl"/>
