Commit message: added shelf mashes

File: iai_shelfs/urdf/shelfs.urdf (robot description, URDF)
Before this commit: robot iai_shelfs, 5 links, 4 joints
Links:
- link shelf1: geometry visual mesh filename=package://iai_shelfs/meshes/Shelf_1.dae
- link shelf2: geometry visual mesh filename=package://iai_shelfs/meshes/Shelf_2_no_texture_center_left_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
- link shelf3: geometry visual mesh filename=package://iai_shelfs/meshes/Shelf_3.dae
- link shelf4: geometry visual mesh filename=package://iai_shelfs/meshes/Shelf_4.dae
