Commit message: updated iai shelves urdf

File: iai_shelves/urdf/shelves.urdf (robot description, URDF)
Before this commit: robot iai_shelves, 5 links, 4 joints
Joints:
- joint shelf1_joint: origin xyz=-1.5 0.0 0.0 rpy=0.0 0.0 0.0 -> xyz=-0.515 0.0 0.0 rpy=0.0 0.0 3.14159265359

Commit message: renamed shelf meshes and changed color to white

File: iai_shelves/urdf/shelves.urdf (robot description, URDF)
Before this commit: robot iai_shelves, 5 links, 4 joints
Links:
- removed link shelf4
- added link shelf0; visual mesh filename=package://iai_shelves/meshes/Shelf_0.dae
- link shelf2: geometry visual mesh filename=package://iai_shelves/meshes/Shelf_2.dae
Joints:
- removed joint shelf4_joint
- added joint shelf0_joint: type fixed, parent room_link, child shelf0, origin xyz=-0.515 0.0 0.0 rpy=0.0 0.0 3.14159265359
- joint shelf1_joint: origin xyz=-0.515 0.0 0.0 rpy=0.0 0.0 3.14159265359 -> xyz=0.0 1.0 0.0 rpy=0.0 0.0 0.0; parent room_link -> shelf0
