Commit message: Added cucumber to cutting world.

File: iai_dlr_cutting_demo/urdf/map.urdf (robot description, URDF)
Before this commit: robot iai_dlr_cutting_map, 4 links, 3 joints
Links:
- added link cucumber; visual mesh filename=package://iai_dlr_cutting_demo/meshes/food-drinks/cucumber/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 scale=0.001 0.001 0.001
Joints:
- added joint cucumber_location_joint: type fixed, parent cutting_board, child cucumber, origin xyz=0.2 0.25 0.03 rpy=0 0 -1
