Commit message: urdf uses obj as collision meshes as well

File: iai_kitchen/urdf_obj/IAI_kitchen_island.urdf.xacro (robot description, xacro)
@@ -19,5 +19,5 @@
         <origin xyz="0 0 0" rpy="0 0 0" />
         <geometry>
-          <mesh filename="package://iai_kitchen/meshes/collision/kitchen_island.stl"/>
+          <mesh filename="package://iai_kitchen/meshes/racks/IslandArea.obj"/>
         </geometry>
       </collision>

File: iai_kitchen/urdf_obj/IAI_oven_area.urdf.xacro (robot description, xacro)
@@ -20,5 +20,5 @@
         <origin xyz="0 0 0" rpy="0 0 0" />
         <geometry>
-          <mesh filename="package://iai_kitchen/meshes/collision/kitchen_oven_area.stl"/>
+          <mesh filename="package://iai_kitchen/meshes/racks/OvenArea.obj"/>
         </geometry>
       </collision>

File: iai_kitchen/urdf_obj/IAI_sink_area.urdf.xacro (robot description, xacro)
@@ -20,5 +20,5 @@
         <origin xyz="0 0 0" rpy="0 0 0" />
         <geometry>
-          <mesh filename="package://iai_kitchen/meshes/collision/kitchen_sink.stl"/>
+          <mesh filename="package://iai_kitchen/meshes/racks/SinkArea.obj"/>
         </geometry>
       </collision>
@@ -33,18 +33,4 @@
     <parent link="${name}_footprint"/>
     <child link="${name}"/>
-  </joint>
-  <link name="${name}_surface">
-    <sphere_inertia radius="0" mass="0"/>
-    <collision>
-      <origin xyz="0 0 0" rpy="0 0 0" />
-      <geometry>
-        <box size="0.575 2.05 0.02"/>
-      </geometry>
-    </collision>
-  </link>
-  <joint name="${name}_surface_joint" type="fixed">
-    <origin xyz="0.0 0. 0.43" rpy="0 0 0" />
-    <parent link="${name}"/>
-    <child link="${name}_surface"/>
   </joint>
   <link name="${name}_sink">
