Commit message: calibrated offsets in obj kitchen urdf

File: iai_kitchen/urdf_obj/IAI_sink_area.urdf.xacro (robot description, xacro)
@@ -69,14 +69,14 @@
   </joint>
   <iai_generic_panel name="${name}_right_panel" parent="${name}" width="60">
-    <origin rpy="0 0 0" xyz="0.28 0.7 0.325 "/>
+    <origin rpy="0 0 0" xyz="0.28 0.7 0.355 "/>
   </iai_generic_panel>
   <iai_drawer_60_58 name="${name}_trash_drawer" parent="${name}">
-    <origin rpy="0 0 0" xyz="0.01 0.7 -0.035 "/>
+    <origin rpy="0 0 0" xyz="0.01 0.7 -0.015 "/>
   </iai_drawer_60_58>
   <iai_drawer_80_14 name="${name}_left_upper_drawer" parent="${name}">
-    <origin rpy="0 0 0" xyz="0.01 -0.6 0.325 "/>
+    <origin rpy="0 0 0" xyz="0.01 -0.6 0.345 "/>
   </iai_drawer_80_14>
   <iai_drawer_80_29 name="${name}_left_middle_drawer" parent="${name}">
-    <origin rpy="0 0 0" xyz="0.01 -0.6 0.11 "/>
+    <origin rpy="0 0 0" xyz="0.01 -0.6 0.12 "/>
   </iai_drawer_80_29>
   <iai_drawer_80_29 name="${name}_left_bottom_drawer" parent="${name}">
@@ -84,5 +84,5 @@
   </iai_drawer_80_29>
   <iai_dish_washer name="${name}_dish_washer" parent="${name}">
-    <origin rpy="0 0 0" xyz="0.01 0.1 0.035 "/>
+    <origin rpy="0 0 0" xyz="0.01 0.1 0.044 "/>
   </iai_dish_washer>
   </macro>

File: iai_kitchen/urdf_obj/iai_kitchen_python.urdf.xacro (robot description, xacro)
@@ -19,5 +19,5 @@
     <link name="world"/>
     <joint name="world_room_joint" type="fixed">
-        <origin xyz="0 0 0 " rpy="0 0 0" />
+        <origin xyz="0.02 -0.01 0 " rpy="0 0 0" />
         <parent link="world"/>
         <child link="room_link"/>

Commit message: added sink surface back to urdf and reduced size to not include sink

File: iai_kitchen/urdf_obj/IAI_sink_area.urdf.xacro (robot description, xacro)
@@ -34,4 +34,18 @@
     <child link="${name}"/>
   </joint>
+  <link name="${name}_surface">
+    <sphere_inertia radius="0" mass="0"/>
+    <collision>
+      <origin xyz="0 -0.225 0" rpy="0 0 0" />
+      <geometry>
+        <box size="0.575 1.6 0.02"/>
+      </geometry>
+    </collision>
+  </link>
+ <joint name="${name}_surface_joint" type="fixed">
+    <origin xyz="0.0 0. 0.43" rpy="0 0 0" />
+    <parent link="${name}"/>
+    <child link="${name}_surface"/>
+ </joint>
   <link name="${name}_sink">
     <sphere_inertia radius="0" mass="0"/>
