Commit message: [obj urdf] RViz in 18.04 complains about numbers without 0 like .3

File: iai_kitchen/urdf_obj/IAI_fridge_area.urdf.xacro (robot description, xacro)
@@ -30,5 +30,5 @@
     </joint>
     <joint name="${name}_main_joint" type="fixed">
-      <origin xyz="0.29 .3 0.74" rpy="0 0 0" />
+      <origin xyz="0.29 0.3 0.74" rpy="0 0 0" />
       <parent link="${name}_footprint"/>
       <child link="${name}"/>

File: iai_kitchen/urdf_obj/IAI_kitchen.urdf (robot description, URDF)
Before this commit: robot iai_oven_area, 60 links, 59 joints
Joints:
- joint fridge_area_main_joint: origin xyz=0.29 .3 0.74 rpy=0 0 0 -> xyz=0.29 0.3 0.74 rpy=0 0 0
