Commit message: added the grids on the left and right sioe

File: iai_kitchen/urdf_obj/IAI_popcorn_table.urdf.xacro (robot description, xacro)
@@ -139,4 +139,28 @@
       </collision>
     </link>
+    <link name="${name}_right_grid">
+      <visual>
+        <geometry>
+          <box size="0.5 0.5 0.015"/>
+        </geometry>
+      </visual>
+      <collision>
+        <geometry>
+          <box size="0.5 0.5 0.015"/>
+        </geometry>
+      </collision>
+    </link>
+    <link name="${name}_left_grid">
+      <visual>
+        <geometry>
+          <box size="0.5 0.5 0.015"/>
+        </geometry>
+      </visual>
+      <collision>
+        <geometry>
+          <box size="0.5 0.5 0.015"/>
+        </geometry>
+      </collision>
+    </link>
     <joint name="${name}_front_left_leg_joint" type="fixed">
       <origin xyz="-0.81 -0.27 0.345"/>
@@ -193,4 +217,14 @@
       <parent link="${name}_footprint"/>
       <child link="${name}_right_wall"/>
+    </joint>
+    <joint name="${name}_right_grid_joint" type="fixed">
+      <origin xyz="-0.55 0 0.18"/>
+      <parent link="${name}_footprint"/>
+      <child link="${name}_right_grid"/>
+    </joint>
+    <joint name="${name}_left_grid_joint" type="fixed">
+      <origin xyz="0.55 0 0.18"/>
+      <parent link="${name}_footprint"/>
+      <child link="${name}_left_grid"/>
     </joint>
     <iai_popcorn_table_drawer name="iai_popcorn_table_drawer_left" parent="${name}_footprint">

Commit message: adjustet the x axis of the drawer

File: iai_kitchen/urdf_obj/IAI_popcorn_table.urdf.xacro (robot description, xacro)
@@ -1,2 +1,3 @@
+<?xml version="1.0"?>
 <robot name="iai_popcorn_table" xmlns:xacro="http://ros.org/wiki/xacro">
   <macro name="iai_popcorn_table" params="name parent *origin">
@@ -229,8 +230,8 @@
     </joint>
     <iai_popcorn_table_drawer name="iai_popcorn_table_drawer_left" parent="${name}_footprint">
-      <origin xyz="0.555 0 0.53"/>
+      <origin xyz="0.555 0 0.53" rpy="0 0 ${0.5 * pi}"/>
     </iai_popcorn_table_drawer>
     <iai_popcorn_table_drawer name="iai_popcorn_table_drawer_right" parent="${name}_footprint">
-      <origin xyz="-0.555 0 0.53"/>
+      <origin xyz="-0.555 0 0.53" rpy="0 0 ${0.5 * pi}"/>
     </iai_popcorn_table_drawer>
     <iai_popcorn_stove_knob name="iai_popcorn_stove_knob_1" parent="${name}_stove">
@@ -247,9 +248,10 @@
   <joint name="${name}_table_joint" type="prismatic">
         <parent link="${parent}"/>
-        <child link="${name}_bottom"/>
+        <child link="${name}_base"/>
         <limit effort="1000.0" lower="0" upper="0.4" velocity="0.5"/>
-        <axis xyz="0 1 0 "/>
+        <axis xyz="1 0 0 "/>
         <xacro:insert_block name="origin"/>
   </joint>
+  <link name="${name}_base" />
   <link name="${name}_bottom">
     <visual>
@@ -312,4 +314,9 @@
     </collision>
   </link>
+  <joint name="${name}_bottom_side_joint" type="fixed">
+    <origin xyz="0 0 0" rpy="0 0 ${1.5*pi}"/>
+    <parent link="${name}_base"/>
+    <child link="${name}_bottom"/>
+  </joint>
   <joint name="${name}_right_side_joint" type="fixed">
     <origin xyz="0.205 0 0.065"/>

Commit message: rotated the drawer so x axis point to the front

File: iai_kitchen/urdf_obj/IAI_popcorn_table.urdf.xacro (robot description, xacro)
@@ -248,12 +248,12 @@
   <joint name="${name}_table_joint" type="prismatic">
         <parent link="${parent}"/>
-        <child link="${name}_base"/>
+        <child link="${name}_main"/>
         <limit effort="1000.0" lower="0" upper="0.4" velocity="0.5"/>
         <axis xyz="1 0 0 "/>
         <xacro:insert_block name="origin"/>
   </joint>
-  <link name="${name}_base" />
-  <link name="${name}_bottom">
-    <visual>
+  <link name="${name}_main">
+    <visual>
+      <origin rpy="0 0 ${1.5 *pi}"/>
       <geometry>
         <box size="0.42 0.52 0.01"/>
@@ -261,4 +261,5 @@
     </visual>
     <collision>
+      <origin rpy="0 0 ${1.5 *pi}"/>
       <geometry>
         <box size="0.42 0.52 0.01"/>
@@ -314,31 +315,26 @@
     </collision>
   </link>
-  <joint name="${name}_bottom_side_joint" type="fixed">
-    <origin xyz="0 0 0" rpy="0 0 ${1.5*pi}"/>
-    <parent link="${name}_base"/>
-    <child link="${name}_bottom"/>
-  </joint>
   <joint name="${name}_right_side_joint" type="fixed">
-    <origin xyz="0.205 0 0.065"/>
-    <parent link="${name}_bottom"/>
+    <origin xyz="0 0.205 0.065" rpy="0 0 ${0.5 * pi}"/>
+    <parent link="${name}_main"/>
     <child link="${name}_right_side"/>
   </joint>
   <joint name="${name}_left_side_joint" type="fixed">
-    <origin xyz="-0.205 0 0.065"/>
-    <parent link="${name}_bottom"/>
+    <origin xyz="0 -0.205 0.065" rpy="0 0 ${0.5 * pi}"/>
+    <parent link="${name}_main"/>
     <child link="${name}_left_side"/>
   </joint>
   <joint name="${name}_back_side_joint" type="fixed">
-    <origin xyz="0 -0.255 0.065"/>
-    <parent link="${name}_bottom"/>
+    <origin xyz=" -0.255 0 0.065" rpy="0 0 ${0.5 * pi}"/>
+    <parent link="${name}_main"/>
     <child link="${name}_back_side"/>
   </joint>
   <joint name="${name}_front_side_joint" type="fixed">
-    <origin xyz="0 0.255 0.075"/>
-    <parent link="${name}_bottom"/>
+    <origin xyz=" 0.255 0 0.075" rpy="0 0 ${1.5 * pi}"/>
+    <parent link="${name}_main"/>
     <child link="${name}_front_side"/>
   </joint>
   <iai_popcorn_table_drawer_handle name="${name}_handle" parent="${name}_front_side">
-    <origin xyz="0 0.03 0"/>
+    <origin xyz="0 0.03 0" rpy="0 0 ${0.5 * pi}"/>
   </iai_popcorn_table_drawer_handle>
   </macro>
@@ -346,4 +342,5 @@
   <link name="${name}_left_part">
     <visual>
+      <origin rpy="0 0  ${1.5 * pi}"/>
       <geometry>
         <box size="0.01 0.03 0.01"/>
@@ -351,4 +348,5 @@
     </visual>
     <collision>
+      <origin rpy="0 0  ${1.5 * pi}"/>
       <geometry>
         <box size="0.01 0.03 0.01"/>
@@ -358,4 +356,5 @@
   <link name="${name}_right_part">
     <visual>
+      <origin rpy="0 0  ${1.5 * pi}"/>
       <geometry>
         <box size="0.01 0.03 0.01"/>
@@ -363,4 +362,5 @@
     </visual>
     <collision>
+      <origin rpy="0 0  ${1.5 * pi}"/>
       <geometry>
         <box size="0.01 0.03 0.01"/>
@@ -370,4 +370,5 @@
   <link name="${name}_middle_part">
     <visual>
+      <origin rpy="0 0  ${1.5 * pi}"/>
       <geometry>
         <box size="0.3 0.01 0.01"/>
@@ -375,4 +376,5 @@
     </visual>
     <collision>
+      <origin rpy="0 0  ${1.5 * pi}"/>
       <geometry>
         <box size="0.3 0.01 0.01"/>
@@ -381,10 +383,10 @@
   </link>
   <joint name="${name}_left_middle_joint" type="fixed">
-    <origin xyz="-0.15 -0.01 0"/>
+    <origin xyz="-0.01 -0.15  0"/>
     <parent link="${name}_middle_part"/>
     <child link="${name}_left_part"/>
   </joint>
   <joint name="${name}_right_middle_joint" type="fixed">
-    <origin xyz="0.15 -0.01 0"/>
+    <origin xyz="-0.01 0.15  0"/>
     <parent link="${name}_middle_part"/>
     <child link="${name}_right_part"/>

Commit message: removed rotation of links

File: iai_kitchen/urdf_obj/IAI_popcorn_table.urdf.xacro (robot description, xacro)
@@ -255,13 +255,11 @@
   <link name="${name}_main">
     <visual>
-      <origin rpy="0 0 ${1.5 *pi}"/>
-      <geometry>
-        <box size="0.42 0.52 0.01"/>
-      </geometry>
-    </visual>
-    <collision>
-      <origin rpy="0 0 ${1.5 *pi}"/>
-      <geometry>
-        <box size="0.42 0.52 0.01"/>
+      <geometry>
+        <box size="0.52 0.42 0.01"/>
+      </geometry>
+    </visual>
+    <collision>
+      <geometry>
+        <box size="0.52 0.42 0.01"/>
       </geometry>
     </collision>
@@ -270,10 +268,10 @@
     <visual>
       <geometry>
-        <box size="0.01 0.52 0.13"/>
-      </geometry>
-    </visual>
-    <collision>
-      <geometry>
-        <box size="0.01 0.52 0.13"/>
+        <box size="0.52 0.01  0.13"/>
+      </geometry>
+    </visual>
+    <collision>
+      <geometry>
+        <box size="0.52 0.01 0.13"/>
       </geometry>
     </collision>
@@ -282,10 +280,10 @@
     <visual>
       <geometry>
-        <box size="0.01 0.52 0.13"/>
-      </geometry>
-    </visual>
-    <collision>
-      <geometry>
-        <box size="0.01 0.52 0.13"/>
+        <box size="0.52 0.01 0.13"/>
+      </geometry>
+    </visual>
+    <collision>
+      <geometry>
+        <box size=" 0.52 0.01 0.13"/>
       </geometry>
     </collision>
@@ -294,10 +292,10 @@
     <visual>
       <geometry>
-        <box size="0.42 0.01 0.13"/>
-      </geometry>
-    </visual>
-    <collision>
-      <geometry>
-        <box size="0.42 0.01 0.13"/>
+        <box size="0.01 0.42  0.13"/>
+      </geometry>
+    </visual>
+    <collision>
+      <geometry>
+        <box size="0.01 0.42 0.13"/>
       </geometry>
     </collision>
@@ -306,35 +304,35 @@
     <visual>
       <geometry>
-        <box size="0.46 0.01 0.13"/>
-      </geometry>
-    </visual>
-    <collision>
-      <geometry>
-        <box size="0.46 0.01 0.15"/>
+        <box size="0.01 0.46  0.13"/>
+      </geometry>
+    </visual>
+    <collision>
+      <geometry>
+        <box size="0.01 0.46 0.15"/>
       </geometry>
     </collision>
   </link>
   <joint name="${name}_right_side_joint" type="fixed">
-    <origin xyz="0 0.205 0.065" rpy="0 0 ${0.5 * pi}"/>
+    <origin xyz="0 0.205 0.065"/>
     <parent link="${name}_main"/>
     <child link="${name}_right_side"/>
   </joint>
   <joint name="${name}_left_side_joint" type="fixed">
-    <origin xyz="0 -0.205 0.065" rpy="0 0 ${0.5 * pi}"/>
+    <origin xyz="0 -0.205 0.065" />
     <parent link="${name}_main"/>
     <child link="${name}_left_side"/>
   </joint>
   <joint name="${name}_back_side_joint" type="fixed">
-    <origin xyz=" -0.255 0 0.065" rpy="0 0 ${0.5 * pi}"/>
+    <origin xyz=" -0.255 0 0.065" />
     <parent link="${name}_main"/>
     <child link="${name}_back_side"/>
   </joint>
   <joint name="${name}_front_side_joint" type="fixed">
-    <origin xyz=" 0.255 0 0.075" rpy="0 0 ${1.5 * pi}"/>
+    <origin xyz=" 0.255 0 0.075" />
     <parent link="${name}_main"/>
     <child link="${name}_front_side"/>
   </joint>
   <iai_popcorn_table_drawer_handle name="${name}_handle" parent="${name}_front_side">
-    <origin xyz="0 0.03 0" rpy="0 0 ${0.5 * pi}"/>
+    <origin xyz="0.03 0 0"/>
   </iai_popcorn_table_drawer_handle>
   </macro>
@@ -342,13 +340,11 @@
   <link name="${name}_left_part">
     <visual>
-      <origin rpy="0 0  ${1.5 * pi}"/>
-      <geometry>
-        <box size="0.01 0.03 0.01"/>
-      </geometry>
-    </visual>
-    <collision>
-      <origin rpy="0 0  ${1.5 * pi}"/>
-      <geometry>
-        <box size="0.01 0.03 0.01"/>
+      <geometry>
+        <box size="0.03 0.01 0.01"/>
+      </geometry>
+    </visual>
+    <collision>
+      <geometry>
+        <box size="0.03 0.01  0.01"/>
       </geometry>
     </collision>
@@ -356,13 +352,11 @@
   <link name="${name}_right_part">
     <visual>
-      <origin rpy="0 0  ${1.5 * pi}"/>
-      <geometry>
-        <box size="0.01 0.03 0.01"/>
-      </geometry>
-    </visual>
-    <collision>
-      <origin rpy="0 0  ${1.5 * pi}"/>
-      <geometry>
-        <box size="0.01 0.03 0.01"/>
+      <geometry>
+        <box size="0.03 0.01 0.01"/>
+      </geometry>
+    </visual>
+    <collision>
+      <geometry>
+        <box size="0.03 0.01 0.01"/>
       </geometry>
     </collision>
@@ -370,13 +364,11 @@
   <link name="${name}_middle_part">
     <visual>
-      <origin rpy="0 0  ${1.5 * pi}"/>
-      <geometry>
-        <box size="0.3 0.01 0.01"/>
-      </geometry>
-    </visual>
-    <collision>
-      <origin rpy="0 0  ${1.5 * pi}"/>
-      <geometry>
-        <box size="0.3 0.01 0.01"/>
+      <geometry>
+        <box size="0.01 0.3 0.01"/>
+      </geometry>
+    </visual>
+    <collision>
+      <geometry>
+        <box size="0.01 0.3 0.01"/>
       </geometry>
     </collision>
