Commit message: increased upper limit for oven door joint

File: iai_kitchen/urdf_obj/IAI_oven.urdf.xacro (robot description, xacro)
@@ -80,5 +80,5 @@
         -->
         <!-- FIXME make the closed position stable -->
-        <limit lower="0" upper="0." effort="0.03" velocity="10"/>
+        <limit lower="0" upper="${0.5*pi}" effort="0.03" velocity="10"/>
         <dynamics damping="100.1"/>
       </joint>
