Commit message: clean up

File: iai_kitchen/urdf_obj/IAI_drawers.urdf.xacro (robot description, xacro)
@@ -40,415 +40,346 @@
   <macro name="iai_vdrawer" params="name parent *origin">
       <joint name="${name}_joint" type="prismatic">
-          <xacro:insert_block name="origin"/>
-          <parent link="${parent}"/>
-          <child link="${name}_main"/>
-    <axis xyz="0.999 0 0.044"/>
-    <!--  the axis needs to be slightly tilted so that the drawers would stay closed in Gazebo-->
-    <limit effort="300" lower="0" upper="0.48" velocity="10"/>
-</joint>
-<link name="${name}_main">
-    <inertial>
-      <mass value="0.1"/>
-      <inertia ixx="4e-08" ixy="0" ixz="0" iyy="4e-08" iyz="0" izz="4e-08"/>
-    </inertial>
-</link>
-<joint name="${name}_front_joint" type="fixed">
-    <origin rpy="0 0. 0" xyz="0.25 0 0"/>
-    <parent link="${name}_main"/>
-    <child link="${name}_front_link"/>
-    <!--
-    <axis xyz="0.999 0 0.044"/>
-     the axis needs to be slightly tilted so that the drawers would stay closed in Gazebo
-    <limit effort="300" lower="0" upper="0.48" velocity="10"/>
-    -->
-</joint>
-<link name="${name}_front_link">
-      <inertial>
-        <mass value="1.0"/>
-        <inertia ixx="0.153554166667" ixy="0" ixz="0" iyy="0.0348041666667" iyz="0" izz="0.173854166667"/>
-      </inertial>
-    <visual>
-      <origin rpy="0 0 0" xyz="0 0 0"/>
-      <geometry>
-        <box size="0.025 0.295 1.325"/>
-      </geometry>
-    </visual>
-    <collision>
-      <origin rpy="0 0 0" xyz="0 0 0"/>
-      <geometry>
-        <box size="0.025 0.3 1.33"/>
-      </geometry>
-    </collision>
-</link>
+        <xacro:insert_block name="origin"/>
+        <parent link="${parent}"/>
+        <child link="${name}_main"/>
+        <axis xyz="0.999 0 0.044"/>
+        <!--  the axis needs to be slightly tilted so that the drawers would stay closed in Gazebo-->
+        <limit effort="300" lower="0" upper="0.48" velocity="10"/>
+    </joint>
+    <link name="${name}_main">
+        <inertial>
+            <mass value="0.1"/>
+            <inertia ixx="4e-08" ixy="0" ixz="0" iyy="4e-08" iyz="0" izz="4e-08"/>
+        </inertial>
+    </link>
+    <joint name="${name}_front_joint" type="fixed">
+        <origin rpy="0 0. 0" xyz="0.25 0 0"/>
+        <parent link="${name}_main"/>
+        <child link="${name}_front_link"/>
+   </joint>
+    <link name="${name}_front_link">
+        <inertial>
+            <mass value="1.0"/>
+            <inertia ixx="0.153554166667" ixy="0" ixz="0" iyy="0.0348041666667" iyz="0" izz="0.173854166667"/>
+        </inertial>
+        <visual>
+            <origin rpy="0 0 0" xyz="0 0 0"/>
+            <geometry>
+                <box size="0.025 0.295 1.325"/>
+            </geometry>
+        </visual>
+        <collision>
+            <origin rpy="0 0 0" xyz="0 0 0"/>
+            <geometry>
+                <box size="0.025 0.3 1.33"/>
+            </geometry>
+        </collision>
+    </link>
 <!-- Board 0 -->
-<link name="${name}_board0_link">
-    <inertial>
-        <mass value="1.0"/>
-        <inertia ixx="0.153554166667" ixy="0" ixz="0" iyy="0.0348041666667" iyz="0" izz="0.173854166667"/>
-      </inertial>
-    <visual>
-        <origin rpy="0 0 0" xyz="0 0 0"/>
-        <geometry>
-            <box size="0.49 0.27 0.025"/>
-        </geometry>
-    </visual>
-    <collision>
-            <origin rpy="0 0 0" xyz="0 0 0"/>
-        <geometry>
-            <box size="0.49 0.27 0.025"/>
-        </geometry>
-    </collision>
-</link>
-<joint name="${name}_board0_joint" type="fixed">
-    <origin xyz="0 0 -0.655"/>
-    <parent link="${name}_main"/>
-    <child link="${name}_board0_link"/>
-    <!--
-    <axis xyz="0.999 0 0.044"/>
-     the axis needs to be slightly tilted so that the drawers would stay closed in Gazebo
-    <limit effort="300" lower="0" upper="0.48" velocity="10"/>
-    -->
-</joint>
-<link name="${name}_board0_barrier_right_link">
-    <inertial>
-        <mass value="1.0"/>
-        <inertia ixx="0.153554166667" ixy="0" ixz="0" iyy="0.0348041666667" iyz="0" izz="0.173854166667"/>
-    </inertial>
-    <visual>
-        <origin rpy="0 0 0" xyz="0 0 0"/>
-        <geometry>
-            <box size="0.49 0.02 0.05"/>
-        </geometry>
-    </visual>
-    <collision>
-            <origin rpy="0 0 0" xyz="0 0 0"/>
-        <geometry>
-            <box size="0.49 0.02 0.05"/>
-        </geometry>
-    </collision>
-</link>
-<joint name="${name}_board0_barrier_right_joint" type="fixed">
-    <origin xyz="0 -0.135 -0.62"/>
-    <parent link="${name}_main"/>
-    <child link="${name}_board0_barrier_right_link"/>
-</joint>
-<link name="${name}_board0_barrier_left_link">
-    <inertial>
-        <mass value="1.0"/>
-        <inertia ixx="0.153554166667" ixy="0" ixz="0" iyy="0.0348041666667" iyz="0" izz="0.173854166667"/>
-    </inertial>
-    <visual>
-        <origin rpy="0 0 0" xyz="0 0 0"/>
-        <geometry>
-            <box size="0.49 0.02 0.05"/>
-        </geometry>
-    </visual>
-    <collision>
-            <origin rpy="0 0 0" xyz="0 0 0"/>
-        <geometry>
-            <box size="0.49 0.02 0.05"/>
-        </geometry>
-    </collision>
-</link>
-<joint name="${name}_board0_barrier_left_joint" type="fixed">
-    <origin xyz="0 0.135 -0.62"/>
-    <parent link="${name}_main"/>
-    <child link="${name}_board0_barrier_left_link"/>
-</joint>
+    <link name="${name}_board0_link">
+        <inertial>
+            <mass value="1.0"/>
+            <inertia ixx="0.153554166667" ixy="0" ixz="0" iyy="0.0348041666667" iyz="0" izz="0.173854166667"/>
+        </inertial>
+        <visual>
+            <origin rpy="0 0 0" xyz="0 0 0"/>
+            <geometry>
+                <box size="0.49 0.27 0.025"/>
+            </geometry>
+        </visual>
+        <collision>
+            <origin rpy="0 0 0" xyz="0 0 0"/>
+            <geometry>
+                <box size="0.49 0.27 0.025"/>
+            </geometry>
+        </collision>
+    </link>
+    <joint name="${name}_board0_joint" type="fixed">
+        <origin xyz="0 0 -0.655"/>
+        <parent link="${name}_main"/>
+        <child link="${name}_board0_link"/>
+    </joint>
+    <link name="${name}_board0_barrier_right_link">
+        <inertial>
+            <mass value="1.0"/>
+            <inertia ixx="0.153554166667" ixy="0" ixz="0" iyy="0.0348041666667" iyz="0" izz="0.173854166667"/>
+        </inertial>
+        <visual>
+            <origin rpy="0 0 0" xyz="0 0 0"/>
+            <geometry>
+                <box size="0.49 0.02 0.05"/>
+            </geometry>
+        </visual>
+        <collision>
+            <origin rpy="0 0 0" xyz="0 0 0"/>
+            <geometry>
+                <box size="0.49 0.02 0.05"/>
+            </geometry>
+        </collision>
+    </link>
+    <joint name="${name}_board0_barrier_right_joint" type="fixed">
+        <origin xyz="0 -0.135 -0.62"/>
+        <parent link="${name}_main"/>
+        <child link="${name}_board0_barrier_right_link"/>
+    </joint>
+    <link name="${name}_board0_barrier_left_link">
+        <inertial>
+            <mass value="1.0"/>
+            <inertia ixx="0.153554166667" ixy="0" ixz="0" iyy="0.0348041666667" iyz="0" izz="0.173854166667"/>
+        </inertial>
+        <visual>
+            <origin rpy="0 0 0" xyz="0 0 0"/>
+            <geometry>
+                <box size="0.49 0.02 0.05"/>
+            </geometry>
+        </visual>
+        <collision>
+            <origin rpy="0 0 0" xyz="0 0 0"/>
+            <geometry>
+                <box size="0.49 0.02 0.05"/>
+            </geometry>
+        </collision>
+    </link>
+    <joint name="${name}_board0_barrier_left_joint" type="fixed">
+        <origin xyz="0 0.135 -0.62"/>
+        <parent link="${name}_main"/>
+        <child link="${name}_board0_barrier_left_link"/>
+    </joint>
 <!-- Board 1 -->
-<link name="${name}_board1_link">
-    <inertial>
-        <mass value="1.0"/>
-        <inertia ixx="0.153554166667" ixy="0" ixz="0" iyy="0.0348041666667" iyz="0" izz="0.173854166667"/>
-      </inertial>
-    <visual>
-        <origin rpy="0 0 0" xyz="0 0 0"/>
-        <geometry>
-            <box size="0.49 0.27 0.025"/>
-        </geometry>
-    </visual>
-    <collision>
-            <origin rpy="0 0 0" xyz="0 0 0"/>
-        <geometry>
-            <box size="0.49 0.27 0.025"/>
-        </geometry>
-    </collision>
-</link>
-<joint name="${name}_board1_joint" type="fixed">
-    <origin xyz="0 0 -0.33"/>
-    <parent link="${name}_main"/>
-    <child link="${name}_board1_link"/>
-</joint>
-<link name="${name}_board1_barrier_right_link">
-    <inertial>
-        <mass value="1.0"/>
-        <inertia ixx="0.153554166667" ixy="0" ixz="0" iyy="0.0348041666667" iyz="0" izz="0.173854166667"/>
-    </inertial>
-    <visual>
-        <origin rpy="0 0 0" xyz="0 0 0"/>
-        <geometry>
-            <box size="0.49 0.02 0.05"/>
-        </geometry>
-    </visual>
-    <collision>
-            <origin rpy="0 0 0" xyz="0 0 0"/>
-        <geometry>
-            <box size="0.49 0.02 0.05"/>
-        </geometry>
-    </collision>
-</link>
-<joint name="${name}_board1_barrier_right_joint" type="fixed">
-    <origin xyz="0 -0.135 -0.295"/>
-    <parent link="${name}_main"/>
-    <child link="${name}_board1_barrier_right_link"/>
-</joint>
-<link name="${name}_board1_barrier_left_link">
-    <inertial>
-        <mass value="1.0"/>
-        <inertia ixx="0.153554166667" ixy="0" ixz="0" iyy="0.0348041666667" iyz="0" izz="0.173854166667"/>
-    </inertial>
-    <visual>
-        <origin rpy="0 0 0" xyz="0 0 0"/>
-        <geometry>
-            <box size="0.49 0.02 0.05"/>
-        </geometry>
-    </visual>
-    <collision>
-            <origin rpy="0 0 0" xyz="0 0 0"/>
-        <geometry>
-            <box size="0.49 0.02 0.05"/>
-        </geometry>
-    </collision>
-</link>
-<joint name="${name}_board1_barrier_left_joint" type="fixed">
-    <origin xyz="0 0.135 -0.295"/>
-    <parent link="${name}_main"/>
-    <child link="${name}_board1_barrier_left_link"/>
-</joint>
+    <link name="${name}_board1_link">
+        <inertial>
+            <mass value="1.0"/>
+            <inertia ixx="0.153554166667" ixy="0" ixz="0" iyy="0.0348041666667" iyz="0" izz="0.173854166667"/>
+        </inertial>
+        <visual>
+            <origin rpy="0 0 0" xyz="0 0 0"/>
+            <geometry>
+                <box size="0.49 0.27 0.025"/>
+            </geometry>
+        </visual>
+        <collision>
+            <origin rpy="0 0 0" xyz="0 0 0"/>
+            <geometry>
+                <box size="0.49 0.27 0.025"/>
+            </geometry>
+        </collision>
+    </link>
+    <joint name="${name}_board1_joint" type="fixed">
+        <origin xyz="0 0 -0.33"/>
+        <parent link="${name}_main"/>
+        <child link="${name}_board1_link"/>
+    </joint>
+    <link name="${name}_board1_barrier_right_link">
+        <inertial>
+            <mass value="1.0"/>
+            <inertia ixx="0.153554166667" ixy="0" ixz="0" iyy="0.0348041666667" iyz="0" izz="0.173854166667"/>
+        </inertial>
+        <visual>
+            <origin rpy="0 0 0" xyz="0 0 0"/>
+            <geometry>
+                <box size="0.49 0.02 0.05"/>
+            </geometry>
+        </visual>
+        <collision>
+            <origin rpy="0 0 0" xyz="0 0 0"/>
+            <geometry>
+                <box size="0.49 0.02 0.05"/>
+            </geometry>
+        </collision>
+    </link>
+    <joint name="${name}_board1_barrier_right_joint" type="fixed">
+        <origin xyz="0 -0.135 -0.295"/>
+        <parent link="${name}_main"/>
+        <child link="${name}_board1_barrier_right_link"/>
+    </joint>
+    <link name="${name}_board1_barrier_left_link">
+        <inertial>
+            <mass value="1.0"/>
+            <inertia ixx="0.153554166667" ixy="0" ixz="0" iyy="0.0348041666667" iyz="0" izz="0.173854166667"/>
+        </inertial>
+        <visual>
+            <origin rpy="0 0 0" xyz="0 0 0"/>
+            <geometry>
+                <box size="0.49 0.02 0.05"/>
+            </geometry>
+        </visual>
+        <collision>
+            <origin rpy="0 0 0" xyz="0 0 0"/>
+            <geometry>
+                <box size="0.49 0.02 0.05"/>
+            </geometry>
+        </collision>
+    </link>
+    <joint name="${name}_board1_barrier_left_joint" type="fixed">
+        <origin xyz="0 0.135 -0.295"/>
+        <parent link="${name}_main"/>
+        <child link="${name}_board1_barrier_left_link"/>
+    </joint>
 <!-- Board 2 -->
-<link name="${name}_board2_link">
-    <inertial>
-        <mass value="1.0"/>
-        <inertia ixx="0.153554166667" ixy="0" ixz="0" iyy="0.0348041666667" iyz="0" izz="0.173854166667"/>
-      </inertial>
-    <visual>
-        <origin rpy="0 0 0" xyz="0 0 0"/>
-        <geometry>
-            <box size="0.49 0.27 0.025"/>
-        </geometry>
-    </visual>
-    <collision>
-            <origin rpy="0 0 0" xyz="0 0 0"/>
-        <geometry>
-            <box size="0.49 0.27 0.025"/>
-        </geometry>
-    </collision>
-</link>
-<joint name="${name}_board2_joint" type="fixed">
-    <origin xyz="0 0 0"/>
-    <parent link="${name}_main"/>
-    <child link="${name}_board2_link"/>
-</joint>
-<link name="${name}_board2_barrier_right_link">
-    <inertial>
-        <mass value="1.0"/>
-        <inertia ixx="0.153554166667" ixy="0" ixz="0" iyy="0.0348041666667" iyz="0" izz="0.173854166667"/>
-    </inertial>
-    <visual>
-        <origin rpy="0 0 0" xyz="0 0 0"/>
-        <geometry>
-            <box size="0.49 0.02 0.05"/>
-        </geometry>
-    </visual>
-    <collision>
-            <origin rpy="0 0 0" xyz="0 0 0"/>
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