Commit message: [iai_kitchen] used a macro to avoid copy paste

File: iai_kitchen/urdf_obj/IAI_drawers.urdf.xacro (robot description, xacro)
@@ -38,400 +38,174 @@
     </iai_generic_drawer>
   </macro>
+  <macro name="iai_vdrawer_board" params="name parent joint_origin_z">
+    <link name="${parent}_${name}_link">
+      <sphere_inertia radius="0" mass="0"/>
+      <visual>
+        <origin rpy="0 0 0" xyz="0 0 0"/>
+        <geometry>
+          <box size="0.49 0.27 0.025"/>
+        </geometry>
+      </visual>
+      <collision>
+        <origin rpy="0 0 0" xyz="0 0 0"/>
+        <geometry>
+          <box size="0.49 0.27 0.025"/>
+        </geometry>
+      </collision>
+    </link>
+    <joint name="${parent}_${name}_joint" type="fixed">
+      <origin xyz="0 0 ${joint_origin_z}"/>
+      <parent link="${parent}_main"/>
+      <child link="${parent}_${name}_link"/>
+    </joint>
+    <link name="${parent}_${name}_barrier_right_link">
+      <sphere_inertia radius="0" mass="0"/>
+      <visual>
+        <origin rpy="0 0 0" xyz="0 0 0"/>
+        <geometry>
+          <box size="0.49 0.02 0.05"/>
+        </geometry>
+      </visual>
+      <collision>
+        <origin rpy="0 0 0" xyz="0 0 0"/>
+        <geometry>
+          <box size="0.49 0.02 0.05"/>
+        </geometry>
+      </collision>
+    </link>
+    <joint name="${parent}_${name}_barrier_right_joint" type="fixed">
+      <origin xyz="0 -0.135 ${joint_origin_z + 0.035}"/>
+      <parent link="${parent}_main"/>
+      <child link="${parent}_${name}_barrier_right_link"/>
+    </joint>
+    <link name="${parent}_${name}_barrier_left_link">
+      <sphere_inertia radius="0" mass="0"/>
+      <visual>
+        <origin rpy="0 0 0" xyz="0 0 0"/>
+        <geometry>
+          <box size="0.49 0.02 0.05"/>
+        </geometry>
+      </visual>
+      <collision>
+        <origin rpy="0 0 0" xyz="0 0 0"/>
+        <geometry>
+          <box size="0.49 0.02 0.05"/>
+        </geometry>
+      </collision>
+    </link>
+    <joint name="${parent}_${name}_barrier_left_joint" type="fixed">
+      <origin xyz="0 0.135 ${joint_origin_z + 0.035}"/>
+      <parent link="${parent}_main"/>
+      <child link="${parent}_${name}_barrier_left_link"/>
+    </joint>
+  </macro>
   <macro name="iai_vdrawer" params="name parent *origin">
-      <joint name="${name}_joint" type="prismatic">
-        <xacro:insert_block name="origin"/>
-        <parent link="${parent}"/>
-        <child link="${name}_main"/>
-        <axis xyz="0.999 0 0.044"/>
-        <!--  the axis needs to be slightly tilted so that the drawers would stay closed in Gazebo-->
-        <limit effort="300" lower="0" upper="0.48" velocity="10"/>
-    </joint>
     <link name="${name}_main">
-        <inertial>
-            <mass value="0.1"/>
-            <inertia ixx="4e-08" ixy="0" ixz="0" iyy="4e-08" iyz="0" izz="4e-08"/>
-        </inertial>
-    </link>
-    <joint name="${name}_front_joint" type="fixed">
-        <origin rpy="0 0. 0" xyz="0.25 0 0"/>
-        <parent link="${name}_main"/>
-        <child link="${name}_front_link"/>
-   </joint>
-    <link name="${name}_front_link">
-        <inertial>
-            <mass value="1.0"/>
-            <inertia ixx="0.153554166667" ixy="0" ixz="0" iyy="0.0348041666667" iyz="0" izz="0.173854166667"/>
-        </inertial>
-        <visual>
-            <origin rpy="0 0 0" xyz="0 0 0"/>
-            <geometry>
-                <box size="0.025 0.295 1.325"/>
-            </geometry>
-        </visual>
-        <collision>
-            <origin rpy="0 0 0" xyz="0 0 0"/>
-            <geometry>
-                <box size="0.025 0.3 1.33"/>
-            </geometry>
-        </collision>
-    </link>
-<!-- Board 0 -->
-    <link name="${name}_board0_link">
-        <inertial>
-            <mass value="1.0"/>
-            <inertia ixx="0.153554166667" ixy="0" ixz="0" iyy="0.0348041666667" iyz="0" izz="0.173854166667"/>
-        </inertial>
-        <visual>
-            <origin rpy="0 0 0" xyz="0 0 0"/>
-            <geometry>
-                <box size="0.49 0.27 0.025"/>
-            </geometry>
-        </visual>
-        <collision>
-            <origin rpy="0 0 0" xyz="0 0 0"/>
-            <geometry>
-                <box size="0.49 0.27 0.025"/>
-            </geometry>
-        </collision>
-    </link>
-    <joint name="${name}_board0_joint" type="fixed">
-        <origin xyz="0 0 -0.655"/>
-        <parent link="${name}_main"/>
-        <child link="${name}_board0_link"/>
-    </joint>
-    <link name="${name}_board0_barrier_right_link">
-        <inertial>
-            <mass value="1.0"/>
-            <inertia ixx="0.153554166667" ixy="0" ixz="0" iyy="0.0348041666667" iyz="0" izz="0.173854166667"/>
-        </inertial>
-        <visual>
-            <origin rpy="0 0 0" xyz="0 0 0"/>
-            <geometry>
-                <box size="0.49 0.02 0.05"/>
-            </geometry>
-        </visual>
-        <collision>
-            <origin rpy="0 0 0" xyz="0 0 0"/>
-            <geometry>
-                <box size="0.49 0.02 0.05"/>
-            </geometry>
-        </collision>
-    </link>
-    <joint name="${name}_board0_barrier_right_joint" type="fixed">
-        <origin xyz="0 -0.135 -0.62"/>
-        <parent link="${name}_main"/>
-        <child link="${name}_board0_barrier_right_link"/>
-    </joint>
-    <link name="${name}_board0_barrier_left_link">
-        <inertial>
-            <mass value="1.0"/>
-            <inertia ixx="0.153554166667" ixy="0" ixz="0" iyy="0.0348041666667" iyz="0" izz="0.173854166667"/>
-        </inertial>
-        <visual>
-            <origin rpy="0 0 0" xyz="0 0 0"/>
-            <geometry>
-                <box size="0.49 0.02 0.05"/>
-            </geometry>
-        </visual>
-        <collision>
-            <origin rpy="0 0 0" xyz="0 0 0"/>
-            <geometry>
-                <box size="0.49 0.02 0.05"/>
-            </geometry>
-        </collision>
-    </link>
-    <joint name="${name}_board0_barrier_left_joint" type="fixed">
-        <origin xyz="0 0.135 -0.62"/>
-        <parent link="${name}_main"/>
-        <child link="${name}_board0_barrier_left_link"/>
-    </joint>
-<!-- Board 1 -->
-    <link name="${name}_board1_link">
-        <inertial>
-            <mass value="1.0"/>
-            <inertia ixx="0.153554166667" ixy="0" ixz="0" iyy="0.0348041666667" iyz="0" izz="0.173854166667"/>
-        </inertial>
-        <visual>
-            <origin rpy="0 0 0" xyz="0 0 0"/>
-            <geometry>
-                <box size="0.49 0.27 0.025"/>
-            </geometry>
-        </visual>
-        <collision>
-            <origin rpy="0 0 0" xyz="0 0 0"/>
-            <geometry>
-                <box size="0.49 0.27 0.025"/>
-            </geometry>
-        </collision>
-    </link>
-    <joint name="${name}_board1_joint" type="fixed">
-        <origin xyz="0 0 -0.33"/>
-        <parent link="${name}_main"/>
-        <child link="${name}_board1_link"/>
-    </joint>
-    <link name="${name}_board1_barrier_right_link">
-        <inertial>
-            <mass value="1.0"/>
-            <inertia ixx="0.153554166667" ixy="0" ixz="0" iyy="0.0348041666667" iyz="0" izz="0.173854166667"/>
-        </inertial>
-        <visual>
-            <origin rpy="0 0 0" xyz="0 0 0"/>
-            <geometry>
-                <box size="0.49 0.02 0.05"/>
-            </geometry>
-        </visual>
-        <collision>
-            <origin rpy="0 0 0" xyz="0 0 0"/>
-            <geometry>
-                <box size="0.49 0.02 0.05"/>
-            </geometry>
-        </collision>
-    </link>
-    <joint name="${name}_board1_barrier_right_joint" type="fixed">
-        <origin xyz="0 -0.135 -0.295"/>
-        <parent link="${name}_main"/>
-        <child link="${name}_board1_barrier_right_link"/>
-    </joint>
-    <link name="${name}_board1_barrier_left_link">
-        <inertial>
-            <mass value="1.0"/>
-            <inertia ixx="0.153554166667" ixy="0" ixz="0" iyy="0.0348041666667" iyz="0" izz="0.173854166667"/>
-        </inertial>
-        <visual>
-            <origin rpy="0 0 0" xyz="0 0 0"/>
-            <geometry>
-                <box size="0.49 0.02 0.05"/>
-            </geometry>
-        </visual>
-        <collision>
-            <origin rpy="0 0 0" xyz="0 0 0"/>
-            <geometry>
-                <box size="0.49 0.02 0.05"/>
-            </geometry>
-        </collision>
-    </link>
-    <joint name="${name}_board1_barrier_left_joint" type="fixed">
-        <origin xyz="0 0.135 -0.295"/>
-        <parent link="${name}_main"/>
-        <child link="${name}_board1_barrier_left_link"/>
-    </joint>
-<!-- Board 2 -->
-    <link name="${name}_board2_link">
-        <inertial>
-            <mass value="1.0"/>
-            <inertia ixx="0.153554166667" ixy="0" ixz="0" iyy="0.0348041666667" iyz="0" izz="0.173854166667"/>
-        </inertial>
-        <visual>
-            <origin rpy="0 0 0" xyz="0 0 0"/>
-            <geometry>
-                <box size="0.49 0.27 0.025"/>
-            </geometry>
-        </visual>
-        <collision>
-            <origin rpy="0 0 0" xyz="0 0 0"/>
-            <geometry>
-                <box size="0.49 0.27 0.025"/>
-            </geometry>
-        </collision>
-    </link>
-    <joint name="${name}_board2_joint" type="fixed">
-        <origin xyz="0 0 0"/>
-        <parent link="${name}_main"/>
-        <child link="${name}_board2_link"/>
-    </joint>
-    <link name="${name}_board2_barrier_right_link">
-        <inertial>
-            <mass value="1.0"/>
-            <inertia ixx="0.153554166667" ixy="0" ixz="0" iyy="0.0348041666667" iyz="0" izz="0.173854166667"/>
-        </inertial>
-        <visual>
-            <origin rpy="0 0 0" xyz="0 0 0"/>
-            <geometry>
-                <box size="0.49 0.02 0.05"/>
-            </geometry>
-        </visual>
-        <collision>
-            <origin rpy="0 0 0" xyz="0 0 0"/>
-            <geometry>
-                <box size="0.49 0.02 0.05"/>
-            </geometry>
-        </collision>
-    </link>
-    <joint name="${name}_board2_barrier_right_joint" type="fixed">
-        <origin xyz="0 -0.135 0.035"/>
-        <parent link="${name}_main"/>
-        <child link="${name}_board2_barrier_right_link"/>
-    </joint>
-    <link name="${name}_board2_barrier_left_link">
-        <inertial>
-            <mass value="1.0"/>
-            <inertia ixx="0.153554166667" ixy="0" ixz="0" iyy="0.0348041666667" iyz="0" izz="0.173854166667"/>
-        </inertial>
-        <visual>
-            <origin rpy="0 0 0" xyz="0 0 0"/>
-            <geometry>
-                <box size="0.49 0.02 0.05"/>
-            </geometry>
-        </visual>
-        <collision>
-            <origin rpy="0 0 0" xyz="0 0 0"/>
-            <geometry>
-                <box size="0.49 0.02 0.05"/>
-            </geometry>
-        </collision>
-    </link>
-    <joint name="${name}_board2_barrier_left_joint" type="fixed">
-        <origin xyz="0 0.135 0.035"/>
-        <parent link="${name}_main"/>
-        <child link="${name}_board2_barrier_left_link"/>
-    </joint>
-<!-- Board 3 -->
-    <link name="${name}_board3_link">
-        <inertial>
-            <mass value="1.0"/>
-            <inertia ixx="0.153554166667" ixy="0" ixz="0" iyy="0.0348041666667" iyz="0" izz="0.173854166667"/>
-        </inertial>
-        <visual>
-            <origin rpy="0 0 0" xyz="0 0 0"/>
-            <geometry>
-                <box size="0.49 0.27 0.025"/>
-            </geometry>
-        </visual>
-        <collision>
-            <origin rpy="0 0 0" xyz="0 0 0"/>
-            <geometry>
-                <box size="0.49 0.27 0.025"/>
-            </geometry>
-        </collision>
-    </link>
-    <joint name="${name}_board3_joint" type="fixed">
-        <origin xyz="0 0 0.33"/>
-        <parent link="${name}_main"/>
-        <child link="${name}_board3_link"/>
-    </joint>
-    <link name="${name}_board3_barrier_right_link">
-        <inertial>
-            <mass value="1.0"/>
-            <inertia ixx="0.153554166667" ixy="0" ixz="0" iyy="0.0348041666667" iyz="0" izz="0.173854166667"/>
-        </inertial>
-        <visual>
-            <origin rpy="0 0 0" xyz="0 0 0"/>
-            <geometry>
-                <box size="0.49 0.02 0.05"/>
-            </geometry>
-        </visual>
-        <collision>
-            <origin rpy="0 0 0" xyz="0 0 0"/>
-            <geometry>
-                <box size="0.49 0.02 0.05"/>
-            </geometry>
-        </collision>
-    </link>
-    <joint name="${name}_board3_barrier_right_joint" type="fixed">
-        <origin xyz="0 -0.135 0.365"/>
-        <parent link="${name}_main"/>
-        <child link="${name}_board3_barrier_right_link"/>
-    </joint>
-    <link name="${name}_board3_barrier_left_link">
-        <inertial>
-            <mass value="1.0"/>
-            <inertia ixx="0.153554166667" ixy="0" ixz="0" iyy="0.0348041666667" iyz="0" izz="0.173854166667"/>
-        </inertial>
-        <visual>
-            <origin rpy="0 0 0" xyz="0 0 0"/>
-            <geometry>
-                <box size="0.49 0.02 0.05"/>
-            </geometry>
-        </visual>
-        <collision>
-            <origin rpy="0 0 0" xyz="0 0 0"/>
-            <geometry>
-                <box size="0.49 0.02 0.05"/>
-            </geometry>
-        </collision>
-    </link>
-    <joint name="${name}_board3_barrier_left_joint" type="fixed">
-        <origin xyz="0 0.135 0.365"/>
-        <parent link="${name}_main"/>
-        <child link="${name}_board3_barrier_left_link"/>
-    </joint>
-    <!-- Joint handle to drawer -->
-    <joint name="${name}_handle_joint" type="fixed">
-        <origin rpy="0 0 0" xyz="0.05 0.0 0.0"/>
-        <parent link="${name}_front_link" />
-        <child link="${name}_handle" />
-    </joint>
+      <sphere_inertia radius="0" mass="0"/>
+    </link>
     <link name="${name}_handle">
-        <inertial>
-            <mass value="0.1"/>
-            <inertia ixx="0.0127110416667" ixy="0" ixz="0" iyy="1.66666666667e-06" iyz="0" izz="0.0127110416667"/>
-        </inertial>
-        <visual>
-            <origin rpy="0 0 0" xyz="0 0 0"/>
-            <geometry>
-                <box size="0.01 0.01 1.235"/>
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
Commit message: [iai_kitchen] added back barrier to vdrawer and some cleanup

File: iai_kitchen/urdf_obj/IAI_drawers.urdf.xacro (robot description, xacro)
@@ -38,4 +38,8 @@
     </iai_generic_drawer>
   </macro>
+  <xacro:property name="board_x" value="0.49"/>
+  <xacro:property name="board_y" value="0.25"/>
+  <xacro:property name="board_z" value="0.016"/>
+  <xacro:property name="barrier_z" value="0.082"/>
   <macro name="iai_vdrawer_board" params="name parent joint_origin_z">
     <link name="${parent}_${name}_link">
@@ -44,11 +48,11 @@
         <origin rpy="0 0 0" xyz="0 0 0"/>
         <geometry>
-          <box size="0.49 0.27 0.025"/>
-        </geometry>
-      </visual>
-      <collision>
-        <origin rpy="0 0 0" xyz="0 0 0"/>
-        <geometry>
-          <box size="0.49 0.27 0.025"/>
+          <box size="${board_x} ${board_y} ${board_z}"/>
+        </geometry>
+      </visual>
+      <collision>
+        <origin rpy="0 0 0" xyz="0 0 0"/>
+        <geometry>
+          <box size="${board_x} ${board_y} ${board_z}"/>
         </geometry>
       </collision>
@@ -64,16 +68,16 @@
         <origin rpy="0 0 0" xyz="0 0 0"/>
         <geometry>
-          <box size="0.49 0.02 0.05"/>
-        </geometry>
-      </visual>
-      <collision>
-        <origin rpy="0 0 0" xyz="0 0 0"/>
-        <geometry>
-          <box size="0.49 0.02 0.05"/>
+          <box size="${board_x} ${board_z} ${barrier_z}"/>
+        </geometry>
+      </visual>
+      <collision>
+        <origin rpy="0 0 0" xyz="0 0 0"/>
+        <geometry>
+          <box size="${board_x} ${board_z} ${barrier_z}"/>
         </geometry>
       </collision>
     </link>
     <joint name="${parent}_${name}_barrier_right_joint" type="fixed">
-      <origin xyz="0 -0.135 ${joint_origin_z + 0.035}"/>
+      <origin xyz="0 ${-board_y / 2 + board_z / 2} ${joint_origin_z + barrier_z/2 - board_z/2}"/>
       <parent link="${parent}_main"/>
       <child link="${parent}_${name}_barrier_right_link"/>
@@ -84,18 +88,38 @@
         <origin rpy="0 0 0" xyz="0 0 0"/>
         <geometry>
-          <box size="0.49 0.02 0.05"/>
-        </geometry>
-      </visual>
-      <collision>
-        <origin rpy="0 0 0" xyz="0 0 0"/>
-        <geometry>
-          <box size="0.49 0.02 0.05"/>
+          <box size="${board_x} ${board_z} ${barrier_z}"/>
+        </geometry>
+      </visual>
+      <collision>
+        <origin rpy="0 0 0" xyz="0 0 0"/>
+        <geometry>
+          <box size="${board_x} ${board_z} ${barrier_z}"/>
         </geometry>
       </collision>
     </link>
     <joint name="${parent}_${name}_barrier_left_joint" type="fixed">
-      <origin xyz="0 0.135 ${joint_origin_z + 0.035}"/>
+      <origin xyz="0 ${board_y / 2 - board_z / 2} ${joint_origin_z + barrier_z/2 - board_z/2}"/>
       <parent link="${parent}_main"/>
       <child link="${parent}_${name}_barrier_left_link"/>
+    </joint>
+    <link name="${parent}_${name}_barrier_back_link">
+      <sphere_inertia radius="0" mass="0"/>
+      <visual>
+        <origin rpy="0 0 0" xyz="0 0 0"/>
+        <geometry>
+          <box size="${board_z} ${board_y} ${barrier_z}"/>
+        </geometry>
+      </visual>
+      <collision>
+        <origin rpy="0 0 0" xyz="0 0 0"/>
+        <geometry>
+          <box size="${board_z} ${board_y} ${barrier_z}"/>
+        </geometry>
+      </collision>
+    </link>
+    <joint name="${parent}_${name}_barrier_back_joint" type="fixed">
+      <origin xyz="${-board_x / 2 + board_z / 2} 0 ${joint_origin_z + barrier_z/2 - board_z/2}"/>
+      <parent link="${parent}_main"/>
+      <child link="${parent}_${name}_barrier_back_link"/>
     </joint>
   </macro>

Commit message: rotated frame of vertical drawer handles such that y axis aligns with handle

File: iai_kitchen/urdf_obj/IAI_drawers.urdf.xacro (robot description, xacro)
@@ -131,5 +131,5 @@
       <sphere_inertia radius="0" mass="0"/>
       <visual>
-        <origin xyz="0 0 0" rpy="0 0 0" />
+        <origin xyz="0 0 0" rpy="${0.5*pi} 0 0" />
         <geometry>
           <mesh filename="package://iai_kitchen/meshes/handles/VHandle130.obj"/>
@@ -137,5 +137,5 @@
       </visual>
       <collision>
-        <origin xyz="0 0 0" rpy="0 0 0" />
+        <origin xyz="0 0 0" rpy="${0.5*pi} 0 0" />
         <geometry>
           <mesh filename="package://iai_kitchen/meshes/handles/VHandle130.obj"/>
@@ -151,5 +151,5 @@
     </joint>
     <joint name="${name}_handle_joint" type="fixed">
-      <origin rpy="0 0 0" xyz="0.05 0.0 0.0"/>
+      <origin rpy="${-0.5*pi} 0 0" xyz="0.05 0.0 0.0"/>
       <parent link="${name}_front_link" />
       <child link="${name}_handle" />
