Commit message: [iai_kitchen] Remove virtual main joint in vdrawer, former front_link is now main.

File: iai_kitchen/urdf_obj/IAI_drawers.urdf.xacro (robot description, xacro)
@@ -59,5 +59,5 @@
     </link>
     <joint name="${parent}_${name}_joint" type="fixed">
-      <origin xyz="0 0 ${joint_origin_z}"/>
+      <origin xyz="-0.25 0 ${joint_origin_z}"/>
       <parent link="${parent}_main"/>
       <child link="${parent}_${name}_link"/>
@@ -79,5 +79,5 @@
     </link>
     <joint name="${parent}_${name}_barrier_right_joint" type="fixed">
-      <origin xyz="0 ${-board_y / 2 + board_z / 2} ${joint_origin_z + barrier_z/2 - board_z/2}"/>
+      <origin xyz="-0.25 ${-board_y / 2 + board_z / 2} ${joint_origin_z + barrier_z/2 - board_z/2}"/>
       <parent link="${parent}_main"/>
       <child link="${parent}_${name}_barrier_right_link"/>
@@ -99,5 +99,5 @@
     </link>
     <joint name="${parent}_${name}_barrier_left_joint" type="fixed">
-      <origin xyz="0 ${board_y / 2 - board_z / 2} ${joint_origin_z + barrier_z/2 - board_z/2}"/>
+      <origin xyz="-0.25 ${board_y / 2 - board_z / 2} ${joint_origin_z + barrier_z/2 - board_z/2}"/>
       <parent link="${parent}_main"/>
       <child link="${parent}_${name}_barrier_left_link"/>
@@ -119,5 +119,5 @@
     </link>
     <joint name="${parent}_${name}_barrier_back_joint" type="fixed">
-      <origin xyz="${-board_x / 2 + board_z / 2} 0 ${joint_origin_z + barrier_z/2 - board_z/2}"/>
+      <origin xyz="${-board_x / 2 + board_z / 2 - 0.25} 0 ${joint_origin_z + barrier_z/2 - board_z/2}"/>
       <parent link="${parent}_main"/>
       <child link="${parent}_${name}_barrier_back_link"/>
@@ -125,22 +125,4 @@
   </macro>
   <macro name="iai_vdrawer" params="name parent *origin">
-    <link name="${name}_main">
-      <sphere_inertia radius="0" mass="0"/>
-    </link>
-    <link name="${name}_handle">
-      <sphere_inertia radius="0" mass="0"/>
-      <visual>
-        <origin xyz="0 0 0" rpy="${0.5*pi} 0 0" />
-        <geometry>
-          <mesh filename="package://iai_kitchen/meshes/handles/VHandle130.obj"/>
-        </geometry>
-      </visual>
-      <collision>
-        <origin xyz="0 0 0" rpy="${0.5*pi} 0 0" />
-        <geometry>
-          <mesh filename="package://iai_kitchen/meshes/handles/VHandle130.obj"/>
-        </geometry>
-      </collision>
-    </link>
     <joint name="${name}_main_joint" type="prismatic">
       <xacro:insert_block name="origin"/>
@@ -150,26 +132,36 @@
       <limit effort="300" lower="0" upper="0.48" velocity="10"/>
     </joint>
+    <link name="${name}_main">
+      <sphere_inertia radius="0" mass="0"/>
+      <visual>
+        <origin rpy="0 0 0" xyz="0 0 0"/>
+        <geometry>
+          <box size="0.025 0.295 1.325"/>
+        </geometry>
+      </visual>
+      <collision>
+        <origin rpy="0 0 0" xyz="0 0 0"/>
+        <geometry>
+          <box size="0.025 0.3 1.33"/>
+        </geometry>
+      </collision>
+    </link>
     <joint name="${name}_handle_joint" type="fixed">
       <origin rpy="${-0.5*pi} 0 0" xyz="0.05 0.0 0.0"/>
-      <parent link="${name}_front_link" />
+      <parent link="${name}_main" />
       <child link="${name}_handle" />
     </joint>
-    <joint name="${name}_front_joint" type="fixed">
-      <origin rpy="0 0. 0" xyz="0.25 0 0"/>
-      <parent link="${name}_main"/>
-      <child link="${name}_front_link"/>
-    </joint>
-    <link name="${name}_front_link">
-      <sphere_inertia radius="0" mass="0"/>
-      <visual>
-        <origin rpy="0 0 0" xyz="0 0 0"/>
-        <geometry>
-          <box size="0.025 0.295 1.325"/>
-        </geometry>
-      </visual>
-      <collision>
-        <origin rpy="0 0 0" xyz="0 0 0"/>
-        <geometry>
-          <box size="0.025 0.3 1.33"/>
+    <link name="${name}_handle">
+      <sphere_inertia radius="0" mass="0"/>
+      <visual>
+        <origin xyz="0 0 0" rpy="${0.5*pi} 0 0" />
+        <geometry>
+          <mesh filename="package://iai_kitchen/meshes/handles/VHandle130.obj"/>
+        </geometry>
+      </visual>
+      <collision>
+        <origin xyz="0 0 0" rpy="${0.5*pi} 0 0" />
+        <geometry>
+          <mesh filename="package://iai_kitchen/meshes/handles/VHandle130.obj"/>
         </geometry>
       </collision>

File: iai_kitchen/urdf_obj/IAI_oven_area.urdf.xacro (robot description, xacro)
@@ -44,8 +44,8 @@
   </iai_drawer_60_58>
   <iai_vdrawer name="${name}_area_left_drawer" parent="${name}_area">
-    <origin rpy="0 0 0" xyz="0.0 -0.45 0.06 "/>
+    <origin rpy="0 0 0" xyz="0.25 -0.45 0.06 "/>
   </iai_vdrawer>
   <iai_vdrawer name="${name}_area_right_drawer" parent="${name}_area">
-    <origin rpy="0 0 0" xyz="0.0 0.45 0.06 "/>
+    <origin rpy="0 0 0" xyz="0.25 0.45 0.06 "/>
   </iai_vdrawer>
   </macro>

Commit message: [iai_kitchen]Refactoring the macro because of issues integrating levels in cram

File: iai_kitchen/urdf_obj/IAI_drawers.urdf.xacro (robot description, xacro)
@@ -43,5 +43,5 @@
   <xacro:property name="barrier_z" value="0.082"/>
   <macro name="iai_vdrawer_board" params="name parent joint_origin_z">
-    <link name="${parent}_${name}_link">
+    <link name="${parent}_board_${name}_link">
       <sphere_inertia radius="0" mass="0"/>
       <visual>
@@ -58,50 +58,50 @@
       </collision>
     </link>
-    <joint name="${parent}_${name}_joint" type="fixed">
+    <joint name="${parent}_board_${name}_joint" type="fixed">
       <origin xyz="0 0 ${joint_origin_z}"/>
       <parent link="${parent}_main"/>
-      <child link="${parent}_${name}_link"/>
-    </joint>
-    <link name="${parent}_${name}_barrier_right_link">
-      <sphere_inertia radius="0" mass="0"/>
-      <visual>
-        <origin rpy="0 0 0" xyz="0 0 0"/>
-        <geometry>
-          <box size="${board_x} ${board_z} ${barrier_z}"/>
-        </geometry>
-      </visual>
-      <collision>
-        <origin rpy="0 0 0" xyz="0 0 0"/>
-        <geometry>
-          <box size="${board_x} ${board_z} ${barrier_z}"/>
-        </geometry>
-      </collision>
-    </link>
-    <joint name="${parent}_${name}_barrier_right_joint" type="fixed">
+      <child link="${parent}_board_${name}_link"/>
+    </joint>
+    <link name="${parent}_barrier_${name}_right_link">
+      <sphere_inertia radius="0" mass="0"/>
+      <visual>
+        <origin rpy="0 0 0" xyz="0 0 0"/>
+        <geometry>
+          <box size="${board_x} ${board_z} ${barrier_z}"/>
+        </geometry>
+      </visual>
+      <collision>
+        <origin rpy="0 0 0" xyz="0 0 0"/>
+        <geometry>
+          <box size="${board_x} ${board_z} ${barrier_z}"/>
+        </geometry>
+      </collision>
+    </link>
+    <joint name="${parent}_barrier_${name}_right_joint" type="fixed">
       <origin xyz="0 ${-board_y / 2 + board_z / 2} ${joint_origin_z + barrier_z/2 - board_z/2}"/>
       <parent link="${parent}_main"/>
-      <child link="${parent}_${name}_barrier_right_link"/>
-    </joint>
-    <link name="${parent}_${name}_barrier_left_link">
-      <sphere_inertia radius="0" mass="0"/>
-      <visual>
-        <origin rpy="0 0 0" xyz="0 0 0"/>
-        <geometry>
-          <box size="${board_x} ${board_z} ${barrier_z}"/>
-        </geometry>
-      </visual>
-      <collision>
-        <origin rpy="0 0 0" xyz="0 0 0"/>
-        <geometry>
-          <box size="${board_x} ${board_z} ${barrier_z}"/>
-        </geometry>
-      </collision>
-    </link>
-    <joint name="${parent}_${name}_barrier_left_joint" type="fixed">
+      <child link="${parent}_barrier_${name}_right_link"/>
+    </joint>
+    <link name="${parent}_barrier_${name}_left_link">
+      <sphere_inertia radius="0" mass="0"/>
+      <visual>
+        <origin rpy="0 0 0" xyz="0 0 0"/>
+        <geometry>
+          <box size="${board_x} ${board_z} ${barrier_z}"/>
+        </geometry>
+      </visual>
+      <collision>
+        <origin rpy="0 0 0" xyz="0 0 0"/>
+        <geometry>
+          <box size="${board_x} ${board_z} ${barrier_z}"/>
+        </geometry>
+      </collision>
+    </link>
+    <joint name="${parent}_barrier_${name}_left_joint" type="fixed">
       <origin xyz="0 ${board_y / 2 - board_z / 2} ${joint_origin_z + barrier_z/2 - board_z/2}"/>
       <parent link="${parent}_main"/>
-      <child link="${parent}_${name}_barrier_left_link"/>
-    </joint>
-    <link name="${parent}_${name}_barrier_back_link">
+      <child link="${parent}_barrier_${name}_left_link"/>
+    </joint>
+    <link name="${parent}_barrier_${name}_back_link">
       <sphere_inertia radius="0" mass="0"/>
       <visual>
@@ -118,8 +118,8 @@
       </collision>
     </link>
-    <joint name="${parent}_${name}_barrier_back_joint" type="fixed">
+    <joint name="${parent}_barrier_${name}_back_joint" type="fixed">
       <origin xyz="${-board_x / 2 + board_z / 2} 0 ${joint_origin_z + barrier_z/2 - board_z/2}"/>
       <parent link="${parent}_main"/>
-      <child link="${parent}_${name}_barrier_back_link"/>
+      <child link="${parent}_barrier_${name}_back_link"/>
     </joint>
   </macro>
@@ -175,8 +175,8 @@
       </collision>
     </link>
-    <iai_vdrawer_board name="board0" parent="${name}" joint_origin_z="-0.655"/>
-    <iai_vdrawer_board name="board1" parent="${name}" joint_origin_z="-0.33"/>
-    <iai_vdrawer_board name="board2" parent="${name}" joint_origin_z="0"/>
-    <iai_vdrawer_board name="board3" parent="${name}" joint_origin_z="0.33"/>
+    <iai_vdrawer_board name="0" parent="${name}" joint_origin_z="-0.655"/>
+    <iai_vdrawer_board name="1" parent="${name}" joint_origin_z="-0.33"/>
+    <iai_vdrawer_board name="2" parent="${name}" joint_origin_z="0"/>
+    <iai_vdrawer_board name="3" parent="${name}" joint_origin_z="0.33"/>
   </macro>
   <macro name="iai_drawer_29" params="name parent width *origin">

Commit message: tweaked kitchen obj urdf

File: iai_kitchen/urdf_obj/IAI_drawers.urdf.xacro (robot description, xacro)
@@ -148,5 +148,5 @@
     </link>
     <joint name="${name}_handle_joint" type="fixed">
-      <origin rpy="${-0.5*pi} 0 0" xyz="0.05 0.0 0.0"/>
+      <origin rpy="${-0.5*pi} 0 0" xyz="0.07 0.0 0.0"/>
       <parent link="${name}_main" />
       <child link="${name}_handle" />
@@ -167,8 +167,8 @@
       </collision>
     </link>
-    <iai_vdrawer_board name="0" parent="${name}" joint_origin_z="-0.655"/>
-    <iai_vdrawer_board name="1" parent="${name}" joint_origin_z="-0.33"/>
-    <iai_vdrawer_board name="2" parent="${name}" joint_origin_z="0"/>
-    <iai_vdrawer_board name="3" parent="${name}" joint_origin_z="0.33"/>
+    <iai_vdrawer_board name="0" parent="${name}" joint_origin_z="-0.6"/>
+    <iai_vdrawer_board name="1" parent="${name}" joint_origin_z="-0.28"/>
+    <iai_vdrawer_board name="2" parent="${name}" joint_origin_z="0.05"/>
+    <iai_vdrawer_board name="3" parent="${name}" joint_origin_z="0.38"/>
   </macro>
   <macro name="iai_drawer_29" params="name parent width *origin">

File: iai_kitchen/urdf_obj/IAI_oven_area.urdf.xacro (robot description, xacro)
@@ -44,8 +44,8 @@
   </iai_drawer_60_58>
   <iai_vdrawer name="${name}_area_left_drawer" parent="${name}_area">
-    <origin rpy="0 0 0" xyz="0.25 -0.45 0.06 "/>
+    <origin rpy="0 0 0" xyz="0.28 -0.45 0.07 "/>
   </iai_vdrawer>
   <iai_vdrawer name="${name}_area_right_drawer" parent="${name}_area">
-    <origin rpy="0 0 0" xyz="0.25 0.45 0.06 "/>
+    <origin rpy="0 0 0" xyz="0.28 0.45 0.07"/>
   </iai_vdrawer>
   </macro>

File: iai_kitchen/urdf_obj/iai_kitchen_python.urdf.xacro (robot description, xacro)
@@ -35,8 +35,8 @@
   <xacro:include filename="$(find iai_kitchen)/urdf_obj/IAI_kitchen_walls.urdf.xacro"/>
   <iai_sink_area name="sink_area" parent="room_link">
-    <origin xyz="1.825 1.32 0" rpy="0 0 ${pi}" />
+    <origin xyz="1.855 1.3 0" rpy="0 0 ${pi}" />
   </iai_sink_area>
   <iai_oven_area name="oven_area" parent="room_link">
-    <origin xyz="1.805 2.52 0" rpy="0 0 ${pi}" />
+    <origin xyz="1.855 2.47 0" rpy="0 0 ${pi}" />
   </iai_oven_area>
   <iai_kitchen_island name="kitchen_island" parent="room_link">
@@ -44,5 +44,5 @@
   </iai_kitchen_island>
   <iai_fridge_area name="fridge_area" parent="room_link">
-    <origin xyz="1.825 -0.74 0" rpy="0 0 ${pi}" />
+    <origin xyz="1.845 -0.73 0" rpy="0 0 ${pi}" />
   </iai_fridge_area>
   <iai_table_1 name="table_area" parent="room_link">

Commit message: [kitchen_Urdf] tweaking numbers

File: iai_kitchen/urdf_obj/IAI_drawers.urdf.xacro (robot description, xacro)
@@ -175,5 +175,5 @@
     <iai_generic_drawer name="${name}" parent="${parent}" width="${width}" height="29">
       <xacro:insert_block name="origin" />
-      <origin xyz="0.3325 0 0.11" rpy="0 0 0" />
+      <origin xyz="0.3525 0 0.11" rpy="0 0 0" />
     </iai_generic_drawer>
   </macro>
@@ -181,5 +181,5 @@
     <iai_generic_drawer name="${name}" parent="${parent}" width="${width}" height="14">
       <xacro:insert_block name="origin" />
-      <origin xyz="0.3325 0 0.0175" rpy="0 0 0" />
+      <origin xyz="0.3525 0 0.0175" rpy="0 0 0" />
     </iai_generic_drawer>
   </macro>

File: iai_kitchen/urdf_obj/IAI_fridge.urdf.xacro (robot description, xacro)
@@ -107,10 +107,10 @@
       <visual>
         <geometry>
-          <box size="0.04 0.523 0.825"/>
-        </geometry>
-      </visual>
-      <collision>
-        <geometry>
-          <box size="0.04 0.523 0.825"/>
+          <box size="0.04 0.523 0.88"/>
+        </geometry>
+      </visual>
+      <collision>
+        <geometry>
+          <box size="0.04 0.523 0.88"/>
         </geometry>
       </collision>
@@ -119,10 +119,10 @@
       <visual>
         <geometry>
-          <box size="0.045 0.015 0.73"/>
-        </geometry>
-      </visual>
-      <collision>
-        <geometry>
-          <box size="0.045 0.015 0.73"/>
+          <box size="0.06 0.015 0.73"/>
+        </geometry>
+      </visual>
+      <collision>
+        <geometry>
+          <box size="0.06 0.015 0.73"/>
         </geometry>
       </collision>
@@ -131,10 +131,10 @@
       <visual>
         <geometry>
-          <box size="0.045 0.015 0.73"/>
-        </geometry>
-      </visual>
-      <collision>
-        <geometry>
-          <box size="0.045 0.015 0.73"/>
+          <box size="0.06 0.015 0.73"/>
+        </geometry>
+      </visual>
+      <collision>
+        <geometry>
+          <box size="0.06 0.015 0.73"/>
         </geometry>
       </collision>
@@ -143,15 +143,15 @@
       <visual>
         <geometry>
-          <box size="0.025 0.46 0.01"/>
-        </geometry>
-      </visual>
-      <collision>
-        <geometry>
-          <box size="0.025 0.46 0.01"/>
+          <box size="0.045 0.46 0.01"/>
+        </geometry>
+      </visual>
+      <collision>
+        <geometry>
+          <box size="0.045 0.46 0.01"/>
         </geometry>
       </collision>
     </link>
     <joint name="${name}_door_block_joint" type="fixed">
-      <origin xyz="-0.025 -0.27 -0.05" />
+      <origin xyz="-0.025 -0.27 -0.01" />
       <parent link="${name}_door"/>
       <child link="${name}_door_block"/>
@@ -176,8 +176,8 @@
     </fridge_door_shelf>
     <fridge_door_shelf name="${name}_door_shelf2" parent="${name}_door_block" height="0.065">
-      <origin xyz="-0.07 0 0.0425"/>
+      <origin xyz="-0.07 0 0.02"/>
     </fridge_door_shelf>
     <fridge_door_shelf name="${name}_door_shelf3" parent="${name}_door_block" height="0.065">
-      <origin xyz="-0.07 0 0.2625 "/>
+      <origin xyz="-0.07 0 0.26"/>
     </fridge_door_shelf>
   </macro>
@@ -203,10 +203,10 @@
       <visual>
         <geometry>
-          <box size="0.105 0.06 ${height}"/>
-        </geometry>
-      </visual>
-      <collision>
-        <geometry>
-          <box size="0.105 0.06 ${height}"/>
+          <box size="0.115 0.06 ${height}"/>
+        </geometry>
+      </visual>
+      <collision>
+        <geometry>
+          <box size="0.115 0.06 ${height}"/>
         </geometry>
       </collision>
@@ -215,10 +215,10 @@
       <visual>
         <geometry>
-          <box size="0.105 0.06 ${height}"/>
-        </geometry>
-      </visual>
-      <collision>
-        <geometry>
-          <box size="0.105 0.06 ${height}"/>
+          <box size="0.115 0.06 ${height}"/>
+        </geometry>
+      </visual>
+      <collision>
+        <geometry>
+          <box size="0.115 0.06 ${height}"/>
         </geometry>
       </collision>
@@ -227,5 +227,5 @@
       <visual>
         <geometry>
-          <box size="0.01 0.35 ${height}"/>
+          <box size="0.02 0.35 ${height}"/>
         </geometry>
       </visual>

Commit message: [kitchen urdf] tweaking oven area

File: iai_kitchen/urdf_obj/IAI_drawers.urdf.xacro (robot description, xacro)
@@ -148,5 +148,5 @@
     </link>
     <joint name="${name}_handle_joint" type="fixed">
-      <origin rpy="${-0.5*pi} 0 0" xyz="0.07 0.0 0.0"/>
+      <origin rpy="${-0.5*pi} 0 0" xyz="0.1 0.0 0.0"/>
       <parent link="${name}_main" />
       <child link="${name}_handle" />

File: iai_kitchen/urdf_obj/IAI_oven_area.urdf.xacro (robot description, xacro)
@@ -44,8 +44,8 @@
   </iai_drawer_60_58>
   <iai_vdrawer name="${name}_area_left_drawer" parent="${name}_area">
-    <origin rpy="0 0 0" xyz="0.28 -0.45 0.07 "/>
+    <origin rpy="0 0 0" xyz="0.29 -0.45 0.07 "/>
   </iai_vdrawer>
   <iai_vdrawer name="${name}_area_right_drawer" parent="${name}_area">
-    <origin rpy="0 0 0" xyz="0.28 0.45 0.07"/>
+    <origin rpy="0 0 0" xyz="0.29 0.45 0.07"/>
   </iai_vdrawer>
   </macro>

File: iai_kitchen/urdf_obj/iai_kitchen_python.urdf.xacro (robot description, xacro)
@@ -35,5 +35,5 @@
   </iai_sink_area>
   <iai_oven_area name="oven_area" parent="room_link">
-    <origin xyz="1.855 2.47 0" rpy="0 0 ${pi}" />
+    <origin xyz="1.855 2.5 0" rpy="0 0 ${pi}" />
     <!-- <origin xyz="-5.27 -6.85 0" rpy="0 0 0" /> -->
   </iai_oven_area>

Commit message: [kitchen urdf] brought oven area 1 cm forward

File: iai_kitchen/urdf_obj/IAI_drawers.urdf.xacro (robot description, xacro)
@@ -148,5 +148,5 @@
     </link>
     <joint name="${name}_handle_joint" type="fixed">
-      <origin rpy="${-0.5*pi} 0 0" xyz="0.1 0.0 0.0"/>
+      <origin rpy="${-0.5*pi} 0 0" xyz="0.08 0.0 0.0"/>
       <parent link="${name}_main" />
       <child link="${name}_handle" />

File: iai_kitchen/urdf_obj/iai_kitchen_python.urdf.xacro (robot description, xacro)
@@ -35,5 +35,5 @@
   </iai_sink_area>
   <iai_oven_area name="oven_area" parent="room_link">
-    <origin xyz="1.855 2.5 0" rpy="0 0 ${pi}" />
+    <origin xyz="1.845 2.5 0" rpy="0 0 ${pi}" />
     <!-- <origin xyz="-5.27 -6.85 0" rpy="0 0 0" /> -->
   </iai_oven_area>
