Commit message: [iai_fridge]Adding a level in the fridge object

File: iai_kitchen/urdf_obj/IAI_fridge.urdf.xacro (robot description, xacro)
@@ -15,4 +15,18 @@
         <geometry>
           <mesh filename="package://iai_kitchen/meshes/misc/Fridge.obj"/>
+        </geometry>
+      </collision>
+    </link>
+    <link name="${name}_main_middle_level">
+      <visual>
+        <origin xyz="-0.01 0 -0.17" rpy="0 0 0" />
+        <geometry>
+          <box size="0.29 0.50 0.01"/>
+        </geometry>
+      </visual>
+      <collision>
+        <origin xyz="-0.01 0 -0.17" rpy="0 0 0" />
+        <geometry>
+          <box size="0.29 0.50 0.01"/>
         </geometry>
       </collision>
@@ -53,4 +67,9 @@
       <child link="${name}_main"/>
     </joint>
+    <joint name="${name}_main_middle_level_joint" type="fixed">
+      <parent link="${name}_main"/>
+      <child link="${name}_main_middle_level"/>
+      <origin xyz="0 0 0.30" rpy="0 0 0" />
+    </joint>
     <joint name="${name}_door_joint" type="revolute">
       <origin xyz="0.29 0.3 0.245" rpy="0 0 0" />

Commit message: [iai_kitchen]Adjusted the origin of the joint to keep visual at 0

File: iai_kitchen/urdf_obj/IAI_fridge.urdf.xacro (robot description, xacro)
@@ -20,5 +20,5 @@
     <link name="${name}_main_middle_level">
       <visual>
-        <origin xyz="-0.01 0 -0.17" rpy="0 0 0" />
+        <origin xyz="0 0 0" rpy="0 0 0" />
         <geometry>
           <box size="0.29 0.50 0.01"/>
@@ -26,5 +26,5 @@
       </visual>
       <collision>
-        <origin xyz="-0.01 0 -0.17" rpy="0 0 0" />
+        <origin xyz="0 0 0" rpy="0 0 0" />
         <geometry>
           <box size="0.29 0.50 0.01"/>
@@ -70,5 +70,5 @@
       <parent link="${name}_main"/>
       <child link="${name}_main_middle_level"/>
-      <origin xyz="0 0 0.30" rpy="0 0 0" />
+      <origin xyz="-0.01 0 0.13" rpy="0 0 0" />
     </joint>
     <joint name="${name}_door_joint" type="revolute">

Commit message: Glued box to fridge door to represent the shleves

File: iai_kitchen/urdf_obj/IAI_fridge.urdf.xacro (robot description, xacro)
@@ -32,5 +32,17 @@
         </geometry>
       </collision>
-    </link>
+  </link>
+    <link name="${name}_door_shelves">
+        <visual>
+            <geometry>
+                <box size="0.1 0.5 0.8"/>
+            </geometry>
+        </visual>
+        <collision>
+            <geometry>
+                <box size="0.1 0.5 0.8"/>
+            </geometry>
+        </collision>
+  </link>
     <link name="${name}_door_handle">
       <sphere_inertia radius="0" mass="0"/>
@@ -63,4 +75,9 @@
 -->
     </joint>
+    <joint name="${name}_door_shelves_joint" type="fixed">
+        <origin xyz="-0.06 -0.29 0"/>
+        <parent link="${name}_door"/>
+        <child link="${name}_door_shelves"/>
+    </joint>
     <joint name="${name}_door_handle_joint" type="fixed">
       <origin xyz="0.06 -0.57 0." rpy="0 0 0" />

Commit message: fixed fridge layer height

File: iai_kitchen/urdf_obj/IAI_fridge.urdf.xacro (robot description, xacro)
@@ -82,5 +82,5 @@
       <parent link="${name}_main"/>
       <child link="${name}_main_middle_level"/>
-      <origin xyz="-0.01 0 0.13" rpy="0 0 0" />
+      <origin xyz="-0.01 0 0.27" rpy="0 0 0" />
     </joint>
     <joint name="${name}_door_joint" type="revolute">

Commit message: fixed fridge shelf box size

File: iai_kitchen/urdf_obj/IAI_fridge.urdf.xacro (robot description, xacro)
@@ -50,10 +50,10 @@
         <visual>
             <geometry>
-                <box size="0.1 0.5 0.8"/>
+                <box size="0.16 0.5 0.8"/>
             </geometry>
         </visual>
         <collision>
             <geometry>
-                <box size="0.1 0.5 0.8"/>
+                <box size="0.16 0.5 0.8"/>
             </geometry>
         </collision>
@@ -95,10 +95,10 @@
     </joint>
     <joint name="${name}_door_shelves_joint" type="fixed">
-        <origin xyz="-0.06 -0.29 0"/>
+        <origin xyz="-0.09 -0.29 0"/>
         <parent link="${name}_door"/>
         <child link="${name}_door_shelves"/>
     </joint>
     <joint name="${name}_door_handle_joint" type="fixed">
-      <origin xyz="0.06 -0.57 0." rpy="0 0 0" />
+      <origin xyz="0.09 -0.57 0." rpy="0 0 0" />
       <parent link="${name}_door"/>
       <child link="${name}_door_handle"/>

Commit message: added fridge ceiling box

File: iai_kitchen/urdf_obj/IAI_fridge.urdf.xacro (robot description, xacro)
@@ -59,4 +59,16 @@
         </collision>
   </link>
+  <link name="${name}_ceiling">
+        <visual>
+            <geometry>
+                <box size="0.48 0.5 0.05"/>
+            </geometry>
+        </visual>
+        <collision>
+            <geometry>
+                <box size="0.48 0.5 0.05"/>
+            </geometry>
+        </collision>
+  </link>
     <link name="${name}_door_handle">
       <sphere_inertia radius="0" mass="0"/>
@@ -99,4 +111,9 @@
         <child link="${name}_door_shelves"/>
     </joint>
+    <joint name="${name}_ceiling_joint" type="fixed">
+        <origin xyz="0.0 0.0 0.64"/>
+        <parent link="${name}_main"/>
+        <child link="${name}_ceiling"/>
+    </joint>
     <joint name="${name}_door_handle_joint" type="fixed">
       <origin xyz="0.09 -0.57 0." rpy="0 0 0" />

Commit message: added macro for fridge door shelf

File: iai_kitchen/urdf_obj/IAI_fridge.urdf.xacro (robot description, xacro)
@@ -68,4 +68,77 @@
       <child link="${name}_door_handle"/>
     </joint>
+    <fridge_door_shelve name="${name}_door_shelf" parent="${name}_door">
+      <origin xyz="-0.05 -0.32 0 "/>
+    </fridge_door_shelve>
+  </macro>
+  <macro name="fridge_door_shelve" params="name parent *origin">
+    <joint name="${name}_to_door" type="fixed">
+      <xacro:insert_block name="origin"/>
+      <child link="${name}_bottom"/>
+      <parent link="${parent}"/>
+    </joint>
+    <link name="${name}_bottom" >
+      <visual>
+        <geometry>
+          <box size="0.1 0.5 0.03"/>
+        </geometry>
+      </visual>
+      <collision>
+        <geometry>
+          <box size="0.1 0.5 0.03"/>
+        </geometry>
+      </collision>
+    </link>
+    <link name="${name}_left_side" >
+      <visual>
+        <geometry>
+          <box size="0.1 0.02 0.1"/>
+        </geometry>
+      </visual>
+      <collision>
+        <geometry>
+          <box size="0.1 0.02 0.1"/>
+        </geometry>
+      </collision>
+    </link>
+    <link name="${name}_right_side" >
+      <visual>
+        <geometry>
+          <box size="0.1 0.02 0.1"/>
+        </geometry>
+      </visual>
+      <collision>
+        <geometry>
+          <box size="0.1 0.02 0.1"/>
+        </geometry>
+      </collision>
+    </link>
+    <link name="${name}_front_side" >
+      <visual>
+        <geometry>
+          <box size="0.02 0.5 0.1"/>
+        </geometry>
+      </visual>
+      <collision>
+        <geometry>
+          <box size="0.02 0.5 0.1"/>
+        </geometry>
+      </collision>
+    </link>
+    <joint name="${name}_left_to_bottom" type="fixed">
+      <origin xyz="0 -0.24 0.05"/>
+      <parent link="${name}_bottom"/>
+      <child link="${name}_left_side"/>
+    </joint>
+    <joint name="${name}_right_to_bottom" type="fixed">
+      <origin xyz="0 0.24 0.05"/>
+      <parent link="${name}_bottom"/>
+      <child link="${name}_right_side"/>
+    </joint>
+    <joint name="${name}_front_to_bottom" type="fixed">
+      <origin xyz="-0.05 0 0.05"/>
+      <parent link="${name}_bottom"/>
+      <child link="${name}_front_side"/>
+    </joint>
   </macro>
 </robot>

Commit message: fixed wrong position of fridge door handle

File: iai_kitchen/urdf_obj/IAI_fridge.urdf.xacro (robot description, xacro)
@@ -100,5 +100,5 @@
     </joint>
     <joint name="${name}_door_handle_joint" type="fixed">
-      <origin xyz="0.09 -0.57 0." rpy="0 0 0" />
+      <origin xyz="0.05 -0.57 0." rpy="0 0 0" />
       <parent link="${name}_door"/>
       <child link="${name}_door_handle"/>

Commit message: Reverted change of handle position

File: iai_kitchen/urdf_obj/IAI_fridge.urdf.xacro (robot description, xacro)
@@ -100,5 +100,5 @@
     </joint>
     <joint name="${name}_door_handle_joint" type="fixed">
-      <origin xyz="0.05 -0.57 0." rpy="0 0 0" />
+      <origin xyz="0.09 -0.57 0." rpy="0 0 0" />
       <parent link="${name}_door"/>
       <child link="${name}_door_handle"/>

Commit message: adjusted urdf to new fridge mesh

File: iai_kitchen/urdf_obj/IAI_fridge.urdf.xacro (robot description, xacro)
@@ -94,8 +94,8 @@
       <parent link="${name}_main"/>
       <child link="${name}_main_middle_level"/>
-      <origin xyz="-0.01 0 0.27" rpy="0 0 0" />
+      <origin xyz="-0.01 0 0.07" rpy="0 0 0" />
     </joint>
     <joint name="${name}_door_joint" type="revolute">
-      <origin xyz="0.29 0.3 0.245" rpy="0 0 0" />
+      <origin xyz="0.29 0.3 0" rpy="0 0 0" />
       <parent link="${name}_main"/>
       <child link="${name}_door"/>
@@ -112,5 +112,5 @@
     </joint>
     <joint name="${name}_ceiling_joint" type="fixed">
-        <origin xyz="0.0 0.0 0.64"/>
+        <origin xyz="0.0 0.0 0.44"/>
         <parent link="${name}_main"/>
         <child link="${name}_ceiling"/>

File: iai_kitchen/urdf_obj/IAI_fridge_area.urdf.xacro (robot description, xacro)
@@ -38,5 +38,5 @@
   </iai_drawer_60_29>
   <iai_fridge name="iai_fridge" parent="${name}">
-    <origin xyz="0 0 0" rpy="0 0 0" />
+    <origin xyz="0 0 0.25" rpy="0 0 0" />
   </iai_fridge>
   </macro>

Commit message: [urdf] fridge handle depth tweak

File: iai_kitchen/urdf_obj/IAI_fridge.urdf.xacro (robot description, xacro)
@@ -100,5 +100,5 @@
     </joint>
     <joint name="${name}_door_handle_joint" type="fixed">
-      <origin xyz="0.09 -0.57 0." rpy="0 0 0" />
+      <origin xyz="0.07 -0.57 0." rpy="0 0 0" />
       <parent link="${name}_door"/>
       <child link="${name}_door_handle"/>
