Commit message: fixed kitchen offsets

File: iai_kitchen/urdf_obj/iai_kitchen_python.urdf.xacro (robot description, xacro)
@@ -19,5 +19,5 @@
     <link name="world"/>
     <joint name="world_room_joint" type="fixed">
-        <origin xyz="0.02 -0.01 0 " rpy="0 0 0" />
+        <origin xyz="0.0 0.0 0 " rpy="0 0 0" />
         <parent link="world"/>
         <child link="room_link"/>
@@ -35,14 +35,14 @@
   <xacro:include filename="$(find iai_kitchen)/urdf_obj/IAI_kitchen_walls.urdf.xacro"/>
   <iai_sink_area name="sink_area" parent="room_link">
-    <origin xyz="1.825 1.3 0" rpy="0 0 ${pi}" />
+    <origin xyz="1.845 1.33 0" rpy="0 0 ${pi}" />
   </iai_sink_area>
   <iai_oven_area name="oven_area" parent="room_link">
-    <origin xyz="1.805 2.5 0" rpy="0 0 ${pi}" />
+    <origin xyz="1.825 2.53 0" rpy="0 0 ${pi}" />
   </iai_oven_area>
   <iai_kitchen_island name="kitchen_island" parent="room_link">
-    <origin xyz="-1.365 0.59 0" rpy="0 0 0" />
+    <origin xyz="-1.345 0.58 0" rpy="0 0 0" />
   </iai_kitchen_island>
   <iai_fridge_area name="fridge_area" parent="room_link">
-    <origin xyz="1.825 -0.76 0" rpy="0 0 ${pi}" />
+    <origin xyz="1.845 -0.74 0" rpy="0 0 ${pi}" />
   </iai_fridge_area>
   <iai_table_1 name="table_area" parent="room_link">

Commit message: fixed no-json-obj.launch

File: iai_kitchen/urdf_obj/iai_kitchen_python.urdf.xacro (robot description, xacro)
@@ -35,14 +35,14 @@
   <xacro:include filename="$(find iai_kitchen)/urdf_obj/IAI_kitchen_walls.urdf.xacro"/>
   <iai_sink_area name="sink_area" parent="room_link">
-    <origin xyz="1.845 1.33 0" rpy="0 0 ${pi}" />
+    <origin xyz="1.845 1.35 0" rpy="0 0 ${pi}" />
   </iai_sink_area>
   <iai_oven_area name="oven_area" parent="room_link">
-    <origin xyz="1.825 2.53 0" rpy="0 0 ${pi}" />
+    <origin xyz="1.825 2.55 0" rpy="0 0 ${pi}" />
   </iai_oven_area>
   <iai_kitchen_island name="kitchen_island" parent="room_link">
-    <origin xyz="-1.345 0.58 0" rpy="0 0 0" />
+    <origin xyz="-1.355 0.58 0" rpy="0 0 0" />
   </iai_kitchen_island>
   <iai_fridge_area name="fridge_area" parent="room_link">
-    <origin xyz="1.845 -0.74 0" rpy="0 0 ${pi}" />
+    <origin xyz="1.845 -0.72 0" rpy="0 0 ${pi}" />
   </iai_fridge_area>
   <iai_table_1 name="table_area" parent="room_link">

Commit message: moved overall kitchen offset from static transform publisher to urdf

File: iai_kitchen/urdf_obj/iai_kitchen_python.urdf.xacro (robot description, xacro)
@@ -19,5 +19,5 @@
     <link name="world"/>
     <joint name="world_room_joint" type="fixed">
-        <origin xyz="0.0 0.0 0 " rpy="0 0 0" />
+        <origin xyz="0.0 0.03 0 " rpy="0 0 0" />
         <parent link="world"/>
         <child link="room_link"/>

Commit message: added the table for the popcorn demo

File: iai_kitchen/urdf_obj/iai_kitchen_python.urdf.xacro (robot description, xacro)
@@ -7,4 +7,5 @@
   <xacro:include filename="$(find iai_kitchen)/urdf_obj/IAI_tables.urdf.xacro"/>
   <xacro:include filename="$(find iai_kitchen)/urdf_obj/IAI_kitchen_walls.urdf.xacro"/>
+  <xacro:include filename="$(find iai_kitchen)/urdf_obj/IAI_popcorn_table.urdf.xacro"/>
   <xacro:property name="pi" value="3.1415926535897931" />
   <xacro:property name="simulated" value="true" />
@@ -55,4 +56,7 @@
     <origin xyz="-0.96 0.65 0" rpy="0.0 0.0 0.0" />
   </iai_kitchen_wall_robohow>
+  <iai_popcorn_table name="iai_popcorn_table" parent="room_link">
+    <origin xyz="-0.05 -1.7 0"/>
+  </iai_popcorn_table>
   <gazebo>
     <static>false</static>

Commit message: [iai_kitchen] gave correct name to the robot in URDF and clean up

File: iai_kitchen/urdf_obj/iai_kitchen_python.urdf.xacro (robot description, xacro)
@@ -1,31 +1,4 @@
 <?xml version="1.0"?>
-<robot name="iai_oven_area" xmlns:xacro="http://ros.org/wiki/xacro">
-  <xacro:property name="pi" value="3.1415926535897931" />
-  <xacro:property name="simulated" value="true" />
-  <macro name="sphere_inertia" params="radius mass">
-        <inertial>
-          <origin xyz="0.0 0.0 0.0" rpy="0 0 0"/>
-          <mass value="1"/>
-          <inertia
-              ixx="1" ixy="0.0" ixz="0.0"
-              iyy="1" iyz="0.0"
-              izz="1"/>
-        </inertial>
-  </macro>
-  <link name="room_link">
-      <sphere_inertia radius="0" mass="0"/>
-  </link>
-  <xacro:if value="${simulated}">
-    <link name="world"/>
-    <joint name="world_room_joint" type="fixed">
-        <origin xyz="0.0 0.03 0 " rpy="0 0 0" />
-        <parent link="world"/>
-        <child link="room_link"/>
-      </joint>
-  </xacro:if>
-  <gazebo>
-      <static>false</static>
-  </gazebo>
-  <!--- FIXME THIS should NOT be here -->
+<robot name="iai_kitchen" xmlns:xacro="http://ros.org/wiki/xacro">
   <xacro:include filename="$(find iai_kitchen)/urdf_obj/IAI_oven_area.urdf.xacro"/>
   <xacro:include filename="$(find iai_kitchen)/urdf_obj/IAI_kitchen_island.urdf.xacro"/>
@@ -34,15 +7,42 @@
   <xacro:include filename="$(find iai_kitchen)/urdf_obj/IAI_tables.urdf.xacro"/>
   <xacro:include filename="$(find iai_kitchen)/urdf_obj/IAI_kitchen_walls.urdf.xacro"/>
+  <xacro:property name="pi" value="3.1415926535897931" />
+  <xacro:property name="simulated" value="true" />
+  <macro name="sphere_inertia" params="radius mass">
+    <inertial>
+      <origin xyz="0.0 0.0 0.0" rpy="0 0 0"/>
+      <mass value="1"/>
+      <inertia
+          ixx="1" ixy="0.0" ixz="0.0"
+          iyy="1" iyz="0.0"
+          izz="1"/>
+    </inertial>
+  </macro>
+  <link name="room_link">
+    <sphere_inertia radius="0" mass="0"/>
+  </link>
+  <xacro:if value="${simulated}">
+    <link name="world"/>
+    <joint name="world_room_joint" type="fixed">
+      <origin xyz="0.0 0.03 0 " rpy="0 0 0" />
+      <parent link="world"/>
+      <child link="room_link"/>
+    </joint>
+  </xacro:if>
   <iai_sink_area name="sink_area" parent="room_link">
     <origin xyz="1.855 1.3 0" rpy="0 0 ${pi}" />
+    <!-- <origin xyz="-5.29 -5.65 0" rpy="0 0 0" /> -->
   </iai_sink_area>
   <iai_oven_area name="oven_area" parent="room_link">
     <origin xyz="1.855 2.47 0" rpy="0 0 ${pi}" />
+    <!-- <origin xyz="-5.27 -6.85 0" rpy="0 0 0" /> -->
   </iai_oven_area>
   <iai_kitchen_island name="kitchen_island" parent="room_link">
     <origin xyz="-1.365 0.59 0" rpy="0 0 0" />
+    <!-- <origin xyz="-2.1 -4.94 0" rpy="0 0 ${pi}" /> -->
   </iai_kitchen_island>
   <iai_fridge_area name="fridge_area" parent="room_link">
     <origin xyz="1.845 -0.73 0" rpy="0 0 ${pi}" />
+    <!-- <origin xyz="-5.29 -3.59 0" rpy="0 0 0" /> -->
   </iai_fridge_area>
   <iai_table_1 name="table_area" parent="room_link">
@@ -52,17 +52,6 @@
     <origin xyz="-0.96 0.65 0" rpy="0.0 0.0 0.0" />
   </iai_kitchen_wall_robohow>
-  <!-- Included above already
-  <iai_sink_area name="sink_area" parent="room_link">
-    <origin xyz="-5.29 -5.65 0" rpy="0 0 0" />
-  </iai_sink_area>
-  <iai_oven_area name="oven_area" parent="room_link">
-    <origin xyz="-5.27 -6.85 0" rpy="0 0 0" />
-  </iai_oven_area>
-  <iai_kitchen_island name="kitchen_island" parent="room_link">
-    <origin xyz="-2.1 -4.94 0" rpy="0 0 ${pi}" />
-  </iai_kitchen_island>
-  <iai_fridge_area name="fridge_area" parent="room_link">
-    <origin xyz="-5.29 -3.59 0" rpy="0 0 0" />
-  </iai_fridge_area>
-  -->
+  <gazebo>
+    <static>false</static>
+  </gazebo>
 </robot>

Commit message: removed obsolete macro and added properties

File: iai_kitchen/urdf_obj/iai_kitchen_python.urdf.xacro (robot description, xacro)
@@ -10,4 +10,5 @@
   <xacro:property name="pi" value="3.1415926535897931" />
   <xacro:property name="simulated" value="true" />
+  <xacro:property name="include_wall_7" value="true"/>
   <macro name="sphere_inertia" params="radius mass">
     <inertial>
@@ -53,10 +54,7 @@
     <origin xyz="-3.38 0.28 0" rpy="0 0 ${pi / 2}" />
   </iai_dining_area>
-  <iai_kitchen_wall_robohow parent="room_link" wall_7="true">
+  <iai_kitchen_wall_robohow parent="room_link" wall_7="${include_wall_7}">
     <origin xyz="-0.96 0.65 0" rpy="0.0 0.0 0.0" />
   </iai_kitchen_wall_robohow>
-  <iai_popcorn_table name="iai_popcorn_table" parent="room_link">
-    <origin xyz="-0.05 -1.7 0"/>
-  </iai_popcorn_table>
   <gazebo>
     <static>false</static>

Commit message: added default parameter

File: iai_kitchen/urdf_obj/iai_kitchen_python.urdf.xacro (robot description, xacro)
@@ -10,5 +10,4 @@
   <xacro:property name="pi" value="3.1415926535897931" />
   <xacro:property name="simulated" value="true" />
-  <xacro:property name="include_wall_7" value="true"/>
   <macro name="sphere_inertia" params="radius mass">
     <inertial>
@@ -54,5 +53,5 @@
     <origin xyz="-3.38 0.28 0" rpy="0 0 ${pi / 2}" />
   </iai_dining_area>
-  <iai_kitchen_wall_robohow parent="room_link" wall_7="${include_wall_7}">
+  <iai_kitchen_wall_robohow parent="room_link">
     <origin xyz="-0.96 0.65 0" rpy="0.0 0.0 0.0" />
   </iai_kitchen_wall_robohow>
