Commit message: added new wall to kitchen obj urdf and fixed position of existing walls

File: iai_kitchen/urdf_obj/IAI_kitchen_walls.urdf.xacro (robot description, xacro)
@@ -68,5 +68,5 @@
         <origin xyz="0 0 0.35" rpy="0 0 0" />
         <geometry>
-            <box size="3.27328 0.15 0.7" />
+            <box size="2.27328 0.15 0.7" />
         </geometry>
      </visual>
@@ -74,5 +74,5 @@
         <origin xyz="0 0 0.35" rpy="0 0 0" />
         <geometry>
-            <box size="3.27328 0.15 0.7" />
+            <box size="2.27328 0.15 0.7" />
         </geometry>
       </collision>
@@ -90,4 +90,19 @@
         <geometry>
             <box size="1 0.15 0.7" />
+        </geometry>
+      </collision>
+    </link>
+    <link name="kitchen_wall_7">
+      <sphere_inertia radius="0" mass="0"/>
+      <visual>
+        <origin xyz="0 0 0.375" rpy="0 0 0" />
+        <geometry>
+            <box size="1.6 0.15 0.75" />
+        </geometry>
+     </visual>
+      <collision>
+        <origin xyz="0 0 0.375" rpy="0 0 0" />
+        <geometry>
+            <box size="1.6 0.15 0.75" />
         </geometry>
       </collision>
@@ -128,12 +143,17 @@
     </joint>
     <joint name="wall_5_joint" type="fixed">
-        <origin xyz="-1.31385 -1.58376 0" rpy="0 -0 0.000157" />
+        <origin xyz="-1.81385 -1.70376 0" rpy="0 -0 0.000157" />
       <parent link="kitchen_walls"/>
       <child link="kitchen_wall_5"/>
     </joint>
     <joint name="wall_6_joint" type="fixed">
-      <origin xyz="0.247785 -2.00851 0" rpy="0 0 -1.5708" />
+      <origin xyz="-0.65 -2.12851 0" rpy="0 0 -1.5708" />
       <parent link="kitchen_walls"/>
       <child link="kitchen_wall_6"/>
+    </joint>
+    <joint name="wall_7_joint" type="fixed">
+      <origin xyz="1.01271 -2.556 0" rpy="0 -0 3.14159" />
+      <parent link="kitchen_walls"/>
+      <child link="kitchen_wall_7"/>
     </joint>
     <gazebo reference="kitchen_wall_6">

File: iai_kitchen/urdf_obj/iai_kitchen_python.urdf.xacro (robot description, xacro)
@@ -47,8 +47,8 @@
   </iai_fridge_area>
   <iai_table_1 name="table_area" parent="room_link">
-    <origin xyz="-1.4 -1.05 0" rpy="0 0 ${pi}" />
+    <origin xyz="-2.4 -1.5 0" rpy="0 0 ${pi}" />
   </iai_table_1>
   <iai_kitchen_wall_robohow parent="room_link">
-    <origin xyz="-1 0.562175 0" rpy="0.0 0.0 0.0" />
+    <origin xyz="-0.96 0.65 0" rpy="0.0 0.0 0.0" />
   </iai_kitchen_wall_robohow>
   <!-- Included above already

Commit message: added the table for the popcorn demo

File: iai_kitchen/urdf_obj/IAI_kitchen_walls.urdf.xacro (robot description, xacro)
@@ -93,4 +93,5 @@
       </collision>
     </link>
+<!--
     <link name="kitchen_wall_7">
       <sphere_inertia radius="0" mass="0"/>
@@ -108,4 +109,5 @@
       </collision>
     </link>
+  -->
     <!-- JOINTS -->
     <link name="kitchen_walls"/>
@@ -152,4 +154,5 @@
       <child link="kitchen_wall_6"/>
     </joint>
+<!--
     <joint name="wall_7_joint" type="fixed">
       <origin xyz="1.01271 -2.556 0" rpy="0 -0 3.14159" />
@@ -157,4 +160,5 @@
       <child link="kitchen_wall_7"/>
     </joint>
+-->
     <gazebo reference="kitchen_wall_6">
         <material>Gazebo/DarkGrey</material>

File: iai_kitchen/urdf_obj/iai_kitchen_python.urdf.xacro (robot description, xacro)
@@ -34,4 +34,5 @@
   <xacro:include filename="$(find iai_kitchen)/urdf_obj/IAI_tables.urdf.xacro"/>
   <xacro:include filename="$(find iai_kitchen)/urdf_obj/IAI_kitchen_walls.urdf.xacro"/>
+  <xacro:include filename="$(find iai_kitchen)/urdf_obj/IAI_popcorn_table.urdf.xacro"/>
   <iai_sink_area name="sink_area" parent="room_link">
     <origin xyz="1.855 1.3 0" rpy="0 0 ${pi}" />
@@ -52,4 +53,7 @@
     <origin xyz="-0.96 0.65 0" rpy="0.0 0.0 0.0" />
   </iai_kitchen_wall_robohow>
+  <iai_popcorn_table name="iai_popcorn_table" parent="room_link">
+    <origin xyz="-0.05 -1.7 0"/>
+  </iai_popcorn_table>
   <!-- Included above already
   <iai_sink_area name="sink_area" parent="room_link">

Commit message: added default parameter

File: iai_kitchen/urdf_obj/IAI_kitchen_walls.urdf.xacro (robot description, xacro)
@@ -1,5 +1,5 @@
 <?xml version="1.0"?>
 <robot name="iai_kitchen_wall_robohow" xmlns:xacro="http://ros.org/wiki/xacro">
-  <macro name="iai_kitchen_wall_robohow" params="parent *origin wall_7">
+  <macro name="iai_kitchen_wall_robohow" params="parent *origin wall_7:=true">
     <!-- LINKS -->
     <link name="kitchen_wall_1">

File: iai_kitchen/urdf_obj/iai_kitchen_python.urdf.xacro (robot description, xacro)
@@ -3,5 +3,4 @@
   <xacro:property name="pi" value="3.1415926535897931" />
   <xacro:property name="simulated" value="true" />
-  <xacro:property name="include_wall_7" value="true"/>
   <macro name="sphere_inertia" params="radius mass">
         <inertial>
@@ -50,5 +49,5 @@
     <origin xyz="-2.4 -1.5 0" rpy="0 0 ${pi}" />
   </iai_table_1>
-  <iai_kitchen_wall_robohow parent="room_link" wall_7="${include_wall_7}">
+  <iai_kitchen_wall_robohow parent="room_link">
     <origin xyz="-0.96 0.65 0" rpy="0.0 0.0 0.0" />
   </iai_kitchen_wall_robohow>

Commit message: changed for noetic and popcorn demo, WARNING: iai_kitchen_python.urdf.xacro includs popcorn atm, on the otherhand iai_kitchen_popcorn_python.urdf.xacro does not work yet this has to be changed!

File: iai_kitchen/urdf_obj/IAI_kitchen_walls.urdf.xacro (robot description, xacro)
@@ -1,5 +1,5 @@
 <?xml version="1.0"?>
 <robot name="iai_kitchen_wall_robohow" xmlns:xacro="http://ros.org/wiki/xacro">
-  <macro name="iai_kitchen_wall_robohow" params="parent *origin include_wall_7:=true">
+  <xacro:macro name="iai_kitchen_wall_robohow" params="parent *origin include_wall_7:=true">
     <!-- LINKS -->
     <link name="kitchen_wall_1">
@@ -164,4 +164,4 @@
         <material>Gazebo/DarkGrey</material>
     </gazebo>
-  </macro>
+  </xacro:macro>
 </robot>

File: iai_kitchen/urdf_obj/IAI_popcorn_table.urdf.xacro (robot description, xacro)
@@ -1,5 +1,5 @@
 <?xml version="1.0"?>
 <robot name="iai_popcorn_table" xmlns:xacro="http://ros.org/wiki/xacro">
-  <macro name="iai_popcorn_table" params="name parent *origin">
+  <xacro:macro name="iai_popcorn_table" params="name parent *origin">
     <link name="${name}_footprint"/>
     <joint name="${name}_footprint_joint" type="fixed">
@@ -244,6 +244,6 @@
       <origin xyz="-0.235 0.12 0.01"/>
     </iai_popcorn_stove_knob>
-  </macro>
-  <macro name="iai_popcorn_table_drawer" params="name parent *origin">
+  </xacro:macro>
+  <xacro:macro name="iai_popcorn_table_drawer" params="name parent *origin">
   <joint name="${name}_table_joint" type="prismatic">
         <parent link="${parent}"/>
@@ -336,6 +336,6 @@
     <origin xyz="0.03 0 0"/>
   </iai_popcorn_table_drawer_handle>
-  </macro>
-  <macro name="iai_popcorn_table_drawer_handle" params="name parent *origin">
+  </xacro:macro>
+  <xacro:macro name="iai_popcorn_table_drawer_handle" params="name parent *origin">
   <link name="${name}_left_part">
     <visual>
@@ -389,6 +389,6 @@
     <child link="${name}_middle_part"/>
   </joint>
-  </macro>
-  <macro name="iai_popcorn_stove_knob" params="name parent *origin">
+  </xacro:macro>
+  <xacro:macro name="iai_popcorn_stove_knob" params="name parent *origin">
   <link name="${name}">
     <sphere_inertia radius="0" mass="0"/>
@@ -413,4 +413,4 @@
     <limit lower="-${pi}" upper="0" effort="300" velocity="10"/>
   </joint>
-  </macro>
+  </xacro:macro>
 </robot>

File: iai_kitchen/urdf_obj/iai_kitchen_popcorn_python.urdf.xacro (robot description, xacro)
@@ -1,8 +1,16 @@
 <?xml version="1.0"?>
 <robot name="iai_oven_area" xmlns:xacro="http://ros.org/wiki/xacro">
+  <!--- FIXME THIS should NOT be here -->
+  <xacro:include filename="$(find iai_kitchen)/urdf_obj/IAI_oven_area.urdf.xacro"/>
+  <xacro:include filename="$(find iai_kitchen)/urdf_obj/IAI_kitchen_island.urdf.xacro"/>
+  <xacro:include filename="$(find iai_kitchen)/urdf_obj/IAI_sink_area.urdf.xacro"/>
+  <xacro:include filename="$(find iai_kitchen)/urdf_obj/IAI_fridge_area.urdf.xacro"/>
+  <xacro:include filename="$(find iai_kitchen)/urdf_obj/IAI_tables.urdf.xacro"/>
+  <xacro:include filename="$(find iai_kitchen)/urdf_obj/IAI_kitchen_walls.urdf.xacro"/>
+  <xacro:include filename="$(find iai_kitchen)/urdf_obj/IAI_popcorn_table.urdf.xacro"/>
   <xacro:property name="pi" value="3.1415926535897931" />
   <xacro:property name="simulated" value="true" />
   <xacro:property name="include_wall_7" value="false"/>
-  <macro name="sphere_inertia" params="radius mass">
+  <xacro:macro name="sphere_inertia" params="radius mass">
         <inertial>
           <origin xyz="0.0 0.0 0.0" rpy="0 0 0"/>
@@ -13,5 +21,5 @@
               izz="1"/>
         </inertial>
-  </macro>
+  </xacro:macro>
   <link name="room_link">
       <sphere_inertia radius="0" mass="0"/>
@@ -28,12 +36,4 @@
       <static>false</static>
   </gazebo>
-  <!--- FIXME THIS should NOT be here -->
-  <xacro:include filename="$(find iai_kitchen)/urdf_obj/IAI_oven_area.urdf.xacro"/>
-  <xacro:include filename="$(find iai_kitchen)/urdf_obj/IAI_kitchen_island.urdf.xacro"/>
-  <xacro:include filename="$(find iai_kitchen)/urdf_obj/IAI_sink_area.urdf.xacro"/>
-  <xacro:include filename="$(find iai_kitchen)/urdf_obj/IAI_fridge_area.urdf.xacro"/>
-  <xacro:include filename="$(find iai_kitchen)/urdf_obj/IAI_tables.urdf.xacro"/>
-  <xacro:include filename="$(find iai_kitchen)/urdf_obj/IAI_kitchen_walls.urdf.xacro"/>
-  <xacro:include filename="$(find iai_kitchen)/urdf_obj/IAI_popcorn_table.urdf.xacro"/>
   <iai_sink_area name="sink_area" parent="room_link">
     <origin xyz="1.855 1.3 0" rpy="0 0 ${pi}" />

File: iai_kitchen/urdf_obj/iai_kitchen_python.urdf.xacro (robot description, xacro)
@@ -10,4 +10,5 @@
   <xacro:property name="pi" value="3.1415926535897931" />
   <xacro:property name="simulated" value="true" />
+  <xacro:property name="include_wall_7" value="false"/>
   <xacro:macro name="sphere_inertia" params="radius mass">
     <inertial>
@@ -56,4 +57,7 @@
     <origin xyz="-0.96 0.65 0" rpy="0.0 0.0 0.0" />
   </xacro:iai_kitchen_wall_robohow>
+    <xacro:iai_popcorn_table name="iai_popcorn_table" parent="room_link">
+    <origin xyz="-0.05 -1.7 0"/>
+    </xacro:iai_popcorn_table>
   <gazebo>
     <static>false</static>
