Commit message: adding fullbuild popcorn kitchen urdf for KnowRob

File: iai_kitchen/urdf_obj/iai_kitchen_popcorn_python.urdf (robot description, URDF)
Before this commit: robot iai_oven_area, 164 links, 163 joints
Links:
- added link dining_area_footprint
- added link dining_area_jokkmokk_left_chair_main; collision mesh filename=package://iai_kitchen/meshes/jokkmokk/JokkmokkChair.obj; visual mesh filename=package://iai_kitchen/meshes/jokkmokk/JokkmokkChair.obj
- added link dining_area_jokkmokk_right_chair_main; collision mesh filename=package://iai_kitchen/meshes/jokkmokk/JokkmokkChair.obj; visual mesh filename=package://iai_kitchen/meshes/jokkmokk/JokkmokkChair.obj
- added link dining_area_jokkmokk_table_main; collision mesh filename=package://iai_kitchen/meshes/jokkmokk/JokkmokkTable.obj; visual mesh filename=package://iai_kitchen/meshes/jokkmokk/JokkmokkTable.obj
Joints:
- added joint dining_area_footprint_joint: type fixed, parent room_link, child dining_area_footprint, origin xyz=-3.38 0.28 0 rpy=0 0 1.5707963267948966
- added joint dining_area_jokkmokk_left_chair_main_joint: type fixed, parent dining_area_footprint, child dining_area_jokkmokk_left_chair_main, origin xyz=-1 0 0.5535 rpy=0 0 0
- added joint dining_area_jokkmokk_right_chair_main_joint: type fixed, parent dining_area_footprint, child dining_area_jokkmokk_right_chair_main, origin xyz=1 0 0.5535 rpy=0 0 -3.141592653589793
- added joint dining_area_jokkmokk_table_main_joint: type fixed, parent dining_area_footprint, child dining_area_jokkmokk_table_main, origin xyz=0 0 0.35 rpy=0 0 0
- joint kitchen_island_footprint_joint: origin xyz=-1.365 0.59 0 rpy=0 0 0 -> xyz=-1.363 0.59 0 rpy=0 0 0
- joint oven_area_footprint_joint: origin xyz=1.855 2.47 0 rpy=0 0 3.141592653589793 -> xyz=1.845 2.5 0 rpy=0 0 3.141592653589793
