Commit message: added macro for a tray in the dishwascher

File: iai_kitchen/urdf_obj/IAI_dish_washer.urdf.xacro (robot description, xacro)
@@ -57,4 +57,5 @@
       <child link="${name}_main"/>
     </joint>
+    <!--
     <xacro:if value="${simulated}">
     <joint name="${name}_door_joint" type="revolute">
@@ -63,9 +64,12 @@
       <child link="${name}_door"/>
       <axis xyz="0 0 1"/>
-      <!-- FIXME make closed position stable instead of forbidding opening... -->
+       FIXME make closed position stable instead of forbidding opening...
       <limit lower="0" upper="0" effort="300" velocity="10"/>
     </joint>
     </xacro:if>
+    -->
+    <!--
     <xacro:unless value="${simulated}">
+    -->
     <joint name="${name}_door_joint" type="revolute">
       <origin xyz="0.27 0. -0.325" rpy="${-0.5*pi} 0 0" />
@@ -78,5 +82,7 @@
       <limit lower="0" upper="${0.5*pi}" effort="300" velocity="10"/>
     </joint>
+    <!--
     </xacro:unless>
+  -->
     <joint name="${name}_door_handle_joint" type="fixed">
       <origin xyz="0.0625 -0.6325 0." rpy="${-0.5*pi} 0 0" />
@@ -84,4 +90,96 @@
       <child link="${name}_door_handle"/>
     </joint>
+    <dishwasher_tray name="${name}_tray" parent="${name}_main">
+      <origin xyu="0 0 0.15"/>
+    </dishwasher_tray>
+  </macro>
+  <macro name="dishwasher_tray" params="name parent *origin">
+    <joint name="${name}_main" type="prismatic">
+      <xacro:insert_block name="origin"/>
+      <parent link="${parent}"/>
+      <child link="${name}_bottom"/>
+      <axis xyz="1 0 0"/>
+      <limit lower="0" upper="0.4" effort="300" velocity="10"/>
+    </joint>
+    <link name="${name}_bottom">
+      <visual>
+        <geometry>
+          <box size="0.5 0.5 0.02"/>
+        </geometry>
+      </visual>
+      <collision>
+        <geometry>
+          <box size="0.5 0.5 0.02"/>
+        </geometry>
+      </collision>
+    </link>
+    <link name="${name}_left_side">
+      <visual>
+        <geometry>
+          <box size="0.5 0.02 0.1"/>
+        </geometry>
+      </visual>
+      <collision>
+        <geometry>
+          <box size="0.5 0.02 0.1"/>
+        </geometry>
+      </collision>
+    </link>
+    <link name="${name}_right_side">
+      <visual>
+        <geometry>
+          <box size="0.5 0.02 0.1"/>
+        </geometry>
+      </visual>
+      <collision>
+        <geometry>
+          <box size="0.5 0.02 0.1"/>
+        </geometry>
+      </collision>
+    </link>
+    <link name="${name}_back_side">
+      <visual>
+        <geometry>
+          <box size="0.02 0.5 0.1"/>
+        </geometry>
+      </visual>
+      <collision>
+        <geometry>
+          <box size="0.02 0.5 0.1"/>
+        </geometry>
+      </collision>
+    </link>
+    <link name="${name}_front_side">
+      <visual>
+        <geometry>
+          <box size="0.02 0.5 0.1"/>
+        </geometry>
+      </visual>
+      <collision>
+        <geometry>
+          <box size="0.02 0.5 0.1"/>
+        </geometry>
+      </collision>
+    </link>
+    <joint name="${name}_bottom_left" type="fixed">
+      <origin xyz="0 -0.24 0.06"/>
+      <child link="${name}_left_side" />
+      <parent link="${name}_bottom"/>
+    </joint>
+    <joint name="${name}_bottom_right" type="fixed">
+      <origin xyz="0 0.24 0.06"/>
+      <child link="${name}_right_side" />
+      <parent link="${name}_bottom"/>
+    </joint>
+    <joint name="${name}_bottom_back" type="fixed">
+      <origin xyz="-0.24 0 0.06"/>
+      <child link="${name}_back_side" />
+      <parent link="${name}_bottom"/>
+    </joint>
+    <joint name="${name}_front_back" type="fixed">
+      <origin xyz="0.24 0 0.06"/>
+      <child link="${name}_front_side" />
+      <parent link="${name}_bottom"/>
+    </joint>
   </macro>
 </robot>

Commit message: Fridge and dishwasher with final messurments

File: iai_kitchen/urdf_obj/IAI_dish_washer.urdf.xacro (robot description, xacro)
@@ -105,10 +105,10 @@
       <visual>
         <geometry>
-          <box size="0.5 0.5 0.02"/>
-        </geometry>
-      </visual>
-      <collision>
-        <geometry>
-          <box size="0.5 0.5 0.02"/>
+          <box size="0.464 0.5 0.02"/>
+        </geometry>
+      </visual>
+      <collision>
+        <geometry>
+          <box size="0.464 0.5 0.02"/>
         </geometry>
       </collision>
@@ -117,10 +117,10 @@
       <visual>
         <geometry>
-          <box size="0.5 0.02 0.1"/>
-        </geometry>
-      </visual>
-      <collision>
-        <geometry>
-          <box size="0.5 0.02 0.1"/>
+          <box size="0.464 0.02 0.17"/>
+        </geometry>
+      </visual>
+      <collision>
+        <geometry>
+          <box size="0.464 0.02 0.17"/>
         </geometry>
       </collision>
@@ -129,10 +129,10 @@
       <visual>
         <geometry>
-          <box size="0.5 0.02 0.1"/>
-        </geometry>
-      </visual>
-      <collision>
-        <geometry>
-          <box size="0.5 0.02 0.1"/>
+          <box size="0.464 0.02 0.17"/>
+        </geometry>
+      </visual>
+      <collision>
+        <geometry>
+          <box size="0.464 0.02 0.17"/>
         </geometry>
       </collision>
@@ -141,10 +141,10 @@
       <visual>
         <geometry>
-          <box size="0.02 0.5 0.1"/>
-        </geometry>
-      </visual>
-      <collision>
-        <geometry>
-          <box size="0.02 0.5 0.1"/>
+          <box size="0.02 0.5 0.17"/>
+        </geometry>
+      </visual>
+      <collision>
+        <geometry>
+          <box size="0.02 0.5 0.17"/>
         </geometry>
       </collision>
@@ -153,32 +153,88 @@
       <visual>
         <geometry>
-          <box size="0.02 0.5 0.1"/>
-        </geometry>
-      </visual>
-      <collision>
-        <geometry>
-          <box size="0.02 0.5 0.1"/>
+          <box size="0.02 0.5 0.17"/>
+        </geometry>
+      </visual>
+      <collision>
+        <geometry>
+          <box size="0.02 0.5 0.17"/>
         </geometry>
       </collision>
     </link>
     <joint name="${name}_bottom_left" type="fixed">
-      <origin xyz="0 -0.24 0.06"/>
+      <origin xyz="0 -0.24 0.075"/>
       <child link="${name}_left_side" />
       <parent link="${name}_bottom"/>
     </joint>
     <joint name="${name}_bottom_right" type="fixed">
-      <origin xyz="0 0.24 0.06"/>
+      <origin xyz="0 0.24 0.075"/>
       <child link="${name}_right_side" />
       <parent link="${name}_bottom"/>
     </joint>
     <joint name="${name}_bottom_back" type="fixed">
-      <origin xyz="-0.24 0 0.06"/>
+      <origin xyz="-0.24 0 0.075"/>
       <child link="${name}_back_side" />
       <parent link="${name}_bottom"/>
     </joint>
     <joint name="${name}_front_back" type="fixed">
-      <origin xyz="0.24 0 0.06"/>
+      <origin xyz="0.24 0 0.075"/>
       <child link="${name}_front_side" />
       <parent link="${name}_bottom"/>
+    </joint>
+    <tray_handle name="${name}_handle" parent="${name}_front_side">
+      <origin xyz="0.0305 0 0"/>
+    </tray_handle>
+  </macro>
+  <macro name="tray_handle" params="name parent *origin">
+    <joint name="${name}_joint" type="fixed">
+      <xacro:insert_block name="origin"/>
+      <child link="${name}_front_side" />
+      <parent link="${parent}"/>
+    </joint>
+    <link name="${name}_left_side">
+      <visual>
+        <geometry>
+          <box size="0.03 0.01 0.01"/>
+        </geometry>
+      </visual>
+      <collision>
+        <geometry>
+          <box size="0.03 0.01 0.01"/>
+        </geometry>
+      </collision>
+    </link>
+    <link name="${name}_right_side">
+      <visual>
+        <geometry>
+          <box size="0.03 0.01 0.01"/>
+        </geometry>
+      </visual>
+      <collision>
+        <geometry>
+          <box size="0.03 0.01 0.01"/>
+        </geometry>
+      </collision>
+    </link>
+    <link name="${name}_front_side">
+      <visual>
+        <geometry>
+          <box size="0.01 0.4 0.01"/>
+        </geometry>
+      </visual>
+      <collision>
+        <geometry>
+          <box size="0.01 0.4 0.01"/>
+        </geometry>
+      </collision>
+    </link>
+    <joint name="${name}_front_left_joint" type="fixed">
+      <origin xyz="-0.01 -0.2 0"/>
+      <child link="${name}_left_side" />
+      <parent link="${name}_front_side"/>
+    </joint>
+    <joint name="${name}_front_right_joint" type="fixed">
+      <origin xyz="-0.01 0.2 0"/>
+      <child link="${name}_right_side" />
+      <parent link="${name}_front_side"/>
     </joint>
   </macro>

File: iai_kitchen/urdf_obj/IAI_fridge.urdf.xacro (robot description, xacro)
@@ -68,9 +68,83 @@
       <child link="${name}_door_handle"/>
     </joint>
-    <fridge_door_shelve name="${name}_door_shelf" parent="${name}_door">
-      <origin xyz="-0.05 -0.32 0 "/>
+    <link name="${name}_door_block" >
+      <visual>
+        <geometry>
+          <box size="0.04 0.523 0.825"/>
+        </geometry>
+      </visual>
+      <collision>
+        <geometry>
+          <box size="0.04 0.523 0.825"/>
+        </geometry>
+      </collision>
+    </link>
+    <link name="${name}_door_block_right_bar" >
+      <visual>
+        <geometry>
+          <box size="0.045 0.015 0.8"/>
+        </geometry>
+      </visual>
+      <collision>
+        <geometry>
+          <box size="0.045 0.015 0.8"/>
+        </geometry>
+      </collision>
+    </link>
+    <link name="${name}_door_block_left_bar" >
+      <visual>
+        <geometry>
+          <box size="0.045 0.015 0.8"/>
+        </geometry>
+      </visual>
+      <collision>
+        <geometry>
+          <box size="0.045 0.015 0.8"/>
+        </geometry>
+      </collision>
+    </link>
+    <link name="${name}_door_block_top_bar" >
+      <visual>
+        <geometry>
+          <box size="0.025 0.365 0.01"/>
+        </geometry>
+      </visual>
+      <collision>
+        <geometry>
+          <box size="0.025 0.0365 0.01"/>
+        </geometry>
+      </collision>
+    </link>
+    <joint name="${name}_door_block_joint" type="fixed">
+      <origin xyz="-0.025 -0.27 0" />
+      <parent link="${name}_door"/>
+      <child link="${name}_door_block"/>
+    </joint>
+    <joint name="${name}_door_block_right_bar_joint" type="fixed">
+      <origin xyz="-0.0425 -0.175 0" />
+      <parent link="${name}_door_block"/>
+      <child link="${name}_door_block_right_bar"/>
+    </joint>
+    <joint name="${name}_door_block_left_bar_joint" type="fixed">
+      <origin xyz="-0.0425 0.175 0" />
+      <parent link="${name}_door_block"/>
+      <child link="${name}_door_block_left_bar"/>
+    </joint>
+    <joint name="${name}_door_block_top_bar_joint" type="fixed">
+      <origin xyz="-0.03 0 0.4" />
+      <parent link="${name}_door_block"/>
+      <child link="${name}_door_block_top_bar"/>
+    </joint>
+    <fridge_door_shelve name="${name}_door_shelf1" parent="${name}_door_block" height="0.1">
+      <origin xyz="-0.07 0 -0.40 "/>
+    </fridge_door_shelve>
+    <fridge_door_shelve name="${name}_door_shelf2" parent="${name}_door_block" height="0.065">
+      <origin xyz="-0.07 0 -0.01"/>
+    </fridge_door_shelve>
+    <fridge_door_shelve name="${name}_door_shelf3" parent="${name}_door_block" height="0.065">
+      <origin xyz="-0.07 0 0.21 "/>
     </fridge_door_shelve>
   </macro>
-  <macro name="fridge_door_shelve" params="name parent *origin">
+  <macro name="fridge_door_shelve" params="name parent height *origin">
     <joint name="${name}_to_door" type="fixed">
       <xacro:insert_block name="origin"/>
@@ -81,10 +155,10 @@
       <visual>
         <geometry>
-          <box size="0.1 0.5 0.03"/>
-        </geometry>
-      </visual>
-      <collision>
-        <geometry>
-          <box size="0.1 0.5 0.03"/>
+          <box size="0.1 0.35 0.01"/>
+        </geometry>
+      </visual>
+      <collision>
+        <geometry>
+          <box size="0.1 0.35 0.01"/>
         </geometry>
       </collision>
@@ -93,10 +167,10 @@
       <visual>
         <geometry>
-          <box size="0.1 0.02 0.1"/>
-        </geometry>
-      </visual>
-      <collision>
-        <geometry>
-          <box size="0.1 0.02 0.1"/>
+          <box size="0.105 0.01 ${height}"/>
+        </geometry>
+      </visual>
+      <collision>
+        <geometry>
+          <box size="0.105 0.01 ${height}"/>
         </geometry>
       </collision>
@@ -105,10 +179,10 @@
       <visual>
         <geometry>
-          <box size="0.1 0.02 0.1"/>
-        </geometry>
-      </visual>
-      <collision>
-        <geometry>
-          <box size="0.1 0.02 0.1"/>
+          <box size="0.105 0.01 ${height}"/>
+        </geometry>
+      </visual>
+      <collision>
+        <geometry>
+          <box size="0.105 0.01 ${height}"/>
         </geometry>
       </collision>
@@ -117,25 +191,25 @@
       <visual>
         <geometry>
-          <box size="0.02 0.5 0.1"/>
-        </geometry>
-      </visual>
-      <collision>
-        <geometry>
-          <box size="0.02 0.5 0.1"/>
+          <box size="0.01 0.35 ${height}"/>
+        </geometry>
+      </visual>
+      <collision>
+        <geometry>
+          <box size="0.01 0.35 ${height}"/>
         </geometry>
       </collision>
     </link>
     <joint name="${name}_left_to_bottom" type="fixed">
-      <origin xyz="0 -0.24 0.05"/>
+      <origin xyz="-0.0025 -0.18 ${ height/2 - 0.005}"/>
       <parent link="${name}_bottom"/>
       <child link="${name}_left_side"/>
     </joint>
     <joint name="${name}_right_to_bottom" type="fixed">
-      <origin xyz="0 0.24 0.05"/>
+      <origin xyz="-0.0025 0.18 ${ height/2 - 0.005}"/>
       <parent link="${name}_bottom"/>
       <child link="${name}_right_side"/>
     </joint>
     <joint name="${name}_front_to_bottom" type="fixed">
-      <origin xyz="-0.05 0 0.05"/>
+      <origin xyz="-0.05 0 ${ height/2 - 0.005}"/>
       <parent link="${name}_bottom"/>
       <child link="${name}_front_side"/>

Commit message: a few changes to the positioning of the macros

File: iai_kitchen/urdf_obj/IAI_dish_washer.urdf.xacro (robot description, xacro)
@@ -91,5 +91,5 @@
     </joint>
     <dishwasher_tray name="${name}_tray" parent="${name}_main">
-      <origin xyu="0 0 0.15"/>
+      <origin xyz="0 0 0.15"/>
     </dishwasher_tray>
   </macro>

File: iai_kitchen/urdf_obj/IAI_fridge.urdf.xacro (robot description, xacro)
@@ -83,10 +83,10 @@
       <visual>
         <geometry>
-          <box size="0.045 0.015 0.8"/>
-        </geometry>
-      </visual>
-      <collision>
-        <geometry>
-          <box size="0.045 0.015 0.8"/>
+          <box size="0.045 0.015 0.73"/>
+        </geometry>
+      </visual>
+      <collision>
+        <geometry>
+          <box size="0.045 0.015 0.73"/>
         </geometry>
       </collision>
@@ -95,10 +95,10 @@
       <visual>
         <geometry>
-          <box size="0.045 0.015 0.8"/>
-        </geometry>
-      </visual>
-      <collision>
-        <geometry>
-          <box size="0.045 0.015 0.8"/>
+          <box size="0.045 0.015 0.73"/>
+        </geometry>
+      </visual>
+      <collision>
+        <geometry>
+          <box size="0.045 0.015 0.73"/>
         </geometry>
       </collision>
@@ -107,41 +107,41 @@
       <visual>
         <geometry>
-          <box size="0.025 0.365 0.01"/>
-        </geometry>
-      </visual>
-      <collision>
-        <geometry>
-          <box size="0.025 0.0365 0.01"/>
+          <box size="0.025 0.46 0.01"/>
+        </geometry>
+      </visual>
+      <collision>
+        <geometry>
+          <box size="0.025 0.46 0.01"/>
         </geometry>
       </collision>
     </link>
     <joint name="${name}_door_block_joint" type="fixed">
-      <origin xyz="-0.025 -0.27 0" />
+      <origin xyz="-0.025 -0.27 -0.05" />
       <parent link="${name}_door"/>
       <child link="${name}_door_block"/>
     </joint>
     <joint name="${name}_door_block_right_bar_joint" type="fixed">
-      <origin xyz="-0.0425 -0.175 0" />
+      <origin xyz="-0.0425 -0.2225 0.01" />
       <parent link="${name}_door_block"/>
       <child link="${name}_door_block_right_bar"/>
     </joint>
     <joint name="${name}_door_block_left_bar_joint" type="fixed">
-      <origin xyz="-0.0425 0.175 0" />
+      <origin xyz="-0.0425 0.2225 0.01" />
       <parent link="${name}_door_block"/>
       <child link="${name}_door_block_left_bar"/>
     </joint>
     <joint name="${name}_door_block_top_bar_joint" type="fixed">
-      <origin xyz="-0.03 0 0.4" />
+      <origin xyz="-0.03 0 0.37" />
       <parent link="${name}_door_block"/>
       <child link="${name}_door_block_top_bar"/>
     </joint>
     <fridge_door_shelve name="${name}_door_shelf1" parent="${name}_door_block" height="0.1">
-      <origin xyz="-0.07 0 -0.40 "/>
+      <origin xyz="-0.07 0 -0.3525 "/>
     </fridge_door_shelve>
     <fridge_door_shelve name="${name}_door_shelf2" parent="${name}_door_block" height="0.065">
-      <origin xyz="-0.07 0 -0.01"/>
+      <origin xyz="-0.07 0 0.0425"/>
     </fridge_door_shelve>
     <fridge_door_shelve name="${name}_door_shelf3" parent="${name}_door_block" height="0.065">
-      <origin xyz="-0.07 0 0.21 "/>
+      <origin xyz="-0.07 0 0.2625 "/>
     </fridge_door_shelve>
   </macro>
@@ -167,10 +167,10 @@
       <visual>
         <geometry>
-          <box size="0.105 0.01 ${height}"/>
-        </geometry>
-      </visual>
-      <collision>
-        <geometry>
-          <box size="0.105 0.01 ${height}"/>
+          <box size="0.105 0.06 ${height}"/>
+        </geometry>
+      </visual>
+      <collision>
+        <geometry>
+          <box size="0.105 0.06 ${height}"/>
         </geometry>
       </collision>
@@ -179,10 +179,10 @@
       <visual>
         <geometry>
-          <box size="0.105 0.01 ${height}"/>
-        </geometry>
-      </visual>
-      <collision>
-        <geometry>
-          <box size="0.105 0.01 ${height}"/>
+          <box size="0.105 0.06 ${height}"/>
+        </geometry>
+      </visual>
+      <collision>
+        <geometry>
+          <box size="0.105 0.06 ${height}"/>
         </geometry>
       </collision>
@@ -201,10 +201,10 @@
     </link>
     <joint name="${name}_left_to_bottom" type="fixed">
-      <origin xyz="-0.0025 -0.18 ${ height/2 - 0.005}"/>
+      <origin xyz="-0.0025 -0.2 ${ height/2 - 0.005}"/>
       <parent link="${name}_bottom"/>
       <child link="${name}_left_side"/>
     </joint>
     <joint name="${name}_right_to_bottom" type="fixed">
-      <origin xyz="-0.0025 0.18 ${ height/2 - 0.005}"/>
+      <origin xyz="-0.0025 0.2 ${ height/2 - 0.005}"/>
       <parent link="${name}_bottom"/>
       <child link="${name}_right_side"/>
