Commit message: [kitchen urdf] tweaking more numbers

File: iai_kitchen/urdf_obj/IAI_dish_washer.urdf.xacro (robot description, xacro)
@@ -86,10 +86,10 @@
   -->
     <joint name="${name}_door_handle_joint" type="fixed">
-      <origin xyz="0.0625 -0.6325 0." rpy="${-0.5*pi} 0 0" />
+      <origin xyz="0.09 -0.65 0.0" rpy="${-0.5*pi} 0 0" />
       <parent link="${name}_door"/>
       <child link="${name}_door_handle"/>
     </joint>
     <dishwasher_tray name="${name}_tray" parent="${name}_main">
-      <origin xyz="0 0 0.15"/>
+      <origin xyz="-0.05 0 0.15"/>
     </dishwasher_tray>
   </macro>
@@ -100,15 +100,15 @@
       <child link="${name}_bottom"/>
       <axis xyz="1 0 0"/>
-      <limit lower="0" upper="0.4" effort="300" velocity="10"/>
+      <limit lower="0" upper="0.40" effort="300" velocity="10"/>
     </joint>
     <link name="${name}_bottom">
       <visual>
         <geometry>
-          <box size="0.464 0.5 0.02"/>
-        </geometry>
-      </visual>
-      <collision>
-        <geometry>
-          <box size="0.464 0.5 0.02"/>
+          <box size="0.32 0.5 0.02"/>
+        </geometry>
+      </visual>
+      <collision>
+        <geometry>
+          <box size="0.32 0.5 0.02"/>
         </geometry>
       </collision>
@@ -117,10 +117,10 @@
       <visual>
         <geometry>
-          <box size="0.464 0.02 0.17"/>
-        </geometry>
-      </visual>
-      <collision>
-        <geometry>
-          <box size="0.464 0.02 0.17"/>
+          <box size="0.32 0.005 0.17"/>
+        </geometry>
+      </visual>
+      <collision>
+        <geometry>
+          <box size="0.32 0.005 0.17"/>
         </geometry>
       </collision>
@@ -129,10 +129,10 @@
       <visual>
         <geometry>
-          <box size="0.464 0.02 0.17"/>
-        </geometry>
-      </visual>
-      <collision>
-        <geometry>
-          <box size="0.464 0.02 0.17"/>
+          <box size="0.32 0.005 0.17"/>
+        </geometry>
+      </visual>
+      <collision>
+        <geometry>
+          <box size="0.32 0.005 0.17"/>
         </geometry>
       </collision>
@@ -141,10 +141,10 @@
       <visual>
         <geometry>
-          <box size="0.02 0.5 0.17"/>
-        </geometry>
-      </visual>
-      <collision>
-        <geometry>
-          <box size="0.02 0.5 0.17"/>
+          <box size="0.005 0.5 0.17"/>
+        </geometry>
+      </visual>
+      <collision>
+        <geometry>
+          <box size="0.005 0.5 0.17"/>
         </geometry>
       </collision>
@@ -153,35 +153,35 @@
       <visual>
         <geometry>
-          <box size="0.02 0.5 0.17"/>
-        </geometry>
-      </visual>
-      <collision>
-        <geometry>
-          <box size="0.02 0.5 0.17"/>
+          <box size="0.005 0.5 0.17"/>
+        </geometry>
+      </visual>
+      <collision>
+        <geometry>
+          <box size="0.005 0.5 0.17"/>
         </geometry>
       </collision>
     </link>
     <joint name="${name}_bottom_left" type="fixed">
-      <origin xyz="0 -0.24 0.075"/>
+      <origin xyz="-0.0 -0.25 0.075"/>
       <child link="${name}_left_side" />
       <parent link="${name}_bottom"/>
     </joint>
     <joint name="${name}_bottom_right" type="fixed">
-      <origin xyz="0 0.24 0.075"/>
+      <origin xyz="-0.0 0.25 0.075"/>
       <child link="${name}_right_side" />
       <parent link="${name}_bottom"/>
     </joint>
     <joint name="${name}_bottom_back" type="fixed">
-      <origin xyz="-0.24 0 0.075"/>
+      <origin xyz="-0.16 0 0.075"/>
       <child link="${name}_back_side" />
       <parent link="${name}_bottom"/>
     </joint>
-    <joint name="${name}_front_back" type="fixed">
-      <origin xyz="0.24 0 0.075"/>
+    <joint name="${name}_bottom_front" type="fixed">
+      <origin xyz="0.16 0 0.075"/>
       <child link="${name}_front_side" />
       <parent link="${name}_bottom"/>
     </joint>
     <tray_handle name="${name}_handle" parent="${name}_front_side">
-      <origin xyz="0.0305 0 0"/>
+      <origin xyz="0.025 0 0.025"/>
     </tray_handle>
   </macro>

File: iai_kitchen/urdf_obj/IAI_drawers.urdf.xacro (robot description, xacro)
@@ -35,5 +35,5 @@
     <iai_generic_drawer name="${name}" parent="${parent}" width="${width}" height="58">
       <xacro:insert_block name="origin" />
-      <origin xyz="0.3325 0 0.2375" rpy="0 0 0" />
+      <origin xyz="0.37 0 0.25" rpy="0 0 0" />
     </iai_generic_drawer>
   </macro>

File: iai_kitchen/urdf_obj/IAI_fridge.urdf.xacro (robot description, xacro)
@@ -50,10 +50,10 @@
         <visual>
             <geometry>
-                <box size="0.48 0.5 0.05"/>
+                <box size="0.56 0.5 0.13"/>
             </geometry>
         </visual>
         <collision>
             <geometry>
-                <box size="0.48 0.5 0.05"/>
+                <box size="0.56 0.5 0.13"/>
             </geometry>
         </collision>
@@ -82,5 +82,5 @@
       <parent link="${name}_main"/>
       <child link="${name}_main_middle_level"/>
-      <origin xyz="-0.01 0 0.07" rpy="0 0 0" />
+      <origin xyz="-0.01 0 0.01" rpy="0 0 0" />
     </joint>
     <joint name="${name}_door_joint" type="revolute">
@@ -179,5 +179,5 @@
     </fridge_door_shelf>
     <fridge_door_shelf name="${name}_door_shelf3" parent="${name}_door_block" height="0.065">
-      <origin xyz="-0.07 0 0.26"/>
+      <origin xyz="-0.07 0 0.23"/>
     </fridge_door_shelf>
   </macro>

Commit message: [kitchen urdf] tweaking

File: iai_kitchen/urdf_obj/IAI_dish_washer.urdf.xacro (robot description, xacro)
@@ -91,5 +91,5 @@
     </joint>
     <dishwasher_tray name="${name}_tray" parent="${name}_main">
-      <origin xyz="-0.05 0 0.15"/>
+      <origin xyz="-0.10 0 0.15"/>
     </dishwasher_tray>
   </macro>
@@ -183,5 +183,5 @@
     </joint>
     <tray_handle name="${name}_handle" parent="${name}_front_side">
-      <origin xyz="0.025 0 0.025"/>
+      <origin xyz="0.025 0 -0.05"/>
     </tray_handle>
   </macro>

File: iai_kitchen/urdf_obj/IAI_sink_area.urdf.xacro (robot description, xacro)
@@ -81,8 +81,8 @@
   </iai_drawer_80_29>
   <iai_drawer_80_29 name="${name}_left_bottom_drawer" parent="${name}">
-    <origin rpy="0 0 0" xyz="0.01 -0.6 -0.18 "/>
+    <origin rpy="0 0 0" xyz="0.01 -0.6 -0.18" />
   </iai_drawer_80_29>
   <iai_dish_washer name="${name}_dish_washer" parent="${name}">
-    <origin rpy="0 0 0" xyz="0.01 0.1 0.044 "/>
+    <origin rpy="0 0 0" xyz="0.01 0.1 0.06" />
   </iai_dish_washer>
   </macro>

Commit message: [kitchen urdf] dishwasher joint tweaking

File: iai_kitchen/urdf_obj/IAI_dish_washer.urdf.xacro (robot description, xacro)
@@ -21,5 +21,5 @@
       <sphere_inertia radius="0" mass="0"/>
       <visual>
-        <origin xyz="0 0 0" rpy="${0.5*pi} 0 0" />
+        <origin xyz="0 0.055 0" rpy="${0.5*pi} 0 0" />
         <geometry>
           <mesh filename="package://iai_kitchen/meshes/misc/DishWasherDoor.obj"/>
@@ -27,5 +27,5 @@
       </visual>
       <collision>
-        <origin xyz="0 0 0" rpy="${0.5*pi} 0 0" />
+        <origin xyz="0 0.055 0" rpy="${0.5*pi} 0 0" />
         <geometry>
           <mesh filename="package://iai_kitchen/meshes/misc/DishWasherDoor.obj"/>
@@ -73,5 +73,5 @@
     -->
     <joint name="${name}_door_joint" type="revolute">
-      <origin xyz="0.27 0. -0.325" rpy="${-0.5*pi} 0 0" />
+      <origin xyz="0.27 0. -0.285" rpy="${-0.5*pi} 0 0" />
       <parent link="${name}_main"/>
       <child link="${name}_door"/>
@@ -86,5 +86,5 @@
   -->
     <joint name="${name}_door_handle_joint" type="fixed">
-      <origin xyz="0.09 -0.65 0.0" rpy="${-0.5*pi} 0 0" />
+      <origin xyz="0.09 -0.575 0.0" rpy="${-0.5*pi} 0 0" />
       <parent link="${name}_door"/>
       <child link="${name}_door_handle"/>

Commit message: [kitchen urdf] tweaking

File: iai_kitchen/urdf_obj/IAI_dish_washer.urdf.xacro (robot description, xacro)
@@ -86,10 +86,10 @@
   -->
     <joint name="${name}_door_handle_joint" type="fixed">
-      <origin xyz="0.09 -0.575 0.0" rpy="${-0.5*pi} 0 0" />
+      <origin xyz="0.085 -0.575 0.0" rpy="${-0.5*pi} 0 0" />
       <parent link="${name}_door"/>
       <child link="${name}_door_handle"/>
     </joint>
     <dishwasher_tray name="${name}_tray" parent="${name}_main">
-      <origin xyz="-0.10 0 0.15"/>
+      <origin xyz="-0.01 0 0.15"/>
     </dishwasher_tray>
   </macro>
@@ -183,5 +183,5 @@
     </joint>
     <tray_handle name="${name}_handle" parent="${name}_front_side">
-      <origin xyz="0.025 0 -0.05"/>
+      <origin xyz="0.04 0 -0.0"/>
     </tray_handle>
   </macro>

File: iai_kitchen/urdf_obj/IAI_drawers.urdf.xacro (robot description, xacro)
@@ -137,16 +137,36 @@
         <origin rpy="0 0 0" xyz="0 0 0"/>
         <geometry>
-          <box size="0.025 0.295 1.325"/>
-        </geometry>
-      </visual>
-      <collision>
-        <origin rpy="0 0 0" xyz="0 0 0"/>
-        <geometry>
           <box size="0.025 0.3 1.33"/>
         </geometry>
+      </visual>
+      <collision>
+        <origin rpy="0 0 0" xyz="0 0 0"/>
+        <geometry>
+          <box size="0.025 0.3 1.33"/>
+        </geometry>
+      </collision>
+    </link>
+    <joint name="${name}_main_padding_joint" type="fixed">
+      <parent link="${name}_main"/>
+      <child link="${name}_main_padding"/>
+      <origin rpy="0 0 0" xyz="-0.03 0.0 0.0"/>
+    </joint>
+    <link name="${name}_main_padding">
+      <sphere_inertia radius="0" mass="0"/>
+      <visual>
+        <origin rpy="0 0 0" xyz="0 0 0"/>
+        <geometry>
+          <box size="0.06 0.3 1.33"/>
+        </geometry>
+      </visual>
+      <collision>
+        <origin rpy="0 0 0" xyz="0 0 0"/>
+        <geometry>
+          <box size="0.06 0.3 1.33"/>
+        </geometry>
       </collision>
     </link>
     <joint name="${name}_handle_joint" type="fixed">
-      <origin rpy="${-0.5*pi} 0 0" xyz="0.08 0.0 0.0"/>
+      <origin rpy="${-0.5*pi} 0 0" xyz="0.08 0.0 0.05"/>
       <parent link="${name}_main" />
       <child link="${name}_handle" />

File: iai_kitchen/urdf_obj/iai_kitchen_python.urdf.xacro (robot description, xacro)
@@ -39,5 +39,5 @@
   </iai_oven_area>
   <iai_kitchen_island name="kitchen_island" parent="room_link">
-    <origin xyz="-1.365 0.59 0" rpy="0 0 0" />
+    <origin xyz="-1.363 0.59 0" rpy="0 0 0" />
     <!-- <origin xyz="-2.1 -4.94 0" rpy="0 0 ${pi}" /> -->
   </iai_kitchen_island>

Commit message: tuned dishwasher for ease demo

File: iai_kitchen/urdf_obj/IAI_dish_washer.urdf.xacro (robot description, xacro)
@@ -91,5 +91,5 @@
     </joint>
     <dishwasher_tray name="${name}_tray" parent="${name}_main">
-      <origin xyz="-0.01 0 0.15"/>
+      <origin xyz="-0.08 0 0.15"/>
     </dishwasher_tray>
   </macro>
@@ -100,15 +100,15 @@
       <child link="${name}_bottom"/>
       <axis xyz="1 0 0"/>
-      <limit lower="0" upper="0.40" effort="300" velocity="10"/>
+      <limit lower="0" upper="0.48" effort="300" velocity="10"/>
     </joint>
     <link name="${name}_bottom">
       <visual>
         <geometry>
-          <box size="0.32 0.5 0.02"/>
-        </geometry>
-      </visual>
-      <collision>
-        <geometry>
-          <box size="0.32 0.5 0.02"/>
+          <box size="0.32 0.5 0.05"/>
+        </geometry>
+      </visual>
+      <collision>
+        <geometry>
+          <box size="0.32 0.5 0.05"/>
         </geometry>
       </collision>
@@ -183,5 +183,5 @@
     </joint>
     <tray_handle name="${name}_handle" parent="${name}_front_side">
-      <origin xyz="0.04 0 -0.0"/>
+      <origin xyz="0.06 -0.1 -0.02"/>
     </tray_handle>
   </macro>
@@ -219,20 +219,20 @@
       <visual>
         <geometry>
-          <box size="0.01 0.4 0.01"/>
-        </geometry>
-      </visual>
-      <collision>
-        <geometry>
-          <box size="0.01 0.4 0.01"/>
+          <box size="0.01 0.2 0.01"/>
+        </geometry>
+      </visual>
+      <collision>
+        <geometry>
+          <box size="0.01 0.2 0.01"/>
         </geometry>
       </collision>
     </link>
     <joint name="${name}_front_left_joint" type="fixed">
-      <origin xyz="-0.01 -0.2 0"/>
+      <origin xyz="-0.01 -0.1 0"/>
       <child link="${name}_left_side" />
       <parent link="${name}_front_side"/>
     </joint>
     <joint name="${name}_front_right_joint" type="fixed">
-      <origin xyz="-0.01 0.2 0"/>
+      <origin xyz="-0.01 0.1 0"/>
       <child link="${name}_right_side" />
       <parent link="${name}_front_side"/>

File: iai_kitchen/urdf_obj/IAI_drawers.urdf.xacro (robot description, xacro)
@@ -40,6 +40,6 @@
   <xacro:property name="board_x" value="0.49"/>
   <xacro:property name="board_y" value="0.25"/>
-  <xacro:property name="board_z" value="0.016"/>
-  <xacro:property name="barrier_z" value="0.082"/>
+  <xacro:property name="board_z" value="0.036"/>
+  <xacro:property name="barrier_z" value="0.1"/>
   <macro name="iai_vdrawer_board" params="name parent joint_origin_z">
     <link name="${parent}_board_${name}_link">
