Commit message: added xacro prefix to kitchen urdf

File: iai_kitchen/urdf_obj/IAI_dish_washer.urdf.xacro (robot description, xacro)
@@ -2,5 +2,5 @@
 <robot name="iai_dish_washer" xmlns:xacro="http://ros.org/wiki/xacro">
   <xacro:property name="pi" value="3.1415926535897931" />
-  <macro name="iai_dish_washer" params="name parent *origin">
+  <xacro:macro name="iai_dish_washer" params="name parent *origin">
      <link name="${name}_main">
       <sphere_inertia radius="0" mass="0"/>
@@ -90,9 +90,9 @@
       <child link="${name}_door_handle"/>
     </joint>
-    <dishwasher_tray name="${name}_tray" parent="${name}_main">
+    <xacro:dishwasher_tray name="${name}_tray" parent="${name}_main">
       <origin xyz="-0.08 0 0.15"/>
-    </dishwasher_tray>
-  </macro>
-  <macro name="dishwasher_tray" params="name parent *origin">
+    </xacro:dishwasher_tray>
+  </xacro:macro>
+  <xacro:macro name="dishwasher_tray" params="name parent *origin">
     <joint name="${name}_main" type="prismatic">
       <xacro:insert_block name="origin"/>
@@ -182,9 +182,9 @@
       <parent link="${name}_bottom"/>
     </joint>
-    <tray_handle name="${name}_handle" parent="${name}_front_side">
+    <xacro:tray_handle name="${name}_handle" parent="${name}_front_side">
       <origin xyz="0.06 -0.1 -0.02"/>
-    </tray_handle>
-  </macro>
-  <macro name="tray_handle" params="name parent *origin">
+    </xacro:tray_handle>
+  </xacro:macro>
+  <xacro:macro name="tray_handle" params="name parent *origin">
     <joint name="${name}_joint" type="fixed">
       <xacro:insert_block name="origin"/>
@@ -238,4 +238,4 @@
       <parent link="${name}_front_side"/>
     </joint>
-  </macro>
+  </xacro:macro>
 </robot>

File: iai_kitchen/urdf_obj/IAI_drawers.urdf.xacro (robot description, xacro)
@@ -2,45 +2,45 @@
 <robot name="iai_drawers" xmlns:xacro="http://ros.org/wiki/xacro">
   <xacro:property name="pi" value="3.1415926535897931" />
-  <macro name="iai_drawer_60_14" params="name parent *origin">
-    <iai_drawer_14 name="${name}" parent="${parent}" width="60">
-      <xacro:insert_block name="origin" />
-    </iai_drawer_14>
-  </macro>
-  <macro name="iai_drawer_80_14" params="name parent *origin">
-    <iai_drawer_14 name="${name}" parent="${parent}" width="80">
-      <xacro:insert_block name="origin" />
-    </iai_drawer_14>
-  </macro>
-  <macro name="iai_drawer_60_29" params="name parent *origin">
-    <iai_drawer_29 name="${name}" parent="${parent}" width="60">
-      <xacro:insert_block name="origin" />
-    </iai_drawer_29>
-  </macro>
-  <macro name="iai_drawer_80_29" params="name parent *origin">
-    <iai_drawer_29 name="${name}" parent="${parent}" width="80">
-      <xacro:insert_block name="origin" />
-    </iai_drawer_29>
-  </macro>
-  <macro name="iai_drawer_100_29" params="name parent *origin">
-    <iai_drawer_29 name="${name}" parent="${parent}" width="100">
-      <xacro:insert_block name="origin" />
-    </iai_drawer_29>
-  </macro>
-  <macro name="iai_drawer_60_58" params="name parent *origin">
-    <iai_drawer_58 name="${name}" parent="${parent}" width="60">
-      <xacro:insert_block name="origin" />
-    </iai_drawer_58>
-  </macro>
-  <macro name="iai_drawer_58" params="name parent width *origin">
-    <iai_generic_drawer name="${name}" parent="${parent}" width="${width}" height="58">
+  <xacro:macro name="iai_drawer_60_14" params="name parent *origin">
+    <xacro:iai_drawer_14 name="${name}" parent="${parent}" width="60">
+      <xacro:insert_block name="origin" />
+    </xacro:iai_drawer_14>
+  </xacro:macro>
+  <xacro:macro name="iai_drawer_80_14" params="name parent *origin">
+    <xacro:iai_drawer_14 name="${name}" parent="${parent}" width="80">
+      <xacro:insert_block name="origin" />
+    </xacro:iai_drawer_14>
+  </xacro:macro>
+  <xacro:macro name="iai_drawer_60_29" params="name parent *origin">
+    <xacro:iai_drawer_29 name="${name}" parent="${parent}" width="60">
+      <xacro:insert_block name="origin" />
+    </xacro:iai_drawer_29>
+  </xacro:macro>
+  <xacro:macro name="iai_drawer_80_29" params="name parent *origin">
+    <xacro:iai_drawer_29 name="${name}" parent="${parent}" width="80">
+      <xacro:insert_block name="origin" />
+    </xacro:iai_drawer_29>
+  </xacro:macro>
+  <xacro:macro name="iai_drawer_100_29" params="name parent *origin">
+    <xacro:iai_drawer_29 name="${name}" parent="${parent}" width="100">
+      <xacro:insert_block name="origin" />
+    </xacro:iai_drawer_29>
+  </xacro:macro>
+  <xacro:macro name="iai_drawer_60_58" params="name parent *origin">
+    <xacro:iai_drawer_58 name="${name}" parent="${parent}" width="60">
+      <xacro:insert_block name="origin" />
+    </xacro:iai_drawer_58>
+  </xacro:macro>
+  <xacro:macro name="iai_drawer_58" params="name parent width *origin">
+    <xacro:iai_generic_drawer name="${name}" parent="${parent}" width="${width}" height="58">
       <xacro:insert_block name="origin" />
       <origin xyz="0.37 0 0.25" rpy="0 0 0" />
-    </iai_generic_drawer>
-  </macro>
+    </xacro:iai_generic_drawer>
+  </xacro:macro>
   <xacro:property name="board_x" value="0.49"/>
   <xacro:property name="board_y" value="0.25"/>
   <xacro:property name="board_z" value="0.036"/>
   <xacro:property name="barrier_z" value="0.1"/>
-  <macro name="iai_vdrawer_board" params="name parent joint_origin_z">
+  <xacro:macro name="iai_vdrawer_board" params="name parent joint_origin_z">
     <link name="${parent}_board_${name}_link">
       <sphere_inertia radius="0" mass="0"/>
@@ -123,6 +123,6 @@
       <child link="${parent}_barrier_${name}_back_link"/>
     </joint>
-  </macro>
-  <macro name="iai_vdrawer" params="name parent *origin">
+  </xacro:macro>
+  <xacro:macro name="iai_vdrawer" params="name parent *origin">
     <joint name="${name}_main_joint" type="prismatic">
       <xacro:insert_block name="origin"/>
@@ -187,22 +187,22 @@
       </collision>
     </link>
-    <iai_vdrawer_board name="0" parent="${name}" joint_origin_z="-0.6"/>
-    <iai_vdrawer_board name="1" parent="${name}" joint_origin_z="-0.28"/>
-    <iai_vdrawer_board name="2" parent="${name}" joint_origin_z="0.05"/>
-    <iai_vdrawer_board name="3" parent="${name}" joint_origin_z="0.38"/>
-  </macro>
-  <macro name="iai_drawer_29" params="name parent width *origin">
-    <iai_generic_drawer name="${name}" parent="${parent}" width="${width}" height="29">
+    <xacro:iai_vdrawer_board name="0" parent="${name}" joint_origin_z="-0.6"/>
+    <xacro:iai_vdrawer_board name="1" parent="${name}" joint_origin_z="-0.28"/>
+    <xacro:iai_vdrawer_board name="2" parent="${name}" joint_origin_z="0.05"/>
+    <xacro:iai_vdrawer_board name="3" parent="${name}" joint_origin_z="0.38"/>
+  </xacro:macro>
+  <xacro:macro name="iai_drawer_29" params="name parent width *origin">
+    <xacro:iai_generic_drawer name="${name}" parent="${parent}" width="${width}" height="29">
       <xacro:insert_block name="origin" />
       <origin xyz="0.3525 0 0.11" rpy="0 0 0" />
-    </iai_generic_drawer>
-  </macro>
-  <macro name="iai_drawer_14" params="name parent width *origin">
-    <iai_generic_drawer name="${name}" parent="${parent}" width="${width}" height="14">
+    </xacro:iai_generic_drawer>
+  </xacro:macro>
+  <xacro:macro name="iai_drawer_14" params="name parent width *origin">
+    <xacro:iai_generic_drawer name="${name}" parent="${parent}" width="${width}" height="14">
       <xacro:insert_block name="origin" />
       <origin xyz="0.3525 0 0.0175" rpy="0 0 0" />
-    </iai_generic_drawer>
-  </macro>
-  <macro name="iai_generic_drawer" params="name parent width height *origin *handle_origin">
+    </xacro:iai_generic_drawer>
+  </xacro:macro>
+  <xacro:macro name="iai_generic_drawer" params="name parent width height *origin *handle_origin">
     <link name="${name}_main">
       <sphere_inertia radius="0" mass="0"/>
@@ -252,6 +252,6 @@
       <limit lower="0" upper="${0.5*pi}" effort="300" velocity="10"/>
     </joint>
-  </macro>
-  <macro name="iai_generic_panel" params="name parent width *origin">
+  </xacro:macro>
+  <xacro:macro name="iai_generic_panel" params="name parent width *origin">
     <link name="${name}">
       <sphere_inertia radius="0" mass="0"/>
@@ -274,5 +274,5 @@
       <child link="${name}"/>
     </joint>
-  </macro>
+  </xacro:macro>
   <!--- FIXME THIS should NOT be here -->
   <!--

File: iai_kitchen/urdf_obj/IAI_fridge.urdf.xacro (robot description, xacro)
@@ -2,5 +2,5 @@
 <robot name="iai_fridge" xmlns:xacro="http://ros.org/wiki/xacro">
   <xacro:property name="pi" value="3.1415926535897931" />
-  <macro name="iai_fridge" params="name parent *origin">
+  <xacro:macro name="iai_fridge" params="name parent *origin">
      <link name="${name}_main">
       <sphere_inertia radius="0" mass="0"/>
@@ -172,15 +172,15 @@
       <child link="${name}_door_block_top_bar"/>
     </joint>
-    <fridge_door_shelf name="${name}_door_shelf1" parent="${name}_door_block" height="0.1">
+    <xacro:fridge_door_shelf name="${name}_door_shelf1" parent="${name}_door_block" height="0.1">
       <origin xyz="-0.07 0 -0.3525 "/>
-    </fridge_door_shelf>
-    <fridge_door_shelf name="${name}_door_shelf2" parent="${name}_door_block" height="0.065">
+    </xacro:fridge_door_shelf>
+    <xacro:fridge_door_shelf name="${name}_door_shelf2" parent="${name}_door_block" height="0.065">
       <origin xyz="-0.07 0 0.02"/>
-    </fridge_door_shelf>
-    <fridge_door_shelf name="${name}_door_shelf3" parent="${name}_door_block" height="0.065">
+    </xacro:fridge_door_shelf>
+    <xacro:fridge_door_shelf name="${name}_door_shelf3" parent="${name}_door_block" height="0.065">
       <origin xyz="-0.07 0 0.23"/>
-    </fridge_door_shelf>
-  </macro>
-  <macro name="fridge_door_shelf" params="name parent height *origin">
+    </xacro:fridge_door_shelf>
+  </xacro:macro>
+  <xacro:macro name="fridge_door_shelf" params="name parent height *origin">
     <joint name="${name}_to_door" type="fixed">
       <xacro:insert_block name="origin"/>
@@ -251,4 +251,4 @@
       <child link="${name}_front_side"/>
     </joint>
-  </macro>
+  </xacro:macro>
 </robot>

File: iai_kitchen/urdf_obj/IAI_fridge_area.urdf.xacro (robot description, xacro)
@@ -4,5 +4,5 @@
   <xacro:include filename="$(find iai_kitchen)/urdf_obj/IAI_drawers.urdf.xacro"/>
   <xacro:include filename="$(find iai_kitchen)/urdf_obj/IAI_fridge.urdf.xacro"/>
-  <macro name="iai_fridge_area" params="parent name *origin">
+  <xacro:macro name="iai_fridge_area" params="parent name *origin">
     <link name="${name}_footprint">
       <sphere_inertia radius="0" mass="0"/>
@@ -34,10 +34,10 @@
       <child link="${name}"/>
     </joint>
-  <iai_drawer_60_29 name="${name}_lower_drawer" parent="${name}">
+  <xacro:iai_drawer_60_29 name="${name}_lower_drawer" parent="${name}">
     <origin rpy="0 0 0" xyz="0.0 -0.0 -0.4175 "/>
-  </iai_drawer_60_29>
-  <iai_fridge name="iai_fridge" parent="${name}">
+  </xacro:iai_drawer_60_29>
+  <xacro:iai_fridge name="iai_fridge" parent="${name}">
     <origin xyz="0 0 0.25" rpy="0 0 0" />
-  </iai_fridge>
-  </macro>
+  </xacro:iai_fridge>
+  </xacro:macro>
 </robot>

File: iai_kitchen/urdf_obj/IAI_kitchen_island.urdf.xacro (robot description, xacro)
@@ -4,5 +4,5 @@
   <!--- FIXME THIS should NOT be here -->
   <xacro:include filename="$(find iai_kitchen)/urdf_obj/IAI_drawers.urdf.xacro"/>
-  <macro name="iai_kitchen_island" params="parent name *origin">
+  <xacro:macro name="iai_kitchen_island" params="parent name *origin">
     <link name="${name}_footprint">
       <sphere_inertia radius="0" mass="0"/>
@@ -67,31 +67,31 @@
       <child link="${name}_stove"/>
     </joint>
-    <iai_generic_panel name="${name}_left_panel" parent="${name}" width="60">
+    <xacro:iai_generic_panel name="${name}_left_panel" parent="${name}" width="60">
       <origin rpy="0 0 0" xyz="0.2725 -0.8 0.329 "/>
-    </iai_generic_panel>
-    <iai_drawer_60_29 name="${name}_left_upper_drawer" parent="${name}">
+    </xacro:iai_generic_panel>
+    <xacro:iai_drawer_60_29 name="${name}_left_upper_drawer" parent="${name}">
       <origin rpy="0 0 0" xyz="0.0025 -0.8 0.114 "/>
-    </iai_drawer_60_29>
-    <iai_drawer_60_29 name="${name}_left_lower_drawer" parent="${name}">
+    </xacro:iai_drawer_60_29>
+    <xacro:iai_drawer_60_29 name="${name}_left_lower_drawer" parent="${name}">
       <origin rpy="0 0 0" xyz="0.0025 -0.8 -0.176 "/>
-    </iai_drawer_60_29>
-    <iai_generic_panel name="${name}_middle_panel" parent="${name}" width="100">
+    </xacro:iai_drawer_60_29>
+    <xacro:iai_generic_panel name="${name}_middle_panel" parent="${name}" width="100">
       <origin rpy="0 0 0" xyz="0.2725 0 0.329 "/>
-    </iai_generic_panel>
-    <iai_drawer_100_29 name="${name}_middle_upper_drawer" parent="${name}">
+    </xacro:iai_generic_panel>
+    <xacro:iai_drawer_100_29 name="${name}_middle_upper_drawer" parent="${name}">
       <origin rpy="0 0 0" xyz="0.0025 0 0.114 "/>
-    </iai_drawer_100_29>
-    <iai_drawer_100_29 name="${name}_middle_lower_drawer" parent="${name}">
+    </xacro:iai_drawer_100_29>
+    <xacro:iai_drawer_100_29 name="${name}_middle_lower_drawer" parent="${name}">
       <origin rpy="0 0 0" xyz="0.0025 0 -0.176 "/>
-    </iai_drawer_100_29>
-    <iai_generic_panel name="${name}_right_panel" parent="${name}" width="60">
+    </xacro:iai_drawer_100_29>
+    <xacro:iai_generic_panel name="${name}_right_panel" parent="${name}" width="60">
       <origin rpy="0 0 0" xyz="0.2725 0.8 0.329 "/>
-    </iai_generic_panel>
-    <iai_drawer_60_29 name="${name}_right_upper_drawer" parent="${name}">
+    </xacro:iai_generic_panel>
+    <xacro:iai_drawer_60_29 name="${name}_right_upper_drawer" parent="${name}">
       <origin rpy="0 0 0" xyz="0.0025 0.8 0.114 "/>
-    </iai_drawer_60_29>
-    <iai_drawer_60_29 name="${name}_right_lower_drawer" parent="${name}">
+    </xacro:iai_drawer_60_29>
+    <xacro:iai_drawer_60_29 name="${name}_right_lower_drawer" parent="${name}">
       <origin rpy="0 0 0" xyz="0.0025 0.8 -0.176 "/>
-    </iai_drawer_60_29>
-  </macro>
+    </xacro:iai_drawer_60_29>
+  </xacro:macro>
 </robot>

File: iai_kitchen/urdf_obj/IAI_kitchen_walls.urdf.xacro (robot description, xacro)
@@ -1,5 +1,5 @@
 <?xml version="1.0"?>
 <robot name="iai_kitchen_wall_robohow" xmlns:xacro="http://ros.org/wiki/xacro">
-  <macro name="iai_kitchen_wall_robohow" params="parent *origin">
+  <xacro:macro name="iai_kitchen_wall_robohow" params="parent *origin">
     <!-- LINKS -->
     <link name="kitchen_wall_1">
@@ -160,4 +160,4 @@
         <material>Gazebo/DarkGrey</material>
     </gazebo>
-  </macro>
+  </xacro:macro>
 </robot>

File: iai_kitchen/urdf_obj/IAI_oven.urdf.xacro (robot description, xacro)
@@ -2,5 +2,5 @@
 <robot name="iai_oven" xmlns:xacro="http://ros.org/wiki/xacro">
   <xacro:property name="pi" value="3.1415926535897931" />
-  <macro name="iai_oven" params="name parent *origin">
+  <xacro:macro name="iai_oven" params="name parent *origin">
     <!-- LINKS -->
     <link name="${name}_main">
@@ -113,11 +113,11 @@
     </joint>
     <!--KNOBS -->
-    <iai_oven_knob name="${name}_knob_stove_1" parent="${name}_panel" xyz="0 -0.21 0"/>
-    <iai_oven_knob name="${name}_knob_stove_2" parent="${name}_panel" xyz="0 -0.14 0"/>
-    <iai_oven_knob name="${name}_knob_stove_3" parent="${name}_panel" xyz="0 -0.07 0"/>
-    <iai_oven_knob name="${name}_knob_stove_4" parent="${name}_panel" xyz="0 -0.0 0"/>
-    <iai_oven_knob name="${name}_knob_oven" parent="${name}_panel" xyz="0 0.16 0"/>
-  </macro>
-  <macro name="iai_oven_knob" params="name parent xyz">
+    <xacro:iai_oven_knob name="${name}_knob_stove_2" parent="${name}_panel" xyz="0 -0.14 0"/>
+    <xacro:iai_oven_knob name="${name}_knob_stove_1" parent="${name}_panel" xyz="0 -0.21 0"/>
+    <xacro:iai_oven_knob name="${name}_knob_stove_3" parent="${name}_panel" xyz="0 -0.07 0"/>
+    <xacro:iai_oven_knob name="${name}_knob_stove_4" parent="${name}_panel" xyz="0 -0.0 0"/>
+    <xacro:iai_oven_knob name="${name}_knob_oven" parent="${name}_panel" xyz="0 0.16 0"/>
+  </xacro:macro>
+  <xacro:macro name="iai_oven_knob" params="name parent xyz">
     <link name="${name}">
       <sphere_inertia radius="0" mass="0"/>
@@ -142,5 +142,5 @@
       <limit lower="0" upper="${pi}" effort="300" velocity="10"/>
     </joint>
-  </macro>
+  </xacro:macro>
   <!--- FIXME THIS should NOT be here -->
 <!--

File: iai_kitchen/urdf_obj/IAI_oven_area.urdf.xacro (robot description, xacro)
@@ -5,5 +5,5 @@
   <xacro:include filename="$(find iai_kitchen)/urdf_obj/IAI_drawers.urdf.xacro"/>
   <xacro:include filename="$(find iai_kitchen)/urdf_obj/IAI_oven.urdf.xacro"/>
-  <macro name="iai_oven_area" params="parent name *origin">
+  <xacro:macro name="iai_oven_area" params="parent name *origin">
   <link name="${name}_area_footprint">
     <sphere_inertia radius="0" mass="0"/>
@@ -34,19 +34,19 @@
     <child link="${name}_area"/>
   </joint>
-  <iai_oven name="${name}_oven" parent="${name}_area">
+  <xacro:iai_oven name="${name}_oven" parent="${name}_area">
     <origin rpy="0 0 0" xyz="0.0 0.0 0.415"/>
-  </iai_oven>
-  <iai_drawer_60_14 name="${name}_area_middle_upper_drawer" parent="${name}_area">
+  </xacro:iai_oven>
+  <xacro:iai_drawer_60_14 name="${name}_area_middle_upper_drawer" parent="${name}_area">
     <origin rpy="0 0 0" xyz="0.0 -0. 0.045 "/>
-  </iai_drawer_60_14>
-  <iai_drawer_60_58 name="${name}_area_middle_lower_drawer" parent="${name}_area">
+  </xacro:iai_drawer_60_14>
+  <xacro:iai_drawer_60_58 name="${name}_area_middle_lower_drawer" parent="${name}_area">
     <origin rpy="0 0 0" xyz="0.0 -0. -0.315 "/>
-  </iai_drawer_60_58>
-  <iai_vdrawer name="${name}_area_left_drawer" parent="${name}_area">
+  </xacro:iai_drawer_60_58>
+  <xacro:iai_vdrawer name="${name}_area_left_drawer" parent="${name}_area">
     <origin rpy="0 0 0" xyz="0.29 -0.45 0.07 "/>
-  </iai_vdrawer>
-  <iai_vdrawer name="${name}_area_right_drawer" parent="${name}_area">
+  </xacro:iai_vdrawer>
+  <xacro:iai_vdrawer name="${name}_area_right_drawer" parent="${name}_area">
     <origin rpy="0 0 0" xyz="0.29 0.45 0.07"/>
-  </iai_vdrawer>
-  </macro>
+  </xacro:iai_vdrawer>
+  </xacro:macro>
 </robot>

File: iai_kitchen/urdf_obj/IAI_sink_area.urdf.xacro (robot description, xacro)
@@ -5,5 +5,5 @@
   <xacro:include filename="$(find iai_kitchen)/urdf_obj/IAI_drawers.urdf.xacro"/>
   <xacro:include filename="$(find iai_kitchen)/urdf_obj/IAI_dish_washer.urdf.xacro"/>
-  <macro name="iai_sink_area" params="parent name *origin">
+  <xacro:macro name="iai_sink_area" params="parent name *origin">
   <link name="${name}_footprint">
     <sphere_inertia radius="0" mass="0"/>
@@ -68,22 +68,22 @@
     <child link="${name}_sink"/>
   </joint>
-  <iai_generic_panel name="${name}_right_panel" parent="${name}" width="60">
+  <xacro:iai_generic_panel name="${name}_right_panel" parent="${name}" width="60">
     <origin rpy="0 0 0" xyz="0.28 0.7 0.355 "/>
-  </iai_generic_panel>
-  <iai_drawer_60_58 name="${name}_trash_drawer" parent="${name}">
+  </xacro:iai_generic_panel>
+  <xacro:iai_drawer_60_58 name="${name}_trash_drawer" parent="${name}">
     <origin rpy="0 0 0" xyz="0.01 0.7 -0.015 "/>
-  </iai_drawer_60_58>
-  <iai_drawer_80_14 name="${name}_left_upper_drawer" parent="${name}">
+  </xacro:iai_drawer_60_58>
+  <xacro:iai_drawer_80_14 name="${name}_left_upper_drawer" parent="${name}">
     <origin rpy="0 0 0" xyz="0.01 -0.6 0.345 "/>
-  </iai_drawer_80_14>
-  <iai_drawer_80_29 name="${name}_left_middle_drawer" parent="${name}">
+  </xacro:iai_drawer_80_14>
+  <xacro:iai_drawer_80_29 name="${name}_left_middle_drawer" parent="${name}">
     <origin rpy="0 0 0" xyz="0.01 -0.6 0.12 "/>
-  </iai_drawer_80_29>
-  <iai_drawer_80_29 name="${name}_left_bottom_drawer" parent="${name}">
+  </xacro:iai_drawer_80_29>
+  <xacro:iai_drawer_80_29 name="${name}_left_bottom_drawer" parent="${name}">
     <origin rpy="0 0 0" xyz="0.01 -0.6 -0.18" />
-  </iai_drawer_80_29>
-  <iai_dish_washer name="${name}_dish_washer" parent="${name}">
+  </xacro:iai_drawer_80_29>
+  <xacro:iai_dish_washer name="${name}_dish_washer" parent="${name}">
     <origin rpy="0 0 0" xyz="0.01 0.1 0.06" />
-  </iai_dish_washer>
-  </macro>
+  </xacro:iai_dish_washer>
+  </xacro:macro>
 </robot>

File: iai_kitchen/urdf_obj/IAI_tables.urdf.xacro (robot description, xacro)
@@ -1,5 +1,5 @@
 <?xml version="1.0"?>
 <robot name="iai_table" xmlns:xacro="http://ros.org/wiki/xacro">
-  <macro name="iai_table_1" params="name parent *origin">
+  <xacro:macro name="iai_table_1" params="name parent *origin">
     <link name="${name}_main">
       <sphere_inertia radius="0" mass="0"/>
@@ -22,6 +22,6 @@
       <child link="${name}_main"/>
     </joint>
-  </macro>
-  <macro name="jokkmokk_table" params="name parent *origin">
+  </xacro:macro>
+  <xacro:macro name="jokkmokk_table" params="name parent *origin">
     <link name="${name}_main">
       <sphere_inertia radius="0" mass="0"/>
@@ -45,6 +45,6 @@
       <origin xyz="0.0 0.0 0.0" rpy="0 0 0" />
     </joint>
-  </macro>
-  <macro name="jokkmokk_chair" params="name parent *origin">
+  </xacro:macro>
+  <xacro:macro name="jokkmokk_chair" params="name parent *origin">
     <link name="${name}_main">
       <sphere_inertia radius="0" mass="0"/>
@@ -67,6 +67,6 @@
       <child link="${name}_main"/>
     </joint>
-  </macro>
-  <macro name="iai_dining_area" params="parent name *origin">
+  </xacro:macro>
+  <xacro:macro name="iai_dining_area" params="parent name *origin">
     <link name="${name}_footprint">
       <sphere_inertia radius="0" mass="0"/>
@@ -77,13 +77,13 @@
       <parent link="${parent}"/>
     </joint>
-    <jokkmokk_table name="${name}_jokkmokk_table" parent="${name}_footprint">
+    <xacro:jokkmokk_table name="${name}_jokkmokk_table" parent="${name}_footprint">
       <origin xyz="0 0 0.35" rpy="0 0 0" />
-    </jokkmokk_table>
-    <jokkmokk_chair name="${name}_jokkmokk_left_chair" parent="${name}_footprint">
+    </xacro:jokkmokk_table>
+    <xacro:jokkmokk_chair name="${name}_jokkmokk_left_chair" parent="${name}_footprint">
       <origin xyz="-1 0 0.5535" rpy="0 0 0" />
-    </jokkmokk_chair>
-    <jokkmokk_chair name="${name}_jokkmokk_right_chair" parent="${name}_footprint">
+    </xacro:jokkmokk_chair>
+    <xacro:jokkmokk_chair name="${name}_jokkmokk_right_chair" parent="${name}_footprint">
       <origin xyz="1 0 0.5535" rpy="0 0 ${-pi}" />
-    </jokkmokk_chair>
-  </macro>
+    </xacro:jokkmokk_chair>
+  </xacro:macro>
 </robot>
