Commit message: added xacro prefix to kitchen urdf

File: iai_kitchen/urdf_obj/iai_kitchen_python.urdf.xacro (robot description, xacro)
@@ -9,5 +9,5 @@
   <xacro:property name="pi" value="3.1415926535897931" />
   <xacro:property name="simulated" value="true" />
-  <macro name="sphere_inertia" params="radius mass">
+  <xacro:macro name="sphere_inertia" params="radius mass">
     <inertial>
       <origin xyz="0.0 0.0 0.0" rpy="0 0 0"/>
@@ -18,5 +18,5 @@
           izz="1"/>
     </inertial>
-  </macro>
+  </xacro:macro>
   <link name="room_link">
     <sphere_inertia radius="0" mass="0"/>
@@ -30,29 +30,29 @@
     </joint>
   </xacro:if>
-  <iai_sink_area name="sink_area" parent="room_link">
+  <xacro:iai_sink_area name="sink_area" parent="room_link">
     <origin xyz="1.855 1.3 0" rpy="0 0 ${pi}" />
     <!-- <origin xyz="-5.29 -5.65 0" rpy="0 0 0" /> -->
-  </iai_sink_area>
-  <iai_oven_area name="oven_area" parent="room_link">
+  </xacro:iai_sink_area>
+  <xacro:iai_oven_area name="oven_area" parent="room_link">
     <origin xyz="1.845 2.5 0" rpy="0 0 ${pi}" />
     <!-- <origin xyz="-5.27 -6.85 0" rpy="0 0 0" /> -->
-  </iai_oven_area>
-  <iai_kitchen_island name="kitchen_island" parent="room_link">
+  </xacro:iai_oven_area>
+  <xacro:iai_kitchen_island name="kitchen_island" parent="room_link">
     <origin xyz="-1.363 0.59 0" rpy="0 0 0" />
     <!-- <origin xyz="-2.1 -4.94 0" rpy="0 0 ${pi}" /> -->
-  </iai_kitchen_island>
-  <iai_fridge_area name="fridge_area" parent="room_link">
+  </xacro:iai_kitchen_island>
+  <xacro:iai_fridge_area name="fridge_area" parent="room_link">
     <origin xyz="1.845 -0.73 0" rpy="0 0 ${pi}" />
     <!-- <origin xyz="-5.29 -3.59 0" rpy="0 0 0" /> -->
-  </iai_fridge_area>
-  <iai_table_1 name="table_area" parent="room_link">
+  </xacro:iai_fridge_area>
+  <xacro:iai_table_1 name="table_area" parent="room_link">
     <origin xyz="-2.4 -1.5 0" rpy="0 0 ${pi}" />
-  </iai_table_1>
-  <iai_dining_area name="dining_area" parent="room_link">
+  </xacro:iai_table_1>
+  <xacro:iai_dining_area name="dining_area" parent="room_link">
     <origin xyz="-3.38 0.28 0" rpy="0 0 ${pi / 2}" />
-  </iai_dining_area>
-  <iai_kitchen_wall_robohow parent="room_link">
+  </xacro:iai_dining_area>
+  <xacro:iai_kitchen_wall_robohow parent="room_link">
     <origin xyz="-0.96 0.65 0" rpy="0.0 0.0 0.0" />
-  </iai_kitchen_wall_robohow>
+  </xacro:iai_kitchen_wall_robohow>
   <gazebo>
     <static>false</static>

Commit message: fixed fixed joint being falsely flagged as revolute

File: iai_kitchen/urdf_obj/IAI_dish_washer.urdf.xacro (robot description, xacro)
@@ -51,6 +51,5 @@
     <xacro:if value="simulated"/>
     -->
-    <joint name="${name}_main_joint" type="revolute">
-      <limit lower="0" upper="0" effort="300" velocity="10"/>
+    <joint name="${name}_main_joint" type="fixed">
       <xacro:insert_block name="origin" />
       <parent link="${parent}"/>

Commit message: Use collada for visual meshes.

File: iai_kitchen/urdf_obj/IAI_dish_washer.urdf.xacro (robot description, xacro)
@@ -4,39 +4,39 @@
   <xacro:macro name="iai_dish_washer" params="name parent *origin">
      <link name="${name}_main">
-      <sphere_inertia radius="0" mass="0"/>
-      <visual>
+      <xacro:sphere_inertia radius="0" mass="0"/>
+      <visual>
+        <origin xyz="0 0 0" rpy="0 0 0" />
+        <geometry>
+          <mesh filename="package://iai_kitchen/meshes/misc/DishWasher.dae"/>
+        </geometry>
+      </visual>
+      <collision>
         <origin xyz="0 0 0" rpy="0 0 0" />
         <geometry>
           <mesh filename="package://iai_kitchen/meshes/misc/DishWasher.obj"/>
         </geometry>
-      </visual>
-      <collision>
-        <origin xyz="0 0 0" rpy="0 0 0" />
-        <geometry>
-          <mesh filename="package://iai_kitchen/meshes/misc/DishWasher.obj"/>
-        </geometry>
       </collision>
     </link>
     <link name="${name}_door">
-      <sphere_inertia radius="0" mass="0"/>
+      <xacro:sphere_inertia radius="0" mass="0"/>
       <visual>
         <origin xyz="0 0.055 0" rpy="${0.5*pi} 0 0" />
         <geometry>
+          <mesh filename="package://iai_kitchen/meshes/misc/DishWasherDoor.dae"/>
+        </geometry>
+      </visual>
+      <collision>
+        <origin xyz="0 0.055 0" rpy="${0.5*pi} 0 0" />
+        <geometry>
           <mesh filename="package://iai_kitchen/meshes/misc/DishWasherDoor.obj"/>
         </geometry>
-      </visual>
-      <collision>
-        <origin xyz="0 0.055 0" rpy="${0.5*pi} 0 0" />
-        <geometry>
-          <mesh filename="package://iai_kitchen/meshes/misc/DishWasherDoor.obj"/>
-        </geometry>
       </collision>
     </link>
     <link name="${name}_door_handle">
-      <sphere_inertia radius="0" mass="0"/>
-      <visual>
-        <origin xyz="0 0 0" rpy="0 0 0" />
-        <geometry>
-          <mesh filename="package://iai_kitchen/meshes/handles/Handle60.obj"/>
+      <xacro:sphere_inertia radius="0" mass="0"/>
+      <visual>
+        <origin xyz="0 0 0" rpy="0 0 0" />
+        <geometry>
+          <mesh filename="package://iai_kitchen/meshes/handles/Handle60.dae"/>
         </geometry>
       </visual>

File: iai_kitchen/urdf_obj/IAI_drawers.urdf.xacro (robot description, xacro)
@@ -44,5 +44,5 @@
   <xacro:macro name="iai_vdrawer_board" params="name parent joint_origin_z">
     <link name="${parent}_board_${name}_link">
-      <sphere_inertia radius="0" mass="0"/>
+      <xacro:sphere_inertia radius="0" mass="0"/>
       <visual>
         <origin rpy="0 0 0" xyz="0 0 0"/>
@@ -64,5 +64,5 @@
     </joint>
     <link name="${parent}_barrier_${name}_right_link">
-      <sphere_inertia radius="0" mass="0"/>
+      <xacro:sphere_inertia radius="0" mass="0"/>
       <visual>
         <origin rpy="0 0 0" xyz="0 0 0"/>
@@ -84,5 +84,5 @@
     </joint>
     <link name="${parent}_barrier_${name}_left_link">
-      <sphere_inertia radius="0" mass="0"/>
+      <xacro:sphere_inertia radius="0" mass="0"/>
       <visual>
         <origin rpy="0 0 0" xyz="0 0 0"/>
@@ -104,5 +104,5 @@
     </joint>
     <link name="${parent}_barrier_${name}_back_link">
-      <sphere_inertia radius="0" mass="0"/>
+      <xacro:sphere_inertia radius="0" mass="0"/>
       <visual>
         <origin rpy="0 0 0" xyz="0 0 0"/>
@@ -133,5 +133,5 @@
     </joint>
     <link name="${name}_main">
-      <sphere_inertia radius="0" mass="0"/>
+      <xacro:sphere_inertia radius="0" mass="0"/>
       <visual>
         <origin rpy="0 0 0" xyz="0 0 0"/>
@@ -139,4 +139,7 @@
           <box size="0.025 0.3 1.33"/>
         </geometry>
+        <material name="KitchenLightGray">
+          <color rgba="0.7 0.7 0.7 1.0"/>
+        </material>
       </visual>
       <collision>
@@ -153,5 +156,5 @@
     </joint>
     <link name="${name}_main_padding">
-      <sphere_inertia radius="0" mass="0"/>
+      <xacro:sphere_inertia radius="0" mass="0"/>
       <visual>
         <origin rpy="0 0 0" xyz="0 0 0"/>
@@ -173,9 +176,9 @@
     </joint>
     <link name="${name}_handle">
-      <sphere_inertia radius="0" mass="0"/>
+      <xacro:sphere_inertia radius="0" mass="0"/>
       <visual>
         <origin xyz="0 0 0" rpy="${0.5*pi} 0 0" />
         <geometry>
-          <mesh filename="package://iai_kitchen/meshes/handles/VHandle130.obj"/>
+          <mesh filename="package://iai_kitchen/meshes/handles/VHandle130.dae"/>
         </geometry>
       </visual>
@@ -206,24 +209,24 @@
   <xacro:macro name="iai_generic_drawer" params="name parent width height *origin *handle_origin">
     <link name="${name}_main">
-      <sphere_inertia radius="0" mass="0"/>
-      <visual>
+      <xacro:sphere_inertia radius="0" mass="0"/>
+      <visual>
+        <origin xyz="0 0 0" rpy="0 0 0" />
+        <geometry>
+          <mesh filename="package://iai_kitchen/meshes/drawers/Drawer_${width}_${height}.dae"/>
+        </geometry>
+      </visual>
+      <collision>
         <origin xyz="0 0 0" rpy="0 0 0" />
         <geometry>
           <mesh filename="package://iai_kitchen/meshes/drawers/Drawer_${width}_${height}.obj"/>
         </geometry>
-      </visual>
-      <collision>
-        <origin xyz="0 0 0" rpy="0 0 0" />
-        <geometry>
-          <mesh filename="package://iai_kitchen/meshes/drawers/Drawer_${width}_${height}.obj"/>
-        </geometry>
       </collision>
     </link>
     <link name="${name}_handle">
-      <sphere_inertia radius="0" mass="0"/>
-      <visual>
-        <origin xyz="0 0 0" rpy="0 0 0" />
-        <geometry>
-          <mesh filename="package://iai_kitchen/meshes/handles/Handle${width}.obj"/>
+      <xacro:sphere_inertia radius="0" mass="0"/>
+      <visual>
+        <origin xyz="0 0 0" rpy="0 0 0" />
+        <geometry>
+          <mesh filename="package://iai_kitchen/meshes/handles/Handle${width}.dae"/>
         </geometry>
       </visual>
@@ -255,9 +258,9 @@
   <xacro:macro name="iai_generic_panel" params="name parent width *origin">
     <link name="${name}">
-      <sphere_inertia radius="0" mass="0"/>
-      <visual>
-        <origin xyz="0 0 0" rpy="0 0 0" />
-        <geometry>
-          <mesh filename="package://iai_kitchen/meshes/drawers/Panel_${width}.obj"/>
+      <xacro:sphere_inertia radius="0" mass="0"/>
+      <visual>
+        <origin xyz="0 0 0" rpy="0 0 0" />
+        <geometry>
+          <mesh filename="package://iai_kitchen/meshes/drawers/Panel_${width}.dae"/>
         </geometry>
       </visual>

File: iai_kitchen/urdf_obj/IAI_fridge.urdf.xacro (robot description, xacro)
@@ -4,16 +4,16 @@
   <xacro:macro name="iai_fridge" params="name parent *origin">
      <link name="${name}_main">
-      <sphere_inertia radius="0" mass="0"/>
-      <visual>
+      <xacro:sphere_inertia radius="0" mass="0"/>
+      <visual>
+        <origin xyz="0 0 0" rpy="0 0 0" />
+        <geometry>
+          <mesh filename="package://iai_kitchen/meshes/misc/Fridge.dae"/>
+        </geometry>
+      </visual>
+      <collision>
         <origin xyz="0 0 0" rpy="0 0 0" />
         <geometry>
           <mesh filename="package://iai_kitchen/meshes/misc/Fridge.obj"/>
         </geometry>
-      </visual>
-      <collision>
-        <origin xyz="0 0 0" rpy="0 0 0" />
-        <geometry>
-          <mesh filename="package://iai_kitchen/meshes/misc/Fridge.obj"/>
-        </geometry>
       </collision>
     </link>
@@ -33,9 +33,9 @@
     </link>
     <link name="${name}_door">
-      <sphere_inertia radius="0" mass="0"/>
-      <visual>
-        <origin xyz="0 0 0" rpy="0 0 0" />
-        <geometry>
-          <mesh filename="package://iai_kitchen/meshes/misc/FridgeDoor.obj"/>
+      <xacro:sphere_inertia radius="0" mass="0"/>
+      <visual>
+        <origin xyz="0 0 0" rpy="0 0 0" />
+        <geometry>
+          <mesh filename="package://iai_kitchen/meshes/misc/FridgeDoor.dae"/>
         </geometry>
       </visual>
@@ -60,9 +60,9 @@
   </link>
     <link name="${name}_door_handle">
-      <sphere_inertia radius="0" mass="0"/>
-      <visual>
-        <origin xyz="0 0 0" rpy="0 0 0" />
-        <geometry>
-          <mesh filename="package://iai_kitchen/meshes/handles/VHandle90.obj"/>
+      <xacro:sphere_inertia radius="0" mass="0"/>
+      <visual>
+        <origin xyz="0 0 0" rpy="0 0 0" />
+        <geometry>
+          <mesh filename="package://iai_kitchen/meshes/handles/VHandle90.dae"/>
         </geometry>
       </visual>

File: iai_kitchen/urdf_obj/IAI_fridge_area.urdf.xacro (robot description, xacro)
@@ -6,12 +6,12 @@
   <xacro:macro name="iai_fridge_area" params="parent name *origin">
     <link name="${name}_footprint">
-      <sphere_inertia radius="0" mass="0"/>
+      <xacro:sphere_inertia radius="0" mass="0"/>
     </link>
     <link name="${name}">
-      <sphere_inertia radius="0" mass="0"/>
+      <xacro:sphere_inertia radius="0" mass="0"/>
       <visual>
     	  <origin xyz="0 0 0.01" rpy="0 0 0" />
     	  <geometry>
-    	    <mesh filename="package://iai_kitchen/meshes/racks/FridgeArea.obj"/>
+    	    <mesh filename="package://iai_kitchen/meshes/racks/FridgeArea.dae"/>
     	  </geometry>
     	</visual>

File: iai_kitchen/urdf_obj/IAI_kitchen_island.urdf.xacro (robot description, xacro)
@@ -6,12 +6,12 @@
   <xacro:macro name="iai_kitchen_island" params="parent name *origin">
     <link name="${name}_footprint">
-      <sphere_inertia radius="0" mass="0"/>
+      <xacro:sphere_inertia radius="0" mass="0"/>
     </link>
     <link name="${name}">
-      <sphere_inertia radius="0" mass="0"/>
+      <xacro:sphere_inertia radius="0" mass="0"/>
       <visual>
         <origin xyz="0 0 0" rpy="0 0 0" />
         <geometry>
-          <mesh filename="package://iai_kitchen/meshes/racks/IslandArea.obj"/>
+          <mesh filename="package://iai_kitchen/meshes/racks/IslandArea.dae"/>
         </geometry>
       </visual>
@@ -34,5 +34,5 @@
     </joint>
     <link name="${name}_surface">
-      <sphere_inertia radius="0" mass="0"/>
+      <xacro:sphere_inertia radius="0" mass="0"/>
       <collision>
           <origin xyz="0 0 0" rpy="0 0 0" />
@@ -48,9 +48,9 @@
     </joint>
     <link name="${name}_stove">
-      <sphere_inertia radius="0" mass="0"/>
+      <xacro:sphere_inertia radius="0" mass="0"/>
       <visual>
           <origin xyz="0 0 0" rpy="0 0 0" />
           <geometry>
-            <mesh filename="package://iai_kitchen/meshes/misc/Stove.obj"/>
+            <mesh filename="package://iai_kitchen/meshes/misc/Stove.dae"/>
           </geometry>
         </visual>

File: iai_kitchen/urdf_obj/IAI_kitchen_walls.urdf.xacro (robot description, xacro)
@@ -4,5 +4,5 @@
     <!-- LINKS -->
     <link name="kitchen_wall_1">
-      <sphere_inertia radius="0" mass="0"/>
+      <xacro:sphere_inertia radius="0" mass="0"/>
       <visual>
         <origin xyz="0 0 1.25" rpy="0 0 0" />
@@ -19,5 +19,5 @@
     </link>
     <link name="kitchen_wall_2">
-      <sphere_inertia radius="0" mass="0"/>
+      <xacro:sphere_inertia radius="0" mass="0"/>
       <visual>
         <origin xyz="0 0 1.25" rpy="0 0 0" />
@@ -34,5 +34,5 @@
     </link>
     <link name="kitchen_wall_3">
-      <sphere_inertia radius="0" mass="0"/>
+      <xacro:sphere_inertia radius="0" mass="0"/>
       <visual>
         <origin xyz="0 0 1.25" rpy="0 0 0" />
@@ -49,5 +49,5 @@
     </link>
     <link name="kitchen_wall_4">
-      <sphere_inertia radius="0" mass="0"/>
+      <xacro:sphere_inertia radius="0" mass="0"/>
       <visual>
         <origin xyz="0 0 0.35" rpy="0 0 0" />
@@ -64,5 +64,5 @@
     </link>
     <link name="kitchen_wall_5">
-      <sphere_inertia radius="0" mass="0"/>
+      <xacro:sphere_inertia radius="0" mass="0"/>
       <visual>
         <origin xyz="0 0 0.35" rpy="0 0 0" />
@@ -79,5 +79,5 @@
     </link>
     <link name="kitchen_wall_6">
-      <sphere_inertia radius="0" mass="0"/>
+      <xacro:sphere_inertia radius="0" mass="0"/>
       <visual>
         <origin xyz="0 0 0.35" rpy="0 0 0" />
@@ -94,5 +94,5 @@
     </link>
     <link name="kitchen_wall_7">
-      <sphere_inertia radius="0" mass="0"/>
+      <xacro:sphere_inertia radius="0" mass="0"/>
       <visual>
         <origin xyz="0 0 0.375" rpy="0 0 0" />

File: iai_kitchen/urdf_obj/IAI_oven.urdf.xacro (robot description, xacro)
@@ -5,9 +5,9 @@
     <!-- LINKS -->
     <link name="${name}_main">
-      <sphere_inertia radius="0" mass="0"/>
+      <xacro:sphere_inertia radius="0" mass="0"/>
       <visual>
         <origin xyz="0 0 0" rpy="0 0 0" />
         <geometry>
-          <mesh filename="package://iai_kitchen/meshes/oven/OvenMain.obj"/>
+          <mesh filename="package://iai_kitchen/meshes/oven/OvenMain.dae"/>
         </geometry>
       </visual>
@@ -20,9 +20,9 @@
     </link>
     <link name="${name}_door">
-      <sphere_inertia radius="0" mass="0"/>
+      <xacro:sphere_inertia radius="0" mass="0"/>
       <visual>
         <origin xyz="0 0 0" rpy="${0.5*pi} 0 0" />
         <geometry>
-          <mesh filename="package://iai_kitchen/meshes/oven/OvenDoor.obj"/>
+          <mesh filename="package://iai_kitchen/meshes/oven/OvenDoor.dae"/>
         </geometry>
       </visual>
@@ -35,9 +35,9 @@
     </link>
     <link name="${name}_door_handle">
-      <sphere_inertia radius="0" mass="0"/>
+      <xacro:sphere_inertia radius="0" mass="0"/>
       <visual>
         <origin xyz="0 0 0" rpy="0 0 0" />
         <geometry>
-          <mesh filename="package://iai_kitchen/meshes/handles/Handle60.obj"/>
+          <mesh filename="package://iai_kitchen/meshes/handles/Handle60.dae"/>
         </geometry>
       </visual>
@@ -50,9 +50,9 @@
     </link>
     <link name="${name}_panel">
-      <sphere_inertia radius="0" mass="0"/>
+      <xacro:sphere_inertia radius="0" mass="0"/>
       <visual>
         <origin xyz="0 0 0" rpy="0 0 0" />
         <geometry>
-          <mesh filename="package://iai_kitchen/meshes/oven/OvenPanel.obj"/>
+          <mesh filename="package://iai_kitchen/meshes/oven/OvenPanel.dae"/>
         </geometry>
       </visual>
@@ -121,5 +121,5 @@
   <xacro:macro name="iai_oven_knob" params="name parent xyz">
     <link name="${name}">
-      <sphere_inertia radius="0" mass="0"/>
+      <xacro:sphere_inertia radius="0" mass="0"/>
       <visual>
         <origin xyz="0 0 0" rpy="0 ${0.5 * pi} 0" />
@@ -146,5 +146,5 @@
 <!--
   <link name="oven_footprint">
-    <sphere_inertia radius="0" mass="0"/>
+    <xacro:sphere_inertia radius="0" mass="0"/>
   </link>
   <iai_oven name="iai_oven" parent="oven_footprint"/>

File: iai_kitchen/urdf_obj/IAI_oven_area.urdf.xacro (robot description, xacro)
@@ -7,12 +7,12 @@
   <xacro:macro name="iai_oven_area" params="parent name *origin">
   <link name="${name}_area_footprint">
-    <sphere_inertia radius="0" mass="0"/>
+    <xacro:sphere_inertia radius="0" mass="0"/>
   </link>
   <link name="${name}_area">
-    <sphere_inertia radius="0" mass="0"/>
+    <xacro:sphere_inertia radius="0" mass="0"/>
     <visual>
         <origin xyz="0 0 0" rpy="0 0 0" />
         <geometry>
-          <mesh filename="package://iai_kitchen/meshes/racks/OvenArea.obj"/>
+          <mesh filename="package://iai_kitchen/meshes/racks/OvenArea.dae"/>
         </geometry>
       </visual>

File: iai_kitchen/urdf_obj/IAI_sink_area.urdf.xacro (robot description, xacro)
@@ -7,12 +7,12 @@
   <xacro:macro name="iai_sink_area" params="parent name *origin">
   <link name="${name}_footprint">
-    <sphere_inertia radius="0" mass="0"/>
+    <xacro:sphere_inertia radius="0" mass="0"/>
   </link>
   <link name="${name}">
-    <sphere_inertia radius="0" mass="0"/>
+    <xacro:sphere_inertia radius="0" mass="0"/>
     <visual>
         <origin xyz="0 0 0" rpy="0 0 0" />
         <geometry>
-          <mesh filename="package://iai_kitchen/meshes/racks/SinkArea.obj"/>
+          <mesh filename="package://iai_kitchen/meshes/racks/SinkArea.dae"/>
         </geometry>
       </visual>
@@ -35,5 +35,5 @@
   </joint>
   <link name="${name}_surface">
-    <sphere_inertia radius="0" mass="0"/>
+    <xacro:sphere_inertia radius="0" mass="0"/>
     <collision>
       <origin xyz="0 -0.225 0" rpy="0 0 0" />
@@ -49,9 +49,9 @@
  </joint>
   <link name="${name}_sink">
-    <sphere_inertia radius="0" mass="0"/>
+    <xacro:sphere_inertia radius="0" mass="0"/>
     <visual>
       <origin xyz="0 0 0" rpy="0 0 0" />
       <geometry>
-        <mesh filename="package://iai_kitchen/meshes/misc/Sink.obj"/>
+        <mesh filename="package://iai_kitchen/meshes/misc/Sink.dae"/>
       </geometry>
     </visual>

File: iai_kitchen/urdf_obj/IAI_tables.urdf.xacro (robot description, xacro)
@@ -3,9 +3,9 @@
   <xacro:macro name="iai_table_1" params="name parent *origin">
     <link name="${name}_main">
-      <sphere_inertia radius="0" mass="0"/>
+      <xacro:sphere_inertia radius="0" mass="0"/>
       <visual>
         <origin xyz="0 0 0.3619" rpy="0 0 0"/>
         <geometry>
-          <mesh filename="package://iai_kitchen/meshes/misc/big_table_1.stl"/>
+          <mesh filename="package://iai_kitchen/meshes/misc/big_table_1.dae"/>
         </geometry>
       </visual>
@@ -25,5 +25,5 @@
   <xacro:macro name="jokkmokk_table" params="name parent *origin">
     <link name="${name}_main">
-      <sphere_inertia radius="0" mass="0"/>
+      <xacro:sphere_inertia radius="0" mass="0"/>
       <visual>
         <origin xyz="0.0 0.0 0.0" rpy="0 0 0" />
@@ -48,5 +48,5 @@
   <xacro:macro name="jokkmokk_chair" params="name parent *origin">
     <link name="${name}_main">
-      <sphere_inertia radius="0" mass="0"/>
+      <xacro:sphere_inertia radius="0" mass="0"/>
       <visual>
         <origin xyz="0.0 0.0 0.0" rpy="0 0 0" />
@@ -70,5 +70,5 @@
   <xacro:macro name="iai_dining_area" params="parent name *origin">
     <link name="${name}_footprint">
-      <sphere_inertia radius="0" mass="0"/>
+      <xacro:sphere_inertia radius="0" mass="0"/>
     </link>
     <joint name="${name}_footprint_joint" type="fixed">

File: iai_kitchen/urdf_obj/iai_kitchen_python.urdf.xacro (robot description, xacro)
@@ -20,5 +20,5 @@
   </xacro:macro>
   <link name="room_link">
-    <sphere_inertia radius="0" mass="0"/>
+    <xacro:sphere_inertia radius="0" mass="0"/>
   </link>
   <xacro:if value="${simulated}">
