Commit message: Use collada for visual meshes.

File: iai_kitchen/urdf_obj/sink_area.urdf.xacro (robot description, xacro)
@@ -1,10 +1,7 @@
 <?xml version="1.0"?>
 <robot name="iai_kitchen_sink_area" xmlns:xacro="http://ros.org/wiki/xacro">
-<!--
-  <xacro:include filename="$(find iai_kitchen)/urdf/drawers.xacro" />
--->
   <xacro:property name="pi" value="3.1415926535897931" />
     <link name="sink_area_footprint">
-      <sphere_inertia radius="0" mass="0"/>
+      <xacro:sphere_inertia radius="0" mass="0"/>
       <!-- ???vizualize footprint??? -->
       <visual>
@@ -16,10 +13,10 @@
     </link>
     <link name="sink_area_main">
-      <sphere_inertia radius="0" mass="0"/>
-      <!-- ???vizualize footprint??? -->
-      <visual>
-        <origin xyz="0 0 0" rpy="0 0 0" />
-        <geometry>
-          <mesh filename="package://iai_kitchen/meshes/SinkArea.obj"/>
+      <xacro:sphere_inertia radius="0" mass="0"/>
+      <!-- ???vizualize footprint??? -->
+      <visual>
+        <origin xyz="0 0 0" rpy="0 0 0" />
+        <geometry>
+          <mesh filename="package://iai_kitchen/meshes/SinkArea.dae"/>
         </geometry>
       </visual>
@@ -38,10 +35,10 @@
     <!-- LEFT BLOCK -->
     <link name="sink_area_drawer_left_bottom">
-      <sphere_inertia radius="0" mass="0"/>
-      <!-- ???vizualize footprint??? -->
-      <visual>
-        <origin xyz="0 0 0" rpy="0 0 0" />
-        <geometry>
-          <mesh filename="package://iai_kitchen/meshes/SinkAreaMedDrawer.obj"/>
+      <xacro:sphere_inertia radius="0" mass="0"/>
+      <!-- ???vizualize footprint??? -->
+      <visual>
+        <origin xyz="0 0 0" rpy="0 0 0" />
+        <geometry>
+          <mesh filename="package://iai_kitchen/meshes/SinkAreaMedDrawer.dae"/>
         </geometry>
       </visual>
@@ -61,10 +58,10 @@
     </joint>
     <link name="sink_area_drawer_left_bottom_handle">
-      <sphere_inertia radius="0" mass="0"/>
-      <!-- ???vizualize footprint??? -->
-      <visual>
-        <origin xyz="0 0 0" rpy="0 0 0" />
-        <geometry>
-          <mesh filename="package://iai_kitchen/meshes/SinkAreaBigHandle.obj"/>
+      <xacro:sphere_inertia radius="0" mass="0"/>
+      <!-- ???vizualize footprint??? -->
+      <visual>
+        <origin xyz="0 0 0" rpy="0 0 0" />
+        <geometry>
+          <mesh filename="package://iai_kitchen/meshes/SinkAreaBigHandle.dae"/>
         </geometry>
       </visual>
@@ -82,10 +79,10 @@
     </joint>
     <link name="sink_area_drawer_left_center">
-      <sphere_inertia radius="0" mass="0"/>
-      <!-- ???vizualize footprint??? -->
-      <visual>
-        <origin xyz="0 0 0" rpy="0 0 0" />
-        <geometry>
-          <mesh filename="package://iai_kitchen/meshes/SinkAreaMedDrawer.obj"/>
+      <xacro:sphere_inertia radius="0" mass="0"/>
+      <!-- ???vizualize footprint??? -->
+      <visual>
+        <origin xyz="0 0 0" rpy="0 0 0" />
+        <geometry>
+          <mesh filename="package://iai_kitchen/meshes/SinkAreaMedDrawer.dae"/>
         </geometry>
       </visual>
@@ -105,9 +102,9 @@
     </joint>
     <link name="sink_area_drawer_left_center_handle">
-      <sphere_inertia radius="0" mass="0"/>
-      <visual>
-        <origin xyz="0 0 0" rpy="0 0 0" />
-        <geometry>
-          <mesh filename="package://iai_kitchen/meshes/SinkAreaBigHandle.obj"/>
+      <xacro:sphere_inertia radius="0" mass="0"/>
+      <visual>
+        <origin xyz="0 0 0" rpy="0 0 0" />
+        <geometry>
+          <mesh filename="package://iai_kitchen/meshes/SinkAreaBigHandle.dae"/>
         </geometry>
       </visual>
@@ -125,10 +122,10 @@
     </joint>
     <link name="sink_area_drawer_left_top">
-      <sphere_inertia radius="0" mass="0"/>
-      <!-- ???vizualize footprint??? -->
-      <visual>
-        <origin xyz="0 0 0" rpy="0 0 0" />
-        <geometry>
-          <mesh filename="package://iai_kitchen/meshes/SinkAreaSmallDrawer.obj"/>
+      <xacro:sphere_inertia radius="0" mass="0"/>
+      <!-- ???vizualize footprint??? -->
+      <visual>
+        <origin xyz="0 0 0" rpy="0 0 0" />
+        <geometry>
+          <mesh filename="package://iai_kitchen/meshes/SinkAreaSmallDrawer.dae"/>
         </geometry>
       </visual>
@@ -148,9 +145,9 @@
     </joint>
     <link name="sink_area_drawer_left_top_handle">
-      <sphere_inertia radius="0" mass="0"/>
-      <visual>
-        <origin xyz="0 0 0" rpy="0 0 0" />
-        <geometry>
-          <mesh filename="package://iai_kitchen/meshes/SinkAreaBigHandle.obj"/>
+      <xacro:sphere_inertia radius="0" mass="0"/>
+      <visual>
+        <origin xyz="0 0 0" rpy="0 0 0" />
+        <geometry>
+          <mesh filename="package://iai_kitchen/meshes/SinkAreaBigHandle.dae"/>
         </geometry>
       </visual>
@@ -169,9 +166,9 @@
     <!-- DISHWASHER BLOCK -->
     <link name="sink_area_inner_dishwasher">
-      <sphere_inertia radius="0" mass="0"/>
-      <visual>
-        <origin xyz="0 0 0" rpy="0 0 0" />
-        <geometry>
-          <mesh filename="package://iai_kitchen/meshes/SinkAreaInnerDishWasher.obj"/>
+      <xacro:sphere_inertia radius="0" mass="0"/>
+      <visual>
+        <origin xyz="0 0 0" rpy="0 0 0" />
+        <geometry>
+          <mesh filename="package://iai_kitchen/meshes/SinkAreaInnerDishWasher.dae"/>
         </geometry>
       </visual>
@@ -189,9 +186,9 @@
     </joint>
     <link name="sink_area_dishwasher_door">
-      <sphere_inertia radius="0" mass="0"/>
-      <visual>
-        <origin xyz="0 0 0" rpy="0 0 0" />
-        <geometry>
-          <mesh filename="package://iai_kitchen/meshes/SinkAreaDishWasherDoor.obj"/>
+      <xacro:sphere_inertia radius="0" mass="0"/>
+      <visual>
+        <origin xyz="0 0 0" rpy="0 0 0" />
+        <geometry>
+          <mesh filename="package://iai_kitchen/meshes/SinkAreaDishWasherDoor.dae"/>
         </geometry>
       </visual>
@@ -211,9 +208,9 @@
     </joint>
     <link name="sink_area_dishwasher_handle">
-      <sphere_inertia radius="0" mass="0"/>
-      <visual>
-        <origin xyz="0 0 0" rpy="0 0 0" />
-        <geometry>
-          <mesh filename="package://iai_kitchen/meshes/SinkAreaSmallHandle.obj"/>
+      <xacro:sphere_inertia radius="0" mass="0"/>
+      <visual>
+        <origin xyz="0 0 0" rpy="0 0 0" />
+        <geometry>
+          <mesh filename="package://iai_kitchen/meshes/SinkAreaSmallHandle.dae"/>
         </geometry>
       </visual>
@@ -232,9 +229,9 @@
     <!-- TRASH AREA -->
     <link name="sink_area_panel">
-      <sphere_inertia radius="0" mass="0"/>
-      <visual>
-        <origin xyz="0 0 0" rpy="0 0 0" />
-        <geometry>
-          <mesh filename="package://iai_kitchen/meshes/SinkAreaPanel.obj"/>
+      <xacro:sphere_inertia radius="0" mass="0"/>
+      <visual>
+        <origin xyz="0 0 0" rpy="0 0 0" />
+        <geometry>
+          <mesh filename="package://iai_kitchen/meshes/SinkAreaPanel.dae"/>
         </geometry>
       </visual>
@@ -252,9 +249,9 @@
     </joint>
     <link name="sink_area_trash">
-      <sphere_inertia radius="0" mass="0"/>
-      <visual>
-        <origin xyz="0 0 0" rpy="0 0 0" />
-        <geometry>
-          <mesh filename="package://iai_kitchen/meshes/SinkAreaTrash.obj"/>
+      <xacro:sphere_inertia radius="0" mass="0"/>
+      <visual>
+        <origin xyz="0 0 0" rpy="0 0 0" />
+        <geometry>
+          <mesh filename="package://iai_kitchen/meshes/SinkAreaTrash.dae"/>
         </geometry>
       </visual>
@@ -274,9 +271,9 @@
     </joint>
     <link name="sink_area_trash_handle">
-      <sphere_inertia radius="0" mass="0"/>
-      <visual>
-        <origin xyz="0 0 0" rpy="0 0 0" />
-        <geometry>
-          <mesh filename="package://iai_kitchen/meshes/SinkAreaSmallHandle.obj"/>
+      <xacro:sphere_inertia radius="0" mass="0"/>
+      <visual>
+        <origin xyz="0 0 0" rpy="0 0 0" />
+        <geometry>
+          <mesh filename="package://iai_kitchen/meshes/SinkAreaSmallHandle.dae"/>
         </geometry>
       </visual>
@@ -294,9 +291,9 @@
     </joint>
     <link name="sink_area_sink">
-      <sphere_inertia radius="0" mass="0"/>
-      <visual>
-        <origin xyz="0 0 0" rpy="0 0 0" />
-        <geometry>
-          <mesh filename="package://iai_kitchen/meshes/SinkAreaSink.obj"/>
+      <xacro:sphere_inertia radius="0" mass="0"/>
+      <visual>
+        <origin xyz="0 0 0" rpy="0 0 0" />
+        <geometry>
+          <mesh filename="package://iai_kitchen/meshes/SinkAreaSink.dae"/>
         </geometry>
       </visual>
