Commit message: Fix meshes

File: iai_kitchen/urdf_obj/IAI_kitchen.urdf (robot description, URDF)
Before this commit: robot iai_oven_area, 60 links, 59 joints
Links:
- link oven_area_oven_knob_oven: geometry visual mesh filename=package://iai_kitchen/meshes/oven/Knob.dae
- link oven_area_oven_knob_stove_1: geometry visual mesh filename=package://iai_kitchen/meshes/oven/Knob.dae
- link oven_area_oven_knob_stove_2: geometry visual mesh filename=package://iai_kitchen/meshes/oven/Knob.dae
- link oven_area_oven_knob_stove_3: geometry visual mesh filename=package://iai_kitchen/meshes/oven/Knob.dae
- link oven_area_oven_knob_stove_4: geometry visual mesh filename=package://iai_kitchen/meshes/oven/Knob.dae

File: iai_kitchen/urdf_obj/IAI_oven.urdf.xacro (robot description, xacro)
@@ -125,5 +125,5 @@
         <origin xyz="0 0 0" rpy="0 ${0.5 * pi} 0" />
         <geometry>
-          <mesh filename="package://iai_kitchen/meshes/oven/Knob.obj"/>
+          <mesh filename="package://iai_kitchen/meshes/oven/Knob.dae"/>
         </geometry>
       </visual>

File: iai_kitchen/urdf_obj/IAI_tables.urdf.xacro (robot description, xacro)
@@ -52,5 +52,5 @@
         <origin xyz="0.0 0.0 0.0" rpy="0 0 0" />
         <geometry>
-          <mesh filename="package://iai_kitchen/meshes/jokkmokk/JokkmokkChair.obj"/>
+          <mesh filename="package://iai_kitchen/meshes/jokkmokk/JokkmokkChair.dae"/>
         </geometry>
       </visual>

Commit message: Revert "Fix meshes"
This reverts commit 47ba345df0ed53e6ac27f4868e70d7c66ffa3c6f.

File: iai_kitchen/urdf_obj/IAI_kitchen.urdf (robot description, URDF)
Before this commit: robot iai_oven_area, 60 links, 59 joints
Links:
- link oven_area_oven_knob_oven: geometry visual mesh filename=package://iai_kitchen/meshes/oven/Knob.obj
- link oven_area_oven_knob_stove_1: geometry visual mesh filename=package://iai_kitchen/meshes/oven/Knob.obj
- link oven_area_oven_knob_stove_2: geometry visual mesh filename=package://iai_kitchen/meshes/oven/Knob.obj
- link oven_area_oven_knob_stove_3: geometry visual mesh filename=package://iai_kitchen/meshes/oven/Knob.obj
- link oven_area_oven_knob_stove_4: geometry visual mesh filename=package://iai_kitchen/meshes/oven/Knob.obj

File: iai_kitchen/urdf_obj/IAI_oven.urdf.xacro (robot description, xacro)
@@ -125,5 +125,5 @@
         <origin xyz="0 0 0" rpy="0 ${0.5 * pi} 0" />
         <geometry>
-          <mesh filename="package://iai_kitchen/meshes/oven/Knob.dae"/>
+          <mesh filename="package://iai_kitchen/meshes/oven/Knob.obj"/>
         </geometry>
       </visual>

File: iai_kitchen/urdf_obj/IAI_tables.urdf.xacro (robot description, xacro)
@@ -52,5 +52,5 @@
         <origin xyz="0.0 0.0 0.0" rpy="0 0 0" />
         <geometry>
-          <mesh filename="package://iai_kitchen/meshes/jokkmokk/JokkmokkChair.dae"/>
+          <mesh filename="package://iai_kitchen/meshes/jokkmokk/JokkmokkChair.obj"/>
         </geometry>
       </visual>
