Commit message: [kitchen urdf] the big table had visiion and collision meshes mixed

File: iai_kitchen/urdf_obj/IAI_tables.urdf.xacro (robot description, xacro)
@@ -8,5 +8,5 @@
         <origin xyz="0 0 0.3619" rpy="0 0 0" />
         <geometry>
-          <mesh filename="package://iai_kitchen/meshes/misc/big_table_1.obj"/>
+          <mesh filename="package://iai_kitchen/meshes/misc/big_table_1.stl"/>
         </geometry>
       </visual>
@@ -14,5 +14,5 @@
         <origin xyz="0 0 0.3619" rpy="0 0 0" />
         <geometry>
-          <mesh filename="package://iai_kitchen/meshes/misc/big_table_1.stl"/>
+          <mesh filename="package://iai_kitchen/meshes/misc/big_table_1.obj"/>
         </geometry>
       </collision>

Commit message: [kitchen urdf] added jokkmokk area with preliminary meshes and poses

File: iai_kitchen/urdf_obj/IAI_tables.urdf.xacro (robot description, xacro)
@@ -2,9 +2,8 @@
 <robot name="iai_table" xmlns:xacro="http://ros.org/wiki/xacro">
   <macro name="iai_table_1" params="name parent *origin">
-    <!-- LINKS -->
     <link name="${name}_main">
       <sphere_inertia radius="0" mass="0"/>
       <visual>
-        <origin xyz="0 0 0.3619" rpy="0 0 0" />
+        <origin xyz="0 0 0.3619" rpy="0 0 0"/>
         <geometry>
           <mesh filename="package://iai_kitchen/meshes/misc/big_table_1.stl"/>
@@ -12,5 +11,5 @@
       </visual>
       <collision>
-        <origin xyz="0 0 0.3619" rpy="0 0 0" />
+        <origin xyz="0 0 0.3619" rpy="0 0 0"/>
         <geometry>
           <mesh filename="package://iai_kitchen/meshes/misc/big_table_1.obj"/>
@@ -18,10 +17,72 @@
       </collision>
     </link>
-    <!-- JOINTS -->
     <joint name="${name}_main_joint" type="fixed">
-      <xacro:insert_block name="origin" />
+      <xacro:insert_block name="origin"/>
       <parent link="${parent}"/>
       <child link="${name}_main"/>
     </joint>
   </macro>
+  <macro name="jokkmokk_table" params="name parent *origin">
+    <link name="${name}_main">
+      <sphere_inertia radius="0" mass="0"/>
+      <visual>
+        <origin xyz="0.0 0.0 0.3978" rpy="0 0 0" />
+        <geometry>
+          <mesh filename="package://iai_kitchen/meshes/jokkmokk/jokkmokkTable.stl"/>
+        </geometry>
+      </visual>
+      <collision>
+        <origin xyz="0.0 0.0 0.3978" rpy="0 0 0" />
+        <geometry>
+          <mesh filename="package://iai_kitchen/meshes/jokkmokk/jokkmokkTable.stl"/>
+        </geometry>
+      </collision>
+    </link>
+    <joint name="${name}_main_joint" type="fixed">
+      <xacro:insert_block name="origin"/>
+      <parent link="${parent}"/>
+      <child link="${name}_main"/>
+    </joint>
+  </macro>
+  <macro name="jokkmokk_chair" params="name parent *origin">
+    <link name="${name}_main">
+      <sphere_inertia radius="0" mass="0"/>
+      <visual>
+        <origin xyz="0.0 0.0 0.5535" rpy="0 0 0" />
+        <geometry>
+          <mesh filename="package://iai_kitchen/meshes/jokkmokk/jokkmokkChair.stl"/>
+        </geometry>
+      </visual>
+      <collision>
+        <origin xyz="0.0 0.0 0.5535" rpy="0 0 0" />
+        <geometry>
+          <mesh filename="package://iai_kitchen/meshes/jokkmokk/jokkmokkChair.stl"/>
+        </geometry>
+      </collision>
+    </link>
+    <joint name="${name}_main_joint" type="fixed">
+      <xacro:insert_block name="origin"/>
+      <parent link="${parent}"/>
+      <child link="${name}_main"/>
+    </joint>
+  </macro>
+  <macro name="iai_dining_area" params="parent name *origin">
+    <link name="${name}_footprint">
+      <sphere_inertia radius="0" mass="0"/>
+    </link>
+    <joint name="${name}_footprint_joint" type="fixed">
+      <xacro:insert_block name="origin" />
+      <child link="${name}_footprint"/>
+      <parent link="${parent}"/>
+    </joint>
+    <jokkmokk_table name="${name}_jokkmokk_table" parent="${name}_footprint">
+      <origin xyz="0 0 0" rpy="0 0 0" />
+    </jokkmokk_table>
+    <jokkmokk_chair name="${name}_jokkmokk_left_chair" parent="${name}_footprint">
+      <origin xyz="-1 0 0" rpy="0 0 0" />
+    </jokkmokk_chair>
+    <jokkmokk_chair name="${name}_jokkmokk_right_chair" parent="${name}_footprint">
+      <origin xyz="1 0 0" rpy="0 0 ${-pi}" />
+    </jokkmokk_chair>
+  </macro>
 </robot>

File: iai_kitchen/urdf_obj/iai_kitchen_python.urdf.xacro (robot description, xacro)
@@ -49,4 +49,7 @@
     <origin xyz="-2.4 -1.5 0" rpy="0 0 ${pi}" />
   </iai_table_1>
+  <iai_dining_area name="dining_area" parent="room_link">
+    <origin xyz="-3.35 0.4 0" rpy="0 0 ${pi / 2}" />
+  </iai_dining_area>
   <iai_kitchen_wall_robohow parent="room_link">
     <origin xyz="-0.96 0.65 0" rpy="0.0 0.0 0.0" />

Commit message: [kitchen urdf] tweaked numbers for dining area

File: iai_kitchen/urdf_obj/IAI_tables.urdf.xacro (robot description, xacro)
@@ -27,5 +27,5 @@
       <sphere_inertia radius="0" mass="0"/>
       <visual>
-        <origin xyz="0.0 0.0 0.3978" rpy="0 0 0" />
+        <origin xyz="0.0 0.0 0.35" rpy="0 0 0" />
         <geometry>
           <mesh filename="package://iai_kitchen/meshes/jokkmokk/jokkmokkTable.stl"/>
@@ -33,5 +33,5 @@
       </visual>
       <collision>
-        <origin xyz="0.0 0.0 0.3978" rpy="0 0 0" />
+        <origin xyz="0.0 0.0 0.35" rpy="0 0 0" />
         <geometry>
           <mesh filename="package://iai_kitchen/meshes/jokkmokk/jokkmokkTable.stl"/>

File: iai_kitchen/urdf_obj/iai_kitchen_python.urdf.xacro (robot description, xacro)
@@ -50,5 +50,5 @@
   </iai_table_1>
   <iai_dining_area name="dining_area" parent="room_link">
-    <origin xyz="-3.35 0.4 0" rpy="0 0 ${pi / 2}" />
+    <origin xyz="-3.38 0.28 0" rpy="0 0 ${pi / 2}" />
   </iai_dining_area>
   <iai_kitchen_wall_robohow parent="room_link">

Commit message: changed kitchen urdf to use new jokkmokk objs

File: iai_kitchen/urdf_obj/IAI_tables.urdf.xacro (robot description, xacro)
@@ -29,5 +29,5 @@
         <origin xyz="0.0 0.0 0.35" rpy="0 0 0" />
         <geometry>
-          <mesh filename="package://iai_kitchen/meshes/jokkmokk/jokkmokkTable.stl"/>
+          <mesh filename="package://iai_kitchen/meshes/jokkmokk/JokkmokkTable.obj"/>
         </geometry>
       </visual>
@@ -35,5 +35,5 @@
         <origin xyz="0.0 0.0 0.35" rpy="0 0 0" />
         <geometry>
-          <mesh filename="package://iai_kitchen/meshes/jokkmokk/jokkmokkTable.stl"/>
+          <mesh filename="package://iai_kitchen/meshes/jokkmokk/JokkmokkTable.obj"/>
         </geometry>
       </collision>
@@ -51,5 +51,5 @@
         <origin xyz="0.0 0.0 0.5535" rpy="0 0 0" />
         <geometry>
-          <mesh filename="package://iai_kitchen/meshes/jokkmokk/jokkmokkChair.stl"/>
+          <mesh filename="package://iai_kitchen/meshes/jokkmokk/JokkmokkChair.obj"/>
         </geometry>
       </visual>
@@ -57,5 +57,5 @@
         <origin xyz="0.0 0.0 0.5535" rpy="0 0 0" />
         <geometry>
-          <mesh filename="package://iai_kitchen/meshes/jokkmokk/jokkmokkChair.stl"/>
+          <mesh filename="package://iai_kitchen/meshes/jokkmokk/JokkmokkChair.obj"/>
         </geometry>
       </collision>

Commit message: Revert "changed kitchen urdf to use new jokkmokk objs"
This reverts commit a5c6ae470b88afc856bd882f416d0cf1c8d8a8b4.

File: iai_kitchen/urdf_obj/IAI_tables.urdf.xacro (robot description, xacro)
@@ -29,5 +29,5 @@
         <origin xyz="0.0 0.0 0.35" rpy="0 0 0" />
         <geometry>
-          <mesh filename="package://iai_kitchen/meshes/jokkmokk/JokkmokkTable.obj"/>
+          <mesh filename="package://iai_kitchen/meshes/jokkmokk/jokkmokkTable.stl"/>
         </geometry>
       </visual>
@@ -35,5 +35,5 @@
         <origin xyz="0.0 0.0 0.35" rpy="0 0 0" />
         <geometry>
-          <mesh filename="package://iai_kitchen/meshes/jokkmokk/JokkmokkTable.obj"/>
+          <mesh filename="package://iai_kitchen/meshes/jokkmokk/jokkmokkTable.stl"/>
         </geometry>
       </collision>
@@ -51,5 +51,5 @@
         <origin xyz="0.0 0.0 0.5535" rpy="0 0 0" />
         <geometry>
-          <mesh filename="package://iai_kitchen/meshes/jokkmokk/JokkmokkChair.obj"/>
+          <mesh filename="package://iai_kitchen/meshes/jokkmokk/jokkmokkChair.stl"/>
         </geometry>
       </visual>
@@ -57,5 +57,5 @@
         <origin xyz="0.0 0.0 0.5535" rpy="0 0 0" />
         <geometry>
-          <mesh filename="package://iai_kitchen/meshes/jokkmokk/JokkmokkChair.obj"/>
+          <mesh filename="package://iai_kitchen/meshes/jokkmokk/jokkmokkChair.stl"/>
         </geometry>
       </collision>

Commit message: Fix meshes

File: iai_kitchen/urdf_obj/IAI_tables.urdf.xacro (robot description, xacro)
@@ -29,5 +29,5 @@
         <origin xyz="0.0 0.0 0.0" rpy="0 0 0" />
         <geometry>
-          <mesh filename="package://iai_kitchen/meshes/jokkmokk/JokkmokkTable.obj"/>
+          <mesh filename="package://iai_kitchen/meshes/jokkmokk/JokkmokkTable.dae"/>
         </geometry>
       </visual>
