Commit message: shelve_1 more details

File: iai_refills_lab/maps/dm_shelves.urdf.xacro (robot description, xacro)
@@ -1,5 +1,56 @@
 <?xml version="1.0"?>
 <robot name="dm_shelves" xmlns:xacro="http://ros.org/wiki/xacro">
-    <macro name="shelve_1_level" params="name parent *origin">
+    <macro name="divider_link" params="parent name *origin">
+        <link name="shelve_1_${name}_link">
+            <visual>
+                <geometry>
+                    <box size="0.004 0.65 0.05"/>
+                </geometry>
+            </visual>
+            <collision>
+                <geometry>
+                    <box size="0.004 0.65 0.05"/>
+                </geometry>
+            </collision>
+        </link>
+        <joint type="fixed" name="shelve_1_${name}_joint">
+            <xacro:insert_block name="origin"/>
+            <parent link="${parent}"/>
+            <child link="shelve_1_${name}_link"/>
+        </joint>
+    </macro>
+    <macro name="shelve_divider" params="parent name dist1 dist2 dist3 dist4 dist5 dist6 dist7 dist8 dist9">
+        <divider_link parent="${parent}" name="${name}_divider_1">
+            <origin xyz="-0.495 0 0.024"/>
+        </divider_link>
+        <divider_link parent="${parent}" name="${name}_divider_2">
+            <origin xyz="${-0.495 + dist1} 0 0.024"/>
+        </divider_link>
+        <divider_link parent="${parent}" name="${name}_divider_3">
+            <origin xyz="${-0.495 + dist1 + dist2} 0 0.024"/>
+        </divider_link>
+        <divider_link parent="${parent}" name="${name}_divider_4">
+            <origin xyz="${-0.495 + dist1 + dist2 + dist3} 0 0.024"/>
+        </divider_link>
+        <divider_link parent="${parent}" name="${name}_divider_5">
+            <origin xyz="${-0.495 + dist1 + dist2 + dist3 + dist4} 0 0.024"/>
+        </divider_link>
+        <divider_link parent="${parent}" name="${name}_divider_6">
+            <origin xyz="${-0.495 + dist1 + dist2 + dist3 + dist4 + dist5} 0 0.024"/>
+        </divider_link>
+        <divider_link parent="${parent}" name="${name}_divider_7">
+            <origin xyz="${-0.495 + dist1 + dist2 + dist3 + dist4 + dist5 + dist6} 0 0.024"/>
+        </divider_link>
+        <divider_link parent="${parent}" name="${name}_divider_8">
+            <origin xyz="${-0.495 + dist1 + dist2 + dist3 + dist4 + dist5 + dist6 + dist7} 0 0.024"/>
+        </divider_link>
+        <divider_link parent="${parent}" name="${name}_divider_9">
+            <origin xyz="${-0.495 + dist1 + dist2 + dist3 + dist4 + dist5 + dist6 + dist7 + dist8} 0 0.024"/>
+        </divider_link>
+        <divider_link parent="${parent}" name="${name}_divider_10">
+            <origin xyz="${-0.495 + dist1 + dist2 + dist3 + dist4 + dist5 + dist6 + dist7 + dist8 + dist9} 0 0.024"/>
+        </divider_link>
+    </macro>
+    <macro name="shelve_1_level" params="name parent *origin dist1 dist2 dist3 dist4 dist5 dist6 dist7 dist8 dist9">
         <link name="shelve_1_${name}_link">
             <visual>
@@ -14,9 +65,44 @@
             </collision>
         </link>
-        <joint type="fixed" name="${name}_joint">
+        <link name="shelve_1_${name}_left_support_link">
+            <visual>
+                <geometry>
+                    <box size="0.004 0.65 0.12"/>
+                </geometry>
+            </visual>
+            <collision>
+                <geometry>
+                    <box size="0.004 0.65 0.12"/>
+                </geometry>
+            </collision>
+        </link>
+        <link name="shelve_1_${name}_right_support_link">
+            <visual>
+                <geometry>
+                    <box size="0.004 0.65 0.12"/>
+                </geometry>
+            </visual>
+            <collision>
+                <geometry>
+                    <box size="0.004 0.65 0.12"/>
+                </geometry>
+            </collision>
+        </link>
+        <joint type="fixed" name="shelve_1_${name}_joint">
             <xacro:insert_block name="origin"/>
             <parent link="${parent}"/>
             <child link="shelve_1_${name}_link"/>
         </joint>
+        <joint type="fixed" name="shelve_1_${name}_right_support_joint">
+            <origin xyz="0.494 0 -0.06"/>
+            <parent link="shelve_1_${name}_link"/>
+            <child link="shelve_1_${name}_right_support_link"/>
+        </joint>
+        <joint type="fixed" name="shelve_1_${name}_left_support_joint">
+            <origin xyz="-0.494 0 -0.06"/>
+            <parent link="shelve_1_${name}_link"/>
+            <child link="shelve_1_${name}_left_support_link"/>
+        </joint>
+        <shelve_divider parent="shelve_1_${name}_link" name="${name}" dist1="${dist1}" dist2="${dist2}" dist3="${dist3}" dist4="${dist4}" dist5="${dist5}" dist6="${dist6}" dist7="${dist7}" dist8="${dist8}" dist9="${dist9}" />
     </macro>
     <link name="room_link"/>
@@ -78,17 +164,17 @@
         <child link="shelve_1_level_0_link"/>
     </joint>
-    <shelve_1_level name="level_1" parent="shelve_1_footprint">
+    <shelve_1_level name="level_1" parent="shelve_1_footprint" dist1="0.15" dist2="0.133" dist3="0.082" dist4="0.167" dist5="0.095" dist6="0.148" dist7="0.095" dist8="0.125" dist9="0" >
         <origin xyz="0 0 0.50965" />
     </shelve_1_level>
-    <shelve_1_level name="level_2" parent="shelve_1_footprint">
+    <shelve_1_level name="level_2" parent="shelve_1_footprint" dist1="0.177" dist2="0.208" dist3="0.147" dist4="0.20" dist5="0.124" dist6="0.14" dist7="0" dist8="0" dist9="0" >
         <origin xyz="0 0 0.84465" />
     </shelve_1_level>
-    <shelve_1_level name="level_3" parent="shelve_1_footprint">
+    <shelve_1_level name="level_3" parent="shelve_1_footprint" dist1="0" dist2="0" dist3="0" dist4="0" dist5="0" dist6="0" dist7="0" dist8="0" dist9="0" >
         <origin xyz="0 0 1.22265" />
     </shelve_1_level>
-    <shelve_1_level name="level_4" parent="shelve_1_footprint">
+    <shelve_1_level name="level_4" parent="shelve_1_footprint" dist1="0" dist2="0" dist3="0" dist4="0" dist5="0" dist6="0" dist7="0" dist8="0" dist9="0" >
         <origin xyz="0 0 1.53565" />
     </shelve_1_level>
-    <shelve_1_level name="level_5" parent="shelve_1_footprint">
+    <shelve_1_level name="level_5" parent="shelve_1_footprint" dist1="0" dist2="0" dist3="0" dist4="0" dist5="0" dist6="0" dist7="0" dist8="0" dist9="0" >
         <origin xyz="0 0 1.86865" />
     </shelve_1_level>

Commit message: shelf 2 and dividers

File: iai_refills_lab/maps/dm_shelves.urdf.xacro (robot description, xacro)
@@ -1,4 +1,5 @@
 <?xml version="1.0"?>
 <robot name="dm_shelves" xmlns:xacro="http://ros.org/wiki/xacro">
+<link name="room_link"/>
     <macro name="divider_link" params="parent name *origin">
         <link name="shelve_1_${name}_link">
@@ -106,9 +107,28 @@
         <shelve_divider parent="shelve_1_${name}_link" name="${name}" dist1="${dist1}" dist2="${dist2}" dist3="${dist3}" dist4="${dist4}" dist5="${dist5}" dist6="${dist6}" dist7="${dist7}" dist8="${dist8}" dist9="${dist9}" />
     </macro>
-    <link name="room_link"/>
+    <macro name="shelve_2_level" params="name parent *origin">
+        <link name="shelve_2_${name}_link">
+            <visual>
+                <geometry>
+                    <box size="0.992 0.435 0.043"/>
+                </geometry>
+            </visual>
+            <collision>
+                <geometry>
+                    <box size="0.992 0.435 0.043"/>
+                </geometry>
+            </collision>
+        </link>
+        <joint type="fixed" name="shelve_2_${name}_joint">
+            <xacro:insert_block name="origin"/>
+            <parent link="${parent}"/>
+            <child link="shelve_2_${name}_link"/>
+        </joint>
+    </macro>
+    <macro name="shelve_1" params="*origin parent">
     <link name="shelve_1_footprint"/>
-    <joint type="fixed" name="romm_shleve1_joint">
-        <origin xyz="1 1 0.08515"/>
-        <parent link="room_link"/>
+    <joint type="fixed" name="romm_shleve_1_joint">
+        <xacro:insert_block name="origin"/>
+        <parent link="${parent}"/>
         <child link="shelve_1_footprint"/>
     </joint>
@@ -179,3 +199,119 @@
         <origin xyz="0 0 1.86865" />
     </shelve_1_level>
+</macro>
+    <!-- Shelve 2 -->
+    <macro name="shelve_2" params="*origin parent">
+     <link name="shelve_2_footprint"/>
+    <joint type="fixed" name="romm_shleve_2_joint">
+        <xacro:insert_block name="origin"/>
+        <parent link="${parent}"/>
+        <child link="shelve_2_footprint"/>
+    </joint>
+     <link name="shelve_2_base">
+        <visual>
+            <geometry>
+                <box size="1 0.6 0.145"/>
+            </geometry>
+        </visual>
+        <collision>
+           <geometry>
+                <box size="1 0.6 0.145"/>
+            </geometry>
+        </collision>
+    </link>
+    <joint type="fixed" name="shelve_2_foot_base_joint">
+        <iorigin xyz="0 0 0"/>
+        <parent link="shelve_2_footprint"/>
+        <child link="shelve_2_base"/>
+    </joint>
+    <link name="shelve_2_left_side">
+        <visual>
+            <geometry>
+                <box size="0.05 0.54 1.3"/>
+            </geometry>
+        </visual>
+        <collision>
+           <geometry>
+                <box size="0.05 0.54 1.3"/>
+            </geometry>
+        </collision>
+    </link>
+    <joint type="fixed" name="shelve_2_foot_left_joint">
+        <origin xyz="-0.475 0 0.7225"/>
+        <parent link="shelve_2_footprint"/>
+        <child link="shelve_2_left_side"/>
+    </joint>
+    <link name="shelve_2_right_side">
+        <visual>
+            <geometry>
+                <box size="0.05 0.54 1.3"/>
+            </geometry>
+        </visual>
+        <collision>
+           <geometry>
+                <box size="0.05 0.54 1.3"/>
+            </geometry>
+        </collision>
+    </link>
+    <joint type="fixed" name="shelve_2_foot_right_joint">
+        <origin xyz="0.475 0 0.7225"/>
+        <parent link="shelve_2_footprint"/>
+        <child link="shelve_2_right_side"/>
+    </joint>
+    <link name="shelve_2_back">
+        <visual>
+            <geometry>
+                <box size="1 0.05 1.4"/>
+            </geometry>
+        </visual>
+        <collision>
+           <geometry>
+                <box size="1 0.05 1.4"/>
+            </geometry>
+        </collision>
+    </link>
+    <joint type="fixed" name="shelve_2_foot_back_joint">
+        <origin xyz="0 0.275 0.7725"/>
+        <parent link="shelve_2_footprint"/>
+        <child link="shelve_2_back"/>
+    </joint>
+    <link name="shelve_2_level_0_link">
+        <visual>
+            <geometry>
+                <box size="0.992 0.54 0.043"/>
+            </geometry>
+        </visual>
+        <collision>
+           <geometry>
+                <box size="0.992 0.54 0.043"/>
+            </geometry>
+        </collision>
+    </link>
+    <joint type="fixed" name="shelve_2_level_0_joint">
+        <origin xyz="0 0 0.0925"/>
+        <parent link="shelve_2_footprint"/>
+        <child link="shelve_2_level_0_link"/>
+    </joint>
+    <shelve_2_level name="level_1" parent="shelve_2_footprint">
+        <origin xyz="0 0.05 0.324"/>
+    </shelve_2_level>
+    <shelve_2_level name="level_2" parent="shelve_2_footprint">
+        <origin xyz="0 0.05 0.574"/>
+    </shelve_2_level>
+    <shelve_2_level name="level_3" parent="shelve_2_footprint">
+        <origin xyz="0 0.05 0.784"/>
+    </shelve_2_level>
+    <shelve_2_level name="level_4" parent="shelve_2_footprint">
+        <origin xyz="0 0.05 1.036"/>
+    </shelve_2_level>
+    <shelve_2_level name="level_5" parent="shelve_2_footprint">
+        <origin xyz="0 0.05 1.245"/>
+    </shelve_2_level>
+</macro>
+<shelve_1 parent="room_link">
+    <origin xyz="1 1 0.08515"/>
+</shelve_1>
+<shelve_2 parent="room_link">
+    <origin xyz="-1 1 0.08515"/>
+</shelve_2>
 </robot>
