Commit message: correct names

File: iai_refills_lab/maps/dm_shelves.urdf.xacro (robot description, xacro)
@@ -3,5 +3,5 @@
 <link name="room_link"/>
     <macro name="divider_link" params="parent name *origin">
-        <link name="shelve_1_${name}_link">
+        <link name="shelf_1_${name}_link">
             <visual>
                 <geometry>
@@ -15,11 +15,11 @@
             </collision>
         </link>
-        <joint type="fixed" name="shelve_1_${name}_joint">
+        <joint type="fixed" name="shelf_1_${name}_joint">
             <xacro:insert_block name="origin"/>
             <parent link="${parent}"/>
-            <child link="shelve_1_${name}_link"/>
+            <child link="shelf_1_${name}_link"/>
         </joint>
     </macro>
-    <macro name="shelve_divider" params="parent name dist1 dist2 dist3 dist4 dist5 dist6 dist7 dist8 dist9">
+    <macro name="shelf_divider" params="parent name dist1 dist2 dist3 dist4 dist5 dist6 dist7 dist8 dist9">
         <divider_link parent="${parent}" name="${name}_divider_1">
             <origin xyz="-0.495 0 0.024"/>
@@ -53,6 +53,6 @@
         </divider_link>
     </macro>
-    <macro name="shelve_1_level" params="name parent *origin dist1 dist2 dist3 dist4 dist5 dist6 dist7 dist8 dist9">
-        <link name="shelve_1_${name}_link">
+    <macro name="shelf_1_level" params="name parent *origin dist1 dist2 dist3 dist4 dist5 dist6 dist7 dist8 dist9">
+        <link name="shelf_1_${name}_link">
             <visual>
                 <geometry>
@@ -66,5 +66,5 @@
             </collision>
         </link>
-        <link name="shelve_1_${name}_left_support_link">
+        <link name="shelf_1_${name}_left_support_link">
             <visual>
                 <geometry>
@@ -78,5 +78,5 @@
             </collision>
         </link>
-        <link name="shelve_1_${name}_right_support_link">
+        <link name="shelf_1_${name}_right_support_link">
             <visual>
                 <geometry>
@@ -90,23 +90,23 @@
             </collision>
         </link>
-        <joint type="fixed" name="shelve_1_${name}_joint">
+        <joint type="fixed" name="shelf_1_${name}_joint">
             <xacro:insert_block name="origin"/>
             <parent link="${parent}"/>
-            <child link="shelve_1_${name}_link"/>
-        </joint>
-        <joint type="fixed" name="shelve_1_${name}_right_support_joint">
+            <child link="shelf_1_${name}_link"/>
+        </joint>
+        <joint type="fixed" name="shelf_1_${name}_right_support_joint">
             <origin xyz="0.494 0 -0.06"/>
-            <parent link="shelve_1_${name}_link"/>
-            <child link="shelve_1_${name}_right_support_link"/>
-        </joint>
-        <joint type="fixed" name="shelve_1_${name}_left_support_joint">
+            <parent link="shelf_1_${name}_link"/>
+            <child link="shelf_1_${name}_right_support_link"/>
+        </joint>
+        <joint type="fixed" name="shelf_1_${name}_left_support_joint">
             <origin xyz="-0.494 0 -0.06"/>
-            <parent link="shelve_1_${name}_link"/>
-            <child link="shelve_1_${name}_left_support_link"/>
-        </joint>
-        <shelve_divider parent="shelve_1_${name}_link" name="${name}" dist1="${dist1}" dist2="${dist2}" dist3="${dist3}" dist4="${dist4}" dist5="${dist5}" dist6="${dist6}" dist7="${dist7}" dist8="${dist8}" dist9="${dist9}" />
+            <parent link="shelf_1_${name}_link"/>
+            <child link="shelf_1_${name}_left_support_link"/>
+        </joint>
+        <shelf_divider parent="shelf_1_${name}_link" name="${name}" dist1="${dist1}" dist2="${dist2}" dist3="${dist3}" dist4="${dist4}" dist5="${dist5}" dist6="${dist6}" dist7="${dist7}" dist8="${dist8}" dist9="${dist9}" />
     </macro>
-    <macro name="shelve_2_level" params="name parent *origin">
-        <link name="shelve_2_${name}_link">
+    <macro name="shelf_2_level" params="name parent *origin">
+        <link name="shelf_2_${name}_link">
             <visual>
                 <geometry>
@@ -120,18 +120,18 @@
             </collision>
         </link>
-        <joint type="fixed" name="shelve_2_${name}_joint">
+        <joint type="fixed" name="shelf_2_${name}_joint">
             <xacro:insert_block name="origin"/>
             <parent link="${parent}"/>
-            <child link="shelve_2_${name}_link"/>
+            <child link="shelf_2_${name}_link"/>
         </joint>
     </macro>
-    <macro name="shelve_1" params="*origin parent">
-    <link name="shelve_1_footprint"/>
+    <macro name="shelf_1" params="*origin parent">
+    <link name="shelf_1_footprint"/>
     <joint type="fixed" name="romm_shleve_1_joint">
         <xacro:insert_block name="origin"/>
         <parent link="${parent}"/>
-        <child link="shelve_1_footprint"/>
-    </joint>
-    <link name="shelve_1_base">
+        <child link="shelf_1_footprint"/>
+    </joint>
+    <link name="shelf_1_base">
         <visual>
             <geometry>
@@ -147,8 +147,8 @@
     <joint type="fixed" name="foot_base_joint">
         <iorigin xyz="0 0 0"/>
-        <parent link="shelve_1_footprint"/>
-        <child link="shelve_1_base"/>
-    </joint>
-    <link name="shelve_1_back">
+        <parent link="shelf_1_footprint"/>
+        <child link="shelf_1_base"/>
+    </joint>
+    <link name="shelf_1_back">
         <visual>
             <geometry>
@@ -164,8 +164,8 @@
     <joint type="fixed" name="foot_back_joint">
         <origin xyz="0 0.365 1"/>
-        <parent link="shelve_1_footprint"/>
-        <child link="shelve_1_back"/>
-    </joint>
-    <link name="shelve_1_level_0_link">
+        <parent link="shelf_1_footprint"/>
+        <child link="shelf_1_back"/>
+    </joint>
+    <link name="shelf_1_level_0_link">
         <visual>
             <geometry>
@@ -179,34 +179,34 @@
         </collision>
     </link>
-    <joint type="fixed" name="shelve_1_level_0_joint">
+    <joint type="fixed" name="shelf_1_level_0_joint">
         <origin xyz="0 -0.06 0.10665"/>
-        <parent link="shelve_1_footprint"/>
-        <child link="shelve_1_level_0_link"/>
-    </joint>
-    <shelve_1_level name="level_1" parent="shelve_1_footprint" dist1="0.15" dist2="0.133" dist3="0.082" dist4="0.167" dist5="0.095" dist6="0.148" dist7="0.095" dist8="0.125" dist9="0" >
+        <parent link="shelf_1_footprint"/>
+        <child link="shelf_1_level_0_link"/>
+    </joint>
+    <shelf_1_level name="level_1" parent="shelf_1_footprint" dist1="0.15" dist2="0.133" dist3="0.082" dist4="0.167" dist5="0.095" dist6="0.148" dist7="0.095" dist8="0.125" dist9="0" >
         <origin xyz="0 0 0.50965" />
-    </shelve_1_level>
-    <shelve_1_level name="level_2" parent="shelve_1_footprint" dist1="0.177" dist2="0.208" dist3="0.147" dist4="0.20" dist5="0.124" dist6="0.14" dist7="0" dist8="0" dist9="0" >
+    </shelf_1_level>
+    <shelf_1_level name="level_2" parent="shelf_1_footprint" dist1="0.177" dist2="0.208" dist3="0.147" dist4="0.20" dist5="0.124" dist6="0.14" dist7="0" dist8="0" dist9="0" >
         <origin xyz="0 0 0.84465" />
-    </shelve_1_level>
-    <shelve_1_level name="level_3" parent="shelve_1_footprint" dist1="0" dist2="0" dist3="0" dist4="0" dist5="0" dist6="0" dist7="0" dist8="0" dist9="0" >
+    </shelf_1_level>
+    <shelf_1_level name="level_3" parent="shelf_1_footprint" dist1="0" dist2="0" dist3="0" dist4="0" dist5="0" dist6="0" dist7="0" dist8="0" dist9="0" >
         <origin xyz="0 0 1.22265" />
-    </shelve_1_level>
-    <shelve_1_level name="level_4" parent="shelve_1_footprint" dist1="0" dist2="0" dist3="0" dist4="0" dist5="0" dist6="0" dist7="0" dist8="0" dist9="0" >
+    </shelf_1_level>
+    <shelf_1_level name="level_4" parent="shelf_1_footprint" dist1="0" dist2="0" dist3="0" dist4="0" dist5="0" dist6="0" dist7="0" dist8="0" dist9="0" >
         <origin xyz="0 0 1.53565" />
-    </shelve_1_level>
-    <shelve_1_level name="level_5" parent="shelve_1_footprint" dist1="0" dist2="0" dist3="0" dist4="0" dist5="0" dist6="0" dist7="0" dist8="0" dist9="0" >
+    </shelf_1_level>
+    <shelf_1_level name="level_5" parent="shelf_1_footprint" dist1="0" dist2="0" dist3="0" dist4="0" dist5="0" dist6="0" dist7="0" dist8="0" dist9="0" >
         <origin xyz="0 0 1.86865" />
-    </shelve_1_level>
+    </shelf_1_level>
 </macro>
     <!-- Shelve 2 -->
-    <macro name="shelve_2" params="*origin parent">
-     <link name="shelve_2_footprint"/>
+    <macro name="shelf_2" params="*origin parent">
+     <link name="shelf_2_footprint"/>
     <joint type="fixed" name="romm_shleve_2_joint">
         <xacro:insert_block name="origin"/>
         <parent link="${parent}"/>
-        <child link="shelve_2_footprint"/>
-    </joint>
-     <link name="shelve_2_base">
+        <child link="shelf_2_footprint"/>
+    </joint>
+     <link name="shelf_2_base">
         <visual>
             <geometry>
@@ -220,10 +220,10 @@
         </collision>
     </link>
-    <joint type="fixed" name="shelve_2_foot_base_joint">
+    <joint type="fixed" name="shelf_2_foot_base_joint">
         <iorigin xyz="0 0 0"/>
-        <parent link="shelve_2_footprint"/>
-        <child link="shelve_2_base"/>
-    </joint>
-    <link name="shelve_2_left_side">
+        <parent link="shelf_2_footprint"/>
+        <child link="shelf_2_base"/>
+    </joint>
+    <link name="shelf_2_left_side">
         <visual>
             <geometry>
@@ -237,10 +237,10 @@
         </collision>
     </link>
-    <joint type="fixed" name="shelve_2_foot_left_joint">
+    <joint type="fixed" name="shelf_2_foot_left_joint">
         <origin xyz="-0.475 0 0.7225"/>
-        <parent link="shelve_2_footprint"/>
-        <child link="shelve_2_left_side"/>
-    </joint>
-    <link name="shelve_2_right_side">
+        <parent link="shelf_2_footprint"/>
+        <child link="shelf_2_left_side"/>
+    </joint>
+    <link name="shelf_2_right_side">
         <visual>
             <geometry>
@@ -254,10 +254,10 @@
         </collision>
     </link>
-    <joint type="fixed" name="shelve_2_foot_right_joint">
+    <joint type="fixed" name="shelf_2_foot_right_joint">
         <origin xyz="0.475 0 0.7225"/>
-        <parent link="shelve_2_footprint"/>
-        <child link="shelve_2_right_side"/>
-    </joint>
-    <link name="shelve_2_back">
+        <parent link="shelf_2_footprint"/>
+        <child link="shelf_2_right_side"/>
+    </joint>
+    <link name="shelf_2_back">
         <visual>
             <geometry>
@@ -271,10 +271,10 @@
         </collision>
     </link>
-    <joint type="fixed" name="shelve_2_foot_back_joint">
+    <joint type="fixed" name="shelf_2_foot_back_joint">
         <origin xyz="0 0.275 0.7725"/>
-        <parent link="shelve_2_footprint"/>
-        <child link="shelve_2_back"/>
-    </joint>
-    <link name="shelve_2_level_0_link">
+        <parent link="shelf_2_footprint"/>
+        <child link="shelf_2_back"/>
+    </joint>
+    <link name="shelf_2_level_0_link">
         <visual>
             <geometry>
@@ -288,30 +288,30 @@
         </collision>
     </link>
-    <joint type="fixed" name="shelve_2_level_0_joint">
+    <joint type="fixed" name="shelf_2_level_0_joint">
         <origin xyz="0 0 0.0925"/>
-        <parent link="shelve_2_footprint"/>
-        <child link="shelve_2_level_0_link"/>
-    </joint>
-    <shelve_2_level name="level_1" parent="shelve_2_footprint">
+        <parent link="shelf_2_footprint"/>
+        <child link="shelf_2_level_0_link"/>
+    </joint>
+    <shelf_2_level name="level_1" parent="shelf_2_footprint">
         <origin xyz="0 0.05 0.324"/>
-    </shelve_2_level>
-    <shelve_2_level name="level_2" parent="shelve_2_footprint">
+    </shelf_2_level>
+    <shelf_2_level name="level_2" parent="shelf_2_footprint">
         <origin xyz="0 0.05 0.574"/>
-    </shelve_2_level>
-    <shelve_2_level name="level_3" parent="shelve_2_footprint">
+    </shelf_2_level>
+    <shelf_2_level name="level_3" parent="shelf_2_footprint">
         <origin xyz="0 0.05 0.784"/>
-    </shelve_2_level>
-    <shelve_2_level name="level_4" parent="shelve_2_footprint">
+    </shelf_2_level>
+    <shelf_2_level name="level_4" parent="shelf_2_footprint">
         <origin xyz="0 0.05 1.036"/>
-    </shelve_2_level>
-    <shelve_2_level name="level_5" parent="shelve_2_footprint">
+    </shelf_2_level>
+    <shelf_2_level name="level_5" parent="shelf_2_footprint">
         <origin xyz="0 0.05 1.245"/>
-    </shelve_2_level>
+    </shelf_2_level>
 </macro>
-<shelve_1 parent="room_link">
+<shelf_1 parent="room_link">
     <origin xyz="1 1 0.08515"/>
-</shelve_1>
-<shelve_2 parent="room_link">
+</shelf_1>
+<shelf_2 parent="room_link">
     <origin xyz="-1 1 0.08515"/>
-</shelve_2>
+</shelf_2>
 </robot>

Commit message: dm shelves coordinate corrections

File: iai_refills_lab/maps/dm_shelves.urdf.xacro (robot description, xacro)
@@ -228,10 +228,10 @@
         <visual>
             <geometry>
-                <box size="0.05 0.54 1.3"/>
-            </geometry>
-        </visual>
-        <collision>
-           <geometry>
-                <box size="0.05 0.54 1.3"/>
+                <box size="0.05 0.54 1.6"/>
+            </geometry>
+        </visual>
+        <collision>
+           <geometry>
+                <box size="0.05 0.54 1.6"/>
             </geometry>
         </collision>
@@ -245,10 +245,10 @@
         <visual>
             <geometry>
-                <box size="0.05 0.54 1.3"/>
-            </geometry>
-        </visual>
-        <collision>
-           <geometry>
-                <box size="0.05 0.54 1.3"/>
+                <box size="0.05 0.54 1.6"/>
+            </geometry>
+        </visual>
+        <collision>
+           <geometry>
+                <box size="0.05 0.54 1.6"/>
             </geometry>
         </collision>
@@ -262,10 +262,10 @@
         <visual>
             <geometry>
-                <box size="1 0.05 1.4"/>
-            </geometry>
-        </visual>
-        <collision>
-           <geometry>
-                <box size="1 0.05 1.4"/>
+                <box size="1 0.05 1.45"/>
+            </geometry>
+        </visual>
+        <collision>
+           <geometry>
+                <box size="1 0.05 1.45"/>
             </geometry>
         </collision>
@@ -294,24 +294,24 @@
     </joint>
     <shelf_2_level name="level_1" parent="shelf_2_footprint">
-        <origin xyz="0 0.05 0.324"/>
+        <origin xyz="0 0.0 0.374"/>
     </shelf_2_level>
     <shelf_2_level name="level_2" parent="shelf_2_footprint">
-        <origin xyz="0 0.05 0.574"/>
+        <origin xyz="0 0.0 0.624"/>
     </shelf_2_level>
     <shelf_2_level name="level_3" parent="shelf_2_footprint">
-        <origin xyz="0 0.05 0.784"/>
+        <origin xyz="0 0.0 0.864"/>
     </shelf_2_level>
     <shelf_2_level name="level_4" parent="shelf_2_footprint">
-        <origin xyz="0 0.05 1.036"/>
+        <origin xyz="0 0.0 1.17"/>
     </shelf_2_level>
     <shelf_2_level name="level_5" parent="shelf_2_footprint">
-        <origin xyz="0 0.05 1.245"/>
+        <origin xyz="0 0.0 1.42"/>
     </shelf_2_level>
 </macro>
 <shelf_1 parent="room_link">
-    <origin xyz="1 1 0.08515"/>
+    <origin xyz="4.3223 -0.2415761 0.08515" rpy="0 0 -1.5756"/>
 </shelf_1>
 <shelf_2 parent="room_link">
-    <origin xyz="-1 1 0.08515"/>
+    <origin xyz="1.7857 -1.52236 0.08515" rpy="0 0 3.09652"/>
 </shelf_2>
 </robot>
