Commit message: changes to sm_shelves to use as macro in other file

File: iai_refills_lab/maps/dm_shelves.urdf.xacro (robot description, xacro)
@@ -1,5 +1,7 @@
 <?xml version="1.0"?>
 <robot name="dm_shelves" xmlns:xacro="http://ros.org/wiki/xacro">
+<!--
 <link name="room_link"/>
+-->
     <macro name="divider_link" params="parent name *origin">
         <link name="shelf_1_${name}_link">
@@ -54,5 +56,5 @@
     </macro>
     <macro name="shelf_1_level" params="name parent *origin dist1 dist2 dist3 dist4 dist5 dist6 dist7 dist8 dist9">
-        <link name="shelf_1_${name}_link">
+        <link name="${name}_link">
             <visual>
                 <geometry>
@@ -66,5 +68,5 @@
             </collision>
         </link>
-        <link name="shelf_1_${name}_left_support_link">
+        <link name="${name}_left_support_link">
             <visual>
                 <geometry>
@@ -78,5 +80,5 @@
             </collision>
         </link>
-        <link name="shelf_1_${name}_right_support_link">
+        <link name="${name}_right_support_link">
             <visual>
                 <geometry>
@@ -90,21 +92,204 @@
             </collision>
         </link>
-        <joint type="fixed" name="shelf_1_${name}_joint">
+        <joint type="fixed" name="${name}_joint">
             <xacro:insert_block name="origin"/>
             <parent link="${parent}"/>
-            <child link="shelf_1_${name}_link"/>
-        </joint>
-        <joint type="fixed" name="shelf_1_${name}_right_support_joint">
+            <child link="${name}_link"/>
+        </joint>
+        <joint type="fixed" name="${name}_right_support_joint">
             <origin xyz="0.494 0 -0.06"/>
-            <parent link="shelf_1_${name}_link"/>
-            <child link="shelf_1_${name}_right_support_link"/>
-        </joint>
-        <joint type="fixed" name="shelf_1_${name}_left_support_joint">
+            <parent link="${name}_link"/>
+            <child link="${name}_right_support_link"/>
+        </joint>
+        <joint type="fixed" name="${name}_left_support_joint">
             <origin xyz="-0.494 0 -0.06"/>
-            <parent link="shelf_1_${name}_link"/>
-            <child link="shelf_1_${name}_left_support_link"/>
-        </joint>
-        <shelf_divider parent="shelf_1_${name}_link" name="${name}" dist1="${dist1}" dist2="${dist2}" dist3="${dist3}" dist4="${dist4}" dist5="${dist5}" dist6="${dist6}" dist7="${dist7}" dist8="${dist8}" dist9="${dist9}" />
+            <parent link="${name}_link"/>
+            <child link="${name}_left_support_link"/>
+        </joint>
+        <shelf_divider parent="${name}_link" name="${name}" dist1="${dist1}" dist2="${dist2}" dist3="${dist3}" dist4="${dist4}" dist5="${dist5}" dist6="${dist6}" dist7="${dist7}" dist8="${dist8}" dist9="${dist9}" />
     </macro>
+    <macro name="shelf_1" params="*origin parent name">
+    <link name="${name}_footprint"/>
+    <joint type="fixed" name="${name}_joint">
+        <xacro:insert_block name="origin"/>
+        <parent link="${parent}"/>
+        <child link="${name}_footprint"/>
+    </joint>
+    <link name="${name}_base">
+        <visual>
+            <geometry>
+                <box size="1.04 0.85 0.173"/>
+            </geometry>
+        </visual>
+        <collision>
+           <geometry>
+                <box size="1.04 0.85 0.173"/>
+            </geometry>
+        </collision>
+    </link>
+    <joint type="fixed" name="${name}_foot_base_joint">
+        <iorigin xyz="0 0 0.0865"/>
+        <parent link="${name}_footprint"/>
+        <child link="${name}_base"/>
+    </joint>
+    <link name="${name}_back">
+        <visual>
+            <geometry>
+                <box size="1.04 0.12 2"/>
+            </geometry>
+        </visual>
+        <collision>
+           <geometry>
+                <box size="1.04 0.12 2"/>
+            </geometry>
+        </collision>
+    </link>
+    <joint type="fixed" name="${name}_foot_back_joint">
+        <origin xyz="0 0.365 1"/>
+        <parent link="${name}_footprint"/>
+        <child link="${name}_back"/>
+    </joint>
+    <link name="${name}_level_0_link">
+        <visual>
+            <geometry>
+                <box size="1 0.78 0.043"/>
+            </geometry>
+        </visual>
+        <collision>
+           <geometry>
+                <box size="1 0.78 0.043"/>
+            </geometry>
+        </collision>
+    </link>
+    <joint type="fixed" name="${name}_level_0_joint">
+        <origin xyz="0 -0.06 0.10665"/>
+        <parent link="${name}_footprint"/>
+        <child link="${name}_level_0_link"/>
+    </joint>
+    <shelf_1_level name="${name}_level_1" parent="${name}_footprint" dist1="0.15" dist2="0.133" dist3="0.082" dist4="0.167" dist5="0.095" dist6="0.148" dist7="0.095" dist8="0.125" dist9="0" >
+        <origin xyz="0 0 0.50965" />
+    </shelf_1_level>
+    <shelf_1_level name="${name}_level_2" parent="${name}_footprint" dist1="0.177" dist2="0.208" dist3="0.147" dist4="0.20" dist5="0.124" dist6="0.14" dist7="0" dist8="0" dist9="0" >
+        <origin xyz="0 0 0.84465" />
+    </shelf_1_level>
+    <shelf_1_level name="${name}_level_3" parent="${name}_footprint" dist1="0" dist2="0" dist3="0" dist4="0" dist5="0" dist6="0" dist7="0" dist8="0" dist9="0" >
+        <origin xyz="0 0 1.22265" />
+    </shelf_1_level>
+    <shelf_1_level name="${name}_level_4" parent="${name}_footprint" dist1="0" dist2="0" dist3="0" dist4="0" dist5="0" dist6="0" dist7="0" dist8="0" dist9="0" >
+        <origin xyz="0 0 1.53565" />
+    </shelf_1_level>
+    <shelf_1_level name="${name}_level_5" parent="${name}_footprint" dist1="0" dist2="0" dist3="0" dist4="0" dist5="0" dist6="0" dist7="0" dist8="0" dist9="0" >
+        <origin xyz="0 0 1.86865" />
+    </shelf_1_level>
+</macro>
+    <!-- Shelve 2 -->
+    <macro name="shelf_2" params="*origin parent name">
+     <link name="${name}_footprint"/>
+    <joint type="fixed" name="${name}_joint">
+        <xacro:insert_block name="origin"/>
+        <parent link="${parent}"/>
+        <child link="${name}_footprint"/>
+    </joint>
+     <link name="${name}_base">
+        <visual>
+            <geometry>
+                <box size="1 0.6 0.145"/>
+            </geometry>
+        </visual>
+        <collision>
+           <geometry>
+                <box size="1 0.6 0.145"/>
+            </geometry>
+        </collision>
+    </link>
+    <joint type="fixed" name="${name}_foot_base_joint">
+        <iorigin xyz="0 0 0.0725"/>
+        <parent link="${name}_footprint"/>
+        <child link="${name}_base"/>
+    </joint>
+    <link name="${name}_left_side">
+        <visual>
+            <geometry>
+                <box size="0.05 0.54 1.6"/>
+            </geometry>
+        </visual>
+        <collision>
+           <geometry>
+                <box size="0.05 0.54 1.6"/>
+            </geometry>
+        </collision>
+    </link>
+    <joint type="fixed" name="${name}_foot_left_joint">
+        <origin xyz="-0.475 0 0.7225"/>
+        <parent link="${name}_footprint"/>
+        <child link="${name}_left_side"/>
+    </joint>
+    <link name="${name}_right_side">
+        <visual>
+            <geometry>
+                <box size="0.05 0.54 1.6"/>
+            </geometry>
+        </visual>
+        <collision>
+           <geometry>
+                <box size="0.05 0.54 1.6"/>
+            </geometry>
+        </collision>
+    </link>
+    <joint type="fixed" name="${name}_foot_right_joint">
+        <origin xyz="0.475 0 0.7225"/>
+        <parent link="${name}_footprint"/>
+        <child link="${name}_right_side"/>
+    </joint>
+    <link name="${name}_back">
+        <visual>
+            <geometry>
+                <box size="1 0.05 1.45"/>
+            </geometry>
+        </visual>
+        <collision>
+           <geometry>
+                <box size="1 0.05 1.45"/>
+            </geometry>
+        </collision>
+    </link>
+    <joint type="fixed" name="${name}_foot_back_joint">
+        <origin xyz="0 0.275 0.7725"/>
+        <parent link="${name}_footprint"/>
+        <child link="${name}_back"/>
+    </joint>
+    <link name="${name}_level_0_link">
+        <visual>
+            <geometry>
+                <box size="0.992 0.54 0.043"/>
+            </geometry>
+        </visual>
+        <collision>
+           <geometry>
+                <box size="0.992 0.54 0.043"/>
+            </geometry>
+        </collision>
+    </link>
+    <joint type="fixed" name="${name}_level_0_joint">
+        <origin xyz="0 0 0.0925"/>
+        <parent link="${name}_footprint"/>
+        <child link="${name}_level_0_link"/>
+    </joint>
+    <shelf_2_level name="${name}_level_1" parent="${name}_footprint">
+        <origin xyz="0 0.0 0.374"/>
+    </shelf_2_level>
+    <shelf_2_level name="${name}_level_2" parent="${name}_footprint">
+        <origin xyz="0 0.0 0.624"/>
+    </shelf_2_level>
+    <shelf_2_level name="${name}_level_3" parent="${name}_footprint">
+        <origin xyz="0 0.0 0.864"/>
+    </shelf_2_level>
+    <shelf_2_level name="${name}_level_4" parent="${name}_footprint">
+        <origin xyz="0 0.0 1.17"/>
+    </shelf_2_level>
+    <shelf_2_level name="${name}_level_5" parent="${name}_footprint">
+        <origin xyz="0 0.0 1.42"/>
+    </shelf_2_level>
+</macro>
     <macro name="shelf_2_level" params="name parent *origin">
         <link name="shelf_2_${name}_link">
@@ -126,187 +311,5 @@
         </joint>
     </macro>
-    <macro name="shelf_1" params="*origin parent">
-    <link name="shelf_1_footprint"/>
-    <joint type="fixed" name="romm_shleve_1_joint">
-        <xacro:insert_block name="origin"/>
-        <parent link="${parent}"/>
-        <child link="shelf_1_footprint"/>
-    </joint>
-    <link name="shelf_1_base">
-        <visual>
-            <geometry>
-                <box size="1.04 0.85 0.173"/>
-            </geometry>
-        </visual>
-        <collision>
-           <geometry>
-                <box size="1.04 0.85 0.173"/>
-            </geometry>
-        </collision>
-    </link>
-    <joint type="fixed" name="foot_base_joint">
-        <iorigin xyz="0 0 0"/>
-        <parent link="shelf_1_footprint"/>
-        <child link="shelf_1_base"/>
-    </joint>
-    <link name="shelf_1_back">
-        <visual>
-            <geometry>
-                <box size="1.04 0.12 2"/>
-            </geometry>
-        </visual>
-        <collision>
-           <geometry>
-                <box size="1.04 0.12 2"/>
-            </geometry>
-        </collision>
-    </link>
-    <joint type="fixed" name="foot_back_joint">
-        <origin xyz="0 0.365 1"/>
-        <parent link="shelf_1_footprint"/>
-        <child link="shelf_1_back"/>
-    </joint>
-    <link name="shelf_1_level_0_link">
-        <visual>
-            <geometry>
-                <box size="1 0.78 0.043"/>
-            </geometry>
-        </visual>
-        <collision>
-           <geometry>
-                <box size="1 0.78 0.043"/>
-            </geometry>
-        </collision>
-    </link>
-    <joint type="fixed" name="shelf_1_level_0_joint">
-        <origin xyz="0 -0.06 0.10665"/>
-        <parent link="shelf_1_footprint"/>
-        <child link="shelf_1_level_0_link"/>
-    </joint>
-    <shelf_1_level name="level_1" parent="shelf_1_footprint" dist1="0.15" dist2="0.133" dist3="0.082" dist4="0.167" dist5="0.095" dist6="0.148" dist7="0.095" dist8="0.125" dist9="0" >
-        <origin xyz="0 0 0.50965" />
-    </shelf_1_level>
-    <shelf_1_level name="level_2" parent="shelf_1_footprint" dist1="0.177" dist2="0.208" dist3="0.147" dist4="0.20" dist5="0.124" dist6="0.14" dist7="0" dist8="0" dist9="0" >
-        <origin xyz="0 0 0.84465" />
-    </shelf_1_level>
-    <shelf_1_level name="level_3" parent="shelf_1_footprint" dist1="0" dist2="0" dist3="0" dist4="0" dist5="0" dist6="0" dist7="0" dist8="0" dist9="0" >
-        <origin xyz="0 0 1.22265" />
-    </shelf_1_level>
-    <shelf_1_level name="level_4" parent="shelf_1_footprint" dist1="0" dist2="0" dist3="0" dist4="0" dist5="0" dist6="0" dist7="0" dist8="0" dist9="0" >
-        <origin xyz="0 0 1.53565" />
-    </shelf_1_level>
-    <shelf_1_level name="level_5" parent="shelf_1_footprint" dist1="0" dist2="0" dist3="0" dist4="0" dist5="0" dist6="0" dist7="0" dist8="0" dist9="0" >
-        <origin xyz="0 0 1.86865" />
-    </shelf_1_level>
-</macro>
-    <!-- Shelve 2 -->
-    <macro name="shelf_2" params="*origin parent">
-     <link name="shelf_2_footprint"/>
-    <joint type="fixed" name="romm_shleve_2_joint">
-        <xacro:insert_block name="origin"/>
-        <parent link="${parent}"/>
-        <child link="shelf_2_footprint"/>
-    </joint>
-     <link name="shelf_2_base">
-        <visual>
-            <geometry>
-                <box size="1 0.6 0.145"/>
-            </geometry>
-        </visual>
-        <collision>
-           <geometry>
-                <box size="1 0.6 0.145"/>
-            </geometry>
-        </collision>
-    </link>
-    <joint type="fixed" name="shelf_2_foot_base_joint">
-        <iorigin xyz="0 0 0"/>
-        <parent link="shelf_2_footprint"/>
-        <child link="shelf_2_base"/>
-    </joint>
-    <link name="shelf_2_left_side">
-        <visual>
-            <geometry>
-                <box size="0.05 0.54 1.6"/>
-            </geometry>
-        </visual>
-        <collision>
-           <geometry>
-                <box size="0.05 0.54 1.6"/>
-            </geometry>
-        </collision>
-    </link>
-    <joint type="fixed" name="shelf_2_foot_left_joint">
-        <origin xyz="-0.475 0 0.7225"/>
-        <parent link="shelf_2_footprint"/>
-        <child link="shelf_2_left_side"/>
-    </joint>
-    <link name="shelf_2_right_side">
-        <visual>
-            <geometry>
-                <box size="0.05 0.54 1.6"/>
-            </geometry>
-        </visual>
-        <collision>
-           <geometry>
-                <box size="0.05 0.54 1.6"/>
-            </geometry>
-        </collision>
-    </link>
-    <joint type="fixed" name="shelf_2_foot_right_joint">
-        <origin xyz="0.475 0 0.7225"/>
-        <parent link="shelf_2_footprint"/>
-        <child link="shelf_2_right_side"/>
-    </joint>
-    <link name="shelf_2_back">
-        <visual>
-            <geometry>
-                <box size="1 0.05 1.45"/>
-            </geometry>
-        </visual>
-        <collision>
-           <geometry>
-                <box size="1 0.05 1.45"/>
-            </geometry>
-        </collision>
-    </link>
-    <joint type="fixed" name="shelf_2_foot_back_joint">
-        <origin xyz="0 0.275 0.7725"/>
-        <parent link="shelf_2_footprint"/>
-        <child link="shelf_2_back"/>
-    </joint>
-    <link name="shelf_2_level_0_link">
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
Commit message: [dm room urdf] reparented the links to go from shelf base

File: iai_refills_lab/maps/dm_shelves.urdf.xacro (robot description, xacro)
@@ -127,25 +127,19 @@
     </macro>
     <macro name="shelf_1" params="*origin parent">
-    <link name="shelf_1_footprint"/>
+    <link name="shelf_1_base">
+        <visual>
+            <geometry>
+                <box size="1.04 0.85 0.173"/>
+            </geometry>
+        </visual>
+        <collision>
+           <geometry>
+                <box size="1.04 0.85 0.173"/>
+            </geometry>
+        </collision>
+    </link>
     <joint type="fixed" name="romm_shleve_1_joint">
         <xacro:insert_block name="origin"/>
         <parent link="${parent}"/>
-        <child link="shelf_1_footprint"/>
-    </joint>
-    <link name="shelf_1_base">
-        <visual>
-            <geometry>
-                <box size="1.04 0.85 0.173"/>
-            </geometry>
-        </visual>
-        <collision>
-           <geometry>
-                <box size="1.04 0.85 0.173"/>
-            </geometry>
-        </collision>
-    </link>
-    <joint type="fixed" name="foot_base_joint">
-        <iorigin xyz="0 0 0"/>
-        <parent link="shelf_1_footprint"/>
         <child link="shelf_1_base"/>
     </joint>
@@ -164,5 +158,5 @@
     <joint type="fixed" name="foot_back_joint">
         <origin xyz="0 0.365 1"/>
-        <parent link="shelf_1_footprint"/>
+        <parent link="shelf_1_base"/>
         <child link="shelf_1_back"/>
     </joint>
@@ -181,20 +175,20 @@
     <joint type="fixed" name="shelf_1_level_0_joint">
         <origin xyz="0 -0.06 0.10665"/>
-        <parent link="shelf_1_footprint"/>
+        <parent link="shelf_1_base"/>
         <child link="shelf_1_level_0_link"/>
     </joint>
-    <shelf_1_level name="level_1" parent="shelf_1_footprint" dist1="0.15" dist2="0.133" dist3="0.082" dist4="0.167" dist5="0.095" dist6="0.148" dist7="0.095" dist8="0.125" dist9="0" >
+    <shelf_1_level name="level_1" parent="shelf_1_base" dist1="0.15" dist2="0.133" dist3="0.082" dist4="0.167" dist5="0.095" dist6="0.148" dist7="0.095" dist8="0.125" dist9="0" >
         <origin xyz="0 0 0.50965" />
     </shelf_1_level>
-    <shelf_1_level name="level_2" parent="shelf_1_footprint" dist1="0.177" dist2="0.208" dist3="0.147" dist4="0.20" dist5="0.124" dist6="0.14" dist7="0" dist8="0" dist9="0" >
+    <shelf_1_level name="level_2" parent="shelf_1_base" dist1="0.177" dist2="0.208" dist3="0.147" dist4="0.20" dist5="0.124" dist6="0.14" dist7="0" dist8="0" dist9="0" >
         <origin xyz="0 0 0.84465" />
     </shelf_1_level>
-    <shelf_1_level name="level_3" parent="shelf_1_footprint" dist1="0" dist2="0" dist3="0" dist4="0" dist5="0" dist6="0" dist7="0" dist8="0" dist9="0" >
+    <shelf_1_level name="level_3" parent="shelf_1_base" dist1="0" dist2="0" dist3="0" dist4="0" dist5="0" dist6="0" dist7="0" dist8="0" dist9="0" >
         <origin xyz="0 0 1.22265" />
     </shelf_1_level>
-    <shelf_1_level name="level_4" parent="shelf_1_footprint" dist1="0" dist2="0" dist3="0" dist4="0" dist5="0" dist6="0" dist7="0" dist8="0" dist9="0" >
+    <shelf_1_level name="level_4" parent="shelf_1_base" dist1="0" dist2="0" dist3="0" dist4="0" dist5="0" dist6="0" dist7="0" dist8="0" dist9="0" >
         <origin xyz="0 0 1.53565" />
     </shelf_1_level>
-    <shelf_1_level name="level_5" parent="shelf_1_footprint" dist1="0" dist2="0" dist3="0" dist4="0" dist5="0" dist6="0" dist7="0" dist8="0" dist9="0" >
+    <shelf_1_level name="level_5" parent="shelf_1_base" dist1="0" dist2="0" dist3="0" dist4="0" dist5="0" dist6="0" dist7="0" dist8="0" dist9="0" >
         <origin xyz="0 0 1.86865" />
     </shelf_1_level>
@@ -202,25 +196,19 @@
     <!-- Shelve 2 -->
     <macro name="shelf_2" params="*origin parent">
-     <link name="shelf_2_footprint"/>
+     <link name="shelf_2_base">
+        <visual>
+            <geometry>
+                <box size="1 0.6 0.145"/>
+            </geometry>
+        </visual>
+        <collision>
+           <geometry>
+                <box size="1 0.6 0.145"/>
+            </geometry>
+        </collision>
+    </link>
     <joint type="fixed" name="romm_shleve_2_joint">
         <xacro:insert_block name="origin"/>
         <parent link="${parent}"/>
-        <child link="shelf_2_footprint"/>
-    </joint>
-     <link name="shelf_2_base">
-        <visual>
-            <geometry>
-                <box size="1 0.6 0.145"/>
-            </geometry>
-        </visual>
-        <collision>
-           <geometry>
-                <box size="1 0.6 0.145"/>
-            </geometry>
-        </collision>
-    </link>
-    <joint type="fixed" name="shelf_2_foot_base_joint">
-        <iorigin xyz="0 0 0"/>
-        <parent link="shelf_2_footprint"/>
         <child link="shelf_2_base"/>
     </joint>
@@ -239,5 +227,5 @@
     <joint type="fixed" name="shelf_2_foot_left_joint">
         <origin xyz="-0.475 0 0.7225"/>
-        <parent link="shelf_2_footprint"/>
+        <parent link="shelf_2_base"/>
         <child link="shelf_2_left_side"/>
     </joint>
@@ -256,5 +244,5 @@
     <joint type="fixed" name="shelf_2_foot_right_joint">
         <origin xyz="0.475 0 0.7225"/>
-        <parent link="shelf_2_footprint"/>
+        <parent link="shelf_2_base"/>
         <child link="shelf_2_right_side"/>
     </joint>
@@ -273,5 +261,5 @@
     <joint type="fixed" name="shelf_2_foot_back_joint">
         <origin xyz="0 0.275 0.7725"/>
-        <parent link="shelf_2_footprint"/>
+        <parent link="shelf_2_base"/>
         <child link="shelf_2_back"/>
     </joint>
@@ -290,20 +278,20 @@
     <joint type="fixed" name="shelf_2_level_0_joint">
         <origin xyz="0 0 0.0925"/>
-        <parent link="shelf_2_footprint"/>
+        <parent link="shelf_2_base"/>
         <child link="shelf_2_level_0_link"/>
     </joint>
-    <shelf_2_level name="level_1" parent="shelf_2_footprint">
+    <shelf_2_level name="level_1" parent="shelf_2_base">
         <origin xyz="0 0.0 0.374"/>
     </shelf_2_level>
-    <shelf_2_level name="level_2" parent="shelf_2_footprint">
+    <shelf_2_level name="level_2" parent="shelf_2_base">
         <origin xyz="0 0.0 0.624"/>
     </shelf_2_level>
-    <shelf_2_level name="level_3" parent="shelf_2_footprint">
+    <shelf_2_level name="level_3" parent="shelf_2_base">
         <origin xyz="0 0.0 0.864"/>
     </shelf_2_level>
-    <shelf_2_level name="level_4" parent="shelf_2_footprint">
+    <shelf_2_level name="level_4" parent="shelf_2_base">
         <origin xyz="0 0.0 1.17"/>
     </shelf_2_level>
-    <shelf_2_level name="level_5" parent="shelf_2_footprint">
+    <shelf_2_level name="level_5" parent="shelf_2_base">
         <origin xyz="0 0.0 1.42"/>
     </shelf_2_level>
