Commit message: [dm lab urdf] manually merged #71 (thx @Tigul), cleaned up, added walls

File: iai_refills_lab/urdf/dm_shelves.urdf.xacro (robot description, xacro)
@@ -1,304 +1,10 @@
 <?xml version="1.0"?>
 <robot name="dm_shelves" xmlns:xacro="http://ros.org/wiki/xacro">
+  <xacro:include filename="$(find iai_refills_lab)/urdf/dm_shelf_macros.urdf.xacro"/>
   <link name="room_link"/>
-  <macro name="divider_link" params="parent name *origin">
-    <link name="shelf_1_${name}_link">
-      <visual>
-        <geometry>
-          <box size="0.004 0.65 0.05"/>
-        </geometry>
-      </visual>
-      <collision>
-        <geometry>
-          <box size="0.004 0.65 0.05"/>
-        </geometry>
-      </collision>
-    </link>
-    <joint type="fixed" name="shelf_1_${name}_joint">
-      <xacro:insert_block name="origin"/>
-      <parent link="${parent}"/>
-      <child link="shelf_1_${name}_link"/>
-    </joint>
-  </macro>
-  <macro name="shelf_divider" params="parent name dist1 dist2 dist3 dist4 dist5 dist6 dist7 dist8 dist9">
-    <divider_link parent="${parent}" name="${name}_divider_1">
-      <origin xyz="-0.495 0 0.024"/>
-    </divider_link>
-    <divider_link parent="${parent}" name="${name}_divider_2">
-      <origin xyz="${-0.495 + dist1} 0 0.024"/>
-    </divider_link>
-    <divider_link parent="${parent}" name="${name}_divider_3">
-      <origin xyz="${-0.495 + dist1 + dist2} 0 0.024"/>
-    </divider_link>
-    <divider_link parent="${parent}" name="${name}_divider_4">
-      <origin xyz="${-0.495 + dist1 + dist2 + dist3} 0 0.024"/>
-    </divider_link>
-    <divider_link parent="${parent}" name="${name}_divider_5">
-      <origin xyz="${-0.495 + dist1 + dist2 + dist3 + dist4} 0 0.024"/>
-    </divider_link>
-    <divider_link parent="${parent}" name="${name}_divider_6">
-      <origin xyz="${-0.495 + dist1 + dist2 + dist3 + dist4 + dist5} 0 0.024"/>
-    </divider_link>
-    <divider_link parent="${parent}" name="${name}_divider_7">
-      <origin xyz="${-0.495 + dist1 + dist2 + dist3 + dist4 + dist5 + dist6} 0 0.024"/>
-    </divider_link>
-    <divider_link parent="${parent}" name="${name}_divider_8">
-      <origin xyz="${-0.495 + dist1 + dist2 + dist3 + dist4 + dist5 + dist6 + dist7} 0 0.024"/>
-    </divider_link>
-    <divider_link parent="${parent}" name="${name}_divider_9">
-      <origin xyz="${-0.495 + dist1 + dist2 + dist3 + dist4 + dist5 + dist6 + dist7 + dist8} 0 0.024"/>
-    </divider_link>
-    <divider_link parent="${parent}" name="${name}_divider_10">
-      <origin xyz="${-0.495 + dist1 + dist2 + dist3 + dist4 + dist5 + dist6 + dist7 + dist8 + dist9} 0 0.024"/>
-    </divider_link>
-  </macro>
-  <macro name="shelf_1_level" params="name parent *origin dist1 dist2 dist3 dist4 dist5 dist6 dist7 dist8 dist9">
-    <link name="shelf_1_${name}_link">
-      <visual>
-        <geometry>
-          <box size="0.988 0.65 0.043"/>
-        </geometry>
-      </visual>
-      <collision>
-        <geometry>
-          <box size="0.988 0.65 0.043"/>
-        </geometry>
-      </collision>
-    </link>
-    <link name="shelf_1_${name}_left_support_link">
-      <visual>
-        <geometry>
-          <box size="0.004 0.65 0.12"/>
-        </geometry>
-      </visual>
-      <collision>
-        <geometry>
-          <box size="0.004 0.65 0.12"/>
-        </geometry>
-      </collision>
-    </link>
-    <link name="shelf_1_${name}_right_support_link">
-      <visual>
-        <geometry>
-          <box size="0.004 0.65 0.12"/>
-        </geometry>
-      </visual>
-      <collision>
-        <geometry>
-          <box size="0.004 0.65 0.12"/>
-        </geometry>
-      </collision>
-    </link>
-    <joint type="fixed" name="shelf_1_${name}_joint">
-      <xacro:insert_block name="origin"/>
-      <parent link="${parent}"/>
-      <child link="shelf_1_${name}_link"/>
-    </joint>
-    <joint type="fixed" name="shelf_1_${name}_right_support_joint">
-      <origin xyz="0.494 0 -0.06"/>
-      <parent link="shelf_1_${name}_link"/>
-      <child link="shelf_1_${name}_right_support_link"/>
-    </joint>
-    <joint type="fixed" name="shelf_1_${name}_left_support_joint">
-      <origin xyz="-0.494 0 -0.06"/>
-      <parent link="shelf_1_${name}_link"/>
-      <child link="shelf_1_${name}_left_support_link"/>
-    </joint>
-    <shelf_divider parent="shelf_1_${name}_link" name="${name}" dist1="${dist1}" dist2="${dist2}" dist3="${dist3}" dist4="${dist4}" dist5="${dist5}" dist6="${dist6}" dist7="${dist7}" dist8="${dist8}" dist9="${dist9}" />
-  </macro>
-  <macro name="shelf_2_level" params="name parent *origin">
-    <link name="shelf_2_${name}_link">
-      <visual>
-        <geometry>
-          <box size="0.992 0.435 0.043"/>
-        </geometry>
-      </visual>
-      <collision>
-        <geometry>
-          <box size="0.992 0.435 0.043"/>
-        </geometry>
-      </collision>
-    </link>
-    <joint type="fixed" name="shelf_2_${name}_joint">
-      <xacro:insert_block name="origin"/>
-      <parent link="${parent}"/>
-      <child link="shelf_2_${name}_link"/>
-    </joint>
-  </macro>
-  <macro name="shelf_1" params="*origin parent">
-    <link name="shelf_1_base">
-      <visual>
-        <geometry>
-          <box size="1.1 1.05 0.173"/>
-        </geometry>
-      </visual>
-      <collision>
-        <geometry>
-          <box size="1.1 1.05 0.173"/>
-        </geometry>
-      </collision>
-    </link>
-    <joint type="fixed" name="romm_shleve_1_joint">
-      <xacro:insert_block name="origin"/>
-      <parent link="${parent}"/>
-      <child link="shelf_1_base"/>
-    </joint>
-    <link name="shelf_1_back">
-      <visual>
-        <geometry>
-          <box size="1.04 0.12 2"/>
-        </geometry>
-      </visual>
-      <collision>
-        <geometry>
-          <box size="1.04 0.12 2"/>
-        </geometry>
-      </collision>
-    </link>
-    <joint type="fixed" name="foot_back_joint">
-      <origin xyz="0 0.365 1"/>
-      <parent link="shelf_1_base"/>
-      <child link="shelf_1_back"/>
-    </joint>
-    <link name="shelf_1_level_0_link">
-      <visual>
-        <geometry>
-          <box size="1 0.78 0.043"/>
-        </geometry>
-      </visual>
-      <collision>
-        <geometry>
-          <box size="1 0.78 0.043"/>
-        </geometry>
-      </collision>
-    </link>
-    <joint type="fixed" name="shelf_1_level_0_joint">
-      <origin xyz="0 -0.06 0.10665"/>
-      <parent link="shelf_1_base"/>
-      <child link="shelf_1_level_0_link"/>
-    </joint>
-    <shelf_1_level name="level_1" parent="shelf_1_base" dist1="0.15" dist2="0.133" dist3="0.082" dist4="0.167" dist5="0.095" dist6="0.148" dist7="0.095" dist8="0.125" dist9="0" >
-      <origin xyz="0 0 0.50965" />
-    </shelf_1_level>
-    <shelf_1_level name="level_2" parent="shelf_1_base" dist1="0.177" dist2="0.208" dist3="0.147" dist4="0.20" dist5="0.124" dist6="0.14" dist7="0" dist8="0" dist9="0" >
-      <origin xyz="0 0 0.84465" />
-    </shelf_1_level>
-    <shelf_1_level name="level_3" parent="shelf_1_base" dist1="0" dist2="0" dist3="0" dist4="0" dist5="0" dist6="0" dist7="0" dist8="0" dist9="0" >
-      <origin xyz="0 0 1.22265" />
-    </shelf_1_level>
-    <shelf_1_level name="level_4" parent="shelf_1_base" dist1="0" dist2="0" dist3="0" dist4="0" dist5="0" dist6="0" dist7="0" dist8="0" dist9="0" >
-      <origin xyz="0 0 1.53565" />
-    </shelf_1_level>
-    <shelf_1_level name="level_5" parent="shelf_1_base" dist1="0" dist2="0" dist3="0" dist4="0" dist5="0" dist6="0" dist7="0" dist8="0" dist9="0" >
-      <origin xyz="0 0 1.86865" />
-    </shelf_1_level>
-  </macro>
-  <!-- Shelve 2 -->
-  <macro name="shelf_2" params="*origin parent">
-    <link name="shelf_2_base">
-      <visual>
-        <geometry>
-          <box size="1.1 0.8 0.145"/>
-        </geometry>
-      </visual>
-      <collision>
-        <geometry>
-          <box size="1.1 0.8 0.145"/>
-        </geometry>
-      </collision>
-    </link>
-    <joint type="fixed" name="romm_shleve_2_joint">
-      <xacro:insert_block name="origin"/>
-      <parent link="${parent}"/>
-      <child link="shelf_2_base"/>
-    </joint>
-    <link name="shelf_2_left_side">
-      <visual>
-        <geometry>
-          <box size="0.05 0.54 1.6"/>
-        </geometry>
-      </visual>
-      <collision>
-        <geometry>
-          <box size="0.05 0.54 1.6"/>
-        </geometry>
-      </collision>
-    </link>
-    <joint type="fixed" name="shelf_2_foot_left_joint">
-      <origin xyz="-0.475 0 0.7225"/>
-      <parent link="shelf_2_base"/>
-      <child link="shelf_2_left_side"/>
-    </joint>
-    <link name="shelf_2_right_side">
-      <visual>
-        <geometry>
-          <box size="0.05 0.54 1.6"/>
-        </geometry>
-      </visual>
-      <collision>
-        <geometry>
-          <box size="0.05 0.54 1.6"/>
-        </geometry>
-      </collision>
-    </link>
-    <joint type="fixed" name="shelf_2_foot_right_joint">
-      <origin xyz="0.475 0 0.7225"/>
-      <parent link="shelf_2_base"/>
-      <child link="shelf_2_right_side"/>
-    </joint>
-    <link name="shelf_2_back">
-      <visual>
-        <geometry>
-          <box size="1 0.05 1.45"/>
-        </geometry>
-      </visual>
-      <collision>
-        <geometry>
-          <box size="1 0.05 1.45"/>
-        </geometry>
-      </collision>
-    </link>
-    <joint type="fixed" name="shelf_2_foot_back_joint">
-      <origin xyz="0 0.275 0.7725"/>
-      <parent link="shelf_2_base"/>
-      <child link="shelf_2_back"/>
-    </joint>
-    <link name="shelf_2_level_0_link">
-      <visual>
-        <geometry>
-          <box size="0.992 0.54 0.043"/>
-        </geometry>
-      </visual>
-      <collision>
-        <geometry>
-          <box size="0.992 0.54 0.043"/>
-        </geometry>
-      </collision>
-    </link>
-    <joint type="fixed" name="shelf_2_level_0_joint">
-      <origin xyz="0 0 0.0925"/>
-      <parent link="shelf_2_base"/>
-      <child link="shelf_2_level_0_link"/>
-    </joint>
-    <shelf_2_level name="level_1" parent="shelf_2_base">
-      <origin xyz="0 0.0 0.374"/>
-    </shelf_2_level>
-    <shelf_2_level name="level_2" parent="shelf_2_base">
-      <origin xyz="0 0.0 0.624"/>
-    </shelf_2_level>
-    <shelf_2_level name="level_3" parent="shelf_2_base">
-      <origin xyz="0 0.0 0.864"/>
-    </shelf_2_level>
-    <shelf_2_level name="level_4" parent="shelf_2_base">
-      <origin xyz="0 0.0 1.17"/>
-    </shelf_2_level>
-    <shelf_2_level name="level_5" parent="shelf_2_base">
-      <origin xyz="0 0.0 1.42"/>
-    </shelf_2_level>
-  </macro>
-  <shelf_1 parent="room_link">
+  <shelf_1 parent="room_link" name="shelf_1">
     <origin xyz="4.3223 -0.2415761 0.08515" rpy="0 0 -1.5756"/>
   </shelf_1>
-  <shelf_2 parent="room_link">
+  <shelf_2 parent="room_link" name="shelf_2">
     <origin xyz="1.75 -1.45 0.08515" rpy="0 0 3.09652"/>
   </shelf_2>
