Commit message: added inertial tag to all links

File: iai_refills_lab/urdf/dm_shelf_macros.urdf.xacro (robot description, xacro)
@@ -13,4 +13,9 @@
         </geometry>
       </collision>
+      <inertial>
+        <mass value="1."/>
+        <inertia ixx="0.1" ixy="0.1" ixz="0.1" iyy="0.1" iyz="0.1" izz="0.1"/>
+        <origin rpy="0 0 0" xyz="0.00312 0 0.11152"/>
+      </inertial>
     </link>
     <joint type="fixed" name="${name}_joint">
@@ -64,4 +69,9 @@
         </geometry>
       </collision>
+      <inertial>
+        <mass value="1."/>
+        <inertia ixx="0.1" ixy="0.1" ixz="0.1" iyy="0.1" iyz="0.1" izz="0.1"/>
+        <origin rpy="0 0 0" xyz="0.00312 0 0.11152"/>
+      </inertial>
     </link>
     <link name="${name}_left_support_link">
@@ -76,4 +86,9 @@
         </geometry>
       </collision>
+      <inertial>
+        <mass value="1."/>
+        <inertia ixx="0.1" ixy="0.1" ixz="0.1" iyy="0.1" iyz="0.1" izz="0.1"/>
+        <origin rpy="0 0 0" xyz="0.00312 0 0.11152"/>
+      </inertial>
     </link>
     <link name="${name}_right_support_link">
@@ -88,4 +103,9 @@
         </geometry>
       </collision>
+      <inertial>
+        <mass value="1."/>
+        <inertia ixx="0.1" ixy="0.1" ixz="0.1" iyy="0.1" iyz="0.1" izz="0.1"/>
+        <origin rpy="0 0 0" xyz="0.00312 0 0.11152"/>
+      </inertial>
     </link>
     <joint type="fixed" name="${name}_joint">
@@ -118,4 +138,9 @@
         </geometry>
       </collision>
+      <inertial>
+        <mass value="1."/>
+        <inertia ixx="0.1" ixy="0.1" ixz="0.1" iyy="0.1" iyz="0.1" izz="0.1"/>
+        <origin rpy="0 0 0" xyz="0.00312 0 0.11152"/>
+      </inertial>
     </link>
     <joint type="fixed" name="${name}_joint">
@@ -135,4 +160,9 @@
         </geometry>
       </collision>
+      <inertial>
+        <mass value="1."/>
+        <inertia ixx="0.1" ixy="0.1" ixz="0.1" iyy="0.1" iyz="0.1" izz="0.1"/>
+        <origin rpy="0 0 0" xyz="0.00312 0 0.11152"/>
+      </inertial>
     </link>
     <joint type="fixed" name="${name}_base_back_joint">
@@ -152,4 +182,9 @@
         </geometry>
       </collision>
+      <inertial>
+        <mass value="1."/>
+        <inertia ixx="0.1" ixy="0.1" ixz="0.1" iyy="0.1" iyz="0.1" izz="0.1"/>
+        <origin rpy="0 0 0" xyz="0.00312 0 0.11152"/>
+      </inertial>
     </link>
     <joint type="fixed" name="${name}_level_0_joint">
@@ -187,4 +222,9 @@
         </geometry>
       </collision>
+      <inertial>
+        <mass value="1."/>
+        <inertia ixx="0.1" ixy="0.1" ixz="0.1" iyy="0.1" iyz="0.1" izz="0.1"/>
+        <origin rpy="0 0 0" xyz="0.00312 0 0.11152"/>
+      </inertial>
     </link>
     <joint type="fixed" name="shelf_2_${name}_joint">
@@ -206,4 +246,9 @@
         </geometry>
       </collision>
+      <inertial>
+        <mass value="1."/>
+        <inertia ixx="0.1" ixy="0.1" ixz="0.1" iyy="0.1" iyz="0.1" izz="0.1"/>
+        <origin rpy="0 0 0" xyz="0.00312 0 0.11152"/>
+      </inertial>
     </link>
     <joint type="fixed" name="${name}_joint">
@@ -223,4 +268,9 @@
         </geometry>
       </collision>
+      <inertial>
+        <mass value="1."/>
+        <inertia ixx="0.1" ixy="0.1" ixz="0.1" iyy="0.1" iyz="0.1" izz="0.1"/>
+        <origin rpy="0 0 0" xyz="0.00312 0 0.11152"/>
+      </inertial>
     </link>
     <joint type="fixed" name="${name}_base_left_joint">
@@ -240,4 +290,9 @@
         </geometry>
       </collision>
+      <inertial>
+        <mass value="1."/>
+        <inertia ixx="0.1" ixy="0.1" ixz="0.1" iyy="0.1" iyz="0.1" izz="0.1"/>
+        <origin rpy="0 0 0" xyz="0.00312 0 0.11152"/>
+      </inertial>
     </link>
     <joint type="fixed" name="${name}_base_right_joint">
@@ -257,4 +312,9 @@
         </geometry>
       </collision>
+      <inertial>
+        <mass value="1."/>
+        <inertia ixx="0.1" ixy="0.1" ixz="0.1" iyy="0.1" iyz="0.1" izz="0.1"/>
+        <origin rpy="0 0 0" xyz="0.00312 0 0.11152"/>
+      </inertial>
     </link>
     <joint type="fixed" name="${name}_base_back_joint">
@@ -274,4 +334,9 @@
         </geometry>
       </collision>
+      <inertial>
+        <mass value="1."/>
+        <inertia ixx="0.1" ixy="0.1" ixz="0.1" iyy="0.1" iyz="0.1" izz="0.1"/>
+        <origin rpy="0 0 0" xyz="0.00312 0 0.11152"/>
+      </inertial>
     </link>
     <joint type="fixed" name="${name}_level_0_joint">
@@ -308,4 +373,9 @@
         </geometry>
       </collision>
+      <inertial>
+        <mass value="1."/>
+        <inertia ixx="0.1" ixy="0.1" ixz="0.1" iyy="0.1" iyz="0.1" izz="0.1"/>
+        <origin rpy="0 0 0" xyz="0.00312 0 0.11152"/>
+      </inertial>
     </link>
     <joint type="fixed" name="${name}_joint">
