Commit message: added xacro namespace because it is needed in noetic

File: iai_refills_lab/urdf/dm_room.urdf.xacro (robot description, xacro)
@@ -3,92 +3,92 @@
   <xacro:include filename="$(find iai_refills_lab)/urdf/dm_shelf_macros.urdf.xacro"/>
   <xacro:include filename="$(find iai_refills_lab)/urdf/dm_shelves.urdf.xacro"/>
-  <!-- <link name="room_link"/> -->
+   <!-- <link name="room_link"/> -->
   <!-- Left side shelves -->
-  <!-- <shelf_1 parent="room_link" name="shelf_1"> -->
+  <!-- <xacro:shelf_1 parent="room_link" name="xacro:shelf_1"> -->
   <!--   <origin xyz="4.3223 -0.2415761 0.08515" rpy="0 0 -1.5756"/> -->
-  <!-- </shelf_1> -->
-  <shelf_1 parent="room_link" name="shelf_left_center_front">
+  <!-- </xacro:shelf_1> -->
+  <xacro:shelf_1 parent="room_link" name="shelf_left_center_front">
     <origin xyz="4.3223 -1.2415761 0.08515" rpy="0 0 -1.5756"/>
-  </shelf_1>
-  <shelf_1 parent="room_link" name="shelf_left_center_back">
+  </xacro:shelf_1>
+  <xacro:shelf_1 parent="room_link" name="shelf_left_center_back">
     <origin xyz="4.3223 -2.2415761 0.08515" rpy="0 0 -1.5756"/>
-  </shelf_1>
-  <shelf_1 parent="room_link" name="shelf_left_back">
+  </xacro:shelf_1>
+  <xacro:shelf_1 parent="room_link" name="shelf_left_back">
     <origin xyz="4.3223 -3.2415761 0.08515" rpy="0 0 -1.5756"/>
-  </shelf_1>
+  </xacro:shelf_1>
   <!-- Center shelves -->
-  <!-- <shelf_2 parent="room_link" name="shelf_2"> -->
+  <!-- <xacro:shelf_2 parent="room_link" name="xacro:shelf_2"> -->
   <!--   <origin xyz="1.75 -1.45 0.08515" rpy="0 0 3.09652"/> -->
-  <!-- </shelf_2> -->
-  <shelf_2 parent="room_link" name="shelf_center_front_middle">
+  <!-- </xacro:shelf_2> -->
+  <xacro:shelf_2 parent="room_link" name="shelf_center_front_middle">
     <origin xyz="0.75 -1.4 0.08515" rpy="0 0 3.09652"/>
-  </shelf_2>
-  <shelf_2 parent="room_link" name="shelf_center_front_right">
+  </xacro:shelf_2>
+  <xacro:shelf_2 parent="room_link" name="shelf_center_front_right">
     <origin xyz="-0.25 -1.35 0.08515" rpy="0 0 3.09652"/>
-  </shelf_2>
-  <shelf_2 parent="room_link" name="shelf_center_back_left">
+  </xacro:shelf_2>
+  <xacro:shelf_2 parent="room_link" name="shelf_center_back_left">
     <origin xyz="1.73 -2.0 0.08515" rpy="0 0 -3.18666530718"/>
-  </shelf_2>
-  <shelf_2 parent="room_link" name="shelf_center_back_middle">
+  </xacro:shelf_2>
+  <xacro:shelf_2 parent="room_link" name="shelf_center_back_middle">
     <origin xyz="0.73 -1.95 0.08515" rpy="0 0 -3.18666530718"/>
-  </shelf_2>
-  <shelf_2 parent="room_link" name="shelf_center_back_right">
+  </xacro:shelf_2>
+  <xacro:shelf_2 parent="room_link" name="shelf_center_back_right">
     <origin xyz="-0.27 -1.9 0.08515" rpy="0 0 -3.18666530718"/>
-  </shelf_2>
+  </xacro:shelf_2>
   <!-- Back shelves -->
-  <shelf_1 parent="room_link" name="shelf_back_1">
+  <xacro:shelf_1 parent="room_link" name="shelf_back_1">
     <origin xyz="3 -4.3 0.08515" rpy="0 0 ${pi}"/>
-  </shelf_1>
-  <shelf_1 parent="room_link" name="shelf_back_2">
+  </xacro:shelf_1>
+  <xacro:shelf_1 parent="room_link" name="shelf_back_2">
     <origin xyz="2 -4.3 0.08515" rpy="0 0 ${pi}"/>
-  </shelf_1>
-  <shelf_1 parent="room_link" name="shelf_back_3">
+  </xacro:shelf_1>
+  <xacro:shelf_1 parent="room_link" name="shelf_back_3">
     <origin xyz="1 -4.3 0.08515" rpy="0 0 ${pi}"/>
-  </shelf_1>
-  <shelf_1 parent="room_link" name="shelf_back_4">
+  </xacro:shelf_1>
+  <xacro:shelf_1 parent="room_link" name="shelf_back_4">
     <origin xyz="0 -4.3 0.08515" rpy="0 0 ${pi}"/>
-  </shelf_1>
-  <shelf_1 parent="room_link" name="shelf_back_5">
+  </xacro:shelf_1>
+  <xacro:shelf_1 parent="room_link" name="shelf_back_5">
     <origin xyz="-1 -4.3 0.08515" rpy="0 0 ${pi}"/>
-  </shelf_1>
-  <shelf_1 parent="room_link" name="shelf_back_6">
+  </xacro:shelf_1>
+  <xacro:shelf_1 parent="room_link" name="shelf_back_6">
     <origin xyz="-2 -4.3 0.08515" rpy="0 0 ${pi}"/>
-  </shelf_1>
+  </xacro:shelf_1>
   <!--Right side shelves -->
-  <shelf_1 parent="room_link" name="shelf_right_front">
+  <xacro:shelf_1 parent="room_link" name="shelf_right_front">
     <origin xyz="-2.6 -1.0 0.08515" rpy="0 0 1.5756"/>
-  </shelf_1>
-  <shelf_1 parent="room_link" name="shelf_right_center">
+  </xacro:shelf_1>
+  <xacro:shelf_1 parent="room_link" name="shelf_right_center">
     <origin xyz="-2.6 -2.0 0.08515" rpy="0 0 1.5756"/>
-  </shelf_1>
-  <shelf_1 parent="room_link" name="shelf_right_back">
+  </xacro:shelf_1>
+  <xacro:shelf_1 parent="room_link" name="shelf_right_back">
     <origin xyz="-2.6 -3.0 0.08515" rpy="0 0 1.5756"/>
-  </shelf_1>
-  <!-- Walls -->
+  </xacro:shelf_1>
+  <!-- xacro:walls -->
   <xacro:property name="wall_thickness" value="0.2" />
   <xacro:property name="wall_height" value="2.4" />
-  <wall parent="room_link" name="back_wall"
+  <xacro:wall parent="room_link" name="back_wall"
         size="8.0 ${wall_thickness} ${wall_height}">
     <origin xyz="1.0 -5.0 ${wall_height/2}" rpy="0 0 0"/>
-  </wall>
-  <wall parent="room_link" name="left_wall"
+  </xacro:wall>
+  <xacro:wall parent="room_link" name="left_wall"
         size="${wall_thickness} 9.6 ${wall_height}">
     <origin xyz="5.0 -0.3 ${wall_height/2}" rpy="0 0 0"/>
-  </wall>
-  <wall parent="room_link" name="front_wall"
+  </xacro:wall>
+  <xacro:wall parent="room_link" name="front_wall"
         size="5.0 ${wall_thickness} ${wall_height}">
     <origin xyz="2.5 4.6 ${wall_height/2}" rpy="0 0 0"/>
-  </wall>
-  <wall parent="room_link" name="right_wall"
+  </xacro:wall>
+  <xacro:wall parent="room_link" name="right_wall"
         size="${wall_thickness} 5.0 ${wall_height}">
     <origin xyz="-3.0 -2.5 ${wall_height/2}" rpy="0 0 0"/>
-  </wall>
-  <wall parent="room_link" name="back_corner_wall"
+  </xacro:wall>
+  <xacro:wall parent="room_link" name="back_corner_wall"
         size="3.0 ${wall_thickness} ${wall_height}">
     <origin xyz="-1.5 0.0 ${wall_height/2}" rpy="0 0 0"/>
-  </wall>
-  <wall parent="room_link" name="right_corner_wall"
+  </xacro:wall>
+  <xacro:wall parent="room_link" name="right_corner_wall"
         size="${wall_thickness} 4.6 ${wall_height}">
     <origin xyz="0 2.3 ${wall_height/2}" rpy="0 0 0"/>
-  </wall>
+  </xacro:wall>
 </robot>

File: iai_refills_lab/urdf/dm_shelf_macros.urdf.xacro (robot description, xacro)
@@ -21,34 +21,34 @@
   </xacro:macro>
   <xacro:macro name="shelf_divider" params="parent name dist1 dist2 dist3 dist4 dist5 dist6 dist7 dist8 dist9">
-    <divider_link parent="${parent}" name="${name}_divider_1">
+    <xacro:divider_link parent="${parent}" name="${name}_divider_1">
       <origin xyz="-0.495 0 0.024"/>
-    </divider_link>
-    <divider_link parent="${parent}" name="${name}_divider_2">
+    </xacro:divider_link>
+    <xacro:divider_link parent="${parent}" name="${name}_divider_2">
       <origin xyz="${-0.495 + dist1} 0 0.024"/>
-    </divider_link>
-    <divider_link parent="${parent}" name="${name}_divider_3">
+    </xacro:divider_link>
+    <xacro:divider_link parent="${parent}" name="${name}_divider_3">
       <origin xyz="${-0.495 + dist1 + dist2} 0 0.024"/>
-    </divider_link>
-    <divider_link parent="${parent}" name="${name}_divider_4">
+    </xacro:divider_link>
+    <xacro:divider_link parent="${parent}" name="${name}_divider_4">
       <origin xyz="${-0.495 + dist1 + dist2 + dist3} 0 0.024"/>
-    </divider_link>
-    <divider_link parent="${parent}" name="${name}_divider_5">
+    </xacro:divider_link>
+    <xacro:divider_link parent="${parent}" name="${name}_divider_5">
       <origin xyz="${-0.495 + dist1 + dist2 + dist3 + dist4} 0 0.024"/>
-    </divider_link>
-    <divider_link parent="${parent}" name="${name}_divider_6">
+    </xacro:divider_link>
+    <xacro:divider_link parent="${parent}" name="${name}_divider_6">
       <origin xyz="${-0.495 + dist1 + dist2 + dist3 + dist4 + dist5} 0 0.024"/>
-    </divider_link>
-    <divider_link parent="${parent}" name="${name}_divider_7">
+    </xacro:divider_link>
+    <xacro:divider_link parent="${parent}" name="${name}_divider_7">
       <origin xyz="${-0.495 + dist1 + dist2 + dist3 + dist4 + dist5 + dist6} 0 0.024"/>
-    </divider_link>
-    <divider_link parent="${parent}" name="${name}_divider_8">
+    </xacro:divider_link>
+    <xacro:divider_link parent="${parent}" name="${name}_divider_8">
       <origin xyz="${-0.495 + dist1 + dist2 + dist3 + dist4 + dist5 + dist6 + dist7} 0 0.024"/>
-    </divider_link>
-    <divider_link parent="${parent}" name="${name}_divider_9">
+    </xacro:divider_link>
+    <xacro:divider_link parent="${parent}" name="${name}_divider_9">
       <origin xyz="${-0.495 + dist1 + dist2 + dist3 + dist4 + dist5 + dist6 + dist7 + dist8} 0 0.024"/>
-    </divider_link>
-    <divider_link parent="${parent}" name="${name}_divider_10">
+    </xacro:divider_link>
+    <xacro:divider_link parent="${parent}" name="${name}_divider_10">
       <origin xyz="${-0.495 + dist1 + dist2 + dist3 + dist4 + dist5 + dist6 + dist7 + dist8 + dist9} 0 0.024"/>
-    </divider_link>
+    </xacro:divider_link>
   </xacro:macro>
   <xacro:macro name="shelf_1_level" params="name parent *origin dist1 dist2 dist3 dist4 dist5 dist6 dist7 dist8 dist9">
@@ -104,5 +104,5 @@
       <child link="${name}_left_support_link"/>
     </joint>
-    <shelf_divider parent="${name}_link" name="${name}" dist1="${dist1}" dist2="${dist2}" dist3="${dist3}" dist4="${dist4}" dist5="${dist5}" dist6="${dist6}" dist7="${dist7}" dist8="${dist8}" dist9="${dist9}" />
+    <xacro:shelf_divider parent="${name}_link" name="${name}" dist1="${dist1}" dist2="${dist2}" dist3="${dist3}" dist4="${dist4}" dist5="${dist5}" dist6="${dist6}" dist7="${dist7}" dist8="${dist8}" dist9="${dist9}" />
   </xacro:macro>
   <xacro:macro name="shelf_1" params="*origin parent name">
@@ -158,19 +158,19 @@
       <child link="${name}_level_0_link"/>
     </joint>
-    <shelf_1_level name="${name}_level_1" parent="${name}_base" dist1="0.15" dist2="0.133" dist3="0.082" dist4="0.167" dist5="0.095" dist6="0.148" dist7="0.095" dist8="0.125" dist9="0" >
+    <xacro:shelf_1_level name="${name}_level_1" parent="${name}_base" dist1="0.15" dist2="0.133" dist3="0.082" dist4="0.167" dist5="0.095" dist6="0.148" dist7="0.095" dist8="0.125" dist9="0" >
       <origin xyz="0 0 0.50965" />
-    </shelf_1_level>
-    <shelf_1_level name="${name}_level_2" parent="${name}_base" dist1="0.177" dist2="0.208" dist3="0.147" dist4="0.20" dist5="0.124" dist6="0.14" dist7="0" dist8="0" dist9="0" >
+    </xacro:shelf_1_level>
+    <xacro:shelf_1_level name="${name}_level_2" parent="${name}_base" dist1="0.177" dist2="0.208" dist3="0.147" dist4="0.20" dist5="0.124" dist6="0.14" dist7="0" dist8="0" dist9="0" >
       <origin xyz="0 0 0.84465" />
-    </shelf_1_level>
-    <shelf_1_level name="${name}_level_3" parent="${name}_base" dist1="0" dist2="0" dist3="0" dist4="0" dist5="0" dist6="0" dist7="0" dist8="0" dist9="0" >
+    </xacro:shelf_1_level>
+    <xacro:shelf_1_level name="${name}_level_3" parent="${name}_base" dist1="0" dist2="0" dist3="0" dist4="0" dist5="0" dist6="0" dist7="0" dist8="0" dist9="0" >
       <origin xyz="0 0 1.22265" />
-    </shelf_1_level>
-    <shelf_1_level name="${name}_level_4" parent="${name}_base" dist1="0" dist2="0" dist3="0" dist4="0" dist5="0" dist6="0" dist7="0" dist8="0" dist9="0" >
+    </xacro:shelf_1_level>
+    <xacro:shelf_1_level name="${name}_level_4" parent="${name}_base" dist1="0" dist2="0" dist3="0" dist4="0" dist5="0" dist6="0" dist7="0" dist8="0" dist9="0" >
       <origin xyz="0 0 1.53565" />
-    </shelf_1_level>
-    <shelf_1_level name="${name}_level_5" parent="${name}_base" dist1="0" dist2="0" dist3="0" dist4="0" dist5="0" dist6="0" dist7="0" dist8="0" dist9="0" >
+    </xacro:shelf_1_level>
+    <xacro:shelf_1_level name="${name}_level_5" parent="${name}_base" dist1="0" dist2="0" dist3="0" dist4="0" dist5="0" dist6="0" dist7="0" dist8="0" dist9="0" >
       <origin xyz="0 0 1.86865" />
-    </shelf_1_level>
+    </xacro:shelf_1_level>
   </xacro:macro>
   <!-- Shelf 2 -->
@@ -280,19 +280,19 @@
       <child link="${name}_level_0_link"/>
     </joint>
-    <shelf_2_level name="${name}_level_1" parent="${name}_base">
+    <xacro:shelf_2_level name="${name}_level_1" parent="${name}_base">
       <origin xyz="0 0.0 0.374"/>
-    </shelf_2_level>
-    <shelf_2_level name="${name}_level_2" parent="${name}_base">
+    </xacro:shelf_2_level>
+    <xacro:shelf_2_level name="${name}_level_2" parent="${name}_base">
       <origin xyz="0 0.0 0.624"/>
-    </shelf_2_level>
-    <shelf_2_level name="${name}_level_3" parent="${name}_base">
+    </xacro:shelf_2_level>
+    <xacro:shelf_2_level name="${name}_level_3" parent="${name}_base">
       <origin xyz="0 0.0 0.864"/>
-    </shelf_2_level>
-    <shelf_2_level name="${name}_level_4" parent="${name}_base">
+    </xacro:shelf_2_level>
+    <xacro:shelf_2_level name="${name}_level_4" parent="${name}_base">
       <origin xyz="0 0.0 1.17"/>
-    </shelf_2_level>
-    <shelf_2_level name="${name}_level_5" parent="${name}_base">
+    </xacro:shelf_2_level>
+    <xacro:shelf_2_level name="${name}_level_5" parent="${name}_base">
       <origin xyz="0 0.0 1.42"/>
-    </shelf_2_level>
+    </xacro:shelf_2_level>
   </xacro:macro>
   <xacro:macro name="wall" params="parent name size *origin">

File: iai_refills_lab/urdf/dm_shelves.urdf.xacro (robot description, xacro)
@@ -3,9 +3,9 @@
   <xacro:include filename="$(find iai_refills_lab)/urdf/dm_shelf_macros.urdf.xacro"/>
   <link name="room_link"/>
-  <shelf_1 parent="room_link" name="shelf_1">
+  <xacro:shelf_1 parent="room_link" name="shelf_1">
     <origin xyz="4.3223 -0.2415761 0.08515" rpy="0 0 -1.5756"/>
-  </shelf_1>
-  <shelf_2 parent="room_link" name="shelf_2">
+  </xacro:shelf_1>
+  <xacro:shelf_2 parent="room_link" name="shelf_2">
     <origin xyz="1.75 -1.45 0.08515" rpy="0 0 3.09652"/>
-  </shelf_2>
+  </xacro:shelf_2>
 </robot>

Commit message: removing dm_room changes from this branch

File: iai_refills_lab/urdf/dm_room.urdf.xacro (robot description, xacro)
@@ -3,9 +3,9 @@
   <xacro:include filename="$(find iai_refills_lab)/urdf/dm_shelf_macros.urdf.xacro"/>
   <xacro:include filename="$(find iai_refills_lab)/urdf/dm_shelves.urdf.xacro"/>
-  <!-- <link name="room_link"/> -->
+   <!-- <link name="room_link"/> -->
   <!-- Left side shelves -->
-  <!-- <shelf_1 parent="room_link" name="shelf_1"> -->
+  <!-- <xacro:shelf_1 parent="room_link" name="xacro:shelf_1"> -->
   <!--   <origin xyz="4.3223 -0.2415761 0.08515" rpy="0 0 -1.5756"/> -->
-  <!-- </shelf_1> -->
+  <!-- </xacro:shelf_1> -->
   <xacro:shelf_1 parent="room_link" name="shelf_left_center_front">
     <origin xyz="4.3223 -1.2415761 0.08515" rpy="0 0 -1.5756"/>
@@ -18,7 +18,7 @@
   </xacro:shelf_1>
   <!-- Center shelves -->
-  <!-- <shelf_2 parent="room_link" name="shelf_2"> -->
+  <!-- <xacro:shelf_2 parent="room_link" name="xacro:shelf_2"> -->
   <!--   <origin xyz="1.75 -1.45 0.08515" rpy="0 0 3.09652"/> -->
-  <!-- </shelf_2> -->
+  <!-- </xacro:shelf_2> -->
   <xacro:shelf_2 parent="room_link" name="shelf_center_front_middle">
     <origin xyz="0.75 -1.4 0.08515" rpy="0 0 3.09652"/>
@@ -65,5 +65,5 @@
     <origin xyz="-2.6 -3.0 0.08515" rpy="0 0 1.5756"/>
   </xacro:shelf_1>
-  <!-- Walls -->
+  <!-- xacro:walls -->
   <xacro:property name="wall_thickness" value="0.2" />
   <xacro:property name="wall_height" value="2.4" />

File: iai_refills_lab/urdf/dm_shelf_macros.urdf.xacro (robot description, xacro)
@@ -13,4 +13,9 @@
         </geometry>
       </collision>
+      <inertial>
+        <mass value="1."/>
+        <inertia ixx="0.1" ixy="0.1" ixz="0.1" iyy="0.1" iyz="0.1" izz="0.1"/>
+        <origin rpy="0 0 0" xyz="0.00312 0 0.11152"/>
+      </inertial>
     </link>
     <joint type="fixed" name="${name}_joint">
@@ -64,4 +69,9 @@
         </geometry>
       </collision>
+      <inertial>
+        <mass value="1."/>
+        <inertia ixx="0.1" ixy="0.1" ixz="0.1" iyy="0.1" iyz="0.1" izz="0.1"/>
+        <origin rpy="0 0 0" xyz="0.00312 0 0.11152"/>
+      </inertial>
     </link>
     <link name="${name}_left_support_link">
@@ -76,4 +86,9 @@
         </geometry>
       </collision>
+      <inertial>
+        <mass value="1."/>
+        <inertia ixx="0.1" ixy="0.1" ixz="0.1" iyy="0.1" iyz="0.1" izz="0.1"/>
+        <origin rpy="0 0 0" xyz="0.00312 0 0.11152"/>
+      </inertial>
     </link>
     <link name="${name}_right_support_link">
@@ -88,4 +103,9 @@
         </geometry>
       </collision>
+      <inertial>
+        <mass value="1."/>
+        <inertia ixx="0.1" ixy="0.1" ixz="0.1" iyy="0.1" iyz="0.1" izz="0.1"/>
+        <origin rpy="0 0 0" xyz="0.00312 0 0.11152"/>
+      </inertial>
     </link>
     <joint type="fixed" name="${name}_joint">
@@ -104,5 +124,5 @@
       <child link="${name}_left_support_link"/>
     </joint>
-    <shelf_divider parent="${name}_link" name="${name}" dist1="${dist1}" dist2="${dist2}" dist3="${dist3}" dist4="${dist4}" dist5="${dist5}" dist6="${dist6}" dist7="${dist7}" dist8="${dist8}" dist9="${dist9}" />
+    <xacro:shelf_divider parent="${name}_link" name="${name}" dist1="${dist1}" dist2="${dist2}" dist3="${dist3}" dist4="${dist4}" dist5="${dist5}" dist6="${dist6}" dist7="${dist7}" dist8="${dist8}" dist9="${dist9}" />
   </xacro:macro>
   <xacro:macro name="shelf_1" params="*origin parent name">
@@ -118,4 +138,9 @@
         </geometry>
       </collision>
+      <inertial>
+        <mass value="1."/>
+        <inertia ixx="0.1" ixy="0.1" ixz="0.1" iyy="0.1" iyz="0.1" izz="0.1"/>
+        <origin rpy="0 0 0" xyz="0.00312 0 0.11152"/>
+      </inertial>
     </link>
     <joint type="fixed" name="${name}_joint">
@@ -135,4 +160,9 @@
         </geometry>
       </collision>
+      <inertial>
+        <mass value="1."/>
+        <inertia ixx="0.1" ixy="0.1" ixz="0.1" iyy="0.1" iyz="0.1" izz="0.1"/>
+        <origin rpy="0 0 0" xyz="0.00312 0 0.11152"/>
+      </inertial>
     </link>
     <joint type="fixed" name="${name}_base_back_joint">
@@ -152,4 +182,9 @@
         </geometry>
       </collision>
+      <inertial>
+        <mass value="1."/>
+        <inertia ixx="0.1" ixy="0.1" ixz="0.1" iyy="0.1" iyz="0.1" izz="0.1"/>
+        <origin rpy="0 0 0" xyz="0.00312 0 0.11152"/>
+      </inertial>
     </link>
     <joint type="fixed" name="${name}_level_0_joint">
@@ -187,4 +222,9 @@
         </geometry>
       </collision>
+      <inertial>
+        <mass value="1."/>
+        <inertia ixx="0.1" ixy="0.1" ixz="0.1" iyy="0.1" iyz="0.1" izz="0.1"/>
+        <origin rpy="0 0 0" xyz="0.00312 0 0.11152"/>
+      </inertial>
     </link>
     <joint type="fixed" name="shelf_2_${name}_joint">
@@ -206,4 +246,9 @@
         </geometry>
       </collision>
+      <inertial>
+        <mass value="1."/>
+        <inertia ixx="0.1" ixy="0.1" ixz="0.1" iyy="0.1" iyz="0.1" izz="0.1"/>
+        <origin rpy="0 0 0" xyz="0.00312 0 0.11152"/>
+      </inertial>
     </link>
     <joint type="fixed" name="${name}_joint">
@@ -223,4 +268,9 @@
         </geometry>
       </collision>
+      <inertial>
+        <mass value="1."/>
+        <inertia ixx="0.1" ixy="0.1" ixz="0.1" iyy="0.1" iyz="0.1" izz="0.1"/>
+        <origin rpy="0 0 0" xyz="0.00312 0 0.11152"/>
+      </inertial>
     </link>
     <joint type="fixed" name="${name}_base_left_joint">
@@ -240,4 +290,9 @@
         </geometry>
       </collision>
+      <inertial>
+        <mass value="1."/>
+        <inertia ixx="0.1" ixy="0.1" ixz="0.1" iyy="0.1" iyz="0.1" izz="0.1"/>
+        <origin rpy="0 0 0" xyz="0.00312 0 0.11152"/>
+      </inertial>
     </link>
     <joint type="fixed" name="${name}_base_right_joint">
@@ -257,4 +312,9 @@
         </geometry>
       </collision>
+      <inertial>
+        <mass value="1."/>
+        <inertia ixx="0.1" ixy="0.1" ixz="0.1" iyy="0.1" iyz="0.1" izz="0.1"/>
+        <origin rpy="0 0 0" xyz="0.00312 0 0.11152"/>
+      </inertial>
     </link>
     <joint type="fixed" name="${name}_base_back_joint">
@@ -274,4 +334,9 @@
         </geometry>
       </collision>
+      <inertial>
+        <mass value="1."/>
+        <inertia ixx="0.1" ixy="0.1" ixz="0.1" iyy="0.1" iyz="0.1" izz="0.1"/>
+        <origin rpy="0 0 0" xyz="0.00312 0 0.11152"/>
+      </inertial>
     </link>
     <joint type="fixed" name="${name}_level_0_joint">
@@ -308,4 +373,9 @@
         </geometry>
       </collision>
+      <inertial>
+        <mass value="1."/>
+        <inertia ixx="0.1" ixy="0.1" ixz="0.1" iyy="0.1" iyz="0.1" izz="0.1"/>
+        <origin rpy="0 0 0" xyz="0.00312 0 0.11152"/>
+      </inertial>
     </link>
     <joint type="fixed" name="${name}_joint">
