Commit message: Revert "removing dm_room changes from this branch"
This reverts commit e8a1e49feb1e7d49fc62b17195623eb162bbbe27.

File: iai_refills_lab/urdf/dm_room.urdf.xacro (robot description, xacro)
@@ -3,9 +3,9 @@
   <xacro:include filename="$(find iai_refills_lab)/urdf/dm_shelf_macros.urdf.xacro"/>
   <xacro:include filename="$(find iai_refills_lab)/urdf/dm_shelves.urdf.xacro"/>
-   <!-- <link name="room_link"/> -->
+  <!-- <link name="room_link"/> -->
   <!-- Left side shelves -->
-  <!-- <xacro:shelf_1 parent="room_link" name="xacro:shelf_1"> -->
+  <!-- <shelf_1 parent="room_link" name="shelf_1"> -->
   <!--   <origin xyz="4.3223 -0.2415761 0.08515" rpy="0 0 -1.5756"/> -->
-  <!-- </xacro:shelf_1> -->
+  <!-- </shelf_1> -->
   <shelf_1 parent="room_link" name="shelf_left_center_front">
     <origin xyz="4.3223 -1.2415761 0.08515" rpy="0 0 -1.5756"/>
@@ -18,7 +18,7 @@
   </shelf_1>
   <!-- Center shelves -->
-  <!-- <xacro:shelf_2 parent="room_link" name="xacro:shelf_2"> -->
+  <!-- <shelf_2 parent="room_link" name="shelf_2"> -->
   <!--   <origin xyz="1.75 -1.45 0.08515" rpy="0 0 3.09652"/> -->
-  <!-- </xacro:shelf_2> -->
+  <!-- </shelf_2> -->
   <shelf_2 parent="room_link" name="shelf_center_front_middle">
     <origin xyz="0.75 -1.4 0.08515" rpy="0 0 3.09652"/>
@@ -65,5 +65,5 @@
     <origin xyz="-2.6 -3.0 0.08515" rpy="0 0 1.5756"/>
   </shelf_1>
-  <!-- xacro:walls -->
+  <!-- Walls -->
   <xacro:property name="wall_thickness" value="0.2" />
   <xacro:property name="wall_height" value="2.4" />

File: iai_refills_lab/urdf/dm_shelf_macros.urdf.xacro (robot description, xacro)
@@ -13,9 +13,4 @@
         </geometry>
       </collision>
-      <inertial>
-        <mass value="1."/>
-        <inertia ixx="0.1" ixy="0.1" ixz="0.1" iyy="0.1" iyz="0.1" izz="0.1"/>
-        <origin rpy="0 0 0" xyz="0.00312 0 0.11152"/>
-      </inertial>
     </link>
     <joint type="fixed" name="${name}_joint">
@@ -69,9 +64,4 @@
         </geometry>
       </collision>
-      <inertial>
-        <mass value="1."/>
-        <inertia ixx="0.1" ixy="0.1" ixz="0.1" iyy="0.1" iyz="0.1" izz="0.1"/>
-        <origin rpy="0 0 0" xyz="0.00312 0 0.11152"/>
-      </inertial>
     </link>
     <link name="${name}_left_support_link">
@@ -86,9 +76,4 @@
         </geometry>
       </collision>
-      <inertial>
-        <mass value="1."/>
-        <inertia ixx="0.1" ixy="0.1" ixz="0.1" iyy="0.1" iyz="0.1" izz="0.1"/>
-        <origin rpy="0 0 0" xyz="0.00312 0 0.11152"/>
-      </inertial>
     </link>
     <link name="${name}_right_support_link">
@@ -103,9 +88,4 @@
         </geometry>
       </collision>
-      <inertial>
-        <mass value="1."/>
-        <inertia ixx="0.1" ixy="0.1" ixz="0.1" iyy="0.1" iyz="0.1" izz="0.1"/>
-        <origin rpy="0 0 0" xyz="0.00312 0 0.11152"/>
-      </inertial>
     </link>
     <joint type="fixed" name="${name}_joint">
@@ -124,5 +104,5 @@
       <child link="${name}_left_support_link"/>
     </joint>
-    <xacro:shelf_divider parent="${name}_link" name="${name}" dist1="${dist1}" dist2="${dist2}" dist3="${dist3}" dist4="${dist4}" dist5="${dist5}" dist6="${dist6}" dist7="${dist7}" dist8="${dist8}" dist9="${dist9}" />
+    <shelf_divider parent="${name}_link" name="${name}" dist1="${dist1}" dist2="${dist2}" dist3="${dist3}" dist4="${dist4}" dist5="${dist5}" dist6="${dist6}" dist7="${dist7}" dist8="${dist8}" dist9="${dist9}" />
   </xacro:macro>
   <xacro:macro name="shelf_1" params="*origin parent name">
@@ -138,9 +118,4 @@
         </geometry>
       </collision>
-      <inertial>
-        <mass value="1."/>
-        <inertia ixx="0.1" ixy="0.1" ixz="0.1" iyy="0.1" iyz="0.1" izz="0.1"/>
-        <origin rpy="0 0 0" xyz="0.00312 0 0.11152"/>
-      </inertial>
     </link>
     <joint type="fixed" name="${name}_joint">
@@ -160,9 +135,4 @@
         </geometry>
       </collision>
-      <inertial>
-        <mass value="1."/>
-        <inertia ixx="0.1" ixy="0.1" ixz="0.1" iyy="0.1" iyz="0.1" izz="0.1"/>
-        <origin rpy="0 0 0" xyz="0.00312 0 0.11152"/>
-      </inertial>
     </link>
     <joint type="fixed" name="${name}_base_back_joint">
@@ -182,9 +152,4 @@
         </geometry>
       </collision>
-      <inertial>
-        <mass value="1."/>
-        <inertia ixx="0.1" ixy="0.1" ixz="0.1" iyy="0.1" iyz="0.1" izz="0.1"/>
-        <origin rpy="0 0 0" xyz="0.00312 0 0.11152"/>
-      </inertial>
     </link>
     <joint type="fixed" name="${name}_level_0_joint">
@@ -222,9 +187,4 @@
         </geometry>
       </collision>
-      <inertial>
-        <mass value="1."/>
-        <inertia ixx="0.1" ixy="0.1" ixz="0.1" iyy="0.1" iyz="0.1" izz="0.1"/>
-        <origin rpy="0 0 0" xyz="0.00312 0 0.11152"/>
-      </inertial>
     </link>
     <joint type="fixed" name="shelf_2_${name}_joint">
@@ -246,9 +206,4 @@
         </geometry>
       </collision>
-      <inertial>
-        <mass value="1."/>
-        <inertia ixx="0.1" ixy="0.1" ixz="0.1" iyy="0.1" iyz="0.1" izz="0.1"/>
-        <origin rpy="0 0 0" xyz="0.00312 0 0.11152"/>
-      </inertial>
     </link>
     <joint type="fixed" name="${name}_joint">
@@ -268,9 +223,4 @@
         </geometry>
       </collision>
-      <inertial>
-        <mass value="1."/>
-        <inertia ixx="0.1" ixy="0.1" ixz="0.1" iyy="0.1" iyz="0.1" izz="0.1"/>
-        <origin rpy="0 0 0" xyz="0.00312 0 0.11152"/>
-      </inertial>
     </link>
     <joint type="fixed" name="${name}_base_left_joint">
@@ -290,9 +240,4 @@
         </geometry>
       </collision>
-      <inertial>
-        <mass value="1."/>
-        <inertia ixx="0.1" ixy="0.1" ixz="0.1" iyy="0.1" iyz="0.1" izz="0.1"/>
-        <origin rpy="0 0 0" xyz="0.00312 0 0.11152"/>
-      </inertial>
     </link>
     <joint type="fixed" name="${name}_base_right_joint">
@@ -312,9 +257,4 @@
         </geometry>
       </collision>
-      <inertial>
-        <mass value="1."/>
-        <inertia ixx="0.1" ixy="0.1" ixz="0.1" iyy="0.1" iyz="0.1" izz="0.1"/>
-        <origin rpy="0 0 0" xyz="0.00312 0 0.11152"/>
-      </inertial>
     </link>
     <joint type="fixed" name="${name}_base_back_joint">
@@ -334,9 +274,4 @@
         </geometry>
       </collision>
-      <inertial>
-        <mass value="1."/>
-        <inertia ixx="0.1" ixy="0.1" ixz="0.1" iyy="0.1" iyz="0.1" izz="0.1"/>
-        <origin rpy="0 0 0" xyz="0.00312 0 0.11152"/>
-      </inertial>
     </link>
     <joint type="fixed" name="${name}_level_0_joint">
@@ -373,9 +308,4 @@
         </geometry>
       </collision>
-      <inertial>
-        <mass value="1."/>
-        <inertia ixx="0.1" ixy="0.1" ixz="0.1" iyy="0.1" iyz="0.1" izz="0.1"/>
-        <origin rpy="0 0 0" xyz="0.00312 0 0.11152"/>
-      </inertial>
     </link>
     <joint type="fixed" name="${name}_joint">
