Commit message: Lots of other cabinets and tap and sink were added.

File: iai_kimchen/urdf/kitchen.urdf (robot description, URDF)
Before this commit: robot kimchen, 20 links, 19 joints
Links:
- added link cabinet10; collision mesh filename=package://iai_kimchen/meshes/cabinet10/IAIKitchenCabinet9W4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; visual mesh filename=package://iai_kimchen/meshes/cabinet10/IAIKitchenCabinet9W4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
- added link cabinet10_drawer_bottom; collision mesh filename=package://iai_kimchen/meshes/cabinet10/IAIKitchenDrawerW40H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; visual mesh filename=package://iai_kimchen/meshes/cabinet10/IAIKitchenDrawerW40H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
- added link cabinet10_drawer_middle; collision mesh filename=package://iai_kimchen/meshes/cabinet10/IAIKitchenDrawerW40H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; visual mesh filename=package://iai_kimchen/meshes/cabinet10/IAIKitchenDrawerW40H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
- added link cabinet10_drawer_top; collision mesh filename=package://iai_kimchen/meshes/cabinet10/IAIKitchenDrawerW40H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; visual mesh filename=package://iai_kimchen/meshes/cabinet10/IAIKitchenDrawerW40H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
- added link cabinet11; collision mesh filename=package://iai_kimchen/meshes/cabinet11/IAIKitchenCabinet11W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; visual mesh filename=package://iai_kimchen/meshes/cabinet11/IAIKitchenCabinet11W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
- added link cabinet11_drawer_bottom; collision mesh filename=package://iai_kimchen/meshes/cabinet11/IAIKitchenDrawerW90H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; visual mesh filename=package://iai_kimchen/meshes/cabinet11/IAIKitchenDrawerW90H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
- added link cabinet11_drawer_middle; collision mesh filename=package://iai_kimchen/meshes/cabinet11/IAIKitchenDrawerW90H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; visual mesh filename=package://iai_kimchen/meshes/cabinet11/IAIKitchenDrawerW90H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
- added link cabinet11_drawer_top; collision mesh filename=package://iai_kimchen/meshes/cabinet11/IAIKitchenDrawerW90H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; visual mesh filename=package://iai_kimchen/meshes/cabinet11/IAIKitchenDrawerW90H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
- added link cabinet5_drawer_bottom; collision mesh filename=package://iai_kimchen/meshes/cabinet05/IAIKitchenDrawerW60H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; visual mesh filename=package://iai_kimchen/meshes/cabinet05/IAIKitchenDrawerW60H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
- added link cabinet5_drawer_middle; collision mesh filename=package://iai_kimchen/meshes/cabinet05/IAIKitchenDrawerW60H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; visual mesh filename=package://iai_kimchen/meshes/cabinet05/IAIKitchenDrawerW60H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
- added link cabinet5_drawer_top; collision mesh filename=package://iai_kimchen/meshes/cabinet05/IAIKitchenDrawerW60H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; visual mesh filename=package://iai_kimchen/meshes/cabinet05/IAIKitchenDrawerW60H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
- added link cabinet6; collision mesh filename=package://iai_kimchen/meshes/cabinet06/IAIKitchenCabinet6W4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; visual mesh filename=package://iai_kimchen/meshes/cabinet06/IAIKitchenCabinet6W4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
- added link cabinet6_drawer_bottom; collision mesh filename=package://iai_kimchen/meshes/cabinet06/IAIKitchenDrawerW40H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; visual mesh filename=package://iai_kimchen/meshes/cabinet06/IAIKitchenDrawerW40H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
- added link cabinet6_drawer_middle; collision mesh filename=package://iai_kimchen/meshes/cabinet06/IAIKitchenDrawerW40H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; visual mesh filename=package://iai_kimchen/meshes/cabinet06/IAIKitchenDrawerW40H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
- added link cabinet6_drawer_top; collision mesh filename=package://iai_kimchen/meshes/cabinet06/IAIKitchenDrawerW40H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; visual mesh filename=package://iai_kimchen/meshes/cabinet06/IAIKitchenDrawerW40H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
- added link cabinet8; collision mesh filename=package://iai_kimchen/meshes/cabinet08/IAIKitchenCabinet8W6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; visual mesh filename=package://iai_kimchen/meshes/cabinet08/IAIKitchenCabinet8W6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
- added link cabinet8_drawer_bottom; collision mesh filename=package://iai_kimchen/meshes/cabinet08/IAIKitchenDrawerW60H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; visual mesh filename=package://iai_kimchen/meshes/cabinet08/IAIKitchenDrawerW60H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
- added link cabinet8_drawer_middle; collision mesh filename=package://iai_kimchen/meshes/cabinet08/IAIKitchenDrawerW56H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; visual mesh filename=package://iai_kimchen/meshes/cabinet08/IAIKitchenDrawerW56H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
- added link cabinet9; collision mesh filename=package://iai_kimchen/meshes/cabinet09/IAIKitchenCabinet9W6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; visual mesh filename=package://iai_kimchen/meshes/cabinet09/IAIKitchenCabinet9W6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
- added link cabinet9_drawer_bottom; collision mesh filename=package://iai_kimchen/meshes/cabinet09/IAIKitchenDrawerW60H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; visual mesh filename=package://iai_kimchen/meshes/cabinet09/IAIKitchenDrawerW60H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
- added link cabinet9_drawer_middle; collision mesh filename=package://iai_kimchen/meshes/cabinet09/IAIKitchenDrawerW60H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; visual mesh filename=package://iai_kimchen/meshes/cabinet09/IAIKitchenDrawerW60H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
- added link cabinet9_drawer_top; collision mesh filename=package://iai_kimchen/meshes/cabinet09/IAIKitchenDrawerW60H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; visual mesh filename=package://iai_kimchen/meshes/cabinet09/IAIKitchenDrawerW60H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
- added link cooktop; collision mesh filename=package://iai_kimchen/meshes/cooktop/IAIKitchenCookTop.stl; visual mesh filename=package://iai_kimchen/meshes/cooktop/IAIKitchenCookTop.dae
- added link side_A
- added link side_B
- added link sink; collision mesh filename=package://iai_kimchen/meshes/sink/IAIKitchenSink.stl; visual mesh filename=package://iai_kimchen/meshes/sink/IAIKitchenSink.dae
- added link tap; collision mesh filename=package://iai_kimchen/meshes/tap/IAIKitchenWaterTap.stl; visual mesh filename=package://iai_kimchen/meshes/tap/IAIKitchenWaterTap.dae
Joints:
- added joint cabinet10_drawer_bottom_joint: type prismatic, parent cabinet10, child cabinet10_drawer_bottom, origin xyz=0.03 0.0 -0.279, axis 1 0 0, limit lower=0.0 upper=0.5 effort=1000.0 velocity=0.5
- added joint cabinet10_drawer_middle_joint: type prismatic, parent cabinet10, child cabinet10_drawer_middle, origin xyz=0.031 0.0 0.104, axis 1 0 0, limit lower=0.0 upper=0.5 effort=1000.0 velocity=0.5
- added joint cabinet10_drawer_top_joint: type prismatic, parent cabinet10, child cabinet10_drawer_top, origin xyz=0.033 0.0 0.326, axis 1 0 0, limit lower=0.0 upper=0.5 effort=1000.0 velocity=0.5
- added joint cabinet10_joint: type fixed, parent side_B, child cabinet10, origin xyz=0.334 2.207 0.394
- added joint cabinet11_drawer_bottom_joint: type prismatic, parent cabinet11, child cabinet11_drawer_bottom, origin xyz=0.045 0.0 -0.286, axis 1 0 0, limit lower=0.0 upper=0.45 effort=1000.0 velocity=0.5
- added joint cabinet11_drawer_middle_joint: type prismatic, parent cabinet11, child cabinet11_drawer_middle, origin xyz=0.027 0.0 0.106, axis 1 0 0, limit lower=0.0 upper=0.45 effort=1000.0 velocity=0.5
- added joint cabinet11_drawer_top_joint: type prismatic, parent cabinet11, child cabinet11_drawer_top, origin xyz=0.03 0.0 0.326, axis 1 0 0, limit lower=0.0 upper=0.45 effort=1000.0 velocity=0.5
- added joint cabinet11_joint: type fixed, parent side_B, child cabinet11, origin xyz=0.334 2.86 0.394
- added joint cabinet5_drawer_bottom_joint: type prismatic, parent cabinet5, child cabinet5_drawer_bottom, origin xyz=0.037 0.0 -0.28, axis 1 0 0, limit lower=0.0 upper=0.45 effort=1000.0 velocity=0.5
- added joint cabinet5_drawer_middle_joint: type prismatic, parent cabinet5, child cabinet5_drawer_middle, origin xyz=0.027 0.0 0.107, axis 1 0 0, limit lower=0.0 upper=0.45 effort=1000.0 velocity=0.5
- added joint cabinet5_drawer_top_joint: type prismatic, parent cabinet5, child cabinet5_drawer_top, origin xyz=0.03 0.0 0.327, axis 1 0 0, limit lower=0.0 upper=0.45 effort=1000.0 velocity=0.5
- added joint cabinet6_drawer_bottom_joint: type prismatic, parent cabinet6, child cabinet6_drawer_bottom, origin xyz=0.047 0.0 -0.28, axis 1 0 0, limit lower=0.0 upper=0.45 effort=1000.0 velocity=0.5
- added joint cabinet6_drawer_middle_joint: type prismatic, parent cabinet6, child cabinet6_drawer_middle, origin xyz=0.03 0.0 0.105, axis 1 0 0, limit lower=0.0 upper=0.45 effort=1000.0 velocity=0.5
- added joint cabinet6_drawer_top_joint: type prismatic, parent cabinet6, child cabinet6_drawer_top, origin xyz=0.033 -0.0125 0.328, axis 1 0 0, limit lower=0.0 upper=0.45 effort=1000.0 velocity=0.5
- added joint cabinet6_joint: type fixed, parent side_A, child cabinet6, origin xyz=-0.121 2.127 0.4
- added joint cabinet8_drawer_bottom_joint: type prismatic, parent cabinet8, child cabinet8_drawer_bottom, origin xyz=0.014 0.0 -0.412, axis 1 0 0, limit lower=0.0 upper=0.45 effort=1000.0 velocity=0.5
- added joint cabinet8_drawer_middle_joint: type prismatic, parent cabinet8, child cabinet8_drawer_middle, origin xyz=-0.05 0.0 -0.047, axis 1 0 0, limit lower=0.0 upper=0.45 effort=1000.0 velocity=0.5
- added joint cabinet8_joint: type fixed, parent side_B, child cabinet8, origin xyz=0.357 1.102 0.524
- added joint cabinet9_drawer_bottom_joint: type prismatic, parent cabinet9, child cabinet9_drawer_bottom, origin xyz=0.036 0.0 -0.281, axis 1 0 0, limit lower=0.0 upper=0.5 effort=1000.0 velocity=0.5
- added joint cabinet9_drawer_middle_joint: type prismatic, parent cabinet9, child cabinet9_drawer_middle, origin xyz=0.027 0.0 0.106, axis 1 0 0, limit lower=0.0 upper=0.5 effort=1000.0 velocity=0.5
- added joint cabinet9_drawer_top_joint: type prismatic, parent cabinet9, child cabinet9_drawer_top, origin xyz=0.03 0.0 0.327, axis 1 0 0, limit lower=0.0 upper=0.5 effort=1000.0 velocity=0.5
- added joint cabinet9_joint: type fixed, parent side_B, child cabinet9, origin xyz=0.334 1.705 0.394
- added joint cooktop_joint: type fixed, parent side_B, child cooktop, origin xyz=0.26 2.86 0.832
- added joint frame_A_joint: type fixed, parent kitchen_root, child side_A, origin xyz=0.5 0.5 0
- added joint frame_B_joint: type fixed, parent kitchen_root, child side_B, origin xyz=3 3 0.0 rpy=0 0 3.14
- added joint sink_joint: type fixed, parent side_B, child sink, origin xyz=0.328 1.1 0.769
- added joint tap_joint: type fixed, parent side_B, child tap, origin xyz=0.1 1.1 0.935
- joint cabinet1_joint: origin xyz=0.5 0.5 1.07 -> xyz=0.01 0.01 1.07; parent kitchen_root -> side_A
- joint cabinet2_joint: origin xyz=0.33 1 0.98 -> xyz=-0.163 0.51 0.975; parent kitchen_root -> side_A
- joint cabinet3_joint: origin xyz=0.22 1.515 1.07 -> xyz=-0.273 1.022 1.07; parent kitchen_root -> side_A
- joint cabinet4_door_bottom_bottom_joint: mimic (none) -> joint=cabinet4_door_top_top_joint multiplier=1.2
- joint cabinet4_door_top_top_joint: limit lower=-1.5708 upper=0.0 effort=1000.0 velocity=1.5708 -> lower=-2.0 upper=0.0 effort=1000.0 velocity=1.5708
- joint cabinet4_joint: origin xyz=0.32 2.32 1.72 -> xyz=-0.175 1.825 1.72; parent kitchen_root -> side_A
- joint cabinet5_joint: origin xyz=0.37 2.12 0.4 -> xyz=-0.121 1.625 0.4; parent kitchen_root -> side_A
- joint cabinet7_door_bottom_left_joint: origin xyz=0.37 -0.3 -0.45 -> xyz=0.372 0 -0.45
- joint cabinet7_joint: origin xyz=2 2 0.47 rpy=0 0 3.15 -> xyz=0.2 0.5 0.47; parent kitchen_root -> side_B
- joint island_joint: origin xyz=2.1 0.7 0.81 rpy=0 0 3.15 -> xyz=0.13 1.8 0.808; parent kitchen_root -> side_B

Commit message: some handles were added.

File: iai_kimchen/urdf/kitchen.urdf (robot description, URDF)
Before this commit: robot kimchen, 47 links, 46 joints
Links:
- removed link cabinet1_drawer_big
- removed link cabinet1_drawer_small
- added link cabinet1_drawer_bottom; collision mesh filename=package://iai_kimchen/meshes/cabinet01/IAIDrawerW60H53.stl; visual mesh filename=package://iai_kimchen/meshes/cabinet01/IAIDrawerW60H53.dae
- added link cabinet1_drawer_middle; collision mesh filename=package://iai_kimchen/meshes/cabinet01/IAIDrawerW60H26.stl; visual mesh filename=package://iai_kimchen/meshes/cabinet01/IAIDrawerW60H26.dae
- added link handle_cab1_drawer_bottom; collision mesh filename=package://iai_kimchen/meshes/handles/handle_horizontal.stl; visual mesh filename=package://iai_kimchen/meshes/handles/handle_horizontal.dae
- added link handle_cab1_drawer_mid; collision mesh filename=package://iai_kimchen/meshes/handles/handle_horizontal.stl; visual mesh filename=package://iai_kimchen/meshes/handles/handle_horizontal.dae
- added link handle_cab2_door; collision mesh filename=package://iai_kimchen/meshes/handles/handle_horizontal.stl; visual mesh filename=package://iai_kimchen/meshes/handles/handle_horizontal.dae
- link cabinet1_handle_top: geometry collision mesh filename=package://iai_kimchen/meshes/handles/handle_horizontal.stl; visual mesh filename=package://iai_kimchen/meshes/handles/handle_horizontal.dae
Joints:
- removed joint cabinet1_drawer_big_joint
- removed joint cabinet1_drawer_small_joint
- added joint cabinet1_drawer_bottom_joint: type prismatic, parent cabinet1, child cabinet1_drawer_bottom, origin xyz=-0.094 0.0 -0.95, axis 1 0 0, limit lower=0.0 upper=0.5 effort=1000.0 velocity=0.5
- added joint cabinet1_drawer_middle_joint: type prismatic, parent cabinet1, child cabinet1_drawer_middle, origin xyz=-0.117 0.0 -0.43, axis 1 0 0, limit lower=0.0 upper=0.5 effort=1000.0 velocity=0.5
- added joint handle_cab1_drawer_bottom_joint: type fixed, parent cabinet1_drawer_bottom, child handle_cab1_drawer_bottom, origin xyz=0.21 0.0 0.35
- added joint handle_cab1_drawer_mid_joint: type fixed, parent cabinet1_drawer_middle, child handle_cab1_drawer_mid, origin xyz=0.232 0.0 0.11
- added joint handle_cab2_drawer_bottom_joint: type fixed, parent cabinet2_door_left, child handle_cab2_door, origin xyz=0.012 0.29 0.05
- joint cabinet1_door_top_left_joint: origin xyz=0.1 -0.3 0.32 -> xyz=0.103 -0.3 0.32
- joint cabinet8_drawer_bottom_joint: origin xyz=0.014 0.0 -0.412 -> xyz=0.114 0.0 0.105
- joint cabinet8_drawer_middle_joint: origin xyz=-0.05 0.0 -0.047 -> xyz=0.05 0.0 0.48
- joint cabinet8_joint: origin xyz=0.357 1.102 0.524 -> xyz=0.256 1.102 0.006

Commit message: All handles are added.

File: iai_kimchen/urdf/kitchen.urdf (robot description, URDF)
Before this commit: robot kimchen, 50 links, 49 joints
Links:
- removed link cabinet3_door_bottom_left
- removed link cabinet3_door_top_left
- removed link cabinet4_door_bottom_bottom
- removed link cabinet4_door_top_top
- added link cabinet3_door_bottom_right; collision mesh filename=package://iai_kimchen/meshes/cabinet03/IAIDoorW60H80.stl; visual mesh filename=package://iai_kimchen/meshes/cabinet03/IAIDoorW60H80.dae
- added link cabinet3_door_top_right; collision mesh filename=package://iai_kimchen/meshes/cabinet03/IAIDoorW60H133.stl; visual mesh filename=package://iai_kimchen/meshes/cabinet03/IAIDoorW60H133.dae
- added link cabinet4_door_bottom; collision mesh filename=package://iai_kimchen/meshes/cabinet04/IAIDoor2W100H40.stl; visual mesh filename=package://iai_kimchen/meshes/cabinet04/IAIDoor2W100H40.dae
- added link cabinet4_door_top; collision mesh filename=package://iai_kimchen/meshes/cabinet04/IAIDoor1W100H40.stl; visual mesh filename=package://iai_kimchen/meshes/cabinet04/IAIDoor1W100H40.dae
- added link handle_cab10_b; collision mesh filename=package://iai_kimchen/meshes/handles/handle_horizontal.stl; visual mesh filename=package://iai_kimchen/meshes/handles/handle_horizontal.dae
- added link handle_cab10_m; collision mesh filename=package://iai_kimchen/meshes/handles/handle_horizontal.stl; visual mesh filename=package://iai_kimchen/meshes/handles/handle_horizontal.dae
- added link handle_cab10_t; collision mesh filename=package://iai_kimchen/meshes/handles/handle_horizontal.stl; visual mesh filename=package://iai_kimchen/meshes/handles/handle_horizontal.dae
- added link handle_cab11_b; collision mesh filename=package://iai_kimchen/meshes/handles/handle_horizontal.stl; visual mesh filename=package://iai_kimchen/meshes/handles/handle_horizontal.dae
- added link handle_cab11_m; collision mesh filename=package://iai_kimchen/meshes/handles/handle_horizontal.stl; visual mesh filename=package://iai_kimchen/meshes/handles/handle_horizontal.dae
- added link handle_cab11_t; collision mesh filename=package://iai_kimchen/meshes/handles/handle_horizontal.stl; visual mesh filename=package://iai_kimchen/meshes/handles/handle_horizontal.dae
- added link handle_cab3_door_bottom; collision mesh filename=package://iai_kimchen/meshes/handles/handle_horizontal.stl; visual mesh filename=package://iai_kimchen/meshes/handles/handle_horizontal.dae
- added link handle_cab3_door_top; collision mesh filename=package://iai_kimchen/meshes/handles/handle_horizontal.stl; visual mesh filename=package://iai_kimchen/meshes/handles/handle_horizontal.dae
- added link handle_cab4_door_bottom; collision mesh filename=package://iai_kimchen/meshes/handles/handle_horizontal.stl; visual mesh filename=package://iai_kimchen/meshes/handles/handle_horizontal.dae
- added link handle_cab5_b; collision mesh filename=package://iai_kimchen/meshes/handles/handle_horizontal.stl; visual mesh filename=package://iai_kimchen/meshes/handles/handle_horizontal.dae
- added link handle_cab5_m; collision mesh filename=package://iai_kimchen/meshes/handles/handle_horizontal.stl; visual mesh filename=package://iai_kimchen/meshes/handles/handle_horizontal.dae
- added link handle_cab5_t; collision mesh filename=package://iai_kimchen/meshes/handles/handle_horizontal.stl; visual mesh filename=package://iai_kimchen/meshes/handles/handle_horizontal.dae
- added link handle_cab6_b; collision mesh filename=package://iai_kimchen/meshes/handles/handle_horizontal.stl; visual mesh filename=package://iai_kimchen/meshes/handles/handle_horizontal.dae
- added link handle_cab6_m; collision mesh filename=package://iai_kimchen/meshes/handles/handle_horizontal.stl; visual mesh filename=package://iai_kimchen/meshes/handles/handle_horizontal.dae
- added link handle_cab6_t; collision mesh filename=package://iai_kimchen/meshes/handles/handle_horizontal.stl; visual mesh filename=package://iai_kimchen/meshes/handles/handle_horizontal.dae
- added link handle_cab7; collision mesh filename=package://iai_kimchen/meshes/handles/handle_horizontal.stl; visual mesh filename=package://iai_kimchen/meshes/handles/handle_horizontal.dae
- added link handle_cab8; collision mesh filename=package://iai_kimchen/meshes/handles/handle_horizontal.stl; visual mesh filename=package://iai_kimchen/meshes/handles/handle_horizontal.dae
- added link handle_cab9_b; collision mesh filename=package://iai_kimchen/meshes/handles/handle_horizontal.stl; visual mesh filename=package://iai_kimchen/meshes/handles/handle_horizontal.dae
- added link handle_cab9_m; collision mesh filename=package://iai_kimchen/meshes/handles/handle_horizontal.stl; visual mesh filename=package://iai_kimchen/meshes/handles/handle_horizontal.dae
- added link handle_cab9_t; collision mesh filename=package://iai_kimchen/meshes/handles/handle_horizontal.stl; visual mesh filename=package://iai_kimchen/meshes/handles/handle_horizontal.dae
Joints:
- removed joint cabinet3_door_bottom_left_joint
- removed joint cabinet3_door_top_left_joint
- added joint cabinet3_door_bottom_right_joint: type revolute, parent cabinet3, child cabinet3_door_bottom_right, origin xyz=0.39 0.3 -0.5, axis 0 0 -1, limit lower=-1.5708 upper=0.0 effort=1000.0 velocity=1.5708
- added joint cabinet3_door_top_right_joint: type revolute, parent cabinet3, child cabinet3_door_top_right, origin xyz=0.39 0.3 0.5, axis 0 0 -1, limit lower=-1.5708 upper=0.0 effort=1000.0 velocity=1.5708
- added joint handle_cab10_bott_joint: type fixed, parent cabinet10_drawer_bottom, child handle_cab10_b, origin xyz=0.217 0 0.245
- added joint handle_cab10_mid_joint: type fixed, parent cabinet10_drawer_middle, child handle_cab10_m, origin xyz=0.217 0 0.13
- added joint handle_cab10_top_joint: type fixed, parent cabinet10_drawer_top, child handle_cab10_t, origin xyz=0.215 0 0.05
- added joint handle_cab11_bott_joint: type fixed, parent cabinet11_drawer_bottom, child handle_cab11_b, origin xyz=0.199 0 0.245
- added joint handle_cab11_mid_joint: type fixed, parent cabinet11_drawer_middle, child handle_cab11_m, origin xyz=0.217 0 0.13
- added joint handle_cab11_top_joint: type fixed, parent cabinet11_drawer_top, child handle_cab11_t, origin xyz=0.215 0 0.05
- added joint handle_cab3_door_bottom_joint: type fixed, parent cabinet3_door_bottom_right, child handle_cab3_door_bottom, origin xyz=0.01 -0.45 0.1
- added joint handle_cab3_door_top_joint: type fixed, parent cabinet3_door_top_right, child handle_cab3_door_top, origin xyz=0.01 -0.45 -0.65
- added joint handle_cab4_door_bottom_joint: type fixed, parent cabinet4_door_bottom, child handle_cab4_door_bottom, origin xyz=0.027 0 -0.35
- added joint handle_cab5_bott_joint: type fixed, parent cabinet5_drawer_bottom, child handle_cab5_b, origin xyz=0.207 0 0.245
- added joint handle_cab5_mid_joint: type fixed, parent cabinet5_drawer_middle, child handle_cab5_m, origin xyz=0.217 0 0.13
- added joint handle_cab5_top_joint: type fixed, parent cabinet5_drawer_top, child handle_cab5_t, origin xyz=0.217 0 0.05
- added joint handle_cab6_bott_joint: type fixed, parent cabinet6_drawer_bottom, child handle_cab6_b, origin xyz=0.199 0 0.245
- added joint handle_cab6_mid_joint: type fixed, parent cabinet6_drawer_middle, child handle_cab6_m, origin xyz=0.217 0 0.13
- added joint handle_cab6_top_joint: type fixed, parent cabinet6_drawer_top, child handle_cab6_t, origin xyz=0.21 0 0.05
- added joint handle_cab7_top_joint: type fixed, parent cabinet7, child handle_cab7, origin xyz=0.38 0 0.29
- added joint handle_cab8_top_joint: type fixed, parent cabinet8_drawer_bottom, child handle_cab8, origin xyz=0.21 0 0.65
- added joint handle_cab9_bott_joint: type fixed, parent cabinet9_drawer_bottom, child handle_cab9_b, origin xyz=0.213 0 0.245
- added joint handle_cab9_mid_joint: type fixed, parent cabinet9_drawer_middle, child handle_cab9_m, origin xyz=0.217 0 0.13
- added joint handle_cab9_top_joint: type fixed, parent cabinet9_drawer_top, child handle_cab9_t, origin xyz=0.217 0 0.05
- joint cabinet4_door_bottom_bottom_joint: child cabinet4_door_bottom_bottom -> cabinet4_door_bottom; parent cabinet4_door_top_top -> cabinet4_door_top
- joint cabinet4_door_top_top_joint: child cabinet4_door_top_top -> cabinet4_door_top

Commit message: Sockets and countertop were added.

File: iai_kimchen/urdf/kitchen.urdf (robot description, URDF)
Before this commit: robot kimchen, 70 links, 69 joints
Links:
- added link countertop; collision mesh filename=package://iai_kimchen/meshes/countertop/IAIKitchenPartW102H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; visual mesh filename=package://iai_kimchen/meshes/countertop/IAIKitchenPartW102H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
- added link sa; collision mesh filename=package://iai_kimchen/meshes/floor_socket_side_a/IAIKitchen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; visual mesh filename=package://iai_kimchen/meshes/floor_socket_side_a/IAIKitchen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
- added link sb; collision mesh filename=package://iai_kimchen/meshes/floor_socket_side_b/IAIKitchen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; visual mesh filename=package://iai_kimchen/meshes/floor_socket_side_b/IAIKitchen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
Joints:
- added joint countertop_joint: type fixed, parent cabinet5, child countertop, origin xyz=-0.027 0.21 0.423
- added joint socket_a_joint: type fixed, parent side_A, child sa, origin xyz=0.095 1.02 -0.03
- added joint socket_b_joint: type fixed, parent side_B, child sb, origin xyz=0.552 1.755 -0.045
- joint cabinet2_door_left_joint: origin xyz=0.27 -0.19 0.0 -> xyz=0.277 -0.19 0.0
- joint frame_A_joint: origin xyz=0.5 0.5 0 -> xyz=0.5 0.5 0.080
- joint frame_B_joint: origin xyz=3 3 0.0 rpy=0 0 3.14 -> xyz=3 3 0.092 rpy=0 0 3.14
- joint handle_cab7_top_joint: origin xyz=0.38 0 0.29 -> xyz=0.01 0 0.74; parent cabinet7 -> cabinet7_door_bottom_left
