Commit message: side panels were added.

File: iai_kimchen/urdf/kitchen.urdf (robot description, URDF)
Before this commit: robot kimchen, 73 links, 72 joints
Links:
- added link island_back; collision mesh filename=package://iai_kimchen/meshes/IAIKitchenPartW314H90/IAIKitch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; visual mesh filename=package://iai_kimchen/meshes/IAIKitchenPartW314H90/IAIKitch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
- added link island_waterfall_left; collision mesh filename=package://iai_kimchen/meshes/IAIKitchenVisiblePartIslandUnd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; visual mesh filename=package://iai_kimchen/meshes/IAIKitchenVisiblePartIslandUnd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
- added link island_waterfall_right; collision mesh filename=package://iai_kimchen/meshes/IAIKitchenVisiblePartIslandUnd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; visual mesh filename=package://iai_kimchen/meshes/IAIKitchenVisiblePartIslandUnd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
- added link side_A_left; collision mesh filename=package://iai_kimchen/meshes/IAIKitchenPartW58H223/IAIKitch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; visual mesh filename=package://iai_kimchen/meshes/IAIKitchenPartW58H223/IAIKitch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
- added link side_A_rb; collision mesh filename=package://iai_kimchen/meshes/IAIKitchenVisiblePartUnderSide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; visual mesh filename=package://iai_kimchen/meshes/IAIKitchenVisiblePartUnderSide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
- added link side_A_rt; collision mesh filename=package://iai_kimchen/meshes/IAIKitchenVisiblePartUpperside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; visual mesh filename=package://iai_kimchen/meshes/IAIKitchenVisiblePartUpperside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
Joints:
- added joint island_back_joint: type fixed, parent side_B, child island_back, origin xyz=-0.026 1.754 0.353 rpy=0 1.57 0
- added joint island_waterfall_left_joint: type fixed, parent side_B, child island_waterfall_left, origin xyz=0.285 0.191 0.354 rpy=1.57 0 1.57
- added joint island_waterfall_right_joint: type fixed, parent side_B, child island_waterfall_right, origin xyz=0.285 3.315 0.354 rpy=1.57 0 1.57
- added joint side_A_left_joint: type fixed, parent side_A, child side_A_left, origin xyz=-0.16 -0.296 1.030 rpy=0 0 1.57
- added joint side_A_right_bott_joint: type fixed, parent side_A, child side_A_rb, origin xyz=-0.159 2.338 0.361 rpy=1.57 0 1.57
- added joint side_A_right_top_joint: type fixed, parent side_A, child side_A_rt, origin xyz=-0.262 2.336 1.74 rpy=0 0 1.57
- joint cabinet10_joint: origin xyz=0.334 2.207 0.394 -> xyz=0.333 2.204 0.394
- joint cabinet11_joint: origin xyz=0.334 2.86 0.394 -> xyz=0.333 2.855 0.394
- joint cabinet7_joint: origin xyz=0.2 0.5 0.47 -> xyz=0.2 0.501 0.47
- joint cabinet9_joint: origin xyz=0.334 1.705 0.394 -> xyz=0.333 1.703 0.394
- joint cooktop_joint: origin xyz=0.26 2.86 0.832 -> xyz=0.26 2.86 0.830
- joint island_joint: origin xyz=0.13 1.8 0.808 -> xyz=0.13 1.786 0.807
- joint sink_joint: origin xyz=0.328 1.1 0.769 -> xyz=0.328 1.088 0.769
- joint tap_joint: origin xyz=0.1 1.1 0.935 -> xyz=0.1 1.085 0.933
