Commit message: renamed package kimchen to kitchen2

File: iai_kitchen2/urdf/kitchen.urdf (robot description, URDF)
Before this commit: robot kimchen, 79 links, 78 joints
Links:
- link cabinet1: geometry collision mesh filename=package://iai_kitchen2/meshes/cabinet01/IAICabinet1W60.stl; visual mesh filename=package://iai_kitchen2/meshes/cabinet01/IAICabinet1W60.dae
- link cabinet10: geometry collision mesh filename=package://iai_kitchen2/meshes/cabinet10/IAIKitchenCabinet9W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; visual mesh filename=package://iai_kitchen2/meshes/cabinet10/IAIKitchenCabinet9W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
- link cabinet10_drawer_bottom: geometry collision mesh filename=package://iai_kitchen2/meshes/cabinet10/IAIKitchenDrawerW40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; visual mesh filename=package://iai_kitchen2/meshes/cabinet10/IAIKitchenDrawerW40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
- link cabinet10_drawer_middle: geometry collision mesh filename=package://iai_kitchen2/meshes/cabinet10/IAIKitchenDrawerW40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; visual mesh filename=package://iai_kitchen2/meshes/cabinet10/IAIKitchenDrawerW40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
- link cabinet10_drawer_top: geometry collision mesh filename=package://iai_kitchen2/meshes/cabinet10/IAIKitchenDrawerW40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; visual mesh filename=package://iai_kitchen2/meshes/cabinet10/IAIKitchenDrawerW40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
- link cabinet11: geometry collision mesh filename=package://iai_kitchen2/meshes/cabinet11/IAIKitchenCabinet11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; visual mesh filename=package://iai_kitchen2/meshes/cabinet11/IAIKitchenCabinet11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
- link cabinet11_drawer_bottom: geometry collision mesh filename=package://iai_kitchen2/meshes/cabinet11/IAIKitchenDrawerW90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; visual mesh filename=package://iai_kitchen2/meshes/cabinet11/IAIKitchenDrawerW90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
- link cabinet11_drawer_middle: geometry collision mesh filename=package://iai_kitchen2/meshes/cabinet11/IAIKitchenDrawerW90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; visual mesh filename=package://iai_kitchen2/meshes/cabinet11/IAIKitchenDrawerW90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
- link cabinet11_drawer_top: geometry collision mesh filename=package://iai_kitchen2/meshes/cabinet11/IAIKitchenDrawerW90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; visual mesh filename=package://iai_kitchen2/meshes/cabinet11/IAIKitchenDrawerW90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
- link cabinet1_door_top_left: geometry collision mesh filename=package://iai_kitchen2/meshes/cabinet01/IAIDoorW60H80.stl; visual mesh filename=package://iai_kitchen2/meshes/cabinet01/IAIDoorW60H80.dae
- link cabinet1_drawer_bottom: geometry collision mesh filename=package://iai_kitchen2/meshes/cabinet01/IAIDrawerW60H53.stl; visual mesh filename=package://iai_kitchen2/meshes/cabinet01/IAIDrawerW60H53.dae
- link cabinet1_drawer_middle: geometry collision mesh filename=package://iai_kitchen2/meshes/cabinet01/IAIDrawerW60H26.stl; visual mesh filename=package://iai_kitchen2/meshes/cabinet01/IAIDrawerW60H26.dae
- link cabinet1_handle_top: geometry collision mesh filename=package://iai_kitchen2/meshes/handles/handle_horizontal.stl; visual mesh filename=package://iai_kitchen2/meshes/handles/handle_horizontal.dae
- link cabinet2: geometry collision mesh filename=package://iai_kitchen2/meshes/cabinet02/IAICabinet2W40H57.s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; visual mesh filename=package://iai_kitchen2/meshes/cabinet02/IAICabinet2W40H57.d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
- link cabinet2_door_left: geometry collision mesh filename=package://iai_kitchen2/meshes/cabinet02/IAIDoorW40H212.stl; visual mesh filename=package://iai_kitchen2/meshes/cabinet02/IAIDoorW40H212.dae
- link cabinet2_drawer_big: geometry collision mesh filename=package://iai_kitchen2/meshes/cabinet02/IAIDrawerW40H22.stl; visual mesh filename=package://iai_kitchen2/meshes/cabinet02/IAIDrawerW40H22.dae
- link cabinet2_drawer_small: geometry collision mesh filename=package://iai_kitchen2/meshes/cabinet02/IAIDrawerW40H10.stl; visual mesh filename=package://iai_kitchen2/meshes/cabinet02/IAIDrawerW40H10.dae
- link cabinet3: geometry collision mesh filename=package://iai_kitchen2/meshes/cabinet03/IAICabinet3W60.stl; visual mesh filename=package://iai_kitchen2/meshes/cabinet03/IAICabinet3W60.dae
- link cabinet3_door_bottom_right: geometry collision mesh filename=package://iai_kitchen2/meshes/cabinet03/IAIDoorW60H80.stl; visual mesh filename=package://iai_kitchen2/meshes/cabinet03/IAIDoorW60H80.dae
- link cabinet3_door_top_right: geometry collision mesh filename=package://iai_kitchen2/meshes/cabinet03/IAIDoorW60H133.stl; visual mesh filename=package://iai_kitchen2/meshes/cabinet03/IAIDoorW60H133.dae
- link cabinet4: geometry collision mesh filename=package://iai_kitchen2/meshes/cabinet04/IAIKitchenCabinet4W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; visual mesh filename=package://iai_kitchen2/meshes/cabinet04/IAIKitchenCabinet4W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
- link cabinet4_door_bottom: geometry collision mesh filename=package://iai_kitchen2/meshes/cabinet04/IAIDoor2W100H40.stl; visual mesh filename=package://iai_kitchen2/meshes/cabinet04/IAIDoor2W100H40.dae
- link cabinet4_door_top: geometry collision mesh filename=package://iai_kitchen2/meshes/cabinet04/IAIDoor1W100H40.stl; visual mesh filename=package://iai_kitchen2/meshes/cabinet04/IAIDoor1W100H40.dae
- link cabinet5: geometry collision mesh filename=package://iai_kitchen2/meshes/cabinet05/IAIKitchenCabinet5W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; visual mesh filename=package://iai_kitchen2/meshes/cabinet05/IAIKitchenCabinet5W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
- link cabinet5_drawer_bottom: geometry collision mesh filename=package://iai_kitchen2/meshes/cabinet05/IAIKitchenDrawerW60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; visual mesh filename=package://iai_kitchen2/meshes/cabinet05/IAIKitchenDrawerW60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
- link cabinet5_drawer_middle: geometry collision mesh filename=package://iai_kitchen2/meshes/cabinet05/IAIKitchenDrawerW60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; visual mesh filename=package://iai_kitchen2/meshes/cabinet05/IAIKitchenDrawerW60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
- link cabinet5_drawer_top: geometry collision mesh filename=package://iai_kitchen2/meshes/cabinet05/IAIKitchenDrawerW60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; visual mesh filename=package://iai_kitchen2/meshes/cabinet05/IAIKitchenDrawerW60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
- link cabinet6: geometry collision mesh filename=package://iai_kitchen2/meshes/cabinet06/IAIKitchenCabinet6W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; visual mesh filename=package://iai_kitchen2/meshes/cabinet06/IAIKitchenCabinet6W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
- link cabinet6_drawer_bottom: geometry collision mesh filename=package://iai_kitchen2/meshes/cabinet06/IAIKitchenDrawerW40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; visual mesh filename=package://iai_kitchen2/meshes/cabinet06/IAIKitchenDrawerW40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
- link cabinet6_drawer_middle: geometry collision mesh filename=package://iai_kitchen2/meshes/cabinet06/IAIKitchenDrawerW40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; visual mesh filename=package://iai_kitchen2/meshes/cabinet06/IAIKitchenDrawerW40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
- link cabinet6_drawer_top: geometry collision mesh filename=package://iai_kitchen2/meshes/cabinet06/IAIKitchenDrawerW40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; visual mesh filename=package://iai_kitchen2/meshes/cabinet06/IAIKitchenDrawerW40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
- link cabinet7: geometry collision mesh filename=package://iai_kitchen2/meshes/cabinet07/IAIKitchenCabinet7W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; visual mesh filename=package://iai_kitchen2/meshes/cabinet07/IAIKitchenCabinet7W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
- link cabinet7_door_bottom_left: geometry collision mesh filename=package://iai_kitchen2/meshes/cabinet07/IAIKitchenDoorW60H8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; visual mesh filename=package://iai_kitchen2/meshes/cabinet07/IAIKitchenDoorW60H8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
- link cabinet8: geometry collision mesh filename=package://iai_kitchen2/meshes/cabinet08/IAIKitchenCabinet8W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; visual mesh filename=package://iai_kitchen2/meshes/cabinet08/IAIKitchenCabinet8W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
- link cabinet8_drawer_bottom: geometry collision mesh filename=package://iai_kitchen2/meshes/cabinet08/IAIKitchenDrawerW60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; visual mesh filename=package://iai_kitchen2/meshes/cabinet08/IAIKitchenDrawerW60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
- link cabinet8_drawer_middle: geometry collision mesh filename=package://iai_kitchen2/meshes/cabinet08/IAIKitchenDrawerW56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; visual mesh filename=package://iai_kitchen2/meshes/cabinet08/IAIKitchenDrawerW56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
- link cabinet9: geometry collision mesh filename=package://iai_kitchen2/meshes/cabinet09/IAIKitchenCabinet9W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; visual mesh filename=package://iai_kitchen2/meshes/cabinet09/IAIKitchenCabinet9W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
- link cabinet9_drawer_bottom: geometry collision mesh filename=package://iai_kitchen2/meshes/cabinet09/IAIKitchenDrawerW60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; visual mesh filename=package://iai_kitchen2/meshes/cabinet09/IAIKitchenDrawerW60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
- link cabinet9_drawer_middle: geometry collision mesh filename=package://iai_kitchen2/meshes/cabinet09/IAIKitchenDrawerW60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; visual mesh filename=package://iai_kitchen2/meshes/cabinet09/IAIKitchenDrawerW60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
- link cabinet9_drawer_top: geometry collision mesh filename=package://iai_kitchen2/meshes/cabinet09/IAIKitchenDrawerW60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; visual mesh filename=package://iai_kitchen2/meshes/cabinet09/IAIKitchenDrawerW60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
- link cooktop: geometry collision mesh filename=package://iai_kitchen2/meshes/cooktop/IAIKitchenCookTop.stl; visual mesh filename=package://iai_kitchen2/meshes/cooktop/IAIKitchenCookTop.dae
- link countertop: geometry collision mesh filename=package://iai_kitchen2/meshes/countertop/IAIKitchenPartW102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; visual mesh filename=package://iai_kitchen2/meshes/countertop/IAIKitchenPartW102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
- link handle_cab10_b: geometry collision mesh filename=package://iai_kitchen2/meshes/handles/handle_horizontal.stl; visual mesh filename=package://iai_kitchen2/meshes/handles/handle_horizontal.dae
- link handle_cab10_m: geometry collision mesh filename=package://iai_kitchen2/meshes/handles/handle_horizontal.stl; visual mesh filename=package://iai_kitchen2/meshes/handles/handle_horizontal.dae
- link handle_cab10_t: geometry collision mesh filename=package://iai_kitchen2/meshes/handles/handle_horizontal.stl; visual mesh filename=package://iai_kitchen2/meshes/handles/handle_horizontal.dae
- link handle_cab11_b: geometry collision mesh filename=package://iai_kitchen2/meshes/handles/handle_horizontal.stl; visual mesh filename=package://iai_kitchen2/meshes/handles/handle_horizontal.dae
- link handle_cab11_m: geometry collision mesh filename=package://iai_kitchen2/meshes/handles/handle_horizontal.stl; visual mesh filename=package://iai_kitchen2/meshes/handles/handle_horizontal.dae
- link handle_cab11_t: geometry collision mesh filename=package://iai_kitchen2/meshes/handles/handle_horizontal.stl; visual mesh filename=package://iai_kitchen2/meshes/handles/handle_horizontal.dae
- link handle_cab1_drawer_bottom: geometry collision mesh filename=package://iai_kitchen2/meshes/handles/handle_horizontal.stl; visual mesh filename=package://iai_kitchen2/meshes/handles/handle_horizontal.dae
- link handle_cab1_drawer_mid: geometry collision mesh filename=package://iai_kitchen2/meshes/handles/handle_horizontal.stl; visual mesh filename=package://iai_kitchen2/meshes/handles/handle_horizontal.dae
- link handle_cab2_door: geometry collision mesh filename=package://iai_kitchen2/meshes/handles/handle_horizontal.stl; visual mesh filename=package://iai_kitchen2/meshes/handles/handle_horizontal.dae
- link handle_cab3_door_bottom: geometry collision mesh filename=package://iai_kitchen2/meshes/handles/handle_horizontal.stl; visual mesh filename=package://iai_kitchen2/meshes/handles/handle_horizontal.dae
- link handle_cab3_door_top: geometry collision mesh filename=package://iai_kitchen2/meshes/handles/handle_horizontal.stl; visual mesh filename=package://iai_kitchen2/meshes/handles/handle_horizontal.dae
- link handle_cab4_door_bottom: geometry collision mesh filename=package://iai_kitchen2/meshes/handles/handle_horizontal.stl; visual mesh filename=package://iai_kitchen2/meshes/handles/handle_horizontal.dae
- link handle_cab5_b: geometry collision mesh filename=package://iai_kitchen2/meshes/handles/handle_horizontal.stl; visual mesh filename=package://iai_kitchen2/meshes/handles/handle_horizontal.dae
- link handle_cab5_m: geometry collision mesh filename=package://iai_kitchen2/meshes/handles/handle_horizontal.stl; visual mesh filename=package://iai_kitchen2/meshes/handles/handle_horizontal.dae
- link handle_cab5_t: geometry collision mesh filename=package://iai_kitchen2/meshes/handles/handle_horizontal.stl; visual mesh filename=package://iai_kitchen2/meshes/handles/handle_horizontal.dae
- link handle_cab6_b: geometry collision mesh filename=package://iai_kitchen2/meshes/handles/handle_horizontal.stl; visual mesh filename=package://iai_kitchen2/meshes/handles/handle_horizontal.dae
- link handle_cab6_m: geometry collision mesh filename=package://iai_kitchen2/meshes/handles/handle_horizontal.stl; visual mesh filename=package://iai_kitchen2/meshes/handles/handle_horizontal.dae
- link handle_cab6_t: geometry collision mesh filename=package://iai_kitchen2/meshes/handles/handle_horizontal.stl; visual mesh filename=package://iai_kitchen2/meshes/handles/handle_horizontal.dae
- link handle_cab7: geometry collision mesh filename=package://iai_kitchen2/meshes/handles/handle_horizontal.stl; visual mesh filename=package://iai_kitchen2/meshes/handles/handle_horizontal.dae
- link handle_cab8: geometry collision mesh filename=package://iai_kitchen2/meshes/handles/handle_horizontal.stl; visual mesh filename=package://iai_kitchen2/meshes/handles/handle_horizontal.dae
- link handle_cab9_b: geometry collision mesh filename=package://iai_kitchen2/meshes/handles/handle_horizontal.stl; visual mesh filename=package://iai_kitchen2/meshes/handles/handle_horizontal.dae
- link handle_cab9_m: geometry collision mesh filename=package://iai_kitchen2/meshes/handles/handle_horizontal.stl; visual mesh filename=package://iai_kitchen2/meshes/handles/handle_horizontal.dae
- link handle_cab9_t: geometry collision mesh filename=package://iai_kitchen2/meshes/handles/handle_horizontal.stl; visual mesh filename=package://iai_kitchen2/meshes/handles/handle_horizontal.dae
- link island: geometry collision mesh filename=package://iai_kitchen2/meshes/island/IAIKitchenIslandAreaTo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; visual mesh filename=package://iai_kitchen2/meshes/island/IAIKitchenIslandAreaTo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
- link island_back: geometry collision mesh filename=package://iai_kitchen2/meshes/IAIKitchenPartW314H90/IAIKitc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; visual mesh filename=package://iai_kitchen2/meshes/IAIKitchenPartW314H90/IAIKitc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
- link island_waterfall_left: geometry collision mesh filename=package://iai_kitchen2/meshes/IAIKitchenVisiblePartIslandUn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; visual mesh filename=package://iai_kitchen2/meshes/IAIKitchenVisiblePartIslandUn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
- link island_waterfall_right: geometry collision mesh filename=package://iai_kitchen2/meshes/IAIKitchenVisiblePartIslandUn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; visual mesh filename=package://iai_kitchen2/meshes/IAIKitchenVisiblePartIslandUn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
- link sa: geometry collision mesh filename=package://iai_kitchen2/meshes/floor_socket_side_a/IAIKitche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; visual mesh filename=package://iai_kitchen2/meshes/floor_socket_side_a/IAIKitche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
- link sb: geometry collision mesh filename=package://iai_kitchen2/meshes/floor_socket_side_b/IAIKitche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; visual mesh filename=package://iai_kitchen2/meshes/floor_socket_side_b/IAIKitche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
- link side_A_left: geometry collision mesh filename=package://iai_kitchen2/meshes/IAIKitchenPartW58H223/IAIKitc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; visual mesh filename=package://iai_kitchen2/meshes/IAIKitchenPartW58H223/IAIKitc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
- link side_A_rb: geometry collision mesh filename=package://iai_kitchen2/meshes/IAIKitchenVisiblePartUnderSid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; visual mesh filename=package://iai_kitchen2/meshes/IAIKitchenVisiblePartUnderSid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
- link side_A_rt: geometry collision mesh filename=package://iai_kitchen2/meshes/IAIKitchenVisiblePartUppersid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; visual mesh filename=package://iai_kitchen2/meshes/IAIKitchenVisiblePartUppersid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
- link sink: geometry collision mesh filename=package://iai_kitchen2/meshes/sink/IAIKitchenSink.stl; visual mesh filename=package://iai_kitchen2/meshes/sink/IAIKitchenSink.dae
- link tap: geometry collision mesh filename=package://iai_kitchen2/meshes/tap/IAIKitchenWaterTap.stl; visual mesh filename=package://iai_kitchen2/meshes/tap/IAIKitchenWaterTap.dae
