Commit message: fixed urdf refs

File: iai_apartment/urdf/kitchen.urdf (robot description, URDF)
Before this commit: robot kitchen2, 79 links, 78 joints
Links:
- link cabinet1: geometry collision mesh filename=package://iai_apartment/meshes/cabinet01/IAICabinet1W60.stl; visual mesh filename=package://iai_apartment/meshes/cabinet01/IAICabinet1W60.dae
- link cabinet10: geometry collision mesh filename=package://iai_apartment/meshes/cabinet10/IAIKitchenCabinet9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; visual mesh filename=package://iai_apartment/meshes/cabinet10/IAIKitchenCabinet9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
- link cabinet10_drawer_bottom: geometry collision mesh filename=package://iai_apartment/meshes/cabinet10/IAIKitchenDrawerW4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; visual mesh filename=package://iai_apartment/meshes/cabinet10/IAIKitchenDrawerW4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
- link cabinet10_drawer_middle: geometry collision mesh filename=package://iai_apartment/meshes/cabinet10/IAIKitchenDrawerW4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; visual mesh filename=package://iai_apartment/meshes/cabinet10/IAIKitchenDrawerW4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
- link cabinet10_drawer_top: geometry collision mesh filename=package://iai_apartment/meshes/cabinet10/IAIKitchenDrawerW4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; visual mesh filename=package://iai_apartment/meshes/cabinet10/IAIKitchenDrawerW4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
- link cabinet11: geometry collision mesh filename=package://iai_apartment/meshes/cabinet11/IAIKitchenCabinet1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; visual mesh filename=package://iai_apartment/meshes/cabinet11/IAIKitchenCabinet1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
- link cabinet11_drawer_bottom: geometry collision mesh filename=package://iai_apartment/meshes/cabinet11/IAIKitchenDrawerW9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; visual mesh filename=package://iai_apartment/meshes/cabinet11/IAIKitchenDrawerW9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
- link cabinet11_drawer_middle: geometry collision mesh filename=package://iai_apartment/meshes/cabinet11/IAIKitchenDrawerW9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; visual mesh filename=package://iai_apartment/meshes/cabinet11/IAIKitchenDrawerW9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
- link cabinet11_drawer_top: geometry collision mesh filename=package://iai_apartment/meshes/cabinet11/IAIKitchenDrawerW9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; visual mesh filename=package://iai_apartment/meshes/cabinet11/IAIKitchenDrawerW9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
- link cabinet1_door_top_left: geometry collision mesh filename=package://iai_apartment/meshes/cabinet01/IAIDoorW60H80.stl; visual mesh filename=package://iai_apartment/meshes/cabinet01/IAIDoorW60H80.dae
- link cabinet1_drawer_bottom: geometry collision mesh filename=package://iai_apartment/meshes/cabinet01/IAIDrawerW60H53.stl; visual mesh filename=package://iai_apartment/meshes/cabinet01/IAIDrawerW60H53.dae
- link cabinet1_drawer_middle: geometry collision mesh filename=package://iai_apartment/meshes/cabinet01/IAIDrawerW60H26.stl; visual mesh filename=package://iai_apartment/meshes/cabinet01/IAIDrawerW60H26.dae
- link cabinet1_handle_top: geometry collision mesh filename=package://iai_apartment/meshes/handles/handle_horizontal.stl; visual mesh filename=package://iai_apartment/meshes/handles/handle_horizontal.dae
- link cabinet2: geometry collision mesh filename=package://iai_apartment/meshes/cabinet02/IAICabinet2W40H57.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; visual mesh filename=package://iai_apartment/meshes/cabinet02/IAICabinet2W40H57.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
- link cabinet2_door_left: geometry collision mesh filename=package://iai_apartment/meshes/cabinet02/IAIDoorW40H212.stl; visual mesh filename=package://iai_apartment/meshes/cabinet02/IAIDoorW40H212.dae
- link cabinet2_drawer_big: geometry collision mesh filename=package://iai_apartment/meshes/cabinet02/IAIDrawerW40H22.stl; visual mesh filename=package://iai_apartment/meshes/cabinet02/IAIDrawerW40H22.dae
- link cabinet2_drawer_small: geometry collision mesh filename=package://iai_apartment/meshes/cabinet02/IAIDrawerW40H10.stl; visual mesh filename=package://iai_apartment/meshes/cabinet02/IAIDrawerW40H10.dae
- link cabinet3: geometry collision mesh filename=package://iai_apartment/meshes/cabinet03/IAICabinet3W60.stl; visual mesh filename=package://iai_apartment/meshes/cabinet03/IAICabinet3W60.dae
- link cabinet3_door_bottom_right: geometry collision mesh filename=package://iai_apartment/meshes/cabinet03/IAIDoorW60H80.stl; visual mesh filename=package://iai_apartment/meshes/cabinet03/IAIDoorW60H80.dae
- link cabinet3_door_top_right: geometry collision mesh filename=package://iai_apartment/meshes/cabinet03/IAIDoorW60H133.stl; visual mesh filename=package://iai_apartment/meshes/cabinet03/IAIDoorW60H133.dae
- link cabinet4: geometry collision mesh filename=package://iai_apartment/meshes/cabinet04/IAIKitchenCabinet4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; visual mesh filename=package://iai_apartment/meshes/cabinet04/IAIKitchenCabinet4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
- link cabinet4_door_bottom: geometry collision mesh filename=package://iai_apartment/meshes/cabinet04/IAIDoor2W100H40.stl; visual mesh filename=package://iai_apartment/meshes/cabinet04/IAIDoor2W100H40.dae
- link cabinet4_door_top: geometry collision mesh filename=package://iai_apartment/meshes/cabinet04/IAIDoor1W100H40.stl; visual mesh filename=package://iai_apartment/meshes/cabinet04/IAIDoor1W100H40.dae
- link cabinet5: geometry collision mesh filename=package://iai_apartment/meshes/cabinet05/IAIKitchenCabinet5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; visual mesh filename=package://iai_apartment/meshes/cabinet05/IAIKitchenCabinet5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
- link cabinet5_drawer_bottom: geometry collision mesh filename=package://iai_apartment/meshes/cabinet05/IAIKitchenDrawerW6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; visual mesh filename=package://iai_apartment/meshes/cabinet05/IAIKitchenDrawerW6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
- link cabinet5_drawer_middle: geometry collision mesh filename=package://iai_apartment/meshes/cabinet05/IAIKitchenDrawerW6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; visual mesh filename=package://iai_apartment/meshes/cabinet05/IAIKitchenDrawerW6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
- link cabinet5_drawer_top: geometry collision mesh filename=package://iai_apartment/meshes/cabinet05/IAIKitchenDrawerW6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; visual mesh filename=package://iai_apartment/meshes/cabinet05/IAIKitchenDrawerW6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
- link cabinet6: geometry collision mesh filename=package://iai_apartment/meshes/cabinet06/IAIKitchenCabinet6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; visual mesh filename=package://iai_apartment/meshes/cabinet06/IAIKitchenCabinet6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
- link cabinet6_drawer_bottom: geometry collision mesh filename=package://iai_apartment/meshes/cabinet06/IAIKitchenDrawerW4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; visual mesh filename=package://iai_apartment/meshes/cabinet06/IAIKitchenDrawerW4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
- link cabinet6_drawer_middle: geometry collision mesh filename=package://iai_apartment/meshes/cabinet06/IAIKitchenDrawerW4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; visual mesh filename=package://iai_apartment/meshes/cabinet06/IAIKitchenDrawerW4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
- link cabinet6_drawer_top: geometry collision mesh filename=package://iai_apartment/meshes/cabinet06/IAIKitchenDrawerW4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; visual mesh filename=package://iai_apartment/meshes/cabinet06/IAIKitchenDrawerW4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
- link cabinet7: geometry collision mesh filename=package://iai_apartment/meshes/cabinet07/IAIKitchenCabinet7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; visual mesh filename=package://iai_apartment/meshes/cabinet07/IAIKitchenCabinet7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
- link cabinet7_door_bottom_left: geometry collision mesh filename=package://iai_apartment/meshes/cabinet07/IAIKitchenDoorW60H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; visual mesh filename=package://iai_apartment/meshes/cabinet07/IAIKitchenDoorW60H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
- link cabinet8: geometry collision mesh filename=package://iai_apartment/meshes/cabinet08/IAIKitchenCabinet8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; visual mesh filename=package://iai_apartment/meshes/cabinet08/IAIKitchenCabinet8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
- link cabinet8_drawer_bottom: geometry collision mesh filename=package://iai_apartment/meshes/cabinet08/IAIKitchenDrawerW6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; visual mesh filename=package://iai_apartment/meshes/cabinet08/IAIKitchenDrawerW6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
- link cabinet8_drawer_middle: geometry collision mesh filename=package://iai_apartment/meshes/cabinet08/IAIKitchenDrawerW5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; visual mesh filename=package://iai_apartment/meshes/cabinet08/IAIKitchenDrawerW5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
- link cabinet9: geometry collision mesh filename=package://iai_apartment/meshes/cabinet09/IAIKitchenCabinet9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; visual mesh filename=package://iai_apartment/meshes/cabinet09/IAIKitchenCabinet9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
- link cabinet9_drawer_bottom: geometry collision mesh filename=package://iai_apartment/meshes/cabinet09/IAIKitchenDrawerW6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; visual mesh filename=package://iai_apartment/meshes/cabinet09/IAIKitchenDrawerW6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
- link cabinet9_drawer_middle: geometry collision mesh filename=package://iai_apartment/meshes/cabinet09/IAIKitchenDrawerW6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; visual mesh filename=package://iai_apartment/meshes/cabinet09/IAIKitchenDrawerW6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
- link cabinet9_drawer_top: geometry collision mesh filename=package://iai_apartment/meshes/cabinet09/IAIKitchenDrawerW6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; visual mesh filename=package://iai_apartment/meshes/cabinet09/IAIKitchenDrawerW6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
- link cooktop: geometry collision mesh filename=package://iai_apartment/meshes/cooktop/IAIKitchenCookTop.stl; visual mesh filename=package://iai_apartment/meshes/cooktop/IAIKitchenCookTop.dae
- link countertop: geometry collision mesh filename=package://iai_apartment/meshes/countertop/IAIKitchenPartW10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; visual mesh filename=package://iai_apartment/meshes/countertop/IAIKitchenPartW10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
- link handle_cab10_b: geometry collision mesh filename=package://iai_apartment/meshes/handles/handle_horizontal.stl; visual mesh filename=package://iai_apartment/meshes/handles/handle_horizontal.dae
- link handle_cab10_m: geometry collision mesh filename=package://iai_apartment/meshes/handles/handle_horizontal.stl; visual mesh filename=package://iai_apartment/meshes/handles/handle_horizontal.dae
- link handle_cab10_t: geometry collision mesh filename=package://iai_apartment/meshes/handles/handle_horizontal.stl; visual mesh filename=package://iai_apartment/meshes/handles/handle_horizontal.dae
- link handle_cab11_b: geometry collision mesh filename=package://iai_apartment/meshes/handles/handle_horizontal.stl; visual mesh filename=package://iai_apartment/meshes/handles/handle_horizontal.dae
- link handle_cab11_m: geometry collision mesh filename=package://iai_apartment/meshes/handles/handle_horizontal.stl; visual mesh filename=package://iai_apartment/meshes/handles/handle_horizontal.dae
- link handle_cab11_t: geometry collision mesh filename=package://iai_apartment/meshes/handles/handle_horizontal.stl; visual mesh filename=package://iai_apartment/meshes/handles/handle_horizontal.dae
- link handle_cab1_drawer_bottom: geometry collision mesh filename=package://iai_apartment/meshes/handles/handle_horizontal.stl; visual mesh filename=package://iai_apartment/meshes/handles/handle_horizontal.dae
- link handle_cab1_drawer_mid: geometry collision mesh filename=package://iai_apartment/meshes/handles/handle_horizontal.stl; visual mesh filename=package://iai_apartment/meshes/handles/handle_horizontal.dae
- link handle_cab2_door: geometry collision mesh filename=package://iai_apartment/meshes/handles/handle_horizontal.stl; visual mesh filename=package://iai_apartment/meshes/handles/handle_horizontal.dae
- link handle_cab3_door_bottom: geometry collision mesh filename=package://iai_apartment/meshes/handles/handle_horizontal.stl; visual mesh filename=package://iai_apartment/meshes/handles/handle_horizontal.dae
- link handle_cab3_door_top: geometry collision mesh filename=package://iai_apartment/meshes/handles/handle_horizontal.stl; visual mesh filename=package://iai_apartment/meshes/handles/handle_horizontal.dae
- link handle_cab4_door_bottom: geometry collision mesh filename=package://iai_apartment/meshes/handles/handle_horizontal.stl; visual mesh filename=package://iai_apartment/meshes/handles/handle_horizontal.dae
- link handle_cab5_b: geometry collision mesh filename=package://iai_apartment/meshes/handles/handle_horizontal.stl; visual mesh filename=package://iai_apartment/meshes/handles/handle_horizontal.dae
- link handle_cab5_m: geometry collision mesh filename=package://iai_apartment/meshes/handles/handle_horizontal.stl; visual mesh filename=package://iai_apartment/meshes/handles/handle_horizontal.dae
- link handle_cab5_t: geometry collision mesh filename=package://iai_apartment/meshes/handles/handle_horizontal.stl; visual mesh filename=package://iai_apartment/meshes/handles/handle_horizontal.dae
- link handle_cab6_b: geometry collision mesh filename=package://iai_apartment/meshes/handles/handle_horizontal.stl; visual mesh filename=package://iai_apartment/meshes/handles/handle_horizontal.dae
- link handle_cab6_m: geometry collision mesh filename=package://iai_apartment/meshes/handles/handle_horizontal.stl; visual mesh filename=package://iai_apartment/meshes/handles/handle_horizontal.dae
- link handle_cab6_t: geometry collision mesh filename=package://iai_apartment/meshes/handles/handle_horizontal.stl; visual mesh filename=package://iai_apartment/meshes/handles/handle_horizontal.dae
- link handle_cab7: geometry collision mesh filename=package://iai_apartment/meshes/handles/handle_horizontal.stl; visual mesh filename=package://iai_apartment/meshes/handles/handle_horizontal.dae
- link handle_cab8: geometry collision mesh filename=package://iai_apartment/meshes/handles/handle_horizontal.stl; visual mesh filename=package://iai_apartment/meshes/handles/handle_horizontal.dae
- link handle_cab9_b: geometry collision mesh filename=package://iai_apartment/meshes/handles/handle_horizontal.stl; visual mesh filename=package://iai_apartment/meshes/handles/handle_horizontal.dae
- link handle_cab9_m: geometry collision mesh filename=package://iai_apartment/meshes/handles/handle_horizontal.stl; visual mesh filename=package://iai_apartment/meshes/handles/handle_horizontal.dae
- link handle_cab9_t: geometry collision mesh filename=package://iai_apartment/meshes/handles/handle_horizontal.stl; visual mesh filename=package://iai_apartment/meshes/handles/handle_horizontal.dae
- link island: geometry collision mesh filename=package://iai_apartment/meshes/island/IAIKitchenIslandAreaT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; visual mesh filename=package://iai_apartment/meshes/island/IAIKitchenIslandAreaT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
- link island_back: geometry collision mesh filename=package://iai_apartment/meshes/IAIKitchenPartW314H90/IAIKit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; visual mesh filename=package://iai_apartment/meshes/IAIKitchenPartW314H90/IAIKit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
- link island_waterfall_left: geometry collision mesh filename=package://iai_apartment/meshes/IAIKitchenVisiblePartIslandU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; visual mesh filename=package://iai_apartment/meshes/IAIKitchenVisiblePartIslandU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
- link island_waterfall_right: geometry collision mesh filename=package://iai_apartment/meshes/IAIKitchenVisiblePartIslandU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; visual mesh filename=package://iai_apartment/meshes/IAIKitchenVisiblePartIslandU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
- link sa: geometry collision mesh filename=package://iai_apartment/meshes/floor_socket_side_a/IAIKitch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; visual mesh filename=package://iai_apartment/meshes/floor_socket_side_a/IAIKitch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
- link sb: geometry collision mesh filename=package://iai_apartment/meshes/floor_socket_side_b/IAIKitch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; visual mesh filename=package://iai_apartment/meshes/floor_socket_side_b/IAIKitch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
- link side_A_left: geometry collision mesh filename=package://iai_apartment/meshes/IAIKitchenPartW58H223/IAIKit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; visual mesh filename=package://iai_apartment/meshes/IAIKitchenPartW58H223/IAIKit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
- link side_A_rb: geometry collision mesh filename=package://iai_apartment/meshes/IAIKitchenVisiblePartUnderSi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; visual mesh filename=package://iai_apartment/meshes/IAIKitchenVisiblePartUnderSi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
- link side_A_rt: geometry collision mesh filename=package://iai_apartment/meshes/IAIKitchenVisiblePartUppersi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; visual mesh filename=package://iai_apartment/meshes/IAIKitchenVisiblePartUppersi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
- link sink: geometry collision mesh filename=package://iai_apartment/meshes/sink/IAIKitchenSink.stl; visual mesh filename=package://iai_apartment/meshes/sink/IAIKitchenSink.dae
- link tap: geometry collision mesh filename=package://iai_apartment/meshes/tap/IAIKitchenWaterTap.stl; visual mesh filename=package://iai_apartment/meshes/tap/IAIKitchenWaterTap.dae

Commit message: Axes were changed.

File: iai_apartment/urdf/kitchen.urdf (robot description, URDF)
Before this commit: robot apartment, 79 links, 78 joints
Links:
- removed link cabinet1_handle_top
- removed link cabinet3_door_bottom_right
- removed link cabinet3_door_top_right
- added link cabinet3_door_bottom_left; collision mesh filename=package://iai_apartment/meshes/cabinet03/IAIDoorW60H80.stl; visual mesh filename=package://iai_apartment/meshes/cabinet03/IAIDoorW60H80.dae
- added link cabinet3_door_top_left; collision mesh filename=package://iai_apartment/meshes/cabinet03/IAIDoorW60H133.stl; visual mesh filename=package://iai_apartment/meshes/cabinet03/IAIDoorW60H133.dae
- added link handle_cab1_top_door; collision mesh filename=package://iai_apartment/meshes/handles/handle_horizontal.stl; visual mesh filename=package://iai_apartment/meshes/handles/handle_horizontal.dae
Joints:
- removed joint cabinet1_handle_top_joint
- removed joint cabinet3_door_bottom_right_joint
- removed joint cabinet3_door_top_right_joint
- added joint cabinet3_door_bottom_left_joint: type revolute, parent cabinet3, child cabinet3_door_bottom_left, origin xyz=0.39 -0.3 -0.5 rpy=0 0 3.14, axis 0 0 -1, limit lower=0.0 upper=1.5708 effort=1000.0 velocity=1.5708
- added joint cabinet3_door_top_left_joint: type revolute, parent cabinet3, child cabinet3_door_top_left, origin xyz=0.39 -0.3 0.5 rpy=0 0 3.14, axis 0 0 -1, limit lower=0.0 upper=1.5708 effort=1000.0 velocity=1.5708
- added joint handle_cab1_top_door_joint: type fixed, parent cabinet1_door_top_left, child handle_cab1_top_door, origin xyz=-0.01 -0.45 0.02 rpy=1.57 0 0
- joint cabinet1_door_top_left_joint: axis 0 0 1 -> 0 0 -1; limit lower=-1.5708 upper=0.0 effort=1000.0 velocity=1.5708 -> lower=0.0 upper=1.5708 effort=1000.0 velocity=1.5708; origin xyz=0.103 -0.3 0.32 -> xyz=0.103 -0.3 0.32 rpy=0 0 3.14
- joint cabinet1_drawer_bottom_joint: axis 1 0 0 -> -1 0 0; limit lower=0.0 upper=0.5 effort=1000.0 velocity=0.5 -> lower=0.0 upper=0.45 effort=1000.0 velocity=0.5; origin xyz=-0.094 0.0 -0.95 -> xyz=-0.094 0.0 -0.95 rpy=0 0 3.14
- joint cabinet1_drawer_middle_joint: axis 1 0 0 -> -1 0 0; limit lower=0.0 upper=0.5 effort=1000.0 velocity=0.5 -> lower=0.0 upper=0.45 effort=1000.0 velocity=0.5; origin xyz=-0.117 0.0 -0.43 -> xyz=-0.117 0.0 -0.43 rpy=0 0 3.14
- joint cabinet2_door_left_joint: axis 0 0 1 -> 0 0 -1; limit lower=-1.5708 upper=0.0 effort=1000.0 velocity=1.5708 -> lower=0.0 upper=1.5708 effort=1000.0 velocity=1.5708; origin xyz=0.277 -0.19 0.0 -> xyz=0.277 -0.19 0.0 rpy=0 0 3.14
- joint cabinet2_drawer_big_joint: axis 1 0 0 -> -1 0 0; origin xyz=0.04 0.0 -0.12 -> xyz=0.04 0.0 -0.12 rpy=0 0 3.14
- joint cabinet2_drawer_small_joint: axis 1 0 0 -> -1 0 0; limit lower=0.0 upper=0.5 effort=500.0 velocity=0.5 -> lower=0.0 upper=0.45 effort=500.0 velocity=0.5; origin xyz=-0.01 0.0 0.17 -> xyz=-0.01 0.0 0.17 rpy=0 0 3.14
- joint handle_cab1_drawer_bottom_joint: origin xyz=0.21 0.0 0.35 -> xyz=-0.21 0.0 0.35 rpy=1.57 0 0
- joint handle_cab1_drawer_mid_joint: origin xyz=0.232 0.0 0.11 -> xyz=-0.232 0.0 0.11 rpy=1.57 0 0
- joint handle_cab3_door_bottom_joint: parent cabinet3_door_bottom_right -> cabinet3_door_bottom_left
- joint handle_cab3_door_top_joint: parent cabinet3_door_top_right -> cabinet3_door_top_left
