Commit message: more axes changed

File: iai_apartment/urdf/kitchen.urdf (robot description, URDF)
Before this commit: robot apartment, 79 links, 78 joints
Joints:
- joint cabinet10_drawer_bottom_joint: axis 1 0 0 -> -1 0 0; limit lower=0.0 upper=0.5 effort=1000.0 velocity=0.5 -> lower=0.0 upper=0.45 effort=1000.0 velocity=0.5; origin xyz=0.03 0.0 -0.279 -> xyz=0.03 0.0 -0.279 rpy=0 0 3.14
- joint cabinet10_drawer_middle_joint: axis 1 0 0 -> -1 0 0; limit lower=0.0 upper=0.5 effort=1000.0 velocity=0.5 -> lower=0.0 upper=0.45 effort=1000.0 velocity=0.5; origin xyz=0.031 0.0 0.104 -> xyz=0.031 0.0 0.104 rpy=0 0 3.14
- joint cabinet10_drawer_top_joint: axis 1 0 0 -> -1 0 0; limit lower=0.0 upper=0.5 effort=1000.0 velocity=0.5 -> lower=0.0 upper=0.45 effort=1000.0 velocity=0.5; origin xyz=0.033 0.0 0.326 -> xyz=0.033 0.0 0.326 rpy=0 0 3.14
- joint cabinet11_drawer_bottom_joint: axis 1 0 0 -> -1 0 0; origin xyz=0.045 0.0 -0.286 -> xyz=0.045 0.0 -0.286 rpy=0 0 3.14
- joint cabinet11_drawer_middle_joint: axis 1 0 0 -> -1 0 0; origin xyz=0.027 0.0 0.106 -> xyz=0.027 0.0 0.106 rpy=0 0 3.14
- joint cabinet11_drawer_top_joint: axis 1 0 0 -> -1 0 0; origin xyz=0.03 0.0 0.326 -> xyz=0.03 0.0 0.326 rpy=0 0 3.14
- joint cabinet2_drawer_big_joint: limit lower=0.0 upper=0.5 effort=500.0 velocity=0.5 -> lower=0.0 upper=0.45 effort=500.0 velocity=0.5
- joint cabinet4_door_bottom_bottom_joint: limit lower=-1.5708 upper=0.0 effort=1000.0 velocity=1.5708 -> lower=0.0 upper=1.5708 effort=1000.0 velocity=1.5708; origin xyz=0.0 0.0 -0.4 -> xyz=0.0 0.0 -0.4 rpy=0 0 0
- joint cabinet4_door_top_top_joint: limit lower=-2.0 upper=0.0 effort=1000.0 velocity=1.5708 -> lower=0 upper=2.0 effort=1000.0 velocity=1.5708; origin xyz=0.07 0 0.42 -> xyz=0.07 0 0.42 rpy=0 0 3.14
- joint cabinet5_drawer_bottom_joint: axis 1 0 0 -> -1 0 0; origin xyz=0.037 0.0 -0.28 -> xyz=0.037 0.0 -0.28 rpy=0 0 3.14
- joint cabinet5_drawer_middle_joint: axis 1 0 0 -> -1 0 0; origin xyz=0.027 0.0 0.107 -> xyz=0.027 0.0 0.107 rpy=0 0 3.14
- joint cabinet5_drawer_top_joint: axis 1 0 0 -> -1 0 0; origin xyz=0.03 0.0 0.327 -> xyz=0.03 0.0 0.327 rpy=0 0 3.14
- joint cabinet6_drawer_bottom_joint: axis 1 0 0 -> -1 0 0; origin xyz=0.047 0.0 -0.28 -> xyz=0.047 0.0 -0.28 rpy=0 0 3.14
- joint cabinet6_drawer_middle_joint: axis 1 0 0 -> -1 0 0; origin xyz=0.03 0.0 0.105 -> xyz=0.03 0.0 0.105 rpy=0 0 3.14
- joint cabinet6_drawer_top_joint: axis 1 0 0 -> -1 0 0; origin xyz=0.033 -0.0125 0.328 -> xyz=0.033 -0.0125 0.328 rpy=0 0 3.14
- joint cabinet7_door_bottom_left_joint: limit lower=-1.5708 upper=0.0 effort=1000.0 velocity=1.5708 -> lower=0.0 upper=1.5708 effort=1000.0 velocity=1.5708; origin xyz=0.372 0 -0.45 -> xyz=0.372 0 -0.45 rpy=0 0 3.14
- joint cabinet8_drawer_bottom_joint: axis 1 0 0 -> -1 0 0; origin xyz=0.114 0.0 0.105 -> xyz=0.114 0.0 0.105 rpy=0 0 3.14
- joint cabinet8_drawer_middle_joint: axis 1 0 0 -> -1 0 0; limit lower=0.0 upper=0.45 effort=1000.0 velocity=0.5 -> lower=0.0 upper=0.40 effort=1000.0 velocity=0.5; origin xyz=0.05 0.0 0.48 -> xyz=0.05 0.0 0.48 rpy=0 0 3.14
- joint cabinet9_drawer_bottom_joint: axis 1 0 0 -> -1 0 0; limit lower=0.0 upper=0.5 effort=1000.0 velocity=0.5 -> lower=0.0 upper=0.45 effort=1000.0 velocity=0.5; origin xyz=0.036 0.0 -0.281 -> xyz=0.036 0.0 -0.281 rpy=0 0 3.14
- joint cabinet9_drawer_middle_joint: axis 1 0 0 -> -1 0 0; limit lower=0.0 upper=0.5 effort=1000.0 velocity=0.5 -> lower=0.0 upper=0.45 effort=1000.0 velocity=0.5; origin xyz=0.027 0.0 0.106 -> xyz=0.027 0.0 0.106 rpy=0 0 3.14
- joint cabinet9_drawer_top_joint: axis 1 0 0 -> -1 0 0; limit lower=0.0 upper=0.5 effort=1000.0 velocity=0.5 -> lower=0.0 upper=0.45 effort=1000.0 velocity=0.5; origin xyz=0.03 0.0 0.327 -> xyz=0.03 0.0 0.327 rpy=0 0 3.14
- joint handle_cab1_drawer_bottom_joint: origin xyz=-0.21 0.0 0.35 rpy=1.57 0 0 -> xyz=-0.237 0.0 0.35 rpy=1.57 0 0
- joint handle_cab1_drawer_mid_joint: origin xyz=-0.232 0.0 0.11 rpy=1.57 0 0 -> xyz=-0.26 0.0 0.11 rpy=1.57 0 0
- joint handle_cab1_top_door_joint: origin xyz=-0.01 -0.45 0.02 rpy=1.57 0 0 -> xyz=-0.038 -0.45 0.02 rpy=1.57 0 0
- joint handle_cab2_drawer_bottom_joint: origin xyz=0.012 0.29 0.05 -> xyz=-0.040 -0.29 0.05 rpy=1.57 0 0
- joint handle_cab3_door_bottom_joint: origin xyz=0.01 -0.45 0.1 -> xyz=-0.036 -0.45 0.1 rpy=1.57 0 0
- joint handle_cab3_door_top_joint: origin xyz=0.01 -0.45 -0.65 -> xyz=-0.036 -0.45 -0.65 rpy=1.57 0 0
- joint handle_cab4_door_bottom_joint: origin xyz=0.027 0 -0.35 -> xyz=-0.055 0 -0.35 rpy=1.57 0 0
- joint handle_cab5_bott_joint: origin xyz=0.207 0 0.245 -> xyz=0.207 0 0.245 rpy=1.57 0 0
- joint handle_cab5_mid_joint: origin xyz=0.217 0 0.13 -> xyz=-0.245 0 0.13 rpy=1.57 0 0
- joint handle_cab5_top_joint: origin xyz=0.217 0 0.05 -> xyz=-0.245 0 0.05 rpy=1.57 0 0

Commit message: All axes of joints and handles are changed to comply with https://ai.uni-bremen.de/wiki/3dmodeling/items

File: iai_apartment/urdf/kitchen.urdf (robot description, URDF)
Before this commit: robot apartment, 79 links, 78 joints
Joints:
- joint handle_cab10_bott_joint: origin xyz=0.217 0 0.245 -> xyz=-0.245 0 0.245 rpy=1.57 0 0
- joint handle_cab10_mid_joint: origin xyz=0.217 0 0.13 -> xyz=-0.245 0 0.13 rpy=1.57 0 0
- joint handle_cab10_top_joint: origin xyz=0.215 0 0.05 -> xyz=-0.243 0 0.05 rpy=1.57 0 0
- joint handle_cab11_bott_joint: origin xyz=0.199 0 0.245 -> xyz=-0.228 0 0.245 rpy=1.57 0 0
- joint handle_cab11_mid_joint: origin xyz=0.217 0 0.13 -> xyz=-0.245 0 0.13 rpy=1.57 0 0
- joint handle_cab11_top_joint: origin xyz=0.215 0 0.05 -> xyz=-0.243 0 0.05 rpy=1.57 0 0
- joint handle_cab5_bott_joint: origin xyz=0.207 0 0.245 rpy=1.57 0 0 -> xyz=-0.235 0 0.245 rpy=1.57 0 0
- joint handle_cab6_bott_joint: origin xyz=0.199 0 0.245 -> xyz=-0.227 0 0.245 rpy=1.57 0 0
- joint handle_cab6_mid_joint: origin xyz=0.217 0 0.13 -> xyz=-0.245 0 0.13 rpy=1.57 0 0
- joint handle_cab6_top_joint: origin xyz=0.21 0 0.05 -> xyz=-0.238 0 0.05 rpy=1.57 0 0
- joint handle_cab7_top_joint: origin xyz=0.01 0 0.74 -> xyz=-0.038 0 0.74 rpy=1.57 0 0
- joint handle_cab8_top_joint: origin xyz=0.21 0 0.65 -> xyz=-0.238 0 0.65 rpy=1.57 0 0
- joint handle_cab9_bott_joint: origin xyz=0.213 0 0.245 -> xyz=-0.24 0 0.245 rpy=1.57 0 0
- joint handle_cab9_mid_joint: origin xyz=0.217 0 0.13 -> xyz=-0.245 0 0.13 rpy=1.57 0 0
- joint handle_cab9_top_joint: origin xyz=0.217 0 0.05 -> xyz=-0.245 0 0.05 rpy=1.57 0 0
