Commit message: added collada mesh for oven

File: iai_apartment/urdf/iai-apartment.urdf (robot description, URDF)
Before this commit: robot apartment, 104 links, 103 joints
Links:
- link oven: geometry collision box size=0.58 0.58 0.59; visual mesh filename=package://iai_apartment/meshes/cabinet01/oven.dae
