Commit message: Add Unreal map

File: iai_apartment/urdf/apartment_unreal.xacro (robot description, xacro)
@@ -4,12 +4,12 @@
   </link>
   <!-- furnitures, including wardrobe, sofa and coffee table -->
-  <xacro:include filename="$(find iai_apartment)/urdf/furnitures.xacro" />
+  <!-- <xacro:include filename="$(find iai_apartment)/urdf/furnitures.xacro" />
   <xacro:furnitures_macro name="furnitures_base" parent="apartment_root">
     <origin xyz="8.85 1.75 0.0" />
-  </xacro:furnitures_macro>
+  </xacro:furnitures_macro> -->
   <!-- kitchen, kitchen on the walls -->
-  <xacro:include filename="$(find iai_apartment)/urdf/kitchen.xacro" />
+  <xacro:include filename="$(find iai_apartment)/urdf/kitchen_unreal.xacro" />
   <xacro:kitchen_macro name="kitchen_base" parent="apartment_root">
-    <origin xyz="-0.03 0.75 0.005" />
+    <origin xyz="0.0 0.0 0.0" />
   </xacro:kitchen_macro>
 </robot>

File: iai_apartment/urdf/furnitures.xacro (robot description, xacro)
@@ -1,4 +1,4 @@
 <robot xmlns:xacro="http://ros.org/wiki/xacro" name="furnitures">
-  <xacro:macro name="kitchen_macro" params="name parent *origin">
+  <xacro:macro name="furnitures_macro" params="name parent *origin">
     <joint name="${name}" type="fixed">
       <xacro:insert_block name="origin" />

Commit message: Fix the door

File: iai_apartment/urdf/apartment_unreal.xacro (robot description, xacro)
@@ -4,8 +4,8 @@
   </link>
   <!-- furnitures, including wardrobe, sofa and coffee table -->
-  <!-- <xacro:include filename="$(find iai_apartment)/urdf/furnitures.xacro" />
+  <xacro:include filename="$(find iai_apartment)/urdf/furnitures.xacro" />
   <xacro:furnitures_macro name="furnitures_base" parent="apartment_root">
     <origin xyz="8.85 1.75 0.0" />
-  </xacro:furnitures_macro> -->
+  </xacro:furnitures_macro>
   <!-- kitchen, kitchen on the walls -->
   <xacro:include filename="$(find iai_apartment)/urdf/kitchen_unreal.xacro" />

File: iai_apartment/urdf/kitchen_unreal.xacro (robot description, xacro)
@@ -77,5 +77,5 @@
     </link>
     <joint name="cabinet1_door_joint" type="revolute">
-      <origin xyz="-0.274 -0.280 0.677" rpy="0.0 0.0 0.0" />
+      <origin xyz="-0.280 -0.280 0.677" rpy="0.0 0.0 0.0" />
       <parent link="cabinet1" />
       <child link="cabinet1_door" />
@@ -90,5 +90,5 @@
       </visual>
       <collision>
-        <origin xyz="0.285091 -0.00064702 0.0" />
+        <origin xyz="0.285091 0.0 0.0" />
         <geometry>
           <box size="0.596936 0.019 0.86681" />
@@ -416,5 +416,5 @@
     </link>
     <joint name="cabinet2_door_joint" type="revolute">
-      <origin xyz="-0.17998091 -0.29852444 0.00105865" rpy="0.0 0.0 0.0" />
+      <origin xyz="-0.18657 -0.28432144 0.00105865" rpy="0.0 0.0 0.0" />
       <parent link="cabinet2" />
       <child link="cabinet2_door" />
@@ -429,7 +429,7 @@
       </visual>
       <collision>
-        <origin xyz="0.180483 0.013597 0.0" />
-        <geometry>
-          <box size="0.395846 0.018678 2.12276" />
+        <origin xyz="0.185074 -0.000653 0.0" />
+        <geometry>
+          <box size="0.396958 0.019 2.12276" />
         </geometry>
       </collision>
@@ -505,5 +505,5 @@
         <origin xyz="-0.170578 -0.003984 0.0" />
         <geometry>
-          <box size="0.016222 0.494978 0.10099" />
+          <box size="0.016 0.494978 0.10099" />
         </geometry>
       </collision>
@@ -511,5 +511,5 @@
         <origin xyz="0.170578 -0.003984 0.0" />
         <geometry>
-          <box size="0.016222 0.494978 0.10099" />
+          <box size="0.016 0.494978 0.10099" />
         </geometry>
       </collision>
@@ -567,5 +567,5 @@
         <origin xyz="-0.170578 -0.003984 0.075342" />
         <geometry>
-          <box size="0.016222 0.494978 0.023298" />
+          <box size="0.016 0.494978 0.023298" />
         </geometry>
       </collision>
@@ -573,5 +573,5 @@
         <origin xyz="0.170578 -0.003984 0.075342" />
         <geometry>
-          <box size="0.016222 0.494978 0.023298" />
+          <box size="0.016 0.494978 0.023298" />
         </geometry>
       </collision>
@@ -579,5 +579,5 @@
         <origin xyz="-0.170578 -0.003984 -0.043743" />
         <geometry>
-          <box size="0.016222 0.494978 0.087106" />
+          <box size="0.016 0.494978 0.087106" />
         </geometry>
       </collision>
@@ -585,5 +585,5 @@
         <origin xyz="0.170578 -0.003984 -0.043743" />
         <geometry>
-          <box size="0.016222 0.494978 0.087106" />
+          <box size="0.016 0.494978 0.087106" />
         </geometry>
       </collision>
@@ -641,5 +641,5 @@
         <origin xyz="-0.170578 -0.003984 0.075342" />
         <geometry>
-          <box size="0.016222 0.494978 0.023298" />
+          <box size="0.016 0.494978 0.023298" />
         </geometry>
       </collision>
@@ -647,5 +647,5 @@
         <origin xyz="0.170578 -0.003984 0.075342" />
         <geometry>
-          <box size="0.016222 0.494978 0.023298" />
+          <box size="0.016 0.494978 0.023298" />
         </geometry>
       </collision>
@@ -653,5 +653,5 @@
         <origin xyz="-0.170578 -0.003984 -0.043743" />
         <geometry>
-          <box size="0.016222 0.494978 0.087106" />
+          <box size="0.016 0.494978 0.087106" />
         </geometry>
       </collision>
@@ -659,5 +659,5 @@
         <origin xyz="0.170578 -0.003984 -0.043743" />
         <geometry>
-          <box size="0.016222 0.494978 0.087106" />
+          <box size="0.016 0.494978 0.087106" />
         </geometry>
       </collision>
@@ -715,5 +715,5 @@
         <origin xyz="-0.170578 -0.003984 0.075342" />
         <geometry>
-          <box size="0.016222 0.494978 0.023298" />
+          <box size="0.016 0.494978 0.023298" />
         </geometry>
       </collision>
@@ -721,5 +721,5 @@
         <origin xyz="0.170578 -0.003984 0.075342" />
         <geometry>
-          <box size="0.016222 0.494978 0.023298" />
+          <box size="0.016 0.494978 0.023298" />
         </geometry>
       </collision>
@@ -727,5 +727,5 @@
         <origin xyz="-0.170578 -0.003984 -0.043743" />
         <geometry>
-          <box size="0.016222 0.494978 0.087106" />
+          <box size="0.016 0.494978 0.087106" />
         </geometry>
       </collision>
@@ -733,5 +733,5 @@
         <origin xyz="0.170578 -0.003984 -0.043743" />
         <geometry>
-          <box size="0.016222 0.494978 0.087106" />
+          <box size="0.016 0.494978 0.087106" />
         </geometry>
       </collision>
@@ -789,5 +789,5 @@
         <origin xyz="-0.170578 -0.003984 0.075342" />
         <geometry>
-          <box size="0.016222 0.494978 0.023298" />
+          <box size="0.016 0.494978 0.023298" />
         </geometry>
       </collision>
@@ -795,5 +795,5 @@
         <origin xyz="0.170578 -0.003984 0.075342" />
         <geometry>
-          <box size="0.016222 0.494978 0.023298" />
+          <box size="0.016 0.494978 0.023298" />
         </geometry>
       </collision>
@@ -801,5 +801,5 @@
         <origin xyz="-0.170578 -0.003984 -0.043743" />
         <geometry>
-          <box size="0.016222 0.494978 0.087106" />
+          <box size="0.016 0.494978 0.087106" />
         </geometry>
       </collision>
@@ -807,5 +807,5 @@
         <origin xyz="0.170578 -0.003984 -0.043743" />
         <geometry>
-          <box size="0.016222 0.494978 0.087106" />
+          <box size="0.016 0.494978 0.087106" />
         </geometry>
       </collision>
@@ -863,5 +863,5 @@
         <origin xyz="-0.170578 -0.003984 0.075342" />
         <geometry>
-          <box size="0.016222 0.494978 0.023298" />
+          <box size="0.016 0.494978 0.023298" />
         </geometry>
       </collision>
@@ -869,5 +869,5 @@
         <origin xyz="0.170578 -0.003984 0.075342" />
         <geometry>
-          <box size="0.016222 0.494978 0.023298" />
+          <box size="0.016 0.494978 0.023298" />
         </geometry>
       </collision>
@@ -875,5 +875,5 @@
         <origin xyz="-0.170578 -0.003984 -0.043743" />
         <geometry>
-          <box size="0.016222 0.494978 0.087106" />
+          <box size="0.016 0.494978 0.087106" />
         </geometry>
       </collision>
@@ -881,5 +881,5 @@
         <origin xyz="0.170578 -0.003984 -0.043743" />
         <geometry>
-          <box size="0.016222 0.494978 0.087106" />
+          <box size="0.016 0.494978 0.087106" />
         </geometry>
       </collision>
@@ -1380,5 +1380,5 @@
         <origin xyz="-0.196311 0.0 0.0" />
         <geometry>
-          <box size="0.016186 0.332816 0.151834" />
+          <box size="0.016 0.332816 0.151834" />
         </geometry>
       </collision>
@@ -1386,5 +1386,5 @@
         <origin xyz="0.196311 0.0 0.0" />
         <geometry>
-          <box size="0.016186 0.332816 0.151834" />
+          <box size="0.016 0.332816 0.151834" />
         </geometry>
       </collision>
@@ -1674,5 +1674,5 @@
         <origin xyz="-0.270267 0.021031 -0.01336" />
         <geometry>
-          <box size="0.01622 0.491014 0.085266" />
+          <box size="0.016 0.491014 0.085266" />
         </geometry>
       </collision>
@@ -1680,5 +1680,5 @@
         <origin xyz="0.270267 0.021031 -0.01336" />
         <geometry>
-          <box size="0.01622 0.491014 0.085266" />
+          <box size="0.016 0.491014 0.085266" />
         </geometry>
       </collision>
@@ -1748,5 +1748,5 @@
         <origin xyz="-0.270267 0.021031 0.041246" />
         <geometry>
-          <box size="0.01622 0.491014 0.023298" />
+          <box size="0.016 0.491014 0.023298" />
         </geometry>
       </collision>
@@ -1754,5 +1754,5 @@
         <origin xyz="0.270267 0.021031 0.041246" />
         <geometry>
-          <box size="0.01622 0.491014 0.023298" />
+          <box size="0.016 0.491014 0.023298" />
         </geometry>
       </collision>
@@ -1760,5 +1760,5 @@
         <origin xyz="-0.270267 0.021031 -0.078968" />
         <geometry>
-          <box size="0.01622 0.491014 0.083496" />
+          <box size="0.016 0.491014 0.083496" />
         </geometry>
       </collision>
@@ -1766,5 +1766,5 @@
         <origin xyz="0.270267 0.021031 -0.078968" />
         <geometry>
-          <box size="0.01622 0.491014 0.083496" />
+          <box size="0.016 0.491014 0.083496" />
         </geometry>
       </collision>
@@ -1834,5 +1834,5 @@
         <origin xyz="-0.270267 0.021031 -0.00926" />
         <geometry>
-          <box size="0.01622 0.491014 0.023276" />
+          <box size="0.016 0.491014 0.023276" />
         </geometry>
       </collision>
@@ -1840,5 +1840,5 @@
         <origin xyz="0.270267 0.021031 -0.00926" />
         <geometry>
-          <box size="0.01622 0.491014 0.023276" />
+          <box size="0.016 0.491014 0.023276" />
         </geometry>
       </collision>
@@ -1846,5 +1846,5 @@
         <origin xyz="-0.270267 0.021031 -0.129424" />
         <geometry>
-          <box size="0.01622 0.491014 0.083422" />
+          <box size="0.016 0.491014 0.083422" />
         </geometry>
       </collision>
@@ -1852,5 +1852,5 @@
         <origin xyz="0.270267 0.021031 -0.129424" />
         <geometry>
-          <box size="0.01622 0.491014 0.083422" />
+          <box size="0.016 0.491014 0.083422" />
         </geometry>
       </collision>
@@ -1963,5 +1963,5 @@
         <origin xyz="-0.170562 0.021031 -0.01336" />
         <geometry>
-          <box size="0.016656 0.491014 0.085266" />
+          <box size="0.016 0.491014 0.085266" />
         </geometry>
       </collision>
@@ -1969,5 +1969,5 @@
         <origin xyz="0.170562 0.021031 -0.01336" />
         <geometry>
-          <box size="0.016656 0.491014 0.085266" />
+          <box size="0.016 0.491014 0.085266" />
         </geometry>
       </collision>
@@ -2037,5 +2037,5 @@
         <origin xyz="-0.170562 0.021031 0.041246" />
         <geometry>
-          <box size="0.016656 0.491014 0.023298" />
+          <box size="0.016 0.491014 0.023298" />
         </geometry>
       </collision>
@@ -2043,5 +2043,5 @@
         <origin xyz="0.170562 0.021031 0.041246" />
         <geometry>
-          <box size="0.016656 0.491014 0.023298" />
+          <box size="0.016 0.491014 0.023298" />
         </geometry>
       </collision>
@@ -2049,5 +2049,5 @@
         <origin xyz="-0.170562 0.021031 -0.078968" />
         <geometry>
-          <box size="0.016656 0.491014 0.083496" />
+          <box size="0.016 0.491014 0.083496" />
         </geometry>
       </collision>
@@ -2055,5 +2055,5 @@
         <origin xyz="0.170562 0.021031 -0.078968" />
         <geometry>
-          <box size="0.016656 0.491014 0.083496" />
+          <box size="0.016 0.491014 0.083496" />
         </geometry>
       </collision>
@@ -2123,5 +2123,5 @@
         <origin xyz="-0.170562 0.021031 -0.00926" />
         <geometry>
-          <box size="0.016656 0.491014 0.023276" />
+          <box size="0.016 0.491014 0.023276" />
         </geometry>
       </collision>
@@ -2129,5 +2129,5 @@
         <origin xyz="0.170562 0.021031 -0.00926" />
         <geometry>
-          <box size="0.016656 0.491014 0.023276" />
+          <box size="0.016 0.491014 0.023276" />
         </geometry>
       </collision>
@@ -2135,5 +2135,5 @@
         <origin xyz="-0.170562 0.021031 -0.129424" />
         <geometry>
-          <box size="0.016656 0.491014 0.083422" />
+          <box size="0.016 0.491014 0.083422" />
         </geometry>
       </collision>
@@ -2141,5 +2141,5 @@
         <origin xyz="0.170562 0.021031 -0.129424" />
         <geometry>
-          <box size="0.016656 0.491014 0.083422" />
+          <box size="0.016 0.491014 0.083422" />
         </geometry>
       </collision>
@@ -2395,5 +2395,11 @@
       <limit effort="1000.0" lower="${-pi/2}" upper="${pi/2}" velocity="${pi}" />
     </joint>
-    <link name="counter_sink_tap_switch" />
+    <link name="counter_sink_tap_switch" >
+      <collision>
+        <geometry>
+          <box size="0.001 0.001 0.001" />
+        </geometry>
+      </collision>
+    </link>
     <joint name="counter_sink_switch_joint" type="revolute">
       <origin xyz="0.0 0.0 0.0" rpy="0.0 0.0 0.0" />
@@ -2435,13 +2441,25 @@
       </visual>
       <collision>
-        <origin xyz="-0.291193 0.183466 0.25785" />
-        <geometry>
-          <box size="0.015448 0.516974 0.841796" />
-        </geometry>
-      </collision>
-      <collision>
-        <origin xyz="0.291193 0.183466 0.25785" />
-        <geometry>
-          <box size="0.015448 0.516974 0.841796" />
+        <origin xyz="-0.291193 0.244142 0.25785" />
+        <geometry>
+          <box size="0.015448 0.395758 0.841796" />
+        </geometry>
+      </collision>
+      <collision>
+        <origin xyz="0.291193 0.244142 0.25785" />
+        <geometry>
+          <box size="0.015448 0.395758 0.841796" />
+        </geometry>
+      </collision>
+      <collision>
+        <origin xyz="-0.291193 -0.018498 0.328806" />
+        <geometry>
+          <box size="0.015448 0.129522 0.703882" />
+        </geometry>
+      </collision>
+      <collision>
+        <origin xyz="0.291193 -0.018498 0.328806" />
+        <geometry>
+          <box size="0.015448 0.129522 0.703882" />
         </geometry>
       </collision>
@@ -2920,5 +2938,5 @@
         <origin xyz="-0.270267 0.021031 -0.01336" />
         <geometry>
-          <box size="0.01622 0.491014 0.085266" />
+          <box size="0.016 0.491014 0.085266" />
         </geometry>
       </collision>
@@ -2926,5 +2944,5 @@
         <origin xyz="0.270267 0.021031 -0.01336" />
         <geometry>
-          <box size="0.01622 0.491014 0.085266" />
+          <box size="0.016 0.491014 0.085266" />
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