Commit message: Fix urdf

File: iai_apartment/urdf/apartment_unreal.urdf (robot description, URDF)
Before this commit: robot apartment, 116 links, 115 joints
Links:
- removed link sink_drawer
- removed link sink_drawer_handle
- added link fridge_door_tray1; collision box size=0.002 0.421854 0.095574; collision box size=0.002 0.421854 0.095574
- added link fridge_door_tray2; collision box size=0.002 0.421954 0.053802; collision box size=0.002 0.421954 0.053802
- added link fridge_egg_tray; collision mesh filename=package://iai_apartment/meshes/unreal/SM_Fridge_Egg_Tray.stl; visual mesh filename=package://iai_apartment/meshes/unreal/SM_Fridge_Egg_Tray.dae
- added link sink_drawer1; collision box size=0.015 0.498056 0.023296; collision box size=0.015 0.498056 0.023296
- added link sink_drawer1_handle; collision box size=0.013 0.173032 0.013; collision box size=0.02 0.013 0.013
- added link sink_drawer2; collision box size=0.016 0.376026 0.08221; collision box size=0.016 0.376026 0.08221
- link armchair: geometry collision mesh filename=package://iai_apartment/meshes/collision/armchair.stl; visual mesh filename=package://iai_apartment/meshes/visual/armchair.dae
- link sofa: geometry collision mesh filename=package://iai_apartment/meshes/collision/sofa.stl; visual mesh filename=package://iai_apartment/meshes/visual/sofa.dae
Joints:
- removed joint sink_drawer_handle_joint
- removed joint sink_drawer_joint
- added joint fridge_door_tray1_joint: type fixed, parent fridge_door1, child fridge_door_tray1, origin xyz=0.29726078 0.10379066 -0.01565247 rpy=0.0 0.0 1.5707963267948966
- added joint fridge_door_tray2_joint: type fixed, parent fridge_door1, child fridge_door_tray2, origin xyz=0.29847088 0.10176933 0.22387222 rpy=0.0 0.0 1.5707963267948966
- added joint fridge_egg_tray_joint: type fixed, parent fridge_door_tray2, child fridge_egg_tray, origin xyz=-0.00226576 0.08530881 0.00069855 rpy=0.0 0.0 0.0
- added joint sink_drawer1_handle_joint: type fixed, parent sink_drawer1, child sink_drawer1_handle, origin xyz=0.00331339 -0.24900223 0.35071747 rpy=0.0 0.0 1.5707963267948966
- added joint sink_drawer1_joint: type prismatic, parent cabinet8, child sink_drawer1, origin xyz=-0.00013535 -0.05086624 0.0032 rpy=0.0 0.0 0.0, axis 0 -1 0, limit lower=0.0 upper=0.45 effort=1000.0 velocity=0.45
- added joint sink_drawer2_joint: type prismatic, parent cabinet8, child sink_drawer2, origin xyz=-0.00142344 -0.07299484 0.16437714 rpy=0.0 0.0 0.0, axis 0 -1 0, limit lower=0.0 upper=0.3 effort=1000.0 velocity=0.3
- joint armchair_joint: origin xyz=7.9688 -0.3791 0.0 rpy=0 0 1.9199 -> xyz=7.9688 -0.3791 0.3559428 rpy=0 0 1.9199
- joint bedside_table_joint: origin xyz=7.2110 0.1296 0.0 rpy=0 0 0 -> xyz=7.2110 0.1296 0.22990467 rpy=0 0 0
- joint sofa_joint: origin xyz=8.1986 2.4096 0.0 rpy=0 0 0 -> xyz=8.1986 2.4096 0.35732983 rpy=0 0 0

Commit message: Calibrate some coordinates

File: iai_apartment/urdf/apartment_unreal.urdf (robot description, URDF)
Before this commit: robot apartment, 120 links, 119 joints
Joints:
- joint cabinet2_door_handle_joint: origin xyz=0.25886013 -0.00184994 -0.05118866 rpy=0.0 0.0 1.5707963267948966 -> xyz=0.25886013 -0.00184994 -0.10518866 rpy=0.0 0.0 1.5707963267948966
- joint fridge_door1_handle_joint: origin xyz=0.46534321 -0.00799103 -0.4736869 rpy=0.0 0.0 1.5707963267948966 -> xyz=0.46534321 -0.00799103 -0.3616 rpy=0.0 0.0 1.5707963267948966
- joint fridge_door2_handle_joint: origin xyz=0.46538265 0.00804657 0.28486839 rpy=0.0 0.0 1.5707963267948966 -> xyz=0.46538265 0.00804657 0.31786839 rpy=0.0 0.0 1.5707963267948966
- joint kitchen2_root_joint: origin xyz=0.0 0.0 0.0 -> xyz=0.1 0.0 0.0

File: iai_apartment/urdf/kitchen_unreal.xacro (robot description, xacro)
@@ -436,5 +436,5 @@
     </link>
     <joint name="cabinet2_door_handle_joint" type="fixed">
-      <origin xyz="0.25886013 -0.00184994 -0.05118866" rpy="0.0 0.0 ${pi/2}" />
+      <origin xyz="0.25886013 -0.00184994 -0.10518866" rpy="0.0 0.0 ${pi/2}" />
       <parent link="cabinet2_door" />
       <child link="cabinet2_door_handle" />
@@ -997,5 +997,5 @@
     </link>
     <joint name="fridge_door1_handle_joint" type="fixed">
-      <origin xyz="0.46534321 -0.00799103 -0.4736869" rpy="0.0 0.0 ${pi/2}" />
+      <origin xyz="0.46534321 -0.00799103 -0.3616" rpy="0.0 0.0 ${pi/2}" />
       <parent link="fridge_door1" />
       <child link="fridge_door1_handle" />
@@ -1154,5 +1154,5 @@
     </link>
     <joint name="fridge_door2_handle_joint" type="fixed">
-      <origin xyz="0.46538265 0.00804657 0.28486839" rpy="0.0 0.0 ${pi/2}" />
+      <origin xyz="0.46538265 0.00804657 0.31786839" rpy="0.0 0.0 ${pi/2}" />
       <parent link="fridge_door2" />
       <child link="fridge_door2_handle" />
@@ -2333,5 +2333,5 @@
     <!-- Second part of the kitchen (island) -->
     <joint name="kitchen2_root_joint" type="fixed">
-      <origin xyz="0.0 0.0 0.0" />
+      <origin xyz="0.1 0.0 0.0" />
       <parent link="kitchen_root" />
       <child link="kitchen2_root" />
