Commit message: Fix issues #106

File: iai_apartment/urdf/furnitures.xacro (robot description, xacro)
@@ -1,450 +1,444 @@
-<robot xmlns:xacro="http://ros.org/wiki/xacro" name="apartment">
-  <link name="apartment_root">
-    <origin rpy="0 0 0" xyz="0 0 0"/>
-  </link>
-  <joint name="middle_of_the_room_joint" type="fixed">
-    <origin rpy="0 0 0" xyz="8.85 1.75 0.0"/>
-    <parent link="apartment_root"/>
-    <child link="middle_of_the_room"/>
-  </joint>
-  <link name="middle_of_the_room"/>
-  <!-- things and stuff -->
+<robot xmlns:xacro="http://ros.org/wiki/xacro" name="furnitures">
+  <xacro:macro name="kitchen_macro" params="name parent *origin">
+    <joint name="${name}" type="fixed">
+      <xacro:insert_block name="origin" />
+      <parent link="${parent}" />
+      <child link="furnitures_root" />
+    </joint>
+    <link name="furnitures_root" />
+    <!-- things and stuff -->
     <joint name="walls_joint" type="fixed">
-      <origin rpy="0 0 0" xyz="0 0 -0.2"/>
-      <parent link="middle_of_the_room"/>
-      <child link="walls"/>
+      <origin rpy="0 0 0" xyz="0 0 -0.2" />
+      <parent link="furnitures_root" />
+      <child link="walls" />
     </joint>
     <link name="walls">
       <visual>
         <geometry>
-          <mesh filename="package://iai_apartment/meshes/visual/walls.dae"/>
+          <mesh filename="package://iai_apartment/meshes/visual/walls.dae" />
         </geometry>
       </visual>
       <!--collision>
-        <geometry>
-          <mesh filename="package://iai_apartment/meshes/collision/walls.stl" />
-        </geometry>
-      </collision-->
+          <geometry>
+            <mesh filename="package://iai_apartment/meshes/collision/walls.stl" />
+          </geometry>
+        </collision-->
     </link>
     <joint name="windows_joint" type="fixed">
-      <origin rpy="0 0 0" xyz="0 0 -0.2"/>
-      <parent link="middle_of_the_room"/>
-      <child link="windows"/>
+      <origin rpy="0 0 0" xyz="0 0 -0.2" />
+      <parent link="furnitures_root" />
+      <child link="windows" />
     </joint>
     <link name="windows">
       <visual>
         <geometry>
-          <mesh filename="package://iai_apartment/meshes/visual/windows.dae"/>
+          <mesh filename="package://iai_apartment/meshes/visual/windows.dae" />
         </geometry>
       </visual>
       <!--collision>
-        <geometry>
-          <mesh filename="package://iai_apartment/meshes/collision/windows.obj"/>
-        </geometry>
-      </collision-->
+          <geometry>
+            <mesh filename="package://iai_apartment/meshes/collision/windows.obj"/>
+          </geometry>
+        </collision-->
     </link>
     <!-- Collision okay Walls -->
     <!-- From the door side being wall 1, turn right and count the walls. -->
-      <joint name="wall_coloksu_wall1_joint" type="fixed">
-        <origin xyz="0.6 -1.615 1.53" rpy="0 0 -1.57"/>
-        <parent link="middle_of_the_room"/>
-        <child link="wall_coloksu_wall1"/>
-      </joint>
-      <link name="wall_coloksu_wall1">
-        <collision>
-          <origin rpy="0 1.57 0"/>
-          <geometry>
-            <box size="3.05 18.95 0.003"/>
-          </geometry>
-        </collision>
-      </link>
-      <joint name="wall_coloksu_wall2_joint" type="fixed">
-        <origin xyz="-8.855 0.782 1.53" rpy="0 0 3.14"/>
-        <parent link="middle_of_the_room"/>
-        <child link="wall_coloksu_wall2"/>
-      </joint>
-      <link name="wall_coloksu_wall2">
-        <collision>
-          <origin rpy="0 1.57 0"/>
-          <geometry>
-            <box size="3.05 4.808 0.003"/>
-          </geometry>
-        </collision>
-      </link>
-      <joint name="wall_coloksu_wall3_joint" type="fixed">
-        <origin xyz="0.6 3.180 1.53" rpy="0 0 1.57"/>
-        <parent link="middle_of_the_room"/>
-        <child link="wall_coloksu_wall3"/>
-      </joint>
-      <link name="wall_coloksu_wall3">
-        <collision>
-          <origin rpy="0 1.57 0"/>
-          <geometry>
-            <box size="3.05 18.95 0.003"/>
-          </geometry>
-        </collision>
-      </link>
-      <joint name="wall_coloksu_wall4_joint" type="fixed">
-        <origin xyz="10.069 0.782 1.53" rpy="0 0 0"/>
-        <parent link="middle_of_the_room"/>
-        <child link="wall_coloksu_wall4"/>
-      </joint>
-      <link name="wall_coloksu_wall4">
-        <collision>
-          <origin rpy="0 1.57 0"/>
-          <geometry>
-            <box size="3.05 4.808 0.003"/>
-          </geometry>
-        </collision>
-      </link>
+    <joint name="wall_coloksu_wall1_joint" type="fixed">
+      <origin xyz="0.6 -1.615 1.53" rpy="0 0 -1.57" />
+      <parent link="furnitures_root" />
+      <child link="wall_coloksu_wall1" />
+    </joint>
+    <link name="wall_coloksu_wall1">
+      <collision>
+        <origin rpy="0 1.57 0" />
+        <geometry>
+          <box size="3.05 18.95 0.003" />
+        </geometry>
+      </collision>
+    </link>
+    <joint name="wall_coloksu_wall2_joint" type="fixed">
+      <origin xyz="-8.855 0.782 1.53" rpy="0 0 3.14" />
+      <parent link="furnitures_root" />
+      <child link="wall_coloksu_wall2" />
+    </joint>
+    <link name="wall_coloksu_wall2">
+      <collision>
+        <origin rpy="0 1.57 0" />
+        <geometry>
+          <box size="3.05 4.808 0.003" />
+        </geometry>
+      </collision>
+    </link>
+    <joint name="wall_coloksu_wall3_joint" type="fixed">
+      <origin xyz="0.6 3.180 1.53" rpy="0 0 1.57" />
+      <parent link="furnitures_root" />
+      <child link="wall_coloksu_wall3" />
+    </joint>
+    <link name="wall_coloksu_wall3">
+      <collision>
+        <origin rpy="0 1.57 0" />
+        <geometry>
+          <box size="3.05 18.95 0.003" />
+        </geometry>
+      </collision>
+    </link>
+    <joint name="wall_coloksu_wall4_joint" type="fixed">
+      <origin xyz="10.069 0.782 1.53" rpy="0 0 0" />
+      <parent link="furnitures_root" />
+      <child link="wall_coloksu_wall4" />
+    </joint>
+    <link name="wall_coloksu_wall4">
+      <collision>
+        <origin rpy="0 1.57 0" />
+        <geometry>
+          <box size="3.05 4.808 0.003" />
+        </geometry>
+      </collision>
+    </link>
     <joint name="wardrobe_joint" type="fixed">
-      <origin rpy="0 0 0" xyz="9.7082 -0.6331 0.0"/>
-      <parent link="middle_of_the_room"/>
-      <child link="wardrobe"/>
+      <origin rpy="0 0 0" xyz="9.7082 -0.6331 0.0" />
+      <parent link="furnitures_root" />
+      <child link="wardrobe" />
     </joint>
     <link name="wardrobe">
       <visual>
         <geometry>
-          <mesh filename="package://iai_apartment/meshes/visual/wardrobe.dae"/>
-        </geometry>
-      </visual>
-      <collision>
-        <origin rpy="0 0 0" xyz="-0.2693 -0.4482 0.0750"/>
-        <geometry>
-          <box size="0.08 0.08 0.15"/>
-        </geometry>
-      </collision>
-      <collision>
-        <origin rpy="0 0 0" xyz="0.10603 -0.4482 0.0750"/>
-        <geometry>
-          <box size="0.08 0.08 0.15"/>
-        </geometry>
-      </collision>
-      <collision>
-        <origin rpy="0 0 0" xyz="-0.2693 0.4482 0.0750"/>
-        <geometry>
-          <box size="0.08 0.08 0.15"/>
-        </geometry>
-      </collision>
-      <collision>
-        <origin rpy="0 0 0" xyz="0.10603 0.4482 0.0750"/>
-        <geometry>
-          <box size="0.08 0.08 0.15"/>
-        </geometry>
-      </collision>
-      <collision>
-        <origin rpy="0 0 0" xyz="-0.0805 0.0000 0.16345"/>
-        <geometry>
-          <box size="0.487 1.0000 0.0269"/>
-        </geometry>
-      </collision>
-      <collision>
-        <origin rpy="0 0 0" xyz="-0.0805 0.48965 0.975"/>
-        <geometry>
-          <box size="0.487 0.0207 1.65"/>
-        </geometry>
-      </collision>
-      <collision>
-        <origin rpy="0 0 0" xyz="-0.0896 0.0000 0.975"/>
-        <geometry>
-          <box size="0.4318 0.018568 1.65"/>
-        </geometry>
-      </collision>
-      <collision>
-        <origin rpy="0 0 0" xyz="-0.0805 -0.48965 0.975"/>
-        <geometry>
-          <box size="0.487 0.0207 1.65"/>
-        </geometry>
-      </collision>
-      <collision>
-        <origin rpy="0 0 0" xyz="0.14465 0.0000 0.975"/>
-        <geometry>
-          <box size="0.0367 1.0000 1.65"/>
-        </geometry>
-      </collision>
-      <collision>
-        <origin rpy="0 0 0" xyz="0.14465 0.0000 0.975"/>
-        <geometry>
-          <box size="0.0367 1.0000 1.65"/>
-        </geometry>
-      </collision>
-      <collision>
-        <origin rpy="0 0 0" xyz="-0.0805 0.0000 1.7865"/>
-        <geometry>
-          <box size="0.487 1.0000 0.027"/>
-        </geometry>
-      </collision>
-      <collision>
-        <origin rpy="0 0 0" xyz="-0.08861 -0.244343 0.5727"/>
-        <geometry>
-          <box size="0.4299 0.469957 0.0118"/>
-        </geometry>
-      </collision>
-      <collision>
-        <origin rpy="0 0 0" xyz="-0.08861 -0.244343 0.974836"/>
-        <geometry>
-          <box size="0.4299 0.469957 0.0118"/>
-        </geometry>
-      </collision>
-      <collision>
-        <origin rpy="0 0 0" xyz="-0.08861 -0.244343 1.37686"/>
-        <geometry>
-          <box size="0.4299 0.469957 0.0118"/>
-        </geometry>
-      </collision>
-      <collision>
-        <origin rpy="1.5708 0 0" xyz="-0.086923 0.244373 1.66898"/>
-        <geometry>
-          <cylinder radius="0.0075" length="0.469897"/>
+          <mesh filename="package://iai_apartment/meshes/visual/wardrobe.dae" />
+        </geometry>
+      </visual>
+      <collision>
+        <origin rpy="0 0 0" xyz="-0.2693 -0.4482 0.0750" />
+        <geometry>
+          <box size="0.08 0.08 0.15" />
+        </geometry>
+      </collision>
+      <collision>
+        <origin rpy="0 0 0" xyz="0.10603 -0.4482 0.0750" />
+        <geometry>
+          <box size="0.08 0.08 0.15" />
+        </geometry>
+      </collision>
+      <collision>
+        <origin rpy="0 0 0" xyz="-0.2693 0.4482 0.0750" />
+        <geometry>
+          <box size="0.08 0.08 0.15" />
+        </geometry>
+      </collision>
+      <collision>
+        <origin rpy="0 0 0" xyz="0.10603 0.4482 0.0750" />
+        <geometry>
+          <box size="0.08 0.08 0.15" />
+        </geometry>
+      </collision>
+      <collision>
+        <origin rpy="0 0 0" xyz="-0.0805 0.0000 0.16345" />
+        <geometry>
+          <box size="0.487 1.0000 0.0269" />
+        </geometry>
+      </collision>
+      <collision>
+        <origin rpy="0 0 0" xyz="-0.0805 0.48965 0.975" />
+        <geometry>
+          <box size="0.487 0.0207 1.65" />
+        </geometry>
+      </collision>
+      <collision>
+        <origin rpy="0 0 0" xyz="-0.0896 0.0000 0.975" />
+        <geometry>
+          <box size="0.4318 0.018568 1.65" />
+        </geometry>
+      </collision>
+      <collision>
+        <origin rpy="0 0 0" xyz="-0.0805 -0.48965 0.975" />
+        <geometry>
+          <box size="0.487 0.0207 1.65" />
+        </geometry>
+      </collision>
+      <collision>
+        <origin rpy="0 0 0" xyz="0.14465 0.0000 0.975" />
+        <geometry>
+          <box size="0.0367 1.0000 1.65" />
+        </geometry>
+      </collision>
+      <collision>
+        <origin rpy="0 0 0" xyz="0.14465 0.0000 0.975" />
+        <geometry>
+          <box size="0.0367 1.0000 1.65" />
+        </geometry>
+      </collision>
+      <collision>
+        <origin rpy="0 0 0" xyz="-0.0805 0.0000 1.7865" />
+        <geometry>
+          <box size="0.487 1.0000 0.027" />
+        </geometry>
+      </collision>
+      <collision>
+        <origin rpy="0 0 0" xyz="-0.08861 -0.244343 0.5727" />
+        <geometry>
+          <box size="0.4299 0.469957 0.0118" />
+        </geometry>
+      </collision>
+      <collision>
+        <origin rpy="0 0 0" xyz="-0.08861 -0.244343 0.974836" />
+        <geometry>
+          <box size="0.4299 0.469957 0.0118" />
+        </geometry>
+      </collision>
+      <collision>
+        <origin rpy="0 0 0" xyz="-0.08861 -0.244343 1.37686" />
+        <geometry>
+          <box size="0.4299 0.469957 0.0118" />
+        </geometry>
+      </collision>
+      <collision>
+        <origin rpy="1.5708 0 0" xyz="-0.086923 0.244373 1.66898" />
+        <geometry>
+          <cylinder radius="0.0075" length="0.469897" />
         </geometry>
       </collision>
     </link>
     <joint name="wardrobe_door_left_joint" type="revolute">
-      <origin rpy="0 0 0" xyz="-0.3246 0.5 0.0000"/>
-      <parent link="wardrobe"/>
-      <child link="wardrobe_door_left"/>
-      <axis xyz="0 0 -1"/>
-      <limit effort="1000.0" lower="0.0" upper="1.5708" velocity="1.5708"/>
+      <origin rpy="0 0 0" xyz="-0.3246 0.5 0.0000" />
+      <parent link="wardrobe" />
+      <child link="wardrobe_door_left" />
+      <axis xyz="0 0 -1" />
+      <limit effort="1000.0" lower="0.0" upper="1.5708" velocity="1.5708" />
     </joint>
     <link name="wardrobe_door_left">
       <visual>
         <geometry>
-          <mesh filename="package://iai_apartment/meshes/visual/wardrobe_door_left.dae"/>
-        </geometry>
-      </visual>
-      <collision>
-        <origin rpy="0 0 0" xyz="-0.006435 -0.2485 0.975"/>
-        <geometry>
-          <box size="0.012967 0.495438 1.64844"/>
+          <mesh filename="package://iai_apartment/meshes/visual/wardrobe_door_left.dae" />
+        </geometry>
+      </visual>
+      <collision>
+        <origin rpy="0 0 0" xyz="-0.006435 -0.2485 0.975" />
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
Commit message: Fix some coordinates

File: iai_apartment/urdf/furnitures.xacro (robot description, xacro)
@@ -299,5 +299,5 @@
     </link>
     <joint name="armchair_joint" type="fixed">
-      <origin rpy="0 0 1.9199" xyz="7.9688 -0.3791 0.0" />
+      <origin rpy="0 0 1.9199" xyz="7.9688 -0.3791 0.3559428" />
       <parent link="furnitures_root" />
       <child link="armchair" />
@@ -311,10 +311,10 @@
       <collision>
         <geometry>
-          <mesh filename="package://iai_apartment/meshes/collision/armchair.obj" />
+          <mesh filename="package://iai_apartment/meshes/collision/armchair.stl" />
         </geometry>
       </collision>
     </link>
     <joint name="sofa_joint" type="fixed">
-      <origin rpy="0 0 0" xyz="8.1986 2.4096 0.0" />
+      <origin rpy="0 0 0" xyz="8.1986 2.4096 0.35732983" />
       <parent link="furnitures_root" />
       <child link="sofa" />
@@ -328,5 +328,5 @@
       <collision>
         <geometry>
-          <mesh filename="package://iai_apartment/meshes/collision/sofa.obj" />
+          <mesh filename="package://iai_apartment/meshes/collision/sofa.stl" />
         </geometry>
       </collision>
@@ -424,5 +424,5 @@
     </link>
     <joint name="bedside_table_joint" type="fixed">
-      <origin rpy="0 0 0" xyz="7.2110 0.1296 0.0" />
+      <origin rpy="0 0 0" xyz="7.2110 0.1296 0.22990467" />
       <parent link="furnitures_root" />
       <child link="bedside_table" />
@@ -435,5 +435,5 @@
       </visual>
       <collision>
-        <origin rpy="0 0 0" xyz="0.0000 0.0000 0.230" />
+        <origin rpy="0 0 0" xyz="0.0000 0.0000 0.22990467" />
         <geometry>
           <box size="0.312 0.312 0.460" />

Commit message: Fix meshes

File: iai_apartment/urdf/furnitures.xacro (robot description, xacro)
@@ -435,5 +435,5 @@
       </visual>
       <collision>
-        <origin rpy="0 0 0" xyz="0.0000 0.0000 0.22990467" />
+        <origin rpy="0 0 0" xyz="0.0 0.0 0.0" />
         <geometry>
           <box size="0.312 0.312 0.460" />
