Commit message: Fix orientation

File: iai_apartment/urdf/kitchen_unreal.xacro (robot description, xacro)
@@ -2380,5 +2380,5 @@
     <!-- Counter sink stove -->
     <joint name="counter_sink_stove_joint" type="fixed">
-      <origin xyz="2.65274353 2.70903961 0.46562927" rpy="0.0 0.0 ${-pi/2}" />
+      <origin xyz="2.65274353 2.70903961 0.46562927" rpy="0.0 0.0 0.0" />
       <parent link="kitchen2_root" />
       <child link="counter_sink_stove" />
@@ -2391,36 +2391,36 @@
       </visual>
       <collision>
-        <origin xyz="1.5755 0.0 0.0" />
-        <geometry>
-          <box size="0.029 1.0 0.934462" />
-        </geometry>
-      </collision>
-      <collision>
-        <origin xyz="0.0 0.262968 0.453637" />
-        <geometry>
-          <box size="3.17704 0.475062 0.03" />
-        </geometry>
-      </collision>
-      <collision>
-        <origin xyz="0.0 -0.451058 0.453637" />
-        <geometry>
-          <box size="3.17704 0.097634 0.03" />
-        </geometry>
-      </collision>
-      <collision>
-        <origin xyz="-1.22213 0.0 0.453637" />
-        <geometry>
-          <box size="0.735422 0.996 0.03" />
-        </geometry>
-      </collision>
-      <collision>
-        <origin xyz="0.560551 0.0 0.453637" />
-        <geometry>
-          <box size="2.05608 0.996 0.03" />
+        <origin xyz="0.0 -1.5755 0.0" />
+        <geometry>
+          <box size="1.0 0.029 0.934462" />
+        </geometry>
+      </collision>
+      <collision>
+        <origin xyz="0.262968 0.0 0.453637" />
+        <geometry>
+          <box size="0.475062 3.17704 0.03" />
+        </geometry>
+      </collision>
+      <collision>
+        <origin xyz="-0.451058 0.0 0.453637" />
+        <geometry>
+          <box size="0.097634 3.17704 0.03" />
+        </geometry>
+      </collision>
+      <collision>
+        <origin xyz="0.0 1.22213 0.453637" />
+        <geometry>
+          <box size="0.996 0.735422 0.03" />
+        </geometry>
+      </collision>
+      <collision>
+        <origin xyz="0.0 -0.560551 0.453637" />
+        <geometry>
+          <box size="0.996 2.05608 0.03" />
         </geometry>
       </collision>
     </link>
     <joint name="stove_joint" type="fixed">
-      <origin xyz="1.08145462 -0.15655746 0.47160622" rpy="0.0 0.0 0.0" />
+      <origin xyz="-0.15655746 -1.08145462 0.47160622" rpy="0.0 0.0 0.0" />
       <parent link="counter_sink_stove" />
       <child link="stove" />
@@ -2435,10 +2435,10 @@
         <origin xyz="0.0 0.0 0.0" />
         <geometry>
-          <box size="0.795 0.516 0.004802" />
+          <box size="0.516 0.795 0.004802" />
         </geometry>
       </collision>
     </link>
     <joint name="counter_sink_joint" type="fixed">
-      <origin xyz="-0.66553391 -0.18887642 0.38240448" rpy="0.0 0.0 0.0" />
+      <origin xyz="-0.18887642 0.66553391 0.38240448" rpy="0.0 0.0 0.0" />
       <parent link="counter_sink_stove" />
       <child link="counter_sink" />
@@ -2451,25 +2451,25 @@
       </visual>
       <collision>
-        <origin xyz="0.0 0.18348 0.0" />
-        <geometry>
-          <box size="0.404212 0.077992 0.177388" />
-        </geometry>
-      </collision>
-      <collision>
-        <origin xyz="0.0 -0.212477 0.0" />
-        <geometry>
-          <box size="0.404212 0.02 0.177388" />
-        </geometry>
-      </collision>
-      <collision>
-        <origin xyz="0.192479 0.0 0.0" />
-        <geometry>
-          <box size="0.02 0.444618 0.177388" />
-        </geometry>
-      </collision>
-      <collision>
-        <origin xyz="-0.192479 0.0 0.0" />
-        <geometry>
-          <box size="0.02 0.444618 0.177388" />
+        <origin xyz="0.18348 0.0 0.0" />
+        <geometry>
+          <box size="0.077992 0.404212 0.177388" />
+        </geometry>
+      </collision>
+      <collision>
+        <origin xyz="-0.212477 0.0 0.0" />
+        <geometry>
+          <box size="0.02 0.404212 0.177388" />
+        </geometry>
+      </collision>
+      <collision>
+        <origin xyz="0.0 -0.192479 0.0" />
+        <geometry>
+          <box size="0.444618 0.02 0.177388" />
+        </geometry>
+      </collision>
+      <collision>
+        <origin xyz="0.0 0.192479 0.0" />
+        <geometry>
+          <box size="0.444618 0.02 0.177388" />
         </geometry>
       </collision>
@@ -2477,10 +2477,10 @@
         <origin xyz="0.0 0.0 -0.074992" />
         <geometry>
-          <box size="0.404212 0.444618 0.027402" />
+          <box size="0.444618 0.404212 0.027402" />
         </geometry>
       </collision>
     </link>
     <joint name="counter_watertab_joint" type="fixed">
-      <origin xyz="0.01961838 0.07677188 0.2389875" rpy="0.0 0.0 0.0" />
+      <origin xyz="0.07677188 -0.01961838 0.2389875" rpy="0.0 0.0 0.0" />
       <parent link="counter_sink" />
       <child link="counter_watertab" />
@@ -2493,5 +2493,5 @@
       </visual>
       <collision>
-        <origin xyz="-0.0195 0.113704 -0.11162" />
+        <origin xyz="0.113704 0.0195 -0.11162" />
         <geometry>
           <cylinder radius="0.022435" length="0.077478" />
@@ -2499,5 +2499,5 @@
       </collision>
       <collision>
-        <origin xyz="-0.0195 0.113704 0.041404" />
+        <origin xyz="0.113704 0.0195 0.041404" />
         <geometry>
           <cylinder radius="0.014" length="0.21816" />
@@ -2505,5 +2505,5 @@
       </collision>
       <collision>
-        <origin xyz="-0.0195 -0.116237 0.121328" />
+        <origin xyz="-0.116237 0.0195 0.121328" />
         <geometry>
           <cylinder radius="0.010966" length="0.007636" />
@@ -2511,5 +2511,5 @@
       </collision>
       <collision>
-        <origin xyz="-0.009 0.113731 -0.073523" rpy="0.0 ${pi/2} 0.0" />
+        <origin xyz="0.113731 0.009 -0.073523" rpy="0.0 ${pi/2} ${pi/2}" />
         <geometry>
           <cylinder radius="0.022466" length="0.08899" />
@@ -2517,5 +2517,5 @@
       </collision>
       <collision>
-        <origin xyz="0.035496 0.113738 -0.073492" />
+        <origin xyz="0.113738 -0.035496 -0.073492" />
         <geometry>
           <sphere radius="0.018" />
@@ -2523,5 +2523,5 @@
       </collision>
       <collision>
-        <origin xyz="-0.019498 -0.00425 0.136485" rpy="${pi/2} 0.0 0.0" />
+        <origin xyz="-0.00425 0.019498 0.136485" rpy="${pi/2} 0.0 ${pi/2}" />
         <geometry>
           <cylinder radius="0.014" length="0.263972" />
@@ -2530,8 +2530,8 @@
     </link>
     <joint name="counter_sink_tap_temperature_joint" type="revolute">
-      <origin xyz="0.04055276 0.11371069 -0.07370445" rpy="0.0 0.0 ${pi}" />
+      <origin xyz="0.11371069 -0.04055276 -0.07370445" rpy="0.0 0.0 ${pi}" />
       <parent link="counter_watertab" />
       <child link="counter_sink_tap_switch" />
-      <axis xyz="1 0 0" />
+      <axis xyz="0 -1 0" />
       <limit effort="1000.0" lower="${-pi/2}" upper="${pi/2}" velocity="${pi}" />
     </joint>
@@ -2547,5 +2547,5 @@
       <parent link="counter_sink_tap_switch" />
       <child link="counter_sink_tap" />
-      <axis xyz="0 -1 0" />
+      <axis xyz="-1 0 0" />
       <limit effort="1000.0" lower="0.0" upper="${pi/8}" velocity="${pi/8}" />
     </joint>
@@ -2557,5 +2557,5 @@
       </visual>
       <collision>
-        <origin xyz="-0.007501 0.0 0.0" rpy="0.0 ${pi/2} 0.0" />
+        <origin xyz="0.0 0.007501 0.0" rpy="0.0 ${pi/2} ${pi/2}" />
         <geometry>
           <cylinder radius="0.022432" length="0.024394" />
@@ -2563,5 +2563,5 @@
       </collision>
       <collision>
-        <origin xyz="-0.012886 0.0 0.048989" />
+        <origin xyz="0.0 0.012886 0.048989" />
         <geometry>
           <cylinder radius="0.005" length="0.055994" />
@@ -2571,5 +2571,5 @@
     <!-- Dishwasher -->
     <joint name="dishwasher_joint" type="fixed">
-      <origin xyz="2.32419296 3.96355377 0.16226444" rpy="0.0 0.0 ${-pi/2}" />
+      <origin xyz="2.32419296 3.96355377 0.16226444" rpy="0.0 0.0 0.0" />
       <parent link="kitchen2_root" />
       <child link="dishwasher" />
@@ -2582,51 +2582,51 @@
       </visual>
       <collision>
-        <origin xyz="-0.291193 0.244142 0.25785" />
-        <geometry>
-          <box size="0.015448 0.395758 0.841796" />
-        </geometry>
-      </collision>
-      <collision>
-        <origin xyz="0.291193 0.244142 0.25785" />
-        <geometry>
-          <box size="0.015448 0.395758 0.841796" />
-        </geometry>
-      </collision>
-      <collision>
-        <origin xyz="-0.291193 -0.018498 0.328806" />
-        <geometry>
-          <box size="0.015448 0.129522 0.703882" />
-        </geometry>
-      </collision>
-      <collision>
-        <origin xyz="0.291193 -0.018498 0.328806" />
-        <geometry>
-          <box size="0.015448 0.129522 0.703882" />
-        </geometry>
-      </collision>
-      <collision>
-        <origin xyz="0.0 0.439555 0.25785" />
-        <geometry>
-          <box size="0.597834 0.004826 0.841796" />
-        </geometry>
-      </collision>
-      <collision>
-        <origin xyz="0.0 0.183466 0.671998" />
-        <geometry>
-          <box size="0.597834 0.516974 0.013498" />
-        </geometry>
-      </collision>
-      <collision>
-        <origin xyz="0.0 0.183466 -0.079608" />
-        <geometry>
-          <box size="0.597834 0.516974 0.167104" />
+        <origin xyz="0.244142 0.291193 0.25785" />
+        <geometry>
+          <box size="0.395758 0.015448 0.841796" />
+        </geometry>
+      </collision>
+      <collision>
+        <origin xyz="0.244142 -0.291193 0.25785" />
+        <geometry>
+          <box size="0.395758 0.015448 0.841796" />
+        </geometry>
+      </collision>
+      <collision>
+        <origin xyz="-0.018498 0.291193 0.328806" />
+        <geometry>
+          <box size="0.129522 0.015448 0.703882" />
+        </geometry>
+      </collision>
+      <collision>
+        <origin xyz="-0.018498 -0.291193 0.328806" />
+        <geometry>
+          <box size="0.129522 0.015448 0.703882" />
+        </geometry>
+      </collision>
+      <collision>
+        <origin xyz="0.439555 0.0 0.25785" />
+        <geometry>
+          <box size="0.004826 0.597834 0.841796" />
+        </geometry>
+      </collision>
+      <collision>
+        <origin xyz="0.183466 0.0 0.671998" />
+        <geometry>
+          <box size="0.516974 0.597834 0.013498" />
+        </geometry>
+      </collision>
+      <collision>
+        <origin xyz="0.183466 0.0 -0.079608" />
+        <geometry>
+          <box size="0.516974 0.597834 0.167104" />
         </geometry>
       </collision>
     </link>
     <joint name="dishwasher_front_joint" type="revolute">
-      <origin xyz="0.00031149 -0.07612121 0.00728645" rpy="0.0 0.0 0.0" />
+      <origin xyz="-0.07612121 0.00031149 0.00728645" rpy="${-pi/2} 0.0 0.0" />
       <parent link="dishwasher" />
       <child link="dishwasher_front" />
-      <axis xyz="1 0 0" />
+      <axis xyz="0 0 -1" />
       <limit effort="1000.0" lower="0.0" upper="${pi/2}" velocity="${pi/2}" />
     </joint>
@@ -2638,18 +2638,18 @@
       </visual>
       <collision>
-        <origin xyz="0.0 -0.04 0.329015" />
-        <geometry>
-          <box size="0.609974 0.018888 0.794358" />
-        </geometry>
-      </collision>
-      <collision>
-        <origin xyz="-0.01 -0.015728 0.334215" />
-        <geometry>
-          <box size="0.574938 0.03 0.679206" />
+        <origin xyz="-0.04 -0.329015 0.0" />
+        <geometry>
+          <box size="0.018888 0.794358 0.609974" />
+        </geometry>
+      </collision>
+      <collision>
+        <origin xyz="-0.01 -0.334215 -0.015728" />
+        <geometry>
+          <box size="0.03 0.679206 0.574938" />
         </geometry>
       </collision>
     </link>
     <joint name="dishwasher_front_handle_joint" type="fixed">
-      <origin xyz="-0.0169432 -0.05493519 0.67884796" rpy="0.0 0.0 ${pi/2}" />
+      <origin xyz="-0.05493519 -0.67884796 0.0" rpy="0.0 0.0 0.0" />
       <parent link="dishwasher_front" />
       <child link="dishwasher_front_handle" />
@@ -2662,11 +2662,11 @@
       </visual>
       <collision>
-        <origin xyz="-0.003891 0.08 0.0" />
-        <geometry>
-          <box size="0.02 0.013 0.013" />
-        </geometry>
-      </collision>
-      <collision>
-        <origin xyz="-0.003891 -0.08 0.0" />
+        <origin xyz="-0.003891 0.0 0.08" />
+        <geometry>
+          <box size="0.02 0.013 0.013" />
+        </geometry>
+      </collision>
+      <collision>
+        <origin xyz="-0.003891 0.0 -0.08" />
         <geometry>
           <box size="0.02 0.013 0.013" />
@@ -2676,13 +2676,13 @@
         <origin xyz="-0.0203895 0.0 0.0" />
         <geometry>
-          <box size="0.013 0.173032  0.013" />
+          <box size="0.013 0.013 0.173032" />
         </geometry>
       </collision>
     </link>
     <joint name="dishwasher_tray1_joint" type="prismatic">
-      <origin xyz="-0.00735926 0.19401426 0.22713593" rpy="0.0 0.0 0.0" />
+      <origin xyz="0.19401426 0.00735926 0.22713593" rpy="0.0 0.0 0.0" />
       <parent link="dishwasher" />
       <child link="dishwasher_tray1" />
-      <axis xyz="0 -1 0" />
+      <axis xyz="-1 0 0" />
       <limit effort="1000.0" lower="0.0" upper="0.5" velocity="0.5" />
     </joint>
@@ -2694,15 +2694,39 @@
       </visual>
       <collision>
-        <origin xyz="0.0 -0.037745 -0.05" />
-        <geometry>
-          <box size="0.54 0.44 0.2" />
+        <origin xyz="-0.03859 0.0 -0.144673" />
+        <geometry>
+          <box size="0.48427 0.538406 0.014224" />
+        </geometry>
+      </collision>
+      <collision>
+        <origin xyz="-0.03859 0.255159 -0.035299" />
+        <geometry>
+          <box size="0.48427 0.010896 0.232972" />
+        </geometry>
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