Commit message: Fix position

File: iai_apartment/urdf/furnitures_with_window4.xacro (robot description, xacro)
@@ -532,5 +532,5 @@
       </visual>
       <collision>
-        <origin rpy="0 0 0" xyz="0.0000 0.0000 0.22990467" />
+        <origin rpy="0 0 0" xyz="0.0 0.0 0.0" />
         <geometry>
           <box size="0.312 0.312 0.460" />

Commit message: Make window handle fixed joint, put axis in middle

File: iai_apartment/urdf/furnitures_with_window4.xacro (robot description, xacro)
@@ -81,4 +81,5 @@
       </collision>
     </link>
+    <!-- right window -->
     <joint name="window4_right_joint" type="revolute">
       <origin xyz="0.916552 0 -0.425471" />
@@ -101,10 +102,8 @@
       </collision>
     </link>
-    <joint name="window4_right_handle_joint" type="revolute">
-      <origin xyz="-0.815383 -0.019236 0.0" />
+    <joint name="window4_right_handle_joint" type="fixed">
+      <origin xyz="-0.815383 -0.06 -0.058" rpy="${pi} 0 ${pi/2}"/>
       <parent link="window4_right" />
       <child link="window4_right_handle" />
-      <axis xyz="0 -1 0" />
-      <limit effort="1000.0" lower="0.0" upper="${pi}" velocity="${pi}" />
     </joint>
     <link name="window4_right_handle">
@@ -115,22 +114,10 @@
       </visual>
       <collision>
-        <origin xyz="0 -0.011369 0" rpy="${pi/2} 0 0" />
-        <geometry>
-          <cylinder length="0.075236" radius="0.008" />
-        </geometry>
-      </collision>
-      <collision>
-        <origin xyz="0 -0.040987 -0.057684" rpy="0 0 0" />
-        <geometry>
-          <cylinder length="0.131626" radius="0.008" />
-        </geometry>
-      </collision>
-      <collision>
-        <origin xyz="0 -0.022511 -0.115497" rpy="${pi/2} 0 0" />
-        <geometry>
-          <cylinder length="0.052952" radius="0.008" />
-        </geometry>
-      </collision>
-    </link>
+        <geometry>
+          <mesh filename="package://iai_apartment/meshes/handles/window_handle.obj" />
+        </geometry>
+      </collision>
+    </link>
+    <!-- left window -->
     <joint name="window4_left_joint" type="revolute">
       <origin xyz="-0.929112 0.00162 -0.425471" />
@@ -153,13 +140,12 @@
       </collision>
     </link>
-    <joint name="window4_left_handle_joint" type="revolute">
-      <origin xyz="0.834107 -0.019236 0.0" />
+    <joint name="window4_left_handle_joint" type="fixed">
+      <origin xyz="0.815383 -0.06 -0.058" rpy="${pi} 0 ${pi/2}"/>
       <parent link="window4_left" />
       <child link="window4_left_handle" />
-      <axis xyz="0 -1 0" />
-      <limit effort="1000.0" lower="0.0" upper="${pi}" velocity="${pi}" />
     </joint>
     <link name="window4_left_handle">
       <visual>
+        <origin rpy="0 0 0"/>
         <geometry>
           <mesh filename="package://iai_apartment/meshes/unreal/SM_Window_Handle.dae" />
@@ -167,19 +153,6 @@
       </visual>
       <collision>
-        <origin xyz="0 -0.011369 0" rpy="${pi/2} 0 0" />
-        <geometry>
-          <cylinder length="0.075236" radius="0.008" />
-        </geometry>
-      </collision>
-      <collision>
-        <origin xyz="0 -0.040987 -0.057684" rpy="0 0 0" />
-        <geometry>
-          <cylinder length="0.131626" radius="0.008" />
-        </geometry>
-      </collision>
-      <collision>
-        <origin xyz="0 -0.022511 -0.115497" rpy="${pi/2} 0 0" />
-        <geometry>
-          <cylinder length="0.052952" radius="0.008" />
+        <geometry>
+          <mesh filename="package://iai_apartment/meshes/handles/window_handle.obj" />
         </geometry>
       </collision>

Commit message: Add rotation joint for window4_handle

File: iai_apartment/urdf/furnitures_with_window4.xacro (robot description, xacro)
@@ -131,7 +131,15 @@
       </collision>
     </link>
+    <joint name="window4_right_handle_rotation_joint" type="revolute">
+      <origin xyz="0.017383 0.834107 0.0" rpy="0 0 0" />
+      <parent link="window4_right" />
+      <child link="window4_right_handle_rotation" />
+      <axis xyz="-1 0 0" />
+      <limit effort="1000.0" lower="0.0" upper="1.5708" velocity="1.5708" />
+    </joint>
+    <link name="window4_right_handle_rotation"/>
     <joint name="window4_right_handle_joint" type="fixed">
-      <origin xyz="0.055 0.834107 -0.057684" rpy="0 0 0" />
-      <parent link="window4_right" />
+      <origin xyz="0.037617 0 -0.057755" rpy="0 0 0" />
+      <parent link="window4_right_handle_rotation" />
       <child link="window4_right_handle" />
     </joint>
@@ -181,7 +189,15 @@
       </collision>
     </link>
+    <joint name="window4_left_handle_rotation_joint" type="revolute">
+      <origin xyz="0.017383 -0.834107 0.0" rpy="0 0 0" />
+      <parent link="window4_left" />
+      <child link="window4_left_handle_rotation" />
+      <axis xyz="1 0 0" />
+      <limit effort="1000.0" lower="0.0" upper="1.5708" velocity="1.5708" />
+    </joint>
+    <link name="window4_left_handle_rotation"/>
     <joint name="window4_left_handle_joint" type="fixed">
-      <origin xyz="0.055 -0.834107 -0.057684" rpy="0 0 0" />
-      <parent link="window4_left" />
+      <origin xyz="0.037617 0 -0.057755" rpy="0 0 0" />
+      <parent link="window4_left_handle_rotation" />
       <child link="window4_left_handle" />
     </joint>
