Commit message: Add cabinet1

File: iai_apartment/urdf/kitchen_unreal.xacro (robot description, xacro)
@@ -11,5 +11,5 @@
     <!-- Cabinet1 -->
     <joint name="cabinet1_joint" type="fixed">
-      <origin xyz="0.0 1.46675873 1.11440605" rpy="0.0 0.0 0.0" />
+      <origin xyz="0.28463219 1.46675873 1.11440605" rpy="0.0 0.0 ${pi/2}" />
       <parent link="kitchen_root" />
       <child link="cabinet1" />
@@ -70,4 +70,238 @@
       </collision>
     </link>
+    <joint name="cabinet1_door_joint" type="revolute">
+      <origin xyz="-0.274 -0.280 0.677" rpy="0.0 0.0 0.0" />
+      <parent link="cabinet1" />
+      <child link="cabinet1_door" />
+      <axis xyz="0 0 1" />
+      <limit effort="1000.0" lower="-${pi/2}" upper="0.0" velocity="${pi/2}" />
+    </joint>
+    <link name="cabinet1_door">
+      <visual>
+        <geometry>
+          <mesh filename="package://iai_apartment/meshes/unreal/cabinet01/SM_Kitchen_01_Door_01.obj" />
+        </geometry>
+      </visual>
+      <collision>
+        <origin xyz="0.285091 -0.00064702 0.0" />
+        <geometry>
+          <box size="0.596936 0.019 0.86681" />
+        </geometry>
+      </collision>
+    </link>
+    <joint name="cabinet1_door_handle_joint" type="fixed">
+      <origin xyz="0.46315559 -0.01559982 -0.38983368" rpy="0.0 0.0 0.0" />
+      <parent link="cabinet1_door" />
+      <child link="cabinet1_door_handle" />
+    </joint>
+    <link name="cabinet1_door_handle">
+      <visual>
+        <geometry>
+          <mesh filename="package://iai_apartment/meshes/unreal/handles/SM_Kitchen_Handle.obj" />
+        </geometry>
+      </visual>
+      <collision>
+        <origin xyz="0.08 -0.003891  0.0" />
+        <geometry>
+          <box size="0.013 0.02 0.013" />
+        </geometry>
+      </collision>
+      <collision>
+        <origin xyz="-0.08 -0.003891  0.0" />
+        <geometry>
+          <box size="0.013 0.02 0.013" />
+        </geometry>
+      </collision>
+      <collision>
+        <origin xyz="0.0 -0.0203895 0.0" />
+        <geometry>
+          <box size="0.173032 0.013 0.013" />
+        </geometry>
+      </collision>
+    </link>
+    <joint name="cabinet1_drawer_middle_joint" type="prismatic">
+      <origin xyz="0.01122015 -0.04679018 -0.48658508" rpy="0.0 0.0 0.0" />
+      <parent link="cabinet1" />
+      <child link="cabinet1_drawer_middle" />
+      <axis xyz="0 -1 0" />
+      <limit effort="1000.0" lower="0.0" upper="0.45" velocity="0.5" />
+    </joint>
+    <link name="cabinet1_drawer_middle">
+      <visual>
+        <geometry>
+          <mesh filename="package://iai_apartment/meshes/unreal/cabinet01/SM_Kitchen_01_Drawer_01.obj" />
+        </geometry>
+      </visual>
+      <collision>
+        <origin xyz="0.0 -0.233977 0.0" />
+        <geometry>
+          <box size="0.596936 0.019 0.262972" />
+        </geometry>
+      </collision>
+      <collision>
+        <origin xyz="0.26865 0.021336 0.0412455" />
+        <geometry>
+          <box size="0.0158442 0.4917 0.0223924" />
+        </geometry>
+      </collision>
+      <collision>
+        <origin xyz="-0.26865 0.021336 0.0412455" />
+        <geometry>
+          <box size="0.0158442 0.4917 0.0223924" />
+        </geometry>
+      </collision>
+      <collision>
+        <origin xyz="0.26865 0.021336 -0.078968" />
+        <geometry>
+          <box size="0.0158442 0.4917 0.083496" />
+        </geometry>
+      </collision>
+      <collision>
+        <origin xyz="-0.26865 0.021336 -0.0941" />
+        <geometry>
+          <box size="0.0158442 0.4917 0.053098" />
+        </geometry>
+      </collision>
+      <collision>
+        <origin xyz="0.0 0.021399 -0.114232" />
+        <geometry>
+          <box size="0.52364 0.49156 0.016" />
+        </geometry>
+      </collision>
+      <collision>
+        <origin xyz="0.0 0.26 -0.038" />
+        <geometry>
+          <box size="0.52364 0.01865384 0.16887" />
+        </geometry>
+      </collision>
+    </link>
+    <joint name="cabinet1_drawer_middle_handle_joint" type="fixed">
+      <origin xyz="0.00091816 -0.24792936 0.08401428" rpy="0.0 0.0 0.0" />
+      <parent link="cabinet1_drawer_middle" />
+      <child link="cabinet1_drawer_middle_handle" />
+    </joint>
+    <link name="cabinet1_drawer_middle_handle">
+      <visual>
+        <geometry>
+          <mesh filename="package://iai_apartment/meshes/unreal/handles/SM_Kitchen_Handle.obj" />
+        </geometry>
+      </visual>
+      <collision>
+        <origin xyz="0.08 -0.003891  0.0" />
+        <geometry>
+          <box size="0.013 0.02 0.013" />
+        </geometry>
+      </collision>
+      <collision>
+        <origin xyz="-0.08 -0.003891  0.0" />
+        <geometry>
+          <box size="0.013 0.02 0.013" />
+        </geometry>
+      </collision>
+      <collision>
+        <origin xyz="0.0 -0.0203895 0.0" />
+        <geometry>
+          <box size="0.173032 0.013 0.013" />
+        </geometry>
+      </collision>
+    </link>
+    <joint name="cabinet1_drawer_bottom_joint" type="prismatic">
+      <origin xyz="0.011 -0.046 -0.816" rpy="0.0 0.0 0.0" />
+      <parent link="cabinet1" />
+      <child link="cabinet1_drawer_bottom" />
+      <axis xyz="0 -1 0" />
+      <limit effort="1000.0" lower="0.0" upper="0.45" velocity="0.5" />
+    </joint>
+    <link name="cabinet1_drawer_bottom">
+      <visual>
+        <geometry>
+          <mesh filename="package://iai_apartment/meshes/unreal/cabinet01/SM_Kitchen_01_Drawer_02.obj" />
+        </geometry>
+      </visual>
+      <collision>
+        <origin xyz="0.0 -0.233977 0.0" />
+        <geometry>
+          <box size="0.596936 0.019 0.39428" />
+        </geometry>
+      </collision>
+      <collision>
+        <origin xyz="0.26865 0.021336 -0.0084109" />
+        <geometry>
+          <box size="0.0158442 0.4917 0.0223924" />
+        </geometry>
+      </collision>
+      <collision>
+        <origin xyz="-0.26865 0.021336 -0.0084109" />
+        <geometry>
+          <box size="0.0158442 0.4917 0.0223924" />
+        </geometry>
+      </collision>
+      <collision>
+        <origin xyz="0.26865 0.021336 -0.12854" />
+        <geometry>
+          <box size="0.0158442 0.4917 0.083502" />
+        </geometry>
+      </collision>
+      <collision>
+        <origin xyz="-0.26865 0.021336 -0.12854" />
+        <geometry>
+          <box size="0.0158442 0.4917 0.083502" />
+        </geometry>
+      </collision>
+      <collision>
+        <origin xyz="0.0 0.021399 -0.16226" />
+        <geometry>
+          <box size="0.52364 0.49156 0.016" />
+        </geometry>
+      </collision>
+      <collision>
+        <origin xyz="0.0 0.26 -0.0797358 " />
+        <geometry>
+          <box size="0.52364 0.01865384 0.1517224" />
+        </geometry>
+      </collision>
+    </link>
+    <joint name="cabinet1_drawer_bottom_handle_joint" type="fixed">
+      <origin xyz="0.00145845 -0.24909416 0.150606" rpy="0.0 0.0 0.0" />
+      <parent link="cabinet1_drawer_bottom" />
+      <child link="cabinet1_drawer_bottom_handle" />
+    </joint>
+    <link name="cabinet1_drawer_bottom_handle">
+      <visual>
+        <geometry>
+          <mesh filename="package://iai_apartment/meshes/unreal/handles/SM_Kitchen_Handle.obj" />
+        </geometry>
+      </visual>
+      <collision>
+        <origin xyz="0.08 -0.003891  0.0" />
+        <geometry>
+          <box size="0.013 0.02 0.013" />
+        </geometry>
+      </collision>
+      <collision>
+        <origin xyz="-0.08 -0.003891  0.0" />
+        <geometry>
+          <box size="0.013 0.02 0.013" />
+        </geometry>
+      </collision>
+      <collision>
+        <origin xyz="0.0 -0.0203895 0.0" />
+        <geometry>
+          <box size="0.173032 0.013 0.013" />
+        </geometry>
+      </collision>
+    </link>
+    <joint name="oven_joint" type="fixed">
+      <origin xyz="0.0123597 -0.27395857 -0.3426725" rpy="0 0 0" />
+      <parent link="cabinet1" />
+      <child link="oven" />
+    </joint>
+    <link name="oven">
+      <visual>
+        <geometry>
+          <mesh filename="package://iai_apartment/meshes/unreal/oven/SM_Oven.obj" />
+        </geometry>
+      </visual>
+    </link>
   </xacro:macro>
 </robot>

Commit message: Add cabinet2 and catbinet3

File: iai_apartment/urdf/kitchen_unreal.xacro (robot description, xacro)
@@ -18,5 +18,5 @@
       <visual>
         <geometry>
-          <mesh filename="package://iai_apartment/meshes/unreal/cabinet01/SM_Kitchen_01_Base.obj" />
+          <mesh filename="package://iai_apartment/meshes/unreal/SM_Kitchen_01_Base.dae" />
         </geometry>
       </visual>
@@ -80,5 +80,5 @@
       <visual>
         <geometry>
-          <mesh filename="package://iai_apartment/meshes/unreal/cabinet01/SM_Kitchen_01_Door_01.obj" />
+          <mesh filename="package://iai_apartment/meshes/unreal/SM_Kitchen_01_Door_01.dae" />
         </geometry>
       </visual>
@@ -98,5 +98,5 @@
       <visual>
         <geometry>
-          <mesh filename="package://iai_apartment/meshes/unreal/handles/SM_Kitchen_Handle.obj" />
+          <mesh filename="package://iai_apartment/meshes/unreal/SM_Kitchen_Handle.dae" />
         </geometry>
       </visual>
@@ -130,5 +130,5 @@
       <visual>
         <geometry>
-          <mesh filename="package://iai_apartment/meshes/unreal/cabinet01/SM_Kitchen_01_Drawer_01.obj" />
+          <mesh filename="package://iai_apartment/meshes/unreal/SM_Kitchen_01_Drawer_01.dae" />
         </geometry>
       </visual>
@@ -184,5 +184,5 @@
       <visual>
         <geometry>
-          <mesh filename="package://iai_apartment/meshes/unreal/handles/SM_Kitchen_Handle.obj" />
+          <mesh filename="package://iai_apartment/meshes/unreal/SM_Kitchen_Handle.dae" />
         </geometry>
       </visual>
@@ -216,5 +216,5 @@
       <visual>
         <geometry>
-          <mesh filename="package://iai_apartment/meshes/unreal/cabinet01/SM_Kitchen_01_Drawer_02.obj" />
+          <mesh filename="package://iai_apartment/meshes/unreal/SM_Kitchen_01_Drawer_02.dae" />
         </geometry>
       </visual>
@@ -270,5 +270,5 @@
       <visual>
         <geometry>
-          <mesh filename="package://iai_apartment/meshes/unreal/handles/SM_Kitchen_Handle.obj" />
+          <mesh filename="package://iai_apartment/meshes/unreal/SM_Kitchen_Handle.dae" />
         </geometry>
       </visual>
@@ -300,7 +300,1031 @@
       <visual>
         <geometry>
-          <mesh filename="package://iai_apartment/meshes/unreal/oven/SM_Oven.obj" />
-        </geometry>
-      </visual>
+          <mesh filename="package://iai_apartment/meshes/unreal/SM_Oven.dae" />
+        </geometry>
+      </visual>
+      <collision>
+        <origin xyz="-0.003055 0.264778 0.50654" />
+        <geometry>
+          <box size="0.58989 0.545666 0.150842" />
+        </geometry>
+      </collision>
+      <collision>
+        <origin xyz="-0.003055 0.264778 0.018039" />
+        <geometry>
+          <box size="0.58989 0.545666 0.045598" />
+        </geometry>
+      </collision>
+      <collision>
+        <origin xyz="-0.2675 0.264778 0.288951" />
+        <geometry>
+          <box size="0.059 0.545666 0.586022" />
+        </geometry>
+      </collision>
+      <collision>
+        <origin xyz="0.264104 0.264778 0.288951" />
+        <geometry>
+          <box size="0.054902 0.545666 0.586022" />
+        </geometry>
+      </collision>
+      <collision>
+        <origin xyz="-0.003055 0.5 0.288951" />
+        <geometry>
+          <box size="0.58989 0.074784 0.586022" />
+        </geometry>
+      </collision>
+    </link>
+    <joint name="oven_door_joint" type="revolute">
+      <origin xyz="0.0 0.0 0.0" rpy="0 0 0" />
+      <parent link="oven" />
+      <child link="oven_door" />
+      <axis xyz="1 0 0" />
+      <limit effort="1000.0" lower="0.0" upper="${pi/2}" velocity="${pi/2}" />
+    </joint>
+    <link name="oven_door">
+      <visual>
+        <geometry>
+          <mesh filename="package://iai_apartment/meshes/unreal/SM_Oven_Door.dae" />
+        </geometry>
+      </visual>
+      <collision>
+        <origin xyz="-0.002993 0.005395 0.226757" />
+        <geometry>
+          <box size="0.590588 0.036998 0.471696" />
+        </geometry>
+      </collision>
+    </link>
+    <!-- Cabinet2 -->
+    <joint name="cabinet2_joint" type="fixed">
+      <origin xyz="0.27990936 1.97705429 1.16238914" rpy="0.0 0.0 ${pi/2}" />
+      <parent link="kitchen_root" />
+      <child link="cabinet2" />
+    </joint>
+    <link name="cabinet2">
+      <visual>
+        <geometry>
+          <mesh filename="package://iai_apartment/meshes/unreal/SM_Kitchen_02_Base.dae" />
+        </geometry>
+      </visual>
+      <collision>
+        <origin xyz="-0.191979 0.005897 0.0" />
+        <geometry>
+          <box size="0.016 0.554718 2.12768" />
+        </geometry>
+      </collision>
+      <collision>
+        <origin xyz="0.191979 0.005897 0.0" />
+        <geometry>
+          <box size="0.016 0.554718 2.12768" />
+        </geometry>
+      </collision>
+      <collision>
+        <origin xyz="0.0 0.005897 1.05584" />
+        <geometry>
+          <box size="0.367764 0.554718 0.016" />
+        </geometry>
+      </collision>
+      <collision>
+        <origin xyz="0.0 0.005897 0.975845" />
+        <geometry>
+          <box size="0.367764 0.554718 0.016" />
+        </geometry>
+      </collision>
+      <collision>
+        <origin xyz="0.0 0.005897 -1.05594" />
+        <geometry>
+          <box size="0.367764 0.554718 0.016" />
+        </geometry>
+      </collision>
+      <collision>
+        <origin xyz="0.0 -0.26039 1.01584" />
+        <geometry>
+          <box size="0.367764 0.014374 0.063992" />
+        </geometry>
+      </collision>
+      <collision>
+        <origin xyz="0.0 0.267372 0.0" />
+        <geometry>
+          <box size="0.367764 0.008 2.09568" />
+        </geometry>
+      </collision>
+    </link>
+    <joint name="cabinet2_shelf_joint" type="fixed">
+      <origin xyz="-0.00043732 -0.00337784 0.79036064" rpy="0.0 0.0 0.0" />
+      <parent link="cabinet2" />
+      <child link="cabinet2_shelf" />
+    </joint>
+    <link name="cabinet2_shelf">
+      <visual>
+        <geometry>
+          <mesh filename="package://iai_apartment/meshes/unreal/SM_Kitchen_02_Shelf.dae" />
+        </geometry>
+      </visual>
+    </link>
+    <joint name="cabinet2_drawer1_joint" type="prismatic">
+      <origin xyz="0.00134538 -0.00464775 0.58046211" rpy="0.0 0.0 0.0" />
+      <parent link="cabinet2" />
+      <child link="cabinet2_drawer1" />
+      <axis xyz="0 -1 0" />
+      <limit effort="1000.0" lower="0.0" upper="0.45" velocity="0.5" />
+    </joint>
+    <link name="cabinet2_drawer1">
+      <visual>
+        <geometry>
+          <mesh filename="package://iai_apartment/meshes/unreal/SM_Kitchen_02_Drawer_01.dae" />
+        </geometry>
+      </visual>
+      <collision>
+        <origin xyz="0.0 -0.242975 0.0" />
+        <geometry>
+          <box size="0.361962 0.017 0.10099" />
+        </geometry>
+      </collision>
+      <collision>
+        <origin xyz="0.0 0.235441 0.0" />
+        <geometry>
+          <box size="0.361962 0.016128 0.10099" />
+        </geometry>
+      </collision>
+      <collision>
+        <origin xyz="-0.170578 -0.003984 0.0" />
+        <geometry>
+          <box size="0.016222 0.494978 0.10099" />
+        </geometry>
+      </collision>
+      <collision>
+        <origin xyz="0.170578 -0.003984 0.0" />
+        <geometry>
+          <box size="0.016222 0.494978 0.10099" />
+        </geometry>
+      </collision>
+      <collision>
+        <origin xyz="0.0 -0.003984 -0.039746" />
+        <geometry>
+          <box size="0.361962 0.494978 0.021498" />
+        </geometry>
+      </collision>
+    </link>
+    <joint name="cabinet2_drawer2_joint" type="prismatic">
+      <origin xyz="0.00134538 -0.00464775 0.4227494" rpy="0.0 0.0 0.0" />
+      <parent link="cabinet2" />
+      <child link="cabinet2_drawer2" />
+      <axis xyz="0 -1 0" />
+      <limit effort="1000.0" lower="0.0" upper="0.45" velocity="0.5" />
+    </joint>
+    <link name="cabinet2_drawer2">
+      <visual>
+        <geometry>
+          <mesh filename="package://iai_apartment/meshes/unreal/SM_Kitchen_02_Drawer_02.dae" />
+        </geometry>
+      </visual>
+      <collision>
+        <origin xyz="0.0 -0.242374 -0.042" />
+        <geometry>
+          <box size="0.361962 0.013796 0.098" />
+        </geometry>
+      </collision>
+      <collision>
+        <origin xyz="0.0 -0.242374 0.060843" />
+        <geometry>
+          <box size="0.361962 0.013796 0.020298" />
+        </geometry>
+      </collision>
+      <collision>
+        <origin xyz="-0.148428 -0.242869 0.0" />
+        <geometry>
+          <box size="0.064882 0.016786 0.18198" />
+        </geometry>
+      </collision>
+      <collision>
+        <origin xyz="0.148428 -0.242869 0.0" />
+        <geometry>
+          <box size="0.064882 0.016786 0.18198" />
+        </geometry>
+      </collision>
+      <collision>
+        <origin xyz="0.0 0.235441 0.0" />
+        <geometry>
+          <box size="0.361962 0.016128 0.181758" />
+        </geometry>
+      </collision>
+      <collision>
+        <origin xyz="-0.170578 -0.003984 0.075342" />
+        <geometry>
+          <box size="0.016222 0.494978 0.023298" />
+        </geometry>
+      </collision>
+      <collision>
+        <origin xyz="0.170578 -0.003984 0.075342" />
+        <geometry>
+          <box size="0.016222 0.494978 0.023298" />
+        </geometry>
+      </collision>
+      <collision>
+        <origin xyz="-0.170578 -0.003984 -0.043743" />
+        <geometry>
+          <box size="0.016222 0.494978 0.087106" />
+        </geometry>
+      </collision>
+      <collision>
+        <origin xyz="0.170578 -0.003984 -0.043743" />
+        <geometry>
+          <box size="0.016222 0.494978 0.087106" />
+        </geometry>
+      </collision>
+      <collision>
+        <origin xyz="0.0 -0.003984 -0.080242" />
+        <geometry>
+          <box size="0.361962 0.494978 0.021498" />
+        </geometry>
+      </collision>
+    </link>
+    <joint name="cabinet2_drawer3_joint" type="prismatic">
+      <origin xyz="0.00134538 -0.00464775 0.1428965" rpy="0.0 0.0 0.0" />
+      <parent link="cabinet2" />
+      <child link="cabinet2_drawer3" />
+      <axis xyz="0 -1 0" />
+      <limit effort="1000.0" lower="0.0" upper="0.45" velocity="0.5" />
+    </joint>
+    <link name="cabinet2_drawer3">
+      <visual>
+        <geometry>
+          <mesh filename="package://iai_apartment/meshes/unreal/SM_Kitchen_02_Drawer_02.dae" />
+        </geometry>
+      </visual>
+      <collision>
+        <origin xyz="0.0 -0.242374 -0.042" />
+        <geometry>
+          <box size="0.361962 0.013796 0.098" />
+        </geometry>
+      </collision>
+      <collision>
+        <origin xyz="0.0 -0.242374 0.060843" />
+        <geometry>
+          <box size="0.361962 0.013796 0.020298" />
+        </geometry>
+      </collision>
+      <collision>
+        <origin xyz="-0.148428 -0.242869 0.0" />
+        <geometry>
+          <box size="0.064882 0.016786 0.18198" />
+        </geometry>
+      </collision>
+      <collision>
+        <origin xyz="0.148428 -0.242869 0.0" />
+        <geometry>
+          <box size="0.064882 0.016786 0.18198" />
+        </geometry>
+      </collision>
+      <collision>
+        <origin xyz="0.0 0.235441 0.0" />
+        <geometry>
+          <box size="0.361962 0.016128 0.181758" />
+        </geometry>
+      </collision>
+      <collision>
+        <origin xyz="-0.170578 -0.003984 0.075342" />
+        <geometry>
+          <box size="0.016222 0.494978 0.023298" />
+        </geometry>
+      </collision>
+      <collision>
+        <origin xyz="0.170578 -0.003984 0.075342" />
+        <geometry>
+          <box size="0.016222 0.494978 0.023298" />
+        </geometry>
+      </collision>
+      <collision>
+        <origin xyz="-0.170578 -0.003984 -0.043743" />
+        <geometry>
+          <box size="0.016222 0.494978 0.087106" />
+        </geometry>
+      </collision>
+      <collision>
+        <origin xyz="0.170578 -0.003984 -0.043743" />
+        <geometry>
+          <box size="0.016222 0.494978 0.087106" />
+        </geometry>
+      </collision>
+      <collision>
+        <origin xyz="0.0 -0.003984 -0.080242" />
+        <geometry>
+          <box size="0.361962 0.494978 0.021498" />
+        </geometry>
+      </collision>
+    </link>
+    <joint name="cabinet2_drawer4_joint" type="prismatic">
+      <origin xyz="0.00134538 -0.00464775 -0.24243713" rpy="0.0 0.0 0.0" />
+      <parent link="cabinet2" />
+      <child link="cabinet2_drawer4" />
+      <axis xyz="0 -1 0" />
+      <limit effort="1000.0" lower="0.0" upper="0.45" velocity="0.5" />
+    </joint>
+    <link name="cabinet2_drawer4">
+      <visual>
+        <geometry>
+          <mesh filename="package://iai_apartment/meshes/unreal/SM_Kitchen_02_Drawer_02.dae" />
+        </geometry>
+      </visual>
+      <collision>
+        <origin xyz="0.0 -0.242374 -0.042" />
+        <geometry>
+          <box size="0.361962 0.013796 0.098" />
+        </geometry>
+      </collision>
+      <collision>
+        <origin xyz="0.0 -0.242374 0.060843" />
+        <geometry>
+          <box size="0.361962 0.013796 0.020298" />
+        </geometry>
+      </collision>
+      <collision>
+        <origin xyz="-0.148428 -0.242869 0.0" />
+        <geometry>
+          <box size="0.064882 0.016786 0.18198" />
+        </geometry>
+      </collision>
+      <collision>
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