Commit message: Add cabinet4

File: iai_apartment/urdf/kitchen_unreal.xacro (robot description, xacro)
@@ -8,5 +8,4 @@
     </joint>
     <link name="kitchen_root" />
-    <!-- - - - - - - - - - - - - Cabinets side A - - - - - - - - - -->
     <!-- Cabinet1 -->
     <joint name="cabinet1_joint" type="fixed">
@@ -74,6 +73,6 @@
       <parent link="cabinet1" />
       <child link="cabinet1_door" />
-      <axis xyz="0 0 1" />
-      <limit effort="1000.0" lower="-${pi/2}" upper="0.0" velocity="${pi/2}" />
+      <axis xyz="0 0 -1" />
+      <limit effort="1000.0" lower="0.0" upper="${pi/2}" velocity="${pi/2}" />
     </joint>
     <link name="cabinet1_door">
@@ -91,5 +90,5 @@
     </link>
     <joint name="cabinet1_door_handle_joint" type="fixed">
-      <origin xyz="0.46315559 -0.01559982 -0.38983368" rpy="0.0 0.0 0.0" />
+      <origin xyz="0.46315559 -0.01559982 -0.38983368" rpy="0.0 0.0 ${pi/2}" />
       <parent link="cabinet1_door" />
       <child link="cabinet1_door_handle" />
@@ -120,12 +119,12 @@
       </collision>
     </link>
-    <joint name="cabinet1_drawer_middle_joint" type="prismatic">
+    <joint name="cabinet1_drawer1_joint" type="prismatic">
       <origin xyz="0.01122015 -0.04679018 -0.48658508" rpy="0.0 0.0 0.0" />
       <parent link="cabinet1" />
-      <child link="cabinet1_drawer_middle" />
+      <child link="cabinet1_drawer1" />
       <axis xyz="0 -1 0" />
       <limit effort="1000.0" lower="0.0" upper="0.45" velocity="0.5" />
     </joint>
-    <link name="cabinet1_drawer_middle">
+    <link name="cabinet1_drawer1">
       <visual>
         <geometry>
@@ -176,10 +175,10 @@
       </collision>
     </link>
-    <joint name="cabinet1_drawer_middle_handle_joint" type="fixed">
-      <origin xyz="0.00091816 -0.24792936 0.08401428" rpy="0.0 0.0 0.0" />
-      <parent link="cabinet1_drawer_middle" />
-      <child link="cabinet1_drawer_middle_handle" />
-    </joint>
-    <link name="cabinet1_drawer_middle_handle">
+    <joint name="cabinet1_drawer1_handle_joint" type="fixed">
+      <origin xyz="0.00091816 -0.24792936 0.08401428" rpy="0.0 0.0 ${pi/2}" />
+      <parent link="cabinet1_drawer1" />
+      <child link="cabinet1_drawer1_handle" />
+    </joint>
+    <link name="cabinet1_drawer1_handle">
       <visual>
         <geometry>
@@ -206,12 +205,12 @@
       </collision>
     </link>
-    <joint name="cabinet1_drawer_bottom_joint" type="prismatic">
+    <joint name="cabinet1_drawer2_joint" type="prismatic">
       <origin xyz="0.011 -0.046 -0.816" rpy="0.0 0.0 0.0" />
       <parent link="cabinet1" />
-      <child link="cabinet1_drawer_bottom" />
+      <child link="cabinet1_drawer2" />
       <axis xyz="0 -1 0" />
       <limit effort="1000.0" lower="0.0" upper="0.45" velocity="0.5" />
     </joint>
-    <link name="cabinet1_drawer_bottom">
+    <link name="cabinet1_drawer2">
       <visual>
         <geometry>
@@ -262,10 +261,10 @@
       </collision>
     </link>
-    <joint name="cabinet1_drawer_bottom_handle_joint" type="fixed">
-      <origin xyz="0.00145845 -0.24909416 0.150606" rpy="0.0 0.0 0.0" />
-      <parent link="cabinet1_drawer_bottom" />
-      <child link="cabinet1_drawer_bottom_handle" />
-    </joint>
-    <link name="cabinet1_drawer_bottom_handle">
+    <joint name="cabinet1_drawer2_handle_joint" type="fixed">
+      <origin xyz="0.00145845 -0.24909416 0.150606" rpy="0.0 0.0 ${pi/2}" />
+      <parent link="cabinet1_drawer2" />
+      <child link="cabinet1_drawer2_handle" />
+    </joint>
+    <link name="cabinet1_drawer2_handle">
       <visual>
         <geometry>
@@ -409,4 +408,54 @@
       </collision>
     </link>
+    <joint name="cabinet2_door_joint" type="revolute">
+      <origin xyz="-0.17998091 -0.29852444 0.00105865" rpy="0.0 0.0 0.0" />
+      <parent link="cabinet2" />
+      <child link="cabinet2_door" />
+      <axis xyz="0 0 -1" />
+      <limit effort="1000.0" lower="0.0" upper="${pi/2}" velocity="${pi/2}" />
+    </joint>
+    <link name="cabinet2_door">
+      <visual>
+        <geometry>
+          <mesh filename="package://iai_apartment/meshes/unreal/SM_Kitchen_02_Door.dae" />
+        </geometry>
+      </visual>
+      <collision>
+        <origin xyz="0.180483 0.013597 0.0" />
+        <geometry>
+          <box size="0.395846 0.018678 2.12276" />
+        </geometry>
+      </collision>
+    </link>
+    <joint name="cabinet2_door_handle_joint" type="fixed">
+      <origin xyz="0.25886013 -0.00184994 -0.05118866" rpy="0.0 0.0 ${pi/2}" />
+      <parent link="cabinet2_door" />
+      <child link="cabinet2_door_handle" />
+    </joint>
+    <link name="cabinet2_door_handle">
+      <visual>
+        <geometry>
+          <mesh filename="package://iai_apartment/meshes/unreal/SM_Kitchen_Handle.dae" />
+        </geometry>
+      </visual>
+      <collision>
+        <origin xyz="0.08 -0.003891  0.0" />
+        <geometry>
+          <box size="0.013 0.02 0.013" />
+        </geometry>
+      </collision>
+      <collision>
+        <origin xyz="-0.08 -0.003891  0.0" />
+        <geometry>
+          <box size="0.013 0.02 0.013" />
+        </geometry>
+      </collision>
+      <collision>
+        <origin xyz="0.0 -0.0203895 0.0" />
+        <geometry>
+          <box size="0.173032 0.013 0.013" />
+        </geometry>
+      </collision>
+    </link>
     <joint name="cabinet2_shelf_joint" type="fixed">
       <origin xyz="-0.00043732 -0.00337784 0.79036064" rpy="0.0 0.0 0.0" />
@@ -835,57 +884,7 @@
       </collision>
     </link>
-    <joint name="cabinet2_door_joint" type="revolute">
-      <origin xyz="-0.17998091 -0.29852444 0.00105865" rpy="0.0 0.0 0.0" />
-      <parent link="cabinet2" />
-      <child link="cabinet2_door" />
-      <axis xyz="0 0 1" />
-      <limit effort="1000.0" lower="-${pi/2}" upper="0.0" velocity="${pi/2}" />
-    </joint>
-    <link name="cabinet2_door">
-      <visual>
-        <geometry>
-          <mesh filename="package://iai_apartment/meshes/unreal/SM_Kitchen_02_Door.dae" />
-        </geometry>
-      </visual>
-      <collision>
-        <origin xyz="0.180483 0.013597 0.0" />
-        <geometry>
-          <box size="0.395846 0.018678 2.12276" />
-        </geometry>
-      </collision>
-    </link>
-    <joint name="cabinet2_door_handle_joint" type="fixed">
-      <origin xyz="0.25886013 -0.00184994 -0.05118866" rpy="0.0 0.0 0.0" />
-      <parent link="cabinet2_door" />
-      <child link="cabinet2_door_handle" />
-    </joint>
-    <link name="cabinet2_door_handle">
-      <visual>
-        <geometry>
-          <mesh filename="package://iai_apartment/meshes/unreal/SM_Kitchen_Handle.dae" />
-        </geometry>
-      </visual>
-      <collision>
-        <origin xyz="0.08 -0.003891  0.0" />
-        <geometry>
-          <box size="0.013 0.02 0.013" />
-        </geometry>
-      </collision>
-      <collision>
-        <origin xyz="-0.08 -0.003891  0.0" />
-        <geometry>
-          <box size="0.013 0.02 0.013" />
-        </geometry>
-      </collision>
-      <collision>
-        <origin xyz="0.0 -0.0203895 0.0" />
-        <geometry>
-          <box size="0.173032 0.013 0.013" />
-        </geometry>
-      </collision>
-    </link>
     <!-- Cabinet3 -->
     <joint name="cabinet3_joint" type="fixed">
-      <origin xyz="0.27498539 2.47989822 1.16287888" rpy="0.0 0.0 ${-pi/2}" />
+      <origin xyz="0.27498539 2.47989822 1.16287888" rpy="0.0 0.0 ${pi/2}" />
       <parent link="kitchen_root" />
       <child link="cabinet3" />
@@ -898,5 +897,5 @@
       </visual>
       <collision>
-        <origin xyz="0.291968 -0.003155 0.0" />
+        <origin xyz="0.291968 0.003155 0.0" />
         <geometry>
           <box size="0.02 0.554386 2.12764" />
@@ -904,5 +903,5 @@
       </collision>
       <collision>
-        <origin xyz="-0.291968 -0.003155 0.0" />
+        <origin xyz="-0.291968 0.003155 0.0" />
         <geometry>
           <box size="0.02 0.554386 2.12764" />
@@ -910,5 +909,5 @@
       </collision>
       <collision>
-        <origin xyz="0.0 -0.003155 1.05584" />
+        <origin xyz="0.0 0.003155 1.05584" />
         <geometry>
           <box size="0.572134 0.554386 0.016" />
@@ -916,5 +915,5 @@
       </collision>
       <collision>
-        <origin xyz="0.0 -0.003155 0.895854" />
+        <origin xyz="0.0 0.003155 0.895854" />
         <geometry>
           <box size="0.572134 0.554386 0.016" />
@@ -922,5 +921,5 @@
       </collision>
       <collision>
-        <origin xyz="0.0 -0.003155 0.819863" />
+        <origin xyz="0.0 0.003155 0.819863" />
         <geometry>
           <box size="0.572134 0.554386 0.016" />
@@ -928,5 +927,5 @@
       </collision>
       <collision>
-        <origin xyz="0.0 -0.003155 -0.980943" />
+        <origin xyz="0.0 0.003155 -0.980943" />
         <geometry>
           <box size="0.572134 0.554386 0.016" />
@@ -934,5 +933,5 @@
       </collision>
       <collision>
-        <origin xyz="0.0 -0.003155 -1.05594" />
+        <origin xyz="0.0 0.003155 -1.05594" />
         <geometry>
           <box size="0.572134 0.554386 0.016" />
@@ -940,5 +939,5 @@
       </collision>
       <collision>
-        <origin xyz="0.0 0.262453 0.975825" />
+        <origin xyz="0.0 -0.262453 0.975825" />
         <geometry>
           <box size="0.572134 0.0209188 0.14402" />
@@ -946,5 +945,5 @@
       </collision>
       <collision>
-        <origin xyz="0.0 0.262453 0.857803" />
+        <origin xyz="0.0 -0.262453 0.857803" />
         <geometry>
           <box size="0.572134 0.0209188 0.06" />
@@ -952,5 +951,5 @@
       </collision>
       <collision>
-        <origin xyz="0.0 0.262453 0.857803" />
+        <origin xyz="0.0 -0.262453 0.857803" />
         <geometry>
           <box size="0.572134 0.0209188 0.06" />
@@ -958,7 +957,119 @@
       </collision>
       <collision>
-        <origin xyz="-0.20788 0.264485 -1.02629" />
+        <origin xyz="0.20788 -0.264485 -1.02629" />
         <geometry>
           <box size="0.147984 0.016 0.074692" />
+        </geometry>
+      </collision>
+    </link>
+    <joint name="fridge_door1_joint" type="revolute">
+      <origin xyz="-0.29914526 -0.29725901 0.25673996" rpy="0.0 0.0 0.0" />
+      <parent link="cabinet3" />
+      <child link="fridge_door1" />
+      <axis xyz="0 0 -1" />
+      <limit effort="1000.0" lower="0.0" upper="${pi/2}" velocity="${pi/2}" />
+    </joint>
+    <link name="fridge_door1">
+      <visual>
+        <geometry>
+          <mesh filename="package://iai_apartment/meshes/unreal/SM_Fridge_Door_01.dae" />
+        </geometry>
+      </visual>
+      <collision>
+        <origin xyz="0.297325 0.006948 0.139709" />
+        <geometry>
+          <box size="0.596492 0.018554 1.336678" />
+        </geometry>
+      </collision>
+      <collision>
+        <origin xyz="0.295455 0.03605 -0.001115" />
+        <geometry>
+          <box size="0.553734 0.025 0.988894" />
+        </geometry>
+      </collision>
+    </link>
+    <joint name="fridge_door1_handle_joint" type="fixed">
+      <origin xyz="0.46534321 -0.00799103 -0.4736869" rpy="0.0 0.0 ${pi/2}" />
+      <parent link="fridge_door1" />
+      <child link="fridge_door1_handle" />
+    </joint>
+    <link name="fridge_door1_handle">
+      <visual>
+        <geometry>
+          <mesh filename="package://iai_apartment/meshes/unreal/SM_Kitchen_Handle.dae" />
+        </geometry>
+      </visual>
+      <collision>
+        <origin xyz="0.08 -0.003891  0.0" />
+        <geometry>
+          <box size="0.013 0.02 0.013" />
+        </geometry>
+      </collision>
+      <collision>
+        <origin xyz="-0.08 -0.003891  0.0" />
+        <geometry>
+          <box size="0.013 0.02 0.013" />
+        </geometry>
+      </collision>
+      <collision>
+        <origin xyz="0.0 -0.0203895 0.0" />
+        <geometry>
+          <box size="0.173032 0.013 0.013" />
+        </geometry>
+      </collision>
+    </link>
+    <joint name="fridge_door2_joint" type="revolute">
+      <origin xyz="-0.2990897 -0.29725901 -0.63800789" rpy="0.0 0.0 0.0" />
+      <parent link="cabinet3" />
+      <child link="fridge_door2" />
+      <axis xyz="0 0 -1" />
+      <limit effort="1000.0" lower="0.0" upper="${pi/2}" velocity="${pi/2}" />
+    </joint>
+    <link name="fridge_door2">
+      <visual>
+        <geometry>
+          <mesh filename="package://iai_apartment/meshes/unreal/SM_Fridge_Door_02.dae" />
+        </geometry>
+      </visual>
+      <collision>
+        <origin xyz="0.297325 0.006948 -0.028308" />
+        <geometry>
+          <box size="0.596492 0.018554 0.78594" />
+        </geometry>
+      </collision>
+      <collision>
+        <origin xyz="0.295455 0.03605 0.019366 " />
+        <geometry>
+          <box size="0.553734 0.025 0.622332" />
+        </geometry>
+      </collision>
+    </link>
+    <joint name="fridge_door2_handle_joint" type="fixed">
+      <origin xyz="0.46538265 0.00804657 0.28486839" rpy="0.0 0.0 ${pi/2}" />
+      <parent link="fridge_door2" />
+      <child link="fridge_door2_handle" />
+    </joint>
+    <link name="fridge_door2_handle">
+      <visual>
+        <geometry>
+          <mesh filename="package://iai_apartment/meshes/unreal/SM_Kitchen_Handle.dae" />
+        </geometry>
+      </visual>
+      <collision>
+        <origin xyz="0.08 -0.003891  0.0" />
+        <geometry>
+          <box size="0.013 0.02 0.013" />
+        </geometry>
+      </collision>
+      <collision>
+        <origin xyz="-0.08 -0.003891  0.0" />
+        <geometry>
+          <box size="0.013 0.02 0.013" />
+        </geometry>
+      </collision>
+      <collision>
+        <origin xyz="0.0 -0.0203895 0.0" />
+        <geometry>
+          <box size="0.173032 0.013 0.013" />
         </geometry>
       </collision>
@@ -976,5 +1087,5 @@
       </visual>
       <collision>
-        <origin xyz="0.257778 -0.016051 0.0" />
+        <origin xyz="0.257778 0.016051 0.0" />
         <geometry>
           <box size="0.043244 0.483652 1.75881" />
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