Commit message: Add dishwasher

File: iai_apartment/urdf/kitchen_unreal.xacro (robot description, xacro)
@@ -8,8 +8,15 @@
     </joint>
     <link name="kitchen_root" />
+    <!-- First part of the kitchen (fridge) -->
+    <joint name="kitchen1_root_joint" type="fixed">
+      <origin xyz="0.0 0.0 0.0" />
+      <parent link="kitchen_root" />
+      <child link="kitchen1_root" />
+    </joint>
+    <link name="kitchen1_root" />
     <!-- Cabinet1 -->
     <joint name="cabinet1_joint" type="fixed">
       <origin xyz="0.28463219 1.46675873 1.11440605" rpy="0.0 0.0 ${pi/2}" />
-      <parent link="kitchen_root" />
+      <parent link="kitchen1_root" />
       <child link="cabinet1" />
     </joint>
@@ -101,19 +108,19 @@
       </visual>
       <collision>
-        <origin xyz="0.08 -0.003891  0.0" />
-        <geometry>
-          <box size="0.013 0.02 0.013" />
-        </geometry>
-      </collision>
-      <collision>
-        <origin xyz="-0.08 -0.003891  0.0" />
-        <geometry>
-          <box size="0.013 0.02 0.013" />
-        </geometry>
-      </collision>
-      <collision>
-        <origin xyz="0.0 -0.0203895 0.0" />
-        <geometry>
-          <box size="0.173032 0.013 0.013" />
+        <origin xyz="-0.003891 0.08 0.0" />
+        <geometry>
+          <box size="0.02 0.013 0.013" />
+        </geometry>
+      </collision>
+      <collision>
+        <origin xyz="-0.003891 -0.08 0.0" />
+        <geometry>
+          <box size="0.02 0.013 0.013" />
+        </geometry>
+      </collision>
+      <collision>
+        <origin xyz="-0.0203895 0.0 0.0" />
+        <geometry>
+          <box size="0.013 0.173032  0.013" />
         </geometry>
       </collision>
@@ -187,19 +194,19 @@
       </visual>
       <collision>
-        <origin xyz="0.08 -0.003891  0.0" />
-        <geometry>
-          <box size="0.013 0.02 0.013" />
-        </geometry>
-      </collision>
-      <collision>
-        <origin xyz="-0.08 -0.003891  0.0" />
-        <geometry>
-          <box size="0.013 0.02 0.013" />
-        </geometry>
-      </collision>
-      <collision>
-        <origin xyz="0.0 -0.0203895 0.0" />
-        <geometry>
-          <box size="0.173032 0.013 0.013" />
+        <origin xyz="-0.003891 0.08 0.0" />
+        <geometry>
+          <box size="0.02 0.013 0.013" />
+        </geometry>
+      </collision>
+      <collision>
+        <origin xyz="-0.003891 -0.08 0.0" />
+        <geometry>
+          <box size="0.02 0.013 0.013" />
+        </geometry>
+      </collision>
+      <collision>
+        <origin xyz="-0.0203895 0.0 0.0" />
+        <geometry>
+          <box size="0.013 0.173032  0.013" />
         </geometry>
       </collision>
@@ -273,19 +280,19 @@
       </visual>
       <collision>
-        <origin xyz="0.08 -0.003891  0.0" />
-        <geometry>
-          <box size="0.013 0.02 0.013" />
-        </geometry>
-      </collision>
-      <collision>
-        <origin xyz="-0.08 -0.003891  0.0" />
-        <geometry>
-          <box size="0.013 0.02 0.013" />
-        </geometry>
-      </collision>
-      <collision>
-        <origin xyz="0.0 -0.0203895 0.0" />
-        <geometry>
-          <box size="0.173032 0.013 0.013" />
+        <origin xyz="-0.003891 0.08 0.0" />
+        <geometry>
+          <box size="0.02 0.013 0.013" />
+        </geometry>
+      </collision>
+      <collision>
+        <origin xyz="-0.003891 -0.08 0.0" />
+        <geometry>
+          <box size="0.02 0.013 0.013" />
+        </geometry>
+      </collision>
+      <collision>
+        <origin xyz="-0.0203895 0.0 0.0" />
+        <geometry>
+          <box size="0.013 0.173032  0.013" />
         </geometry>
       </collision>
@@ -356,5 +363,5 @@
     <joint name="cabinet2_joint" type="fixed">
       <origin xyz="0.27990936 1.97705429 1.16238914" rpy="0.0 0.0 ${pi/2}" />
-      <parent link="kitchen_root" />
+      <parent link="kitchen1_root" />
       <child link="cabinet2" />
     </joint>
@@ -440,19 +447,19 @@
       </visual>
       <collision>
-        <origin xyz="0.08 -0.003891  0.0" />
-        <geometry>
-          <box size="0.013 0.02 0.013" />
-        </geometry>
-      </collision>
-      <collision>
-        <origin xyz="-0.08 -0.003891  0.0" />
-        <geometry>
-          <box size="0.013 0.02 0.013" />
-        </geometry>
-      </collision>
-      <collision>
-        <origin xyz="0.0 -0.0203895 0.0" />
-        <geometry>
-          <box size="0.173032 0.013 0.013" />
+        <origin xyz="-0.003891 0.08 0.0" />
+        <geometry>
+          <box size="0.02 0.013 0.013" />
+        </geometry>
+      </collision>
+      <collision>
+        <origin xyz="-0.003891 -0.08 0.0" />
+        <geometry>
+          <box size="0.02 0.013 0.013" />
+        </geometry>
+      </collision>
+      <collision>
+        <origin xyz="-0.0203895 0.0 0.0" />
+        <geometry>
+          <box size="0.013 0.173032  0.013" />
         </geometry>
       </collision>
@@ -887,5 +894,5 @@
     <joint name="cabinet3_joint" type="fixed">
       <origin xyz="0.27498539 2.47989822 1.16287888" rpy="0.0 0.0 ${pi/2}" />
-      <parent link="kitchen_root" />
+      <parent link="kitchen1_root" />
       <child link="cabinet3" />
     </joint>
@@ -1001,19 +1008,19 @@
       </visual>
       <collision>
-        <origin xyz="0.08 -0.003891  0.0" />
-        <geometry>
-          <box size="0.013 0.02 0.013" />
-        </geometry>
-      </collision>
-      <collision>
-        <origin xyz="-0.08 -0.003891  0.0" />
-        <geometry>
-          <box size="0.013 0.02 0.013" />
-        </geometry>
-      </collision>
-      <collision>
-        <origin xyz="0.0 -0.0203895 0.0" />
-        <geometry>
-          <box size="0.173032 0.013 0.013" />
+        <origin xyz="-0.003891 0.08 0.0" />
+        <geometry>
+          <box size="0.02 0.013 0.013" />
+        </geometry>
+      </collision>
+      <collision>
+        <origin xyz="-0.003891 -0.08 0.0" />
+        <geometry>
+          <box size="0.02 0.013 0.013" />
+        </geometry>
+      </collision>
+      <collision>
+        <origin xyz="-0.0203895 0.0 0.0" />
+        <geometry>
+          <box size="0.013 0.173032  0.013" />
         </geometry>
       </collision>
@@ -1057,19 +1064,19 @@
       </visual>
       <collision>
-        <origin xyz="0.08 -0.003891  0.0" />
-        <geometry>
-          <box size="0.013 0.02 0.013" />
-        </geometry>
-      </collision>
-      <collision>
-        <origin xyz="-0.08 -0.003891  0.0" />
-        <geometry>
-          <box size="0.013 0.02 0.013" />
-        </geometry>
-      </collision>
-      <collision>
-        <origin xyz="0.0 -0.0203895 0.0" />
-        <geometry>
-          <box size="0.173032 0.013 0.013" />
+        <origin xyz="-0.003891 0.08 0.0" />
+        <geometry>
+          <box size="0.02 0.013 0.013" />
+        </geometry>
+      </collision>
+      <collision>
+        <origin xyz="-0.003891 -0.08 0.0" />
+        <geometry>
+          <box size="0.02 0.013 0.013" />
+        </geometry>
+      </collision>
+      <collision>
+        <origin xyz="-0.0203895 0.0 0.0" />
+        <geometry>
+          <box size="0.013 0.173032  0.013" />
         </geometry>
       </collision>
@@ -1442,5 +1449,5 @@
     <joint name="cabinet4_joint" type="fixed">
       <origin xyz="0.18224365 3.29388123 1.82711395" rpy="0.0 0.0 ${pi/2}" />
-      <parent link="kitchen_root" />
+      <parent link="kitchen1_root" />
       <child link="cabinet4" />
     </joint>
@@ -1506,4 +1513,1039 @@
       </collision>
     </link>
+    <joint name="cabinet4_door2_joint" type="fixed">
+      <origin xyz="-0.0093109 -0.15042921 -0.19994873" rpy="0.0 0.0 0.0" />
+      <parent link="cabinet4" />
+      <child link="cabinet4_door2" />
+    </joint>
+    <link name="cabinet4_door2">
+      <visual>
+        <geometry>
+          <mesh filename="package://iai_apartment/meshes/unreal/SM_Kitchen_04_Door_02.dae" />
+        </geometry>
+      </visual>
+      <collision>
+        <origin xyz="0.0 -0.025359 0.0" />
+        <geometry>
+          <box size="0.994892 0.019 0.395736" />
+        </geometry>
+      </collision>
+    </link>
+    <joint name="cabinet4_door2_handle_joint" type="fixed">
+      <origin xyz="0.01415195 -0.04103859 -0.13357088" rpy="0.0 0.0 ${pi/2}" />
+      <parent link="cabinet4_door2" />
+      <child link="cabinet4_door2_handle" />
+    </joint>
+    <link name="cabinet4_door2_handle">
+      <visual>
+        <geometry>
+          <mesh filename="package://iai_apartment/meshes/unreal/SM_Kitchen_Handle.dae" />
+        </geometry>
+      </visual>
+      <collision>
+        <origin xyz="-0.003891 0.08 0.0" />
+        <geometry>
+          <box size="0.02 0.013 0.013" />
+        </geometry>
+      </collision>
+      <collision>
+        <origin xyz="-0.003891 -0.08 0.0" />
+        <geometry>
+          <box size="0.02 0.013 0.013" />
+        </geometry>
+      </collision>
+      <collision>
+        <origin xyz="-0.0203895 0.0 0.0" />
+        <geometry>
+          <box size="0.013 0.173032  0.013" />
+        </geometry>
+      </collision>
+    </link>
+    <joint name="cabinet4_shelf1_joint" type="fixed">
+      <origin xyz="-0.01016479 0.00833792 0.12500641" rpy="0.0 0.0 ${pi}" />
+      <parent link="cabinet4" />
+      <child link="cabinet4_shelf1" />
+    </joint>
+    <link name="cabinet4_shelf1">
+      <visual>
+        <geometry>
+          <mesh filename="package://iai_apartment/meshes/unreal/SM_Kitchen_04_Shelf.dae" />
+        </geometry>
+      </visual>
+      <collision>
+        <origin xyz="0.0 0.0 0.0" />
+        <geometry>
+          <box size="0.967896 0.307078 0.008084" />
+        </geometry>
+      </collision>
+    </link>
+    <joint name="cabinet4_shelf2_joint" type="fixed">
+      <origin xyz="-0.01016479 0.00833792 -0.09840179" rpy="0.0 0.0 ${pi}" />
+      <parent link="cabinet4" />
+      <child link="cabinet4_shelf2" />
+    </joint>
+    <link name="cabinet4_shelf2">
+      <visual>
+        <geometry>
+          <mesh filename="package://iai_apartment/meshes/unreal/SM_Kitchen_04_Shelf.dae" />
+        </geometry>
+      </visual>
+      <collision>
+        <origin xyz="0.0 0.0 0.0" />
+        <geometry>
+          <box size="0.967896 0.307078 0.008084" />
+        </geometry>
+      </collision>
+    </link>
+    <!-- Cabinet5 -->
+    <joint name="cabinet5_joint" type="fixed">
+      <origin xyz="0.27476608 3.08411682 0.49420666" rpy="0.0 0.0 ${pi/2}" />
+      <parent link="kitchen1_root" />
+      <child link="cabinet5" />
+    </joint>
+    <link name="cabinet5">
+      <visual>
+        <geometry>
+          <mesh filename="package://iai_apartment/meshes/unreal/SM_Kitchen_05_Base.dae" />
+        </geometry>
+      </visual>
+      <collision>
+        <origin xyz="-0.291968 0.0 0.0" />
+        <geometry>
+          <box size="0.016 0.55452 0.798012" />
+        </geometry>
+      </collision>
+      <collision>
+        <origin xyz="0.291968 0.0 0.0" />
+        <geometry>
+          <box size="0.016 0.55452 0.798012" />
+        </geometry>
+      </collision>
+      <collision>
+        <origin xyz="0.0 0.0 -0.391006" />
+        <geometry>
+          <box size="0.568134 0.55452 0.016" />
+        </geometry>
+      </collision>
+      <collision>
+        <origin xyz="0.0 0.217476 0.390909" />
+        <geometry>
+          <box size="0.568134 0.08 0.016" />
+        </geometry>
+      </collision>
+      <collision>
+        <origin xyz="0.0 0.261473 0.0" />
+        <geometry>
+          <box size="0.568134 0.008 0.76582" />
+        </geometry>
+      </collision>
+    </link>
+    <joint name="cabinet5_drawer1_joint" type="prismatic">
+      <origin xyz="0.00100026 -0.05262699 0.33177837" rpy="0.0 0.0 0.0" />
+      <parent link="cabinet5" />
+      <child link="cabinet5_drawer1" />
+      <axis xyz="0 -1 0" />
+      <limit effort="1000.0" lower="0.0" upper="0.45" velocity="0.5" />
+    </joint>
+    <link name="cabinet5_drawer1">
+      <visual>
+        <geometry>
+          <mesh filename="package://iai_apartment/meshes/unreal/SM_Kitchen_05_Drawer_01.dae" />
+        </geometry>
+      </visual>
+      <collision>
+        <origin xyz="-0.270267 0.021031 -0.01336" />
+        <geometry>
+          <box size="0.01622 0.491014 0.085266" />
+        </geometry>
+      </collision>
+      <collision>
+        <origin xyz="0.270267 0.021031 -0.01336" />
+        <geometry>
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