Commit message: Fix xacro

File: iai_apartment/urdf/kitchen_unreal.xacro (robot description, xacro)
@@ -1598,4 +1598,22 @@
     </link>
     <!-- Cabinet5 -->
+    <joint name="counter_wall_joint" type="fixed">
+      <origin xyz="0.28142776 3.29494293 0.90892097" rpy="0.0 0.0 ${-pi/2}" />
+      <parent link="kitchen1_root" />
+      <child link="counter_wall" />
+    </joint>
+    <link name="counter_wall">
+      <visual>
+        <geometry>
+          <mesh filename="package://iai_apartment/meshes/unreal/SM_Counter_Wall.dae" />
+        </geometry>
+      </visual>
+      <collision>
+        <origin xyz="0.0 0.0 0.0" />
+        <geometry>
+          <box size="1.031064 0.599 0.026778" />
+        </geometry>
+      </collision>
+    </link>
     <joint name="cabinet5_joint" type="fixed">
       <origin xyz="0.27476608 3.08411682 0.49420666" rpy="0.0 0.0 ${pi/2}" />
@@ -1929,22 +1947,4 @@
       </collision>
     </link>
-    <joint name="counter_wall_joint" type="fixed">
-      <origin xyz="-0.28889557 0.00673351 0.41436802" rpy="0.0 0.0 ${pi}" />
-      <parent link="cabinet6" />
-      <child link="counter_wall" />
-    </joint>
-    <link name="counter_wall">
-      <visual>
-        <geometry>
-          <mesh filename="package://iai_apartment/meshes/unreal/SM_Counter_Wall.dae" />
-        </geometry>
-      </visual>
-      <collision>
-        <origin xyz="0.0 0.0 0.0" />
-        <geometry>
-          <box size="1.031064 0.599 0.026778" />
-        </geometry>
-      </collision>
-    </link>
     <joint name="cabinet6_drawer1_joint" type="prismatic">
       <origin xyz="0.00032649 -0.05329598 0.33177837" rpy="0.0 0.0 0.0" />
@@ -2194,28 +2194,15 @@
     </link>
     <joint name="island_cover4_joint" type="fixed">
-      <origin xyz="0.21131807 0.00210169 -0.04853619" rpy="0.0 0.0 0.0" />
-      <parent link="cabinet6" />
+      <origin xyz="0.27259209 3.79515656 0.44601677" rpy="0.0 0.0 ${pi/2}" />
+      <parent link="kitchen1_root" />
       <child link="island_cover4" />
     </joint>
-    <link name="island_cover4">
-      <visual>
-        <geometry>
-          <mesh filename="package://iai_apartment/meshes/unreal/SM_Kitchen_Island_Cover_04.dae" />
-        </geometry>
-      </visual>
-      <collision>
-        <origin xyz="0.0 0.0 0.0" />
-        <geometry>
-          <box size="0.019108 0.592148 0.897013" />
-        </geometry>
-      </collision>
-    </link>
-    <!-- Base board -->
-    <joint name="base_board_joint" type="fixed">
+    <!-- Kitchen1 base board, island cover -->
+    <joint name="kitchen1_base_board_joint" type="fixed">
       <origin xyz="0.55976036 2.47825577 0.05168431" rpy="0.0 0.0 ${-pi/2}" />
       <parent link="kitchen1_root" />
-      <child link="base_board" />
-    </joint>
-    <link name="base_board">
+      <child link="kitchen1_base_board" />
+    </joint>
+    <link name="kitchen1_base_board">
       <visual>
         <geometry>
@@ -2227,4 +2214,17 @@
         <geometry>
           <box size="2.60316 0.019778 0.1" />
+        </geometry>
+      </collision>
+    </link>
+    <link name="island_cover4">
+      <visual>
+        <geometry>
+          <mesh filename="package://iai_apartment/meshes/unreal/SM_Kitchen_Island_Cover_04.dae" />
+        </geometry>
+      </visual>
+      <collision>
+        <origin xyz="0.0 0.0 0.0" />
+        <geometry>
+          <box size="0.019108 0.592148 0.897013" />
         </geometry>
       </collision>
@@ -2318,5 +2318,5 @@
         <origin xyz="0.0 -0.212477 0.0" />
         <geometry>
-          <box size="0.404212 0.01 0.177388" />
+          <box size="0.404212 0.02 0.177388" />
         </geometry>
       </collision>
@@ -2491,4 +2491,34 @@
       </collision>
     </link>
+    <joint name="dishwasher_front_handle_joint" type="fixed">
+      <origin xyz="-0.0169432 -0.05493519 0.67884796" rpy="0.0 0.0 ${pi/2}" />
+      <parent link="dishwasher_front" />
+      <child link="dishwasher_front_handle" />
+    </joint>
+    <link name="dishwasher_front_handle">
+      <visual>
+        <geometry>
+          <mesh filename="package://iai_apartment/meshes/unreal/SM_Kitchen_Handle.dae" />
+        </geometry>
+      </visual>
+      <collision>
+        <origin xyz="-0.003891 0.08 0.0" />
+        <geometry>
+          <box size="0.02 0.013 0.013" />
+        </geometry>
+      </collision>
+      <collision>
+        <origin xyz="-0.003891 -0.08 0.0" />
+        <geometry>
+          <box size="0.02 0.013 0.013" />
+        </geometry>
+      </collision>
+      <collision>
+        <origin xyz="-0.0203895 0.0 0.0" />
+        <geometry>
+          <box size="0.013 0.173032  0.013" />
+        </geometry>
+      </collision>
+    </link>
     <joint name="dishwasher_tray1_joint" type="prismatic">
       <origin xyz="-0.00735926 0.19401426 0.22713593" rpy="0.0 0.0 0.0" />
@@ -2548,4 +2578,1227 @@
       </collision>
     </link>
+    <!-- Cabinet8 -->
+    <joint name="cabinet8_joint" type="fixed">
+      <origin xyz="2.49268082 3.37232117 0.49448143" rpy="0.0 0.0 ${-pi/2}" />
+      <parent link="kitchen2_root" />
+      <child link="cabinet8" />
+    </joint>
+    <link name="cabinet8">
+      <visual>
+        <geometry>
+          <mesh filename="package://iai_apartment/meshes/unreal/SM_Kitchen_08_Sink_Base.dae" />
+        </geometry>
+      </visual>
+      <collision>
+        <origin xyz="-0.291912 0.0 0.0" />
+        <geometry>
+          <box size="0.015884 0.55405 0.79779" />
+        </geometry>
+      </collision>
+      <collision>
+        <origin xyz="0.291912 0.0 0.0" />
+        <geometry>
+          <box size="0.015884 0.55405 0.79779" />
+        </geometry>
+      </collision>
+      <collision>
+        <origin xyz="0.0 0.26153 0.0" />
+        <geometry>
+          <box size="0.568134 0.007888 0.765818" />
+        </geometry>
+      </collision>
+      <collision>
+        <origin xyz="0.0 0.217476 0.39091" />
+        <geometry>
+          <box size="0.568134 0.08 0.016" />
+        </geometry>
+      </collision>
+      <collision>
+        <origin xyz="0.0 0.0 -0.391005 " />
+        <geometry>
+          <box size="0.568134 0.55405 0.016" />
+        </geometry>
+      </collision>
+    </link>
+    <joint name="sink_drawer_joint" type="prismatic">
+      <origin xyz="-0.00013535 -0.05086624 0.0032" rpy="0.0 0.0 0.0" />
+      <parent link="cabinet8" />
+      <child link="sink_drawer" />
+      <axis xyz="0 -1 0" />
+      <limit effort="1000.0" lower="0.0" upper="0.45" velocity="0.45" />
+    </joint>
+    <link name="sink_drawer">
+      <visual>
+        <geometry>
+          <mesh filename="package://iai_apartment/meshes/unreal/SM_Kitchen_08_Sink_Drawer_01.dae" />
+        </geometry>
+      </visual>
+      <collision>
+        <origin xyz="0.0 -0.233976 0.0" />
+        <geometry>
+          <box size="0.596516 0.018776 0.794026" />
+        </geometry>
+      </collision>
+      <collision>
+        <origin xyz="0.0 0.259483 -0.288887" />
+        <geometry>
+          <box size="0.539508 0.018034 0.169484" />
+        </geometry>
+      </collision>
+      <collision>
+        <origin xyz="0.268047 0.025012 -0.08949" />
+        <geometry>
+          <box size="0.015 0.498056 0.084" />
+        </geometry>
+      </collision>
+      <collision>
+        <origin xyz="-0.268047 0.025012 -0.08949" />
+        <geometry>
+          <box size="0.015 0.498056 0.084" />
+        </geometry>
+      </collision>
+      <collision>
+        <origin xyz="0.268047 0.025012 -0.208727" />
+        <geometry>
+          <box size="0.015 0.498056 0.023296" />
+        </geometry>
+      </collision>
+      <collision>
+        <origin xyz="-0.268047 0.025012 -0.208727" />
+        <geometry>
+          <box size="0.015 0.498056 0.023296" />
+        </geometry>
+      </collision>
+      <collision>
+        <origin xyz="0.268047 0.025012 -0.33085" />
+        <geometry>
+          <box size="0.015 0.498056 0.087218" />
+        </geometry>
+      </collision>
+      <collision>
+        <origin xyz="-0.268047 0.025012 -0.33085" />
+        <geometry>
+          <box size="0.015 0.498056 0.087218" />
+        </geometry>
+      </collision>
+      <collision>
+        <origin xyz="0.246033 0.025012 -0.04" />
+        <geometry>
+          <box size="0.062024 0.498056 0.016" />
+        </geometry>
+      </collision>
+      <collision>
+        <origin xyz="-0.246033 0.025012 -0.04" />
+        <geometry>
+          <box size="0.062024 0.498056 0.016" />
+        </geometry>
+      </collision>
+      <collision>
+        <origin xyz="0.0 -0.213959 -0.04" />
+        <geometry>
+          <box size="0.554092 0.021008 0.016" />
+        </geometry>
+      </collision>
+      <collision>
+        <origin xyz="0.0 0.21583 -0.04" />
+        <geometry>
+          <box size="0.554092 0.117306 0.016" />
+        </geometry>
+      </collision>
+      <!-- Trash can 1 -->
+      <collision>
+        <origin xyz="-0.00535 0.086505 -0.198155 " />
+        <geometry>
+          <box size="0.016852 0.149578 0.34661" />
+        </geometry>
+      </collision>
+      <collision>
+        <origin xyz="-0.211412 0.086505 -0.198155" />
+        <geometry>
+          <box size="0.016852 0.149578 0.34661" />
+        </geometry>
+      </collision>
+      <collision>
+        <origin xyz="-0.109826 0.152938 -0.198155" />
+        <geometry>
+          <box size="0.219652 0.016712 0.34661" />
+        </geometry>
+      </collision>
+      <collision>
+        <origin xyz="-0.109826 0.02 -0.198155" />
+        <geometry>
+          <box size="0.219652 0.016712 0.34661" />
+        </geometry>
+      </collision>
+      <collision>
+        <origin xyz="-0.109826 0.086505 -0.372315" />
+        <geometry>
+          <box size="0.219652 0.149578 0.0017" />
+        </geometry>
+      </collision>
+      <!-- Trash can 2 -->
+      <collision>
+        <origin xyz="0.00535 0.086505 -0.198155 " />
+        <geometry>
+          <box size="0.016852 0.149578 0.34661" />
+        </geometry>
+      </collision>
+      <collision>
+        <origin xyz="0.211412 0.086505 -0.198155" />
+        <geometry>
+          <box size="0.016852 0.149578 0.34661" />
+        </geometry>
+      </collision>
+      <collision>
+        <origin xyz="0.109826 0.152938 -0.198155" />
+        <geometry>
+          <box size="0.219652 0.016852 0.34661" />
+        </geometry>
+      </collision>
+      <collision>
+        <origin xyz="0.109826 0.02 -0.198155" />
+        <geometry>
+          <box size="0.219652 0.016852 0.34661" />
+        </geometry>
+      </collision>
+      <collision>
+        <origin xyz="0.109826 0.086505 -0.372315" />
+        <geometry>
+          <box size="0.219652 0.149578 0.0017" />
+        </geometry>
+      </collision>
+      <!-- Trash can 3 -->
+      <collision>
+        <origin xyz="-0.221355 -0.098209 -0.198155" />
+        <geometry>
+          <box size="0.016852 0.219458 0.34661" />
+        </geometry>
+      </collision>
+      <collision>
+        <origin xyz="-0.088435 -0.098209 -0.198155" />
+        <geometry>
+          <box size="0.016852 0.219458 0.34661" />
+        </geometry>
+      </collision>
+      <collision>
+        <origin xyz="-0.155 0.003041 -0.198155 " />
+        <geometry>
+          <box size="0.149382 0.016852 0.34661" />
+        </geometry>
+      </collision>
+      <collision>
+        <origin xyz="-0.155 -0.199821 -0.198155" />
+        <geometry>
+          <box size="0.149382 0.016852 0.34661" />
+        </geometry>
+      </collision>
+      <collision>
+        <origin xyz="-0.155 -0.098209 -0.372315" />
+        <geometry>
+          <box size="0.149382 0.219458 0.0017" />
+        </geometry>
+      </collision>
+      <!-- Trash can 4 -->
+      <collision>
+        <origin xyz="0.221355 -0.098209 -0.198155" />
+        <geometry>
+          <box size="0.016852 0.219458 0.34661" />
+        </geometry>
+      </collision>
+      <collision>
+        <origin xyz="-0.071323 -0.098209 -0.198155" />
+        <geometry>
+          <box size="0.016852 0.219458 0.34661" />
+        </geometry>
+      </collision>
+      <collision>
+        <origin xyz="0.075302 0.003041 -0.198155 " />
+        <geometry>
+          <box size="0.309498 0.016852 0.34661" />
+        </geometry>
+      </collision>
+      <collision>
+        <origin xyz="0.075302 -0.199821 -0.198155" />
+        <geometry>
+          <box size="0.309498 0.016852 0.34661" />
+        </geometry>
+      </collision>
+      <collision>
+        <origin xyz="0.075302 -0.098209 -0.372315" />
+        <geometry>
+          <box size="0.309498 0.219458 0.0017" />
+        </geometry>
+      </collision>
+    </link>
+    <joint name="sink_drawer_handle_joint" type="fixed">
+      <origin xyz="0.00331339 -0.24900223 0.35071747" rpy="0.0 0.0 ${pi/2}" />
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
Commit message: Fix textures

File: iai_apartment/urdf/kitchen_unreal.xacro (robot description, xacro)
@@ -1026,4 +1026,105 @@
       </collision>
     </link>
+    <joint name="fridge_door_tray1_joint" type="fixed">
+      <origin xyz="0.29726078 0.10379066 -0.01565247" rpy="0.0 0.0 ${pi/2}" />
+      <parent link="fridge_door1" />
+      <child link="fridge_door_tray1" />
+    </joint>
+    <link name="fridge_door_tray1">
+      <visual>
+        <geometry>
+          <mesh filename="package://iai_apartment/meshes/unreal/SM_Fridge_Door_Tray_01.dae" />
+        </geometry>
+      </visual>
+      <collision>
+        <origin xyz="0.054273 0.0 0.0" />
+        <geometry>
+          <box size="0.002 0.421854 0.095574" />
+        </geometry>
+      </collision>
+      <collision>
+        <origin xyz="-0.054273 0.0 0.0" />
+        <geometry>
+          <box size="0.002 0.421854 0.095574" />
+        </geometry>
+      </collision>
+      <collision>
+        <origin xyz="0.0 0.209978 0.0" />
+        <geometry>
+          <box size="0.10942 0.002 0.095574" />
+        </geometry>
+      </collision>
+      <collision>
+        <origin xyz="0.0 -0.209978 0.0" />
+        <geometry>
+          <box size="0.10942 0.002 0.095574" />
+        </geometry>
+      </collision>
+      <collision>
+        <origin xyz="0.0 0.0 -0.047166" />
+        <geometry>
+          <box size="0.10942 0.421854 0.002" />
+        </geometry>
+      </collision>
+    </link>
+    <joint name="fridge_door_tray2_joint" type="fixed">
+      <origin xyz="0.29847088 0.10176933 0.22387222" rpy="0.0 0.0 ${pi/2}" />
+      <parent link="fridge_door1" />
+      <child link="fridge_door_tray2" />
+    </joint>
+    <link name="fridge_door_tray2">
+      <visual>
+        <geometry>
+          <mesh filename="package://iai_apartment/meshes/unreal/SM_Fridge_Door_Tray_02.dae" />
+        </geometry>
+      </visual>
+      <collision>
+        <origin xyz="0.054019 0.0 0.0" />
+        <geometry>
+          <box size="0.002 0.421954 0.053802" />
+        </geometry>
+      </collision>
+      <collision>
+        <origin xyz="-0.054019 0.0 0.0" />
+        <geometry>
+          <box size="0.002 0.421954 0.053802" />
+        </geometry>
+      </collision>
+      <collision>
+        <origin xyz="0.0 0.209978 0.0" />
+        <geometry>
+          <box size="0.109988 0.002 0.053802" />
+        </geometry>
+      </collision>
+      <collision>
+        <origin xyz="0.0 -0.209978 0.0" />
+        <geometry>
+          <box size="0.109988 0.002 0.053802" />
+        </geometry>
+      </collision>
+      <collision>
+        <origin xyz="0.0 0.0 -0.025903" />
+        <geometry>
+          <box size="0.109988 0.421954 0.002" />
+        </geometry>
+      </collision>
+    </link>
+    <joint name="fridge_egg_tray_joint" type="fixed">
+      <origin xyz="-0.00226576 0.08530881 0.00069855" rpy="0.0 0.0 0.0" />
+      <parent link="fridge_door_tray2" />
+      <child link="fridge_egg_tray" />
+    </joint>
+    <link name="fridge_egg_tray">
+      <visual>
+        <geometry>
+          <mesh filename="package://iai_apartment/meshes/unreal/SM_Fridge_Egg_Tray.dae" />
+        </geometry>
+      </visual>
+      <collision>
+        <geometry>
+          <mesh filename="package://iai_apartment/meshes/unreal/SM_Fridge_Egg_Tray.stl" />
+        </geometry>
+      </collision>
+    </link>
     <joint name="fridge_door2_joint" type="revolute">
       <origin xyz="-0.2990897 -0.29725901 -0.63800789" rpy="0.0 0.0 0.0" />
@@ -2395,5 +2496,5 @@
       <limit effort="1000.0" lower="${-pi/2}" upper="${pi/2}" velocity="${pi}" />
     </joint>
-    <link name="counter_sink_tap_switch" >
+    <link name="counter_sink_tap_switch">
       <collision>
         <geometry>
@@ -2639,12 +2740,12 @@
       </collision>
     </link>
-    <joint name="sink_drawer_joint" type="prismatic">
+    <joint name="sink_drawer1_joint" type="prismatic">
       <origin xyz="-0.00013535 -0.05086624 0.0032" rpy="0.0 0.0 0.0" />
       <parent link="cabinet8" />
-      <child link="sink_drawer" />
+      <child link="sink_drawer1" />
       <axis xyz="0 -1 0" />
       <limit effort="1000.0" lower="0.0" upper="0.45" velocity="0.45" />
     </joint>
-    <link name="sink_drawer">
+    <link name="sink_drawer1">
       <visual>
         <geometry>
@@ -2849,10 +2950,10 @@
       </collision>
     </link>
-    <joint name="sink_drawer_handle_joint" type="fixed">
+    <joint name="sink_drawer1_handle_joint" type="fixed">
       <origin xyz="0.00331339 -0.24900223 0.35071747" rpy="0.0 0.0 ${pi/2}" />
-      <parent link="sink_drawer" />
-      <child link="sink_drawer_handle" />
-    </joint>
-    <link name="sink_drawer_handle">
+      <parent link="sink_drawer1" />
+      <child link="sink_drawer1_handle" />
+    </joint>
+    <link name="sink_drawer1_handle">
       <visual>
         <geometry>
@@ -2876,4 +2977,60 @@
         <geometry>
           <box size="0.013 0.173032  0.013" />
+        </geometry>
+      </collision>
+    </link>
+    <joint name="sink_drawer2_joint" type="prismatic">
+      <origin xyz="-0.00142344 -0.07299484 0.16437714" rpy="0.0 0.0 0.0" />
+      <parent link="cabinet8" />
+      <child link="sink_drawer2" />
+      <axis xyz="0 -1 0" />
+      <limit effort="1000.0" lower="0.0" upper="0.3" velocity="0.3" />
+    </joint>
+    <link name="sink_drawer2">
+      <visual>
+        <geometry>
+          <mesh filename="package://iai_apartment/meshes/unreal/SM_Kitchen_08_Sink_Drawer_02.dae" />
+        </geometry>
+      </visual>
+      <collision>
+        <origin xyz="-0.270604 0.002535 -0.000733" />
+        <geometry>
+          <box size="0.016 0.376026 0.08221" />
+        </geometry>
+      </collision>
+      <collision>
+        <origin xyz="0.270604 0.002535 -0.000733" />
+        <geometry>
+          <box size="0.016 0.376026 0.08221" />
+        </geometry>
+      </collision>
+      <collision>
+        <origin xyz="-0.248473 -0.191981 0.000834" />
+        <geometry>
+          <box size="0.064994 0.017 0.099322" />
+        </geometry>
+      </collision>
+      <collision>
+        <origin xyz="0.248473 -0.191981 0.000834" />
+        <geometry>
+          <box size="0.064994 0.017 0.099322" />
+        </geometry>
+      </collision>
+      <collision>
+        <origin xyz="0.0 -0.191981 -0.0015" />
+        <geometry>
+          <box size="0.433954 0.017 0.098" />
+        </geometry>
+      </collision>
+      <collision>
+        <origin xyz="0.0 0.184382 -0.0024" />
+        <geometry>
+          <box size="0.557356 0.016 0.083" />
+        </geometry>
+      </collision>
+      <collision>
+        <origin xyz="0.0 0.002535 -0.036496" />
+        <geometry>
+          <box size="0.557356 0.376026 0.016" />
         </geometry>
       </collision>

Commit message: Add cabinet1_shelf1 and cabinet1_shelf2

File: iai_apartment/urdf/kitchen_unreal.xacro (robot description, xacro)
@@ -64,11 +64,44 @@
       </collision>
       <collision>
-        <origin xyz="0.009901 0.0005 0.249501" />
-        <geometry>
-          <box size="0.561938 0.540942 0.015" />
-        </geometry>
-      </collision>
-      <collision>
         <origin xyz="0.009901 0.0005 -0.361161 " />
+        <geometry>
+          <box size="0.561938 0.534942 0.015" />
+        </geometry>
+      </collision>
+    </link>
+    <material name="white">
+      <color rgba="1 1 1 1" />
+    </material>
+    <joint name="cabinet1_shelf1_joint" type="fixed">
+      <origin xyz="0.009901 0.0005 0.560" />
+      <parent link="cabinet1" />
+      <child link="cabinet1_shelf1" />
+    </joint>
+    <link name="cabinet1_shelf1">
+      <visual>
+        <geometry>
+          <box size="0.561938 0.534942 0.015" />
+        </geometry>
+        <material name="white" />
+      </visual>
+      <collision>
+        <geometry>
+          <box size="0.561938 0.534942 0.015" />
+        </geometry>
+      </collision>
+    </link>
+    <joint name="cabinet1_shelf2_joint" type="fixed">
+      <origin xyz="0.009901 0.0005 0.249501" />
+      <parent link="cabinet1" />
+      <child link="cabinet1_shelf2" />
+    </joint>
+    <link name="cabinet1_shelf2">
+      <visual>
+        <geometry>
+          <box size="0.561938 0.534942 0.015" />
+        </geometry>
+        <material name="white" />
+      </visual>
+      <collision>
         <geometry>
           <box size="0.561938 0.534942 0.015" />
