Commit message: Fix orientation

File: iai_apartment/urdf/kitchen_unreal.xacro (robot description, xacro)
@@ -17,5 +17,5 @@
     <!-- Cabinet1 -->
     <joint name="cabinet1_joint" type="fixed">
-      <origin xyz="0.28463219 1.46675873 1.11440605" rpy="0.0 0.0 ${pi/2}" />
+      <origin xyz="0.28463219 1.46675873 1.11440605" rpy="0.0 0.0 ${pi}" />
       <parent link="kitchen1_root" />
       <child link="cabinet1" />
@@ -28,43 +28,43 @@
       </visual>
       <collision>
-        <origin xyz="0.3 0.010499 0.05" />
-        <geometry>
-          <box size="0.019 0.55494 2.12778" />
-        </geometry>
-      </collision>
-      <collision>
-        <origin xyz="-0.280469 0.010499 0.05" />
-        <geometry>
-          <box size="0.019 0.55494 2.12778" />
-        </geometry>
-      </collision>
-      <collision>
-        <origin xyz="0.009901 0.271973 0.041995" />
-        <geometry>
-          <box size="0.561938 0.008 2.11178" />
-        </geometry>
-      </collision>
-      <collision>
-        <origin xyz="-0.299967 0.0 0.0" />
-        <geometry>
-          <box size="0.02092 0.575938 2.22776" />
-        </geometry>
-      </collision>
-      <collision>
-        <origin xyz="0.009901 -0.254976 1.06578" />
-        <geometry>
-          <box size="0.561938 0.016 0.064" />
-        </geometry>
-      </collision>
-      <collision>
-        <origin xyz="0.009901 0.0055 1.10578" />
-        <geometry>
-          <box size="0.561938 0.540942 0.016" />
-        </geometry>
-      </collision>
-      <collision>
-        <origin xyz="0.009901 0.0005 -0.361161 " />
-        <geometry>
-          <box size="0.561938 0.534942 0.015" />
+        <origin xyz="0.010499 -0.3 0.05" />
+        <geometry>
+          <box size="0.55494 0.019 2.12778" />
+        </geometry>
+      </collision>
+      <collision>
+        <origin xyz="0.010499 0.280469 0.05" />
+        <geometry>
+          <box size="0.55494 0.019 2.12778" />
+        </geometry>
+      </collision>
+      <collision>
+        <origin xyz="0.271973 -0.009901 0.041995" />
+        <geometry>
+          <box size="0.008 0.561938 2.11178" />
+        </geometry>
+      </collision>
+      <collision>
+        <origin xyz="0.0 0.299967 0.0" />
+        <geometry>
+          <box size="0.575938 0.02092 2.22776" />
+        </geometry>
+      </collision>
+      <collision>
+        <origin xyz="-0.254976 -0.009901 1.06578" />
+        <geometry>
+          <box size="0.016 0.561938 0.064" />
+        </geometry>
+      </collision>
+      <collision>
+        <origin xyz="0.0055 -0.009901 1.10578" />
+        <geometry>
+          <box size="0.540942 0.561938 0.016" />
+        </geometry>
+      </collision>
+      <collision>
+        <origin xyz="0.0005 -0.009901 0.249501" />
+        <geometry>
+          <box size="0.540942 0.561938 0.015" />
         </geometry>
       </collision>
@@ -104,11 +104,12 @@
       </visual>
       <collision>
-        <geometry>
-          <box size="0.561938 0.534942 0.015" />
+        <origin xyz="0.0005 -0.009901 -0.361161 " />
+        <geometry>
+          <box size="0.534942 0.561938 0.015" />
         </geometry>
       </collision>
     </link>
     <joint name="cabinet1_door_joint" type="revolute">
-      <origin xyz="-0.280 -0.280 0.677" rpy="0.0 0.0 0.0" />
+      <origin xyz="-0.280 0.280 0.677" rpy="0.0 0.0 0.0" />
       <parent link="cabinet1" />
       <child link="cabinet1_door" />
@@ -123,12 +124,12 @@
       </visual>
       <collision>
-        <origin xyz="0.285091 0.0 0.0" />
-        <geometry>
-          <box size="0.596936 0.019 0.86681" />
+        <origin xyz="0.0 -0.285091 0.0" />
+        <geometry>
+          <box size="0.019 0.596936 0.86681" />
         </geometry>
       </collision>
     </link>
     <joint name="cabinet1_door_handle_joint" type="fixed">
-      <origin xyz="0.46315559 -0.01559982 -0.38983368" rpy="0.0 0.0 ${pi/2}" />
+      <origin xyz="-0.01559982 -0.46315559 -0.38983368" rpy="${pi/2} 0.0 0.0" />
       <parent link="cabinet1_door" />
       <child link="cabinet1_door_handle" />
@@ -141,11 +142,11 @@
       </visual>
       <collision>
-        <origin xyz="-0.003891 0.08 0.0" />
-        <geometry>
-          <box size="0.02 0.013 0.013" />
-        </geometry>
-      </collision>
-      <collision>
-        <origin xyz="-0.003891 -0.08 0.0" />
+        <origin xyz="-0.003891 0.0 0.08" />
+        <geometry>
+          <box size="0.02 0.013 0.013" />
+        </geometry>
+      </collision>
+      <collision>
+        <origin xyz="-0.003891 0.0 -0.08" />
         <geometry>
           <box size="0.02 0.013 0.013" />
@@ -155,13 +156,13 @@
         <origin xyz="-0.0203895 0.0 0.0" />
         <geometry>
-          <box size="0.013 0.173032  0.013" />
+          <box size="0.013 0.013 0.173032" />
         </geometry>
       </collision>
     </link>
     <joint name="cabinet1_drawer1_joint" type="prismatic">
-      <origin xyz="0.01122015 -0.04679018 -0.48658508" rpy="0.0 0.0 0.0" />
+      <origin xyz="-0.04679018 -0.01122015 -0.48658508" rpy="0.0 0.0 0.0" />
       <parent link="cabinet1" />
       <child link="cabinet1_drawer1" />
-      <axis xyz="0 -1 0" />
+      <axis xyz="-1 0 0" />
       <limit effort="1000.0" lower="0.0" upper="0.45" velocity="0.5" />
     </joint>
@@ -173,48 +174,48 @@
       </visual>
       <collision>
-        <origin xyz="0.0 -0.233977 0.0" />
-        <geometry>
-          <box size="0.596936 0.019 0.262972" />
-        </geometry>
-      </collision>
-      <collision>
-        <origin xyz="0.26865 0.021336 0.0412455" />
-        <geometry>
-          <box size="0.0158442 0.4917 0.0223924" />
-        </geometry>
-      </collision>
-      <collision>
-        <origin xyz="-0.26865 0.021336 0.0412455" />
-        <geometry>
-          <box size="0.0158442 0.4917 0.0223924" />
-        </geometry>
-      </collision>
-      <collision>
-        <origin xyz="0.26865 0.021336 -0.078968" />
-        <geometry>
-          <box size="0.0158442 0.4917 0.083496" />
-        </geometry>
-      </collision>
-      <collision>
-        <origin xyz="-0.26865 0.021336 -0.0941" />
-        <geometry>
-          <box size="0.0158442 0.4917 0.053098" />
-        </geometry>
-      </collision>
-      <collision>
-        <origin xyz="0.0 0.021399 -0.114232" />
-        <geometry>
-          <box size="0.52364 0.49156 0.016" />
-        </geometry>
-      </collision>
-      <collision>
-        <origin xyz="0.0 0.26 -0.038" />
-        <geometry>
-          <box size="0.52364 0.01865384 0.16887" />
+        <origin xyz="-0.233977 0.0 0.0" />
+        <geometry>
+          <box size="0.019 0.596936 0.262972" />
+        </geometry>
+      </collision>
+      <collision>
+        <origin xyz="0.021336 -0.26865 0.0412455" />
+        <geometry>
+          <box size="0.4917 0.0158442 0.0223924" />
+        </geometry>
+      </collision>
+      <collision>
+        <origin xyz="0.021336 0.26865 0.0412455" />
+        <geometry>
+          <box size="0.4917 0.0158442 0.0223924" />
+        </geometry>
+      </collision>
+      <collision>
+        <origin xyz="0.021336 -0.26865 -0.078968" />
+        <geometry>
+          <box size="0.4917 0.0158442 0.083496" />
+        </geometry>
+      </collision>
+      <collision>
+        <origin xyz="0.021336 0.26865 -0.0941" />
+        <geometry>
+          <box size="0.4917 0.0158442 0.053098" />
+        </geometry>
+      </collision>
+      <collision>
+        <origin xyz="0.021399 0.0 -0.114232" />
+        <geometry>
+          <box size="0.49156 0.52364 0.016" />
+        </geometry>
+      </collision>
+      <collision>
+        <origin xyz="0.26 0.0 -0.038" />
+        <geometry>
+          <box size="0.01865384 0.52364 0.16887" />
         </geometry>
       </collision>
     </link>
     <joint name="cabinet1_drawer1_handle_joint" type="fixed">
-      <origin xyz="0.00091816 -0.24792936 0.08401428" rpy="0.0 0.0 ${pi/2}" />
+      <origin xyz="-0.24792936 0.00091816 0.08401428" rpy="${pi/2} 0.0 0.0" />
       <parent link="cabinet1_drawer1" />
       <child link="cabinet1_drawer1_handle" />
@@ -227,11 +228,11 @@
       </visual>
       <collision>
-        <origin xyz="-0.003891 0.08 0.0" />
-        <geometry>
-          <box size="0.02 0.013 0.013" />
-        </geometry>
-      </collision>
-      <collision>
-        <origin xyz="-0.003891 -0.08 0.0" />
+        <origin xyz="-0.003891 0.0 0.08" />
+        <geometry>
+          <box size="0.02 0.013 0.013" />
+        </geometry>
+      </collision>
+      <collision>
+        <origin xyz="-0.003891 0.0 -0.08" />
         <geometry>
           <box size="0.02 0.013 0.013" />
@@ -241,13 +242,13 @@
         <origin xyz="-0.0203895 0.0 0.0" />
         <geometry>
-          <box size="0.013 0.173032  0.013" />
+          <box size="0.013 0.013 0.173032" />
         </geometry>
       </collision>
     </link>
     <joint name="cabinet1_drawer2_joint" type="prismatic">
-      <origin xyz="0.011 -0.046 -0.816" rpy="0.0 0.0 0.0" />
+      <origin xyz="-0.046 -0.011 -0.816" rpy="0.0 0.0 0.0" />
       <parent link="cabinet1" />
       <child link="cabinet1_drawer2" />
-      <axis xyz="0 -1 0" />
+      <axis xyz="-1 0 0" />
       <limit effort="1000.0" lower="0.0" upper="0.45" velocity="0.5" />
     </joint>
@@ -259,48 +260,48 @@
       </visual>
       <collision>
-        <origin xyz="0.0 -0.233977 0.0" />
-        <geometry>
-          <box size="0.596936 0.019 0.39428" />
-        </geometry>
-      </collision>
-      <collision>
-        <origin xyz="0.26865 0.021336 -0.0084109" />
-        <geometry>
-          <box size="0.0158442 0.4917 0.0223924" />
-        </geometry>
-      </collision>
-      <collision>
-        <origin xyz="-0.26865 0.021336 -0.0084109" />
-        <geometry>
-          <box size="0.0158442 0.4917 0.0223924" />
-        </geometry>
-      </collision>
-      <collision>
-        <origin xyz="0.26865 0.021336 -0.12854" />
-        <geometry>
-          <box size="0.0158442 0.4917 0.083502" />
-        </geometry>
-      </collision>
-      <collision>
-        <origin xyz="-0.26865 0.021336 -0.12854" />
-        <geometry>
-          <box size="0.0158442 0.4917 0.083502" />
-        </geometry>
-      </collision>
-      <collision>
-        <origin xyz="0.0 0.021399 -0.16226" />
-        <geometry>
-          <box size="0.52364 0.49156 0.016" />
-        </geometry>
-      </collision>
-      <collision>
-        <origin xyz="0.0 0.26 -0.0797358 " />
-        <geometry>
-          <box size="0.52364 0.01865384 0.1517224" />
+        <origin xyz="-0.233977 0.0 0.0" />
+        <geometry>
+          <box size="0.019 0.596936 0.39428" />
+        </geometry>
+      </collision>
+      <collision>
+        <origin xyz="0.021336 -0.26865 -0.0084109" />
+        <geometry>
+          <box size="0.4917 0.0158442 0.0223924" />
+        </geometry>
+      </collision>
+      <collision>
+        <origin xyz="0.021336 0.26865 -0.0084109" />
+        <geometry>
+          <box size="0.4917 0.0158442 0.0223924" />
+        </geometry>
+      </collision>
+      <collision>
+        <origin xyz="0.021336 -0.26865 -0.12854" />
+        <geometry>
+          <box size="0.4917 0.0158442 0.083502" />
+        </geometry>
+      </collision>
+      <collision>
+        <origin xyz="0.021336 0.26865 -0.12854" />
+        <geometry>
+          <box size="0.4917 0.0158442 0.083502" />
+        </geometry>
+      </collision>
+      <collision>
+        <origin xyz="0.021399 0.0 -0.16226" />
+        <geometry>
+          <box size="0.49156 0.52364 0.016" />
+        </geometry>
+      </collision>
+      <collision>
+        <origin xyz="0.26 0.0 -0.0797358 " />
+        <geometry>
+          <box size="0.01865384 0.52364 0.1517224" />
         </geometry>
       </collision>
     </link>
     <joint name="cabinet1_drawer2_handle_joint" type="fixed">
-      <origin xyz="0.00145845 -0.24909416 0.150606" rpy="0.0 0.0 ${pi/2}" />
+      <origin xyz="-0.24909416 -0.00145845 0.150606" rpy="${pi/2} 0.0 0.0" />
       <parent link="cabinet1_drawer2" />
       <child link="cabinet1_drawer2_handle" />
@@ -313,11 +314,11 @@
       </visual>
       <collision>
-        <origin xyz="-0.003891 0.08 0.0" />
-        <geometry>
-          <box size="0.02 0.013 0.013" />
-        </geometry>
-      </collision>
-      <collision>
-        <origin xyz="-0.003891 -0.08 0.0" />
+        <origin xyz="-0.003891 0.0 0.08" />
+        <geometry>
+          <box size="0.02 0.013 0.013" />
+        </geometry>
+      </collision>
+      <collision>
+        <origin xyz="-0.003891 0.0 -0.08" />
         <geometry>
           <box size="0.02 0.013 0.013" />
@@ -327,10 +328,10 @@
         <origin xyz="-0.0203895 0.0 0.0" />
         <geometry>
-          <box size="0.013 0.173032  0.013" />
+          <box size="0.013 0.013 0.173032" />
         </geometry>
       </collision>
     </link>
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
Commit message: Fix typo

File: iai_apartment/urdf/kitchen_unreal.xacro (robot description, xacro)
@@ -631,5 +631,5 @@
         <origin xyz="-0.003984 0.0 -0.080242" />
         <geometry>
-          <box size="0.494978 -0.361962 0.021498" />
+          <box size="0.494978 0.361962 0.021498" />
         </geometry>
       </collision>
@@ -705,5 +705,5 @@
         <origin xyz="-0.003984 0.0 -0.080242" />
         <geometry>
-          <box size="0.494978 -0.361962 0.021498" />
+          <box size="0.494978 0.361962 0.021498" />
         </geometry>
       </collision>
@@ -779,5 +779,5 @@
         <origin xyz="-0.003984 0.0 -0.080242" />
         <geometry>
-          <box size="0.494978 -0.361962 0.021498" />
+          <box size="0.494978 0.361962 0.021498" />
         </geometry>
       </collision>
@@ -853,5 +853,5 @@
         <origin xyz="-0.003984 0.0 -0.080242" />
         <geometry>
-          <box size="0.494978 -0.361962 0.021498" />
+          <box size="0.494978 0.361962 0.021498" />
         </geometry>
       </collision>
@@ -927,5 +927,5 @@
         <origin xyz="-0.003984 0.0 -0.080242" />
         <geometry>
-          <box size="0.494978 -0.361962 0.021498" />
+          <box size="0.494978 0.361962 0.021498" />
         </geometry>
       </collision>
@@ -1261,5 +1261,5 @@
         <origin xyz="0.011034 0.0 0.855407" />
         <geometry>
-          <box size="0.49339 -0.556434 0.047996" />
+          <box size="0.49339 0.556434 0.047996" />
         </geometry>
       </collision>
@@ -1267,5 +1267,5 @@
         <origin xyz="-0.029351 0.0 0.839695" />
         <geometry>
-          <box size="0.392848 -0.469566 0.07542" />
+          <box size="0.392848 0.469566 0.07542" />
         </geometry>
       </collision>
@@ -2078,5 +2078,5 @@
         <origin xyz="0.217476 0.0 0.390909" />
         <geometry>
-          <box size="0.08 -0.369666 0.016" />
+          <box size="0.08 0.369666 0.016" />
         </geometry>
       </collision>

Commit message: Remove shelf collision offset

File: iai_apartment/urdf/kitchen_unreal.xacro (robot description, xacro)
@@ -104,5 +104,4 @@
       </visual>
       <collision>
-        <origin xyz="0.0005 -0.009901 -0.361161 " />
         <geometry>
           <box size="0.534942 0.561938 0.015" />
