Commit message: Add left window

File: iai_apartment/urdf/apartment_unreal_with_window4.urdf (robot description, URDF)
Before this commit: robot apartment, 123 links, 122 joints
Links:
- added link window4_right; collision box size=0.843426 0.02 2.05976; visual mesh filename=package://iai_apartment/meshes/unreal/SM_Window_Right.dae
- added link window4_right_handle; collision cylinder length=0.052952 radius=0.008; collision cylinder length=0.075236 radius=0.008
Joints:
- added joint window4_right_handle_joint: type revolute, parent window4_right, child window4_right_handle, origin xyz=-0.823253 -0.026228 0.0, axis 0 -1 0, limit lower=0.0 upper=3.141592653589793 effort=1000.0 velocity=3.141592653589793
- added joint window4_right_joint: type revolute, parent window4_frame, child window4_right, origin xyz=0.924416 -0.00162 -0.42549, axis 0 0 1, limit lower=0.0 upper=1.5708 effort=1000.0 velocity=1.5708
- joint window4_left_handle_joint: origin xyz=-0.823253 -0.026228 0.0 -> xyz=0.841963 -0.026228 0.0
- joint window4_left_joint: axis 0 0 1 -> 0 0 -1; origin xyz=0.924416 -0.00162 -0.42549 -> xyz=-0.9369 0.00162 -0.42549

File: iai_apartment/urdf/furnitures_with_window4.xacro (robot description, xacro)
@@ -81,11 +81,63 @@
       </collision>
     </link>
-    <joint name="window4_left_joint" type="revolute">
+    <joint name="window4_right_joint" type="revolute">
       <origin xyz="0.924416 -0.00162 -0.42549" />
       <parent link="window4_frame" />
-      <child link="window4_left" />
+      <child link="window4_right" />
       <axis xyz="0 0 1" />
       <limit effort="1000.0" lower="0.0" upper="1.5708" velocity="1.5708" />
     </joint>
+    <link name="window4_right">
+      <visual>
+        <geometry>
+          <mesh filename="package://iai_apartment/meshes/unreal/SM_Window_Right.dae" />
+        </geometry>
+      </visual>
+      <collision>
+        <origin xyz="-0.429577 0.000856 0" />
+        <geometry>
+          <box size="0.843426 0.02 2.05976" />
+        </geometry>
+      </collision>
+    </link>
+    <joint name="window4_right_handle_joint" type="revolute">
+      <origin xyz="-0.823253 -0.026228 0.0" />
+      <parent link="window4_right" />
+      <child link="window4_right_handle" />
+      <axis xyz="0 -1 0" />
+      <limit effort="1000.0" lower="0.0" upper="${pi}" velocity="${pi}" />
+    </joint>
+    <link name="window4_right_handle">
+      <visual>
+        <geometry>
+          <mesh filename="package://iai_apartment/meshes/unreal/SM_Window_Handle.dae" />
+        </geometry>
+      </visual>
+      <collision>
+        <origin xyz="0 -0.011369 0" rpy="${pi/2} 0 0" />
+        <geometry>
+          <cylinder length="0.075236" radius="0.008" />
+        </geometry>
+      </collision>
+      <collision>
+        <origin xyz="0 -0.040987 -0.057684" rpy="0 0 0" />
+        <geometry>
+          <cylinder length="0.131626" radius="0.008" />
+        </geometry>
+      </collision>
+      <collision>
+        <origin xyz="0 -0.022511 -0.115497" rpy="${pi/2} 0 0" />
+        <geometry>
+          <cylinder length="0.052952" radius="0.008" />
+        </geometry>
+      </collision>
+    </link>
+    <joint name="window4_left_joint" type="revolute">
+      <origin xyz="-0.9369 0.00162 -0.42549" />
+      <parent link="window4_frame" />
+      <child link="window4_left" />
+      <axis xyz="0 0 -1" />
+      <limit effort="1000.0" lower="0.0" upper="1.5708" velocity="1.5708" />
+    </joint>
     <link name="window4_left">
       <visual>
@@ -95,5 +147,5 @@
       </visual>
       <collision>
-        <origin xyz="-0.429577 0.000856 0" />
+        <origin xyz="0.429577 0.000856 0" />
         <geometry>
           <box size="0.843426 0.02 2.05976" />
@@ -102,5 +154,5 @@
     </link>
     <joint name="window4_left_handle_joint" type="revolute">
-      <origin xyz="-0.823253 -0.026228 0.0" />
+      <origin xyz="0.841963 -0.026228 0.0" />
       <parent link="window4_left" />
       <child link="window4_left_handle" />

Commit message: Fix window meshes

File: iai_apartment/urdf/apartment_unreal_with_window4.urdf (robot description, URDF)
Before this commit: robot apartment, 125 links, 124 joints
Links:
- link window4_left: geometry collision box size=0.86406 0.02 2.0631; visual mesh filename=package://iai_apartment/meshes/unreal/SM_Window_Left.dae
- link window4_right: geometry collision box size=0.843426 0.02 2.0631; visual mesh filename=package://iai_apartment/meshes/unreal/SM_Window_Right.dae
Joints:
- joint window4_left_handle_joint: origin xyz=0.841963 -0.026228 0.0 -> xyz=0.834107 -0.019236 0.0
- joint window4_left_joint: origin xyz=-0.9369 0.00162 -0.42549 -> xyz=-0.929112 0.00162 -0.425471
- joint window4_right_handle_joint: origin xyz=-0.823253 -0.026228 0.0 -> xyz=-0.815383 -0.019236 0.0
- joint window4_right_joint: origin xyz=0.924416 -0.00162 -0.42549 -> xyz=0.916552 0 -0.425471

File: iai_apartment/urdf/furnitures_with_window4.xacro (robot description, xacro)
@@ -82,5 +82,5 @@
     </link>
     <joint name="window4_right_joint" type="revolute">
-      <origin xyz="0.924416 -0.00162 -0.42549" />
+      <origin xyz="0.916552 0 -0.425471" />
       <parent link="window4_frame" />
       <child link="window4_right" />
@@ -95,12 +95,12 @@
       </visual>
       <collision>
-        <origin xyz="-0.429577 0.000856 0" />
-        <geometry>
-          <box size="0.843426 0.02 2.05976" />
+        <origin xyz="-0.421713 0 0" />
+        <geometry>
+          <box size="0.843426 0.02 2.0631" />
         </geometry>
       </collision>
     </link>
     <joint name="window4_right_handle_joint" type="revolute">
-      <origin xyz="-0.823253 -0.026228 0.0" />
+      <origin xyz="-0.815383 -0.019236 0.0" />
       <parent link="window4_right" />
       <child link="window4_right_handle" />
@@ -134,5 +134,5 @@
     </link>
     <joint name="window4_left_joint" type="revolute">
-      <origin xyz="-0.9369 0.00162 -0.42549" />
+      <origin xyz="-0.929112 0.00162 -0.425471" />
       <parent link="window4_frame" />
       <child link="window4_left" />
@@ -147,12 +147,12 @@
       </visual>
       <collision>
-        <origin xyz="0.429577 0.000856 0" />
-        <geometry>
-          <box size="0.843426 0.02 2.05976" />
+        <origin xyz="0.43203 0 0" />
+        <geometry>
+          <box size="0.86406 0.02 2.0631" />
         </geometry>
       </collision>
     </link>
     <joint name="window4_left_handle_joint" type="revolute">
-      <origin xyz="0.841963 -0.026228 0.0" />
+      <origin xyz="0.834107 -0.019236 0.0" />
       <parent link="window4_left" />
       <child link="window4_left_handle" />

Commit message: Update apartment

File: iai_apartment/urdf/apartment_unreal_with_window4.urdf (robot description, URDF)
Before this commit: robot apartment, 125 links, 124 joints
Links:
- added link window4_left_handle_center
- added link window4_right_handle_center
- link dishwasher_tray1: geometry visual mesh filename=package://iai_apartment/meshes/unreal/SM_Dishwasher_Tray_01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
- link dishwasher_tray2: geometry visual mesh filename=package://iai_apartment/meshes/unreal/SM_Dishwasher_Tray_02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
- link dishwasher_tray3: geometry visual mesh filename=package://iai_apartment/meshes/unreal/SM_Dishwasher_Tray_03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
- link fridge_egg_tray: geometry visual mesh filename=package://iai_apartment/meshes/unreal/SM_Fridge_Egg_Tray.dae
Joints:
- added joint window4_left_handle_center_joint: type fixed, parent window4_left_handle, child window4_left_handle_center, origin xyz=0.0 -0.040987 -0.057684 rpy=3.141592653589793 0 1.5707963267948966
- added joint window4_right_handle_center_joint: type fixed, parent window4_right_handle, child window4_right_handle_center, origin xyz=0.0 -0.040987 -0.057684 rpy=3.141592653589793 0 1.5707963267948966
- joint window4_left_handle_joint: axis 0 -1 0 -> (none); limit lower=0.0 upper=3.141592653589793 effort=1000.0 velocity=3.141592653589793 -> (none); origin xyz=0.834107 -0.019236 0.0 -> xyz=0.834107 -0.019236 0.0 rpy=0 1.5707963267948966 0; type revolute -> fixed
- joint window4_right_handle_joint: axis 0 -1 0 -> (none); limit lower=0.0 upper=3.141592653589793 effort=1000.0 velocity=3.141592653589793 -> (none); origin xyz=-0.815383 -0.019236 0.0 -> xyz=-0.815383 -0.019236 0.0 rpy=0 -1.5707963267948966 0; type revolute -> fixed

File: iai_apartment/urdf/furnitures_with_window4.xacro (robot description, xacro)
@@ -81,5 +81,4 @@
       </collision>
     </link>
-    <!-- right window -->
     <joint name="window4_right_joint" type="revolute">
       <origin xyz="0.916552 0 -0.425471" />
@@ -103,5 +102,5 @@
     </link>
     <joint name="window4_right_handle_joint" type="fixed">
-      <origin xyz="-0.815383 -0.06 -0.058" rpy="${pi} 0 ${pi/2}"/>
+      <origin xyz="-0.815383 -0.019236 0.0" rpy="0 ${-pi/2} 0" />
       <parent link="window4_right" />
       <child link="window4_right_handle" />
@@ -114,10 +113,28 @@
       </visual>
       <collision>
-        <geometry>
-          <mesh filename="package://iai_apartment/meshes/handles/window_handle.obj" />
-        </geometry>
-      </collision>
-    </link>
-    <!-- left window -->
+        <origin xyz="0 -0.011369 0" rpy="${pi/2} 0 0" />
+        <geometry>
+          <cylinder length="0.075236" radius="0.008" />
+        </geometry>
+      </collision>
+      <collision>
+        <origin xyz="0 -0.040987 -0.057684" rpy="0 0 0" />
+        <geometry>
+          <cylinder length="0.131626" radius="0.008" />
+        </geometry>
+      </collision>
+      <collision>
+        <origin xyz="0 -0.022511 -0.115497" rpy="${pi/2} 0 0" />
+        <geometry>
+          <cylinder length="0.052952" radius="0.008" />
+        </geometry>
+      </collision>
+    </link>
+    <joint name="window4_right_handle_center_joint" type="fixed">
+      <origin xyz="0.0 -0.040987 -0.057684" rpy="${pi} 0 ${pi/2}" />
+      <parent link="window4_right_handle" />
+      <child link="window4_right_handle_center" />
+    </joint>
+    <link name="window4_right_handle_center" />
     <joint name="window4_left_joint" type="revolute">
       <origin xyz="-0.929112 0.00162 -0.425471" />
@@ -141,5 +158,5 @@
     </link>
     <joint name="window4_left_handle_joint" type="fixed">
-      <origin xyz="0.815383 -0.06 -0.058" rpy="${pi} 0 ${pi/2}"/>
+      <origin xyz="0.834107 -0.019236 0.0" rpy="0 ${pi/2} 0" />
       <parent link="window4_left" />
       <child link="window4_left_handle" />
@@ -147,5 +164,4 @@
     <link name="window4_left_handle">
       <visual>
-        <origin rpy="0 0 0"/>
         <geometry>
           <mesh filename="package://iai_apartment/meshes/unreal/SM_Window_Handle.dae" />
@@ -153,9 +169,28 @@
       </visual>
       <collision>
-        <geometry>
-          <mesh filename="package://iai_apartment/meshes/handles/window_handle.obj" />
-        </geometry>
-      </collision>
-    </link>
+        <origin xyz="0 -0.011369 0" rpy="${pi/2} 0 0" />
+        <geometry>
+          <cylinder length="0.075236" radius="0.008" />
+        </geometry>
+      </collision>
+      <collision>
+        <origin xyz="0 -0.040987 -0.057684" rpy="0 0 0" />
+        <geometry>
+          <cylinder length="0.131626" radius="0.008" />
+        </geometry>
+      </collision>
+      <collision>
+        <origin xyz="0 -0.022511 -0.115497" rpy="${pi/2} 0 0" />
+        <geometry>
+          <cylinder length="0.052952" radius="0.008" />
+        </geometry>
+      </collision>
+    </link>
+    <joint name="window4_left_handle_center_joint" type="fixed">
+      <origin xyz="0.0 -0.040987 -0.057684" rpy="${pi} 0 ${pi/2}" />
+      <parent link="window4_left_handle" />
+      <child link="window4_left_handle_center" />
+    </joint>
+    <link name="window4_left_handle_center" />
     <!-- Collision okay Walls -->
     <!-- From the door side being wall 1, turn right and count the walls. -->

File: iai_apartment/urdf/kitchen_unreal.xacro (robot description, xacro)
@@ -64,44 +64,11 @@
       </collision>
       <collision>
+        <origin xyz="0.009901 0.0005 0.249501" />
+        <geometry>
+          <box size="0.561938 0.540942 0.015" />
+        </geometry>
+      </collision>
+      <collision>
         <origin xyz="0.009901 0.0005 -0.361161 " />
-        <geometry>
-          <box size="0.561938 0.534942 0.015" />
-        </geometry>
-      </collision>
-    </link>
-    <material name="white">
-      <color rgba="1 1 1 1" />
-    </material>
-    <joint name="cabinet1_shelf1_joint" type="fixed">
-      <origin xyz="0.009901 0.0005 0.560" />
-      <parent link="cabinet1" />
-      <child link="cabinet1_shelf1" />
-    </joint>
-    <link name="cabinet1_shelf1">
-      <visual>
-        <geometry>
-          <box size="0.561938 0.534942 0.015" />
-        </geometry>
-        <material name="white" />
-      </visual>
-      <collision>
-        <geometry>
-          <box size="0.561938 0.534942 0.015" />
-        </geometry>
-      </collision>
-    </link>
-    <joint name="cabinet1_shelf2_joint" type="fixed">
-      <origin xyz="0.009901 0.0005 0.249501" />
-      <parent link="cabinet1" />
-      <child link="cabinet1_shelf2" />
-    </joint>
-    <link name="cabinet1_shelf2">
-      <visual>
-        <geometry>
-          <box size="0.561938 0.534942 0.015" />
-        </geometry>
-        <material name="white" />
-      </visual>
-      <collision>
         <geometry>
           <box size="0.561938 0.534942 0.015" />
@@ -1154,9 +1121,9 @@
         </geometry>
       </visual>
-      <collision>
+      <!-- <collision>
         <geometry>
           <mesh filename="package://iai_apartment/meshes/unreal/SM_Fridge_Egg_Tray.stl" />
         </geometry>
-      </collision>
+      </collision> -->
     </link>
     <joint name="fridge_door2_joint" type="revolute">
@@ -2687,6 +2654,7 @@
       </visual>
       <collision>
-        <geometry>
-          <mesh filename="package://iai_apartment/meshes/unreal/SM_Dishwasher_Tray_01.stl" />
+        <origin xyz="0.0 -0.037745 -0.05" />
+        <geometry>
+          <box size="0.54 0.44 0.2" />
         </geometry>
       </collision>
@@ -2706,6 +2674,7 @@
       </visual>
       <collision>
-        <geometry>
-          <mesh filename="package://iai_apartment/meshes/unreal/SM_Dishwasher_Tray_02.stl" />
+        <origin xyz="0.0 0.0 0.0" />
+        <geometry>
+          <box size="0.54 0.44 0.22" />
         </geometry>
       </collision>
@@ -2725,6 +2694,7 @@
       </visual>
       <collision>
-        <geometry>
-          <mesh filename="package://iai_apartment/meshes/unreal/SM_Dishwasher_Tray_03.stl" />
+        <origin xyz="0.0 0.0 0.0" />
+        <geometry>
+          <box size="0.54 0.44 0.072" />
         </geometry>
       </collision>

Commit message: Fix urdf

File: iai_apartment/urdf/apartment_unreal_with_window4.urdf (robot description, URDF)
Before this commit: robot apartment, 125 links, 124 joints
Links:
- link cabinet2_drawer2: geometry collision box size=0.013796 0.361962 0.020298; collision box size=0.013796 0.361962 0.098
- link cabinet2_drawer3: geometry collision box size=0.013796 0.361962 0.020298; collision box size=0.013796 0.361962 0.098
- link cabinet2_drawer4: geometry collision box size=0.013796 0.361962 0.020298; collision box size=0.013796 0.361962 0.098
- link cabinet2_drawer5: geometry collision box size=0.013796 0.361962 0.020298; collision box size=0.013796 0.361962 0.098
- link cabinet2_drawer6: geometry collision box size=0.013796 0.361962 0.020298; collision box size=0.013796 0.361962 0.098
- link cabinet6: geometry collision box size=0.008 0.369666 0.76582; collision box size=0.08 0.369666 0.016
- link fridge_base: geometry collision box size=0.01564 0.469566 0.929316; collision box size=0.116796 0.469566 0.56255

Commit message: Split wall

File: iai_apartment/urdf/apartment_unreal_with_window4.urdf (robot description, URDF)
Before this commit: robot apartment, 125 links, 124 joints
Links:
- removed link walls
- removed link windows
- added link wall1; collision box size=18.76044 0.1285 3.0517; visual mesh filename=package://iai_apartment/meshes/unreal/SM_Wall_01.dae
- added link wall2; collision box size=0.189552 4.9669 3.0517; visual mesh filename=package://iai_apartment/meshes/unreal/SM_Wall_02.dae
- added link wall3; collision box size=8.2886 0.1285 3.0517; collision box size=8.47354 0.1285 3.0517
- added link wall4; collision box size=0.189552 4.9669 3.0517; visual mesh filename=package://iai_apartment/meshes/unreal/SM_Wall_04.dae
Joints:
- removed joint walls_joint
- removed joint windows_joint
- added joint wall1_joint: type fixed, parent envelope_root, child wall1, origin xyz=0 0 -0.2 rpy=0 0 0
- added joint wall2_joint: type fixed, parent envelope_root, child wall2, origin xyz=0 0 -0.2 rpy=0 0 0
- added joint wall3_joint: type fixed, parent envelope_root, child wall3, origin xyz=0 0 -0.2 rpy=0 0 0
- added joint wall4_joint: type fixed, parent envelope_root, child wall4, origin xyz=0 0 -0.2 rpy=0 0 0
- joint window4_frame_joint: origin xyz=0.671098 3.37273 1.72145 rpy=0.0 0.0 -1.5707963267948966 -> xyz=0.671098 3.37273 1.92145 rpy=0.0 0.0 -1.5707963267948966; parent walls -> furnitures_root

File: iai_apartment/urdf/furnitures_with_window4.xacro (robot description, xacro)
@@ -8,13 +8,13 @@
     <link name="furnitures_root" />
     <!-- things and stuff -->
-    <joint name="walls_joint" type="fixed">
+    <joint name="wall1_joint" type="fixed">
       <origin rpy="0 0 0" xyz="0 0 -0.2" />
       <parent link="furnitures_root" />
-      <child link="walls" />
-    </joint>
-    <link name="walls">
-      <visual>
-        <geometry>
-          <mesh filename="package://iai_apartment/meshes/visual/walls.dae" />
+      <child link="wall1" />
+    </joint>
+    <link name="wall1">
+      <visual>
+        <geometry>
+          <mesh filename="package://iai_apartment/meshes/unreal/SM_Wall_01.dae" />
         </geometry>
       </visual>
@@ -25,4 +25,34 @@
         </geometry>
       </collision>
+    </link>
+    <joint name="wall2_joint" type="fixed">
+      <origin rpy="0 0 0" xyz="0 0 -0.2" />
+      <parent link="furnitures_root" />
+      <child link="wall2" />
+    </joint>
+    <link name="wall2">
+      <visual>
+        <geometry>
+          <mesh filename="package://iai_apartment/meshes/unreal/SM_Wall_02.dae" />
+        </geometry>
+      </visual>
+      <collision>
+        <origin xyz="-8.875 0.713447 1.73439" />
+        <geometry>
+          <box size="0.189552 4.9669 3.0517" />
+        </geometry>
+      </collision>
+    </link>
+    <joint name="wall3_joint" type="fixed">
+      <origin rpy="0 0 0" xyz="0 0 -0.2" />
+      <parent link="furnitures_root" />
+      <child link="wall3" />
+    </joint>
+    <link name="wall3">
+      <visual>
+        <geometry>
+          <mesh filename="package://iai_apartment/meshes/unreal/SM_Wall_03.dae" />
+        </geometry>
+      </visual>
       <collision>
         <origin xyz="-4.63823 3.27776 1.73439" />
@@ -37,4 +67,16 @@
         </geometry>
       </collision>
+    </link>
+    <joint name="wall4_joint" type="fixed">
+      <origin rpy="0 0 0" xyz="0 0 -0.2" />
+      <parent link="furnitures_root" />
+      <child link="wall4" />
+    </joint>
+    <link name="wall4">
+      <visual>
+        <geometry>
+          <mesh filename="package://iai_apartment/meshes/unreal/SM_Wall_04.dae" />
+        </geometry>
+      </visual>
       <collision>
         <origin xyz="9.98022 0.713447 1.73439" />
@@ -43,27 +85,9 @@
         </geometry>
       </collision>
-      <collision>
-        <origin xyz="-8.875 0.713447 1.73439" />
-        <geometry>
-          <box size="0.189552 4.9669 3.0517" />
-        </geometry>
-      </collision>
-    </link>
-    <joint name="windows_joint" type="fixed">
-      <origin rpy="0 0 0" xyz="0 0 -0.2" />
-      <parent link="furnitures_root" />
-      <child link="windows" />
-    </joint>
-    <link name="windows">
-      <visual>
-        <geometry>
-          <mesh filename="package://iai_apartment/meshes/visual/windows_without_4.dae" />
-        </geometry>
-      </visual>
     </link>
     <!-- Window 4 -->
     <joint name="window4_frame_joint" type="fixed">
-      <origin xyz="0.671098 3.37273 1.72145" rpy="0.0 0.0 ${-pi/2}"/>
-      <parent link="walls" />
+      <origin xyz="0.671098 3.37273 1.52145" rpy="0.0 0.0 ${-pi/2}"/>
+      <parent link="furnitures_root" />
       <child link="window4_frame" />
     </joint>

Commit message: Move dishwasher tray to avoid collision

File: iai_apartment/urdf/apartment_unreal_with_window4.urdf (robot description, URDF)
Before this commit: robot apartment, 127 links, 126 joints
Joints:
- joint dishwasher_tray1_joint: origin xyz=0.19401426 0.00735926 0.22713593 rpy=0.0 0.0 0.0 -> xyz=0.22401426 0.00735926 0.22713593 rpy=0.0 0.0 0.0
- joint dishwasher_tray2_joint: origin xyz=0.17742002 0.00735798 0.40232784 rpy=0.0 0.0 0.0 -> xyz=0.20742002 0.00735798 0.40232784 rpy=0.0 0.0 0.0
- joint dishwasher_tray3_joint: origin xyz=0.19787212 0.01312525 0.61131351 rpy=0.0 0.0 0.0 -> xyz=0.22787212 0.01312525 0.61131351 rpy=0.0 0.0 0.0
- joint wall1_joint: parent envelope_root -> furnitures_root
- joint wall2_joint: parent envelope_root -> furnitures_root
- joint wall3_joint: parent envelope_root -> furnitures_root
- joint wall4_joint: parent envelope_root -> furnitures_root
- joint window4_frame_joint: origin xyz=0.671098 3.37273 1.92145 rpy=0.0 0.0 -1.5707963267948966 -> xyz=0.671098 3.37273 1.52145 rpy=0.0 0.0 -1.5707963267948966

File: iai_apartment/urdf/kitchen_unreal.xacro (robot description, xacro)
@@ -2680,5 +2680,5 @@
     </link>
     <joint name="dishwasher_tray1_joint" type="prismatic">
-      <origin xyz="0.19401426 0.00735926 0.22713593" rpy="0.0 0.0 0.0" />
+      <origin xyz="0.22401426 0.00735926 0.22713593" rpy="0.0 0.0 0.0" />
       <parent link="dishwasher" />
       <child link="dishwasher_tray1" />
@@ -2724,5 +2724,5 @@
     </link>
     <joint name="dishwasher_tray2_joint" type="prismatic">
-      <origin xyz="0.17742002 0.00735798 0.40232784" rpy="0.0 0.0 0.0" />
+      <origin xyz="0.20742002 0.00735798 0.40232784" rpy="0.0 0.0 0.0" />
       <parent link="dishwasher" />
       <child link="dishwasher_tray2" />
@@ -2768,5 +2768,5 @@
     </link>
     <joint name="dishwasher_tray3_joint" type="prismatic">
-      <origin xyz="0.19787212 0.01312525 0.61131351" rpy="0.0 0.0 0.0" />
+      <origin xyz="0.22787212 0.01312525 0.61131351" rpy="0.0 0.0 0.0" />
       <parent link="dishwasher" />
       <child link="dishwasher_tray3" />
