Commit message: Renamed links and joints for kitchen to be more expressive

File: iai_apartment/urdf/kitchen.xacro (robot description, xacro)
@@ -23,11 +23,11 @@
     <link name="side_B" />
     <!-- - - - - - - - - - - - - Cabinets side A - - - - - - - - - -->
-    <!-- Cabinet 1 -->
-    <joint name="cabinet1_joint" type="fixed">
+    <!-- oven_area -->
+    <joint name="oven_area_joint" type="fixed">
       <origin xyz="0.01 0.01 1.02" />
       <parent link="side_A" />
-      <child link="cabinet1" />
-    </joint>
-    <link name="cabinet1">
+      <child link="oven_area" />
+    </joint>
+    <link name="oven_area">
       <visual>
         <origin xyz="0.0 0.0 0.0" />
@@ -43,12 +43,12 @@
       </collision>
     </link>
-    <joint name="cabinet1_door_top_left_joint" type="revolute">
+    <joint name="oven_area_door_top_left_joint" type="revolute">
       <origin xyz="0.103 -0.3 0.32" rpy="0 0 3.14" />
-      <parent link="cabinet1" />
-      <child link="cabinet1_door_top_left" />
+      <parent link="oven_area" />
+      <child link="oven_area_door_top_left" />
       <axis xyz="0 0 -1" />
       <limit effort="1000.0" lower="0.0" upper="1.5708" velocity="1.5708" />
     </joint>
-    <link name="cabinet1_door_top_left">
+    <link name="oven_area_door_top_left">
       <visual>
         <origin xyz="0.001 -0.305 0.35" rpy="0 0 3.14" />
@@ -64,10 +64,10 @@
       </collision>
     </link>
-    <joint name="handle_cab1_top_door_joint" type="fixed">
+    <joint name="oven_area_door_top_left_handle_joint" type="fixed">
       <origin xyz="-0.055 -0.5 0.0" rpy="1.57 0 0" />
-      <parent link="cabinet1_door_top_left" />
-      <child link="handle_cab1_top_door" />
-    </joint>
-    <link name="handle_cab1_top_door">
+      <parent link="oven_area_door_top_left" />
+      <child link="oven_area_door_top_left_handle" />
+    </joint>
+    <link name="oven_area_door_top_left_handle">
       <visual>
         <geometry>
@@ -84,5 +84,5 @@
       <origin xyz="-0.175 0.0 -0.025" rpy="0 0 0" />
       <!-- <origin xyz="-0.125 0.0 -0.025" rpy="0 0 0"/> -->
-      <parent link="cabinet1" />
+      <parent link="oven_area" />
       <child link="oven" />
     </joint>
@@ -104,12 +104,12 @@
       </collision>
     </link>
-    <joint name="cabinet1_drawer_middle_joint" type="prismatic">
+    <joint name="oven_area_drawer_middle_joint" type="prismatic">
       <origin xyz="-0.117 0.0 -0.43" rpy="0 0 3.14" />
-      <parent link="cabinet1" />
-      <child link="cabinet1_drawer_middle" />
-      <axis xyz="-1 0 0" />
-      <limit effort="1000.0" lower="0.0" upper="0.45" velocity="0.5" />
-    </joint>
-    <link name="cabinet1_drawer_middle">
+      <parent link="oven_area" />
+      <child link="oven_area_drawer_middle" />
+      <axis xyz="-1 0 0" />
+      <limit effort="1000.0" lower="0.0" upper="0.45" velocity="0.5" />
+    </joint>
+    <link name="oven_area_drawer_middle">
       <visual>
         <origin rpy="0 0 3.14" />
@@ -125,29 +125,29 @@
       </collision>
     </link>
-    <joint name="handle_cab1_drawer_mid_joint" type="fixed">
+    <joint name="oven_area_drawer_middle_handle_joint" type="fixed">
       <origin xyz="-0.26 0.0 0.11" rpy="1.57 0 0" />
-      <parent link="cabinet1_drawer_middle" />
-      <child link="handle_cab1_drawer_mid" />
-    </joint>
-    <link name="handle_cab1_drawer_mid">
-      <visual>
-        <geometry>
-          <mesh filename="package://iai_apartment/meshes/handles/handle_horizontal.dae" />
-        </geometry>
-      </visual>
-      <collision>
-        <geometry>
-          <mesh filename="package://iai_apartment/meshes/handles/handle_horizontal.obj" />
-        </geometry>
-      </collision>
-    </link>
-    <joint name="cabinet1_drawer_bottom_joint" type="prismatic">
+      <parent link="oven_area_drawer_middle" />
+      <child link="oven_area_drawer_middle_handle" />
+    </joint>
+    <link name="oven_area_drawer_middle_handle">
+      <visual>
+        <geometry>
+          <mesh filename="package://iai_apartment/meshes/handles/handle_horizontal.dae" />
+        </geometry>
+      </visual>
+      <collision>
+        <geometry>
+          <mesh filename="package://iai_apartment/meshes/handles/handle_horizontal.obj" />
+        </geometry>
+      </collision>
+    </link>
+    <joint name="oven_area_drawer_bottom_joint" type="prismatic">
       <origin xyz="-0.094 0.0 -0.95" rpy="0 0 3.14" />
-      <parent link="cabinet1" />
-      <child link="cabinet1_drawer_bottom" />
-      <axis xyz="-1 0 0" />
-      <limit effort="1000.0" lower="0.0" upper="0.45" velocity="0.5" />
-    </joint>
-    <link name="cabinet1_drawer_bottom">
+      <parent link="oven_area" />
+      <child link="oven_area_drawer_bottom" />
+      <axis xyz="-1 0 0" />
+      <limit effort="1000.0" lower="0.0" upper="0.45" velocity="0.5" />
+    </joint>
+    <link name="oven_area_drawer_bottom">
       <visual>
         <origin rpy="0 0 -3.14" />
@@ -163,10 +163,10 @@
       </collision>
     </link>
-    <joint name="handle_cab1_drawer_bottom_joint" type="fixed">
+    <joint name="oven_area_drawer_bottom_handle_joint" type="fixed">
       <origin xyz="-0.237 0.0 0.35" rpy="1.57 0 0" />
-      <parent link="cabinet1_drawer_bottom" />
-      <child link="handle_cab1_drawer_bottom" />
-    </joint>
-    <link name="handle_cab1_drawer_bottom">
+      <parent link="oven_area_drawer_bottom" />
+      <child link="oven_area_drawer_bottom_handle" />
+    </joint>
+    <link name="oven_area_drawer_bottom_handle">
       <visual>
         <geometry>
@@ -184,10 +184,10 @@
       <color rgba="1 1 1 1" />
     </material>
-    <joint name="cabinet1_coloksu_level4_joint" type="fixed">
+    <joint name="oven_area_coloksu_level4_joint" type="fixed">
       <origin xyz="-0.172 0.005 0.281" />
-      <parent link="cabinet1" />
-      <child link="cabinet1_coloksu_level4" />
-    </joint>
-    <link name="cabinet1_coloksu_level4">
+      <parent link="oven_area" />
+      <child link="oven_area_coloksu_level4" />
+    </joint>
+    <link name="oven_area_coloksu_level4">
       <visual>
         <geometry>
@@ -202,12 +202,12 @@
       </collision>
     </link>
-    <joint name="cabinet1_coloksu_level5_joint" type="fixed">
+    <joint name="oven_area_coloksu_level5_joint" type="fixed">
       <!-- actually this should align with the CAD model but the CAD model is incorrect. -->
       <!-- <origin xyz="-0.172 0.005 0.672"/> -->
       <origin xyz="-0.172 0.005 0.56" />
-      <parent link="cabinet1" />
-      <child link="cabinet1_coloksu_level5" />
-    </joint>
-    <link name="cabinet1_coloksu_level5">
+      <parent link="oven_area" />
+      <child link="oven_area_coloksu_level5" />
+    </joint>
+    <link name="oven_area_coloksu_level5">
       <visual>
         <geometry>
@@ -222,11 +222,11 @@
       </collision>
     </link>
-    <!-- Cabinet 2 -->
-    <joint name="cabinet2_joint" type="fixed">
+    <!-- oven_area_right -->
+    <joint name="oven_area_right_joint" type="fixed">
       <origin xyz="-0.163 0.51 0.975" />
       <parent link="side_A" />
-      <child link="cabinet2" />
-    </joint>
-    <link name="cabinet2">
+      <child link="oven_area_right" />
+    </joint>
+    <link name="oven_area_right">
       <visual>
         <geometry>
@@ -240,20 +240,20 @@
       </collision>
     </link>
-    <joint name="cabinet2_door_out_joint" type="prismatic">
+    <joint name="oven_area_right_door_out_joint" type="prismatic">
       <origin xyz="0.277 -0.19 0.0" rpy="0 0 3.14" />
-      <parent link="cabinet2" />
-      <child link="cabinet2_door_out_fancy" />
+      <parent link="oven_area_right" />
+      <child link="oven_area_right_door_out_fancy" />
       <axis xyz="-1 0 0" />
       <limit effort="1.0" lower="0.0" upper="0.02" velocity="1.5708" />
-      <mimic joint="cabinet2_door_left_joint" multiplier="0.01" />
-    </joint>
-    <link name="cabinet2_door_out_fancy" />
-    <joint name="cabinet2_door_left_joint" type="revolute">
-      <parent link="cabinet2_door_out_fancy" />
-      <child link="cabinet2_door_left" />
+      <mimic joint="oven_area_right_door_left_joint" multiplier="0.01" />
+    </joint>
+    <link name="oven_area_right_door_out_fancy" />
+    <joint name="oven_area_right_door_left_joint" type="revolute">
+      <parent link="oven_area_right_door_out_fancy" />
+      <child link="oven_area_right_door" />
       <axis xyz="0 0 -1" />
       <limit effort="1000.0" lower="0.0" upper="1.5708" velocity="1.5708" />
     </joint>
-    <link name="cabinet2_door_left">
+    <link name="oven_area_right_door">
       <visual>
         <origin xyz="0 -0.2 0.145" rpy="0 0 3.14" />
@@ -271,27 +271,27 @@
     <joint name="handle_cab2_drawer_bottom_joint" type="fixed">
       <origin xyz="-0.040 -0.29 0.05" rpy="1.57 0 0" />
-      <parent link="cabinet2_door_left" />
-      <child link="handle_cab2_door" />
-    </joint>
-    <link name="handle_cab2_door">
-      <visual>
-        <geometry>
-          <mesh filename="package://iai_apartment/meshes/handles/handle_horizontal.dae" />
-        </geometry>
-      </visual>
-      <collision>
-        <geometry>
-          <mesh filename="package://iai_apartment/meshes/handles/handle_horizontal.obj" />
-        </geometry>
-      </collision>
-    </link>
-    <joint name="cabinet2_drawer_small_joint" type="prismatic">
+      <parent link="oven_area_right_door" />
+      <child link="oven_area_right_handle" />
+    </joint>
+    <link name="oven_area_right_handle">
+      <visual>
+        <geometry>
+          <mesh filename="package://iai_apartment/meshes/handles/handle_horizontal.dae" />
+        </geometry>
+      </visual>
+      <collision>
+        <geometry>
+          <mesh filename="package://iai_apartment/meshes/handles/handle_horizontal.obj" />
+        </geometry>
+      </collision>
+    </link>
+    <joint name="oven_area_right_drawer_small_joint" type="prismatic">
       <origin xyz="-0.01 0.0 0.17" rpy="0 0 3.14" />
-      <parent link="cabinet2" />
-      <child link="cabinet2_drawer_small" />
+      <parent link="oven_area_right" />
+      <child link="oven_area_right_drawer_small" />
       <axis xyz="-1 0 0" />
       <limit effort="500.0" lower="0.0" upper="0.45" velocity="0.5" />
     </joint>
-    <link name="cabinet2_drawer_small">
+    <link name="oven_area_right_drawer_small">
       <visual>
         <origin rpy="0 0 3.14" />
@@ -307,12 +307,12 @@
       </collision>
     </link>
-    <joint name="cabinet2_drawer_big_joint" type="prismatic">
+    <joint name="oven_area_right_drawer_big_joint" type="prismatic">
       <origin xyz="0.04 0.0 -0.12" rpy="0 0 3.14" />
-      <parent link="cabinet2" />
-      <child link="cabinet2_drawer_big" />
+      <parent link="oven_area_right" />
+      <child link="oven_area_right_drawer_big" />
       <axis xyz="-1 0 0" />
       <limit effort="500.0" lower="0.0" upper="0.45" velocity="0.5" />
     </joint>
-    <link name="cabinet2_drawer_big">
+    <link name="oven_area_right_drawer_big">
       <visual>
         <origin rpy="0 0 3.14" />
@@ -328,11 +328,11 @@
       </collision>
     </link>
-    <!-- Cabinet 3 -->
-    <joint name="cabinet3_joint" type="fixed">
+    <!-- fridge_area -->
+    <joint name="fridge_area_joint" type="fixed">
       <origin xyz="-0.273 1.022 1.07" />
       <parent link="side_A" />
-      <child link="cabinet3" />
-    </joint>
-    <link name="cabinet3">
+      <child link="fridge_area" />
+    </joint>
+    <link name="fridge_area">
       <visual>
         <geometry>
@@ -346,20 +346,20 @@
       </collision>
     </link>
-    <joint name="cabinet3_door_top_out_joint" type="revolute">
+    <joint name="fridge_area_door_top_out_joint" type="revolute">
       <origin xyz="0.39 -0.3 0.5" rpy="0 0 3.14" />
-      <parent link="cabinet3" />
-      <child link="cabinet3_door_top_out_fancy" />
+      <parent link="fridge_area" />
+      <child link="fridge_area_door_top_out_fancy" />
       <axis xyz="-1 0 0" />
       <limit effort="1.0" lower="0.0" upper="1.5708" velocity="1.5708" />
-      <mimic joint="cabinet3_door_top_left_joint" multiplier="0.01" />
-    </joint>
-    <link name="cabinet3_door_top_out_fancy" />
-    <joint name="cabinet3_door_top_left_joint" type="revolute">
-      <parent link="cabinet3_door_top_out_fancy" />
-      <child link="cabinet3_door_top_left" />
+      <mimic joint="fridge_area_door_top_left_joint" multiplier="0.01" />
+    </joint>
+    <link name="fridge_area_door_top_out_fancy" />
+    <joint name="fridge_area_door_top_left_joint" type="revolute">
+      <parent link="fridge_area_door_top_out_fancy" />
+      <child link="fridge_area_top_door" />
       <axis xyz="0 0 -1" />
       <limit effort="1000.0" lower="0.0" upper="1.5708" velocity="1.5708" />
     </joint>
-    <link name="cabinet3_door_top_left">
+    <link name="fridge_area_top_door">
       <visual>
         <origin xyz="0.001 -0.3 -0.1" rpy="0 0 3.14" />
@@ -375,37 +375,37 @@
       </collision>
     </link>
-    <joint name="handle_cab3_door_top_joint" type="fixed">
+    <joint name="fridge_area_door_top_left_handle_joint" type="fixed">
       <origin xyz="-0.036 -0.45 -0.65" rpy="1.57 0 0" />
-      <parent link="cabinet3_door_top_left" />
-      <child link="handle_cab3_door_top" />
-    </joint>
-    <link name="handle_cab3_door_top">
-      <visual>
-        <geometry>
-          <mesh filename="package://iai_apartment/meshes/handles/handle_horizontal.dae" />
-        </geometry>
-      </visual>
-      <collision>
-        <geometry>
-          <mesh filename="package://iai_apartment/meshes/handles/handle_horizontal.obj" />
-        </geometry>
-      </collision>
-    </link>
-    <joint name="cabinet3_door_bottom_out_joint" type="prismatic">
+      <parent link="fridge_area_top_door" />
+      <child link="fridge_area_top_door_handle" />
+    </joint>
+    <link name="fridge_area_top_door_handle">
+      <visual>
+        <geometry>
+          <mesh filename="package://iai_apartment/meshes/handles/handle_horizontal.dae" />
+        </geometry>
+      </visual>
+      <collision>
+        <geometry>
+          <mesh filename="package://iai_apartment/meshes/handles/handle_horizontal.obj" />
+        </geometry>
+      </collision>
+    </link>
+    <joint name="fridge_area_door_bottom_out_joint" type="prismatic">
       <origin xyz="0.39 -0.3 -0.5" rpy="0 0 3.14" />
-      <parent link="cabinet3" />
-      <child link="cabinet3_door_bottom_out_fancy" />
+      <parent link="fridge_area" />
+      <child link="fridge_area_door_bottom_out_fancy" />
       <axis xyz="-1 0 0" />
       <limit effort="1.0" lower="0.0" upper="0.02" velocity="1.5708" />
-      <mimic joint="cabinet3_door_bottom_left_joint" multiplier="0.01" />
-    </joint>
-    <link name="cabinet3_door_bottom_out_fancy" />
-    <joint name="cabinet3_door_bottom_left_joint" type="revolute">
-      <parent link="cabinet3_door_bottom_out_fancy" />
-      <child link="cabinet3_door_bottom_left" />
+      <mimic joint="fridge_area_door_bottom_left_joint" multiplier="0.01" />
+    </joint>
+    <link name="fridge_area_door_bottom_out_fancy" />
+    <joint name="fridge_area_door_bottom_left_joint" type="revolute">
+      <parent link="fridge_area_door_bottom_out_fancy" />
+      <child link="fridge_area_bottom_door" />
       <axis xyz="0 0 -1" />
       <limit effort="1000.0" lower="0.0" upper="1.5708" velocity="1.5708" />
     </joint>
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
Commit message: Added a simple fridge

File: iai_apartment/urdf/kitchen.xacro (robot description, xacro)
@@ -361,4 +361,112 @@
       <limit effort="1000.0" lower="0.0" upper="1.5708" velocity="1.5708" />
     </joint>
+    <link name="fridge_main" />
+    <joint name="fridge_main_joint" type="fixed">
+      <origin xyz="0 0 0" rpy="0 0 0" />
+      <parent link="fridge_area" />
+      <child link="fridge_main" />
+    </joint>
+    <link name="fridge_back">
+      <visual>
+        <geometry>
+          <box size="0.036 0.56 1.2" />
+        </geometry>
+      </visual>
+      <collision>
+        <geometry>
+          <box size="0.036 0.56 1.2" />
+        </geometry>
+      </collision>
+    </link>
+    <joint name="fridge_back_joint" type="fixed">
+      <origin xyz="-0.1 0 0.4" rpy="0 0 0" />
+      <parent link="fridge_main" />
+      <child link="fridge_back" />
+    </joint>
+    <link name="fridge_left_side">
+      <visual>
+        <geometry>
+          <box size="0.036 0.5 1.2" />
+        </geometry>
+      </visual>
+      <collision>
+        <geometry>
+          <box size="0.036 0.5 1.2" />
+        </geometry>
+      </collision>
+    </link>
+    <joint name="fridge_left_side_joint" type="fixed">
+      <origin xyz="0.1 -0.25 0.4" rpy="0 0 -1.57" />
+      <parent link="fridge_main" />
+      <child link="fridge_left_side" />
+    </joint>
+        <link name="fridge_right_side">
+      <visual>
+        <geometry>
+          <box size="0.036 0.5 1.2" />
+        </geometry>
+      </visual>
+      <collision>
+        <geometry>
+          <box size="0.036 0.5 1.2" />
+        </geometry>
+      </collision>
+    </link>
+    <joint name="fridge_right_side_joint" type="fixed">
+      <origin xyz="0.1 0.25 0.4" rpy="0 0 -1.57" />
+      <parent link="fridge_main" />
+      <child link="fridge_right_side" />
+    </joint>
+     <link name="fridge_top_side">
+      <visual>
+        <geometry>
+          <box size="0.5 0.535 0.036" />
+        </geometry>
+      </visual>
+      <collision>
+        <geometry>
+         <box size="0.5 0.535 0.036" />
+        </geometry>
+      </collision>
+    </link>
+    <joint name="fridge_top_side_joint" type="fixed">
+      <origin xyz="0.1 0. 1." rpy="0 0 0" />
+      <parent link="fridge_main" />
+      <child link="fridge_top_side" />
+    </joint>
+     <link name="fridge_bottom_side">
+      <visual>
+        <geometry>
+          <box size="0.5 0.535 0.036" />
+        </geometry>
+      </visual>
+      <collision>
+        <geometry>
+         <box size="0.5 0.535 0.036" />
+        </geometry>
+      </collision>
+    </link>
+    <joint name="fridge_bottom_side_joint" type="fixed">
+      <origin xyz="0.1 0. -0.2" rpy="0 0 0" />
+      <parent link="fridge_main" />
+      <child link="fridge_bottom_side" />
+    </joint>
+    <link name="fridge_level1">
+      <visual>
+        <geometry>
+          <box size="0.5 0.535 0.036" />
+        </geometry>
+      </visual>
+      <collision>
+        <geometry>
+         <box size="0.5 0.535 0.036" />
+        </geometry>
+      </collision>
+    </link>
+    <joint name="fridge_level1_joint" type="fixed">
+      <origin xyz="0.1 0. 0.1" rpy="0 0 0" />
+      <parent link="fridge_main" />
+      <child link="fridge_level1" />
+    </joint>
     <link name="fridge_area_top_door">
       <visual>
