Commit message: Put the fridge_door under fridge_main

File: iai_apartment/urdf/kitchen.xacro (robot description, xacro)
@@ -346,7 +346,115 @@
       </collision>
     </link>
+    <link name="fridge_main" />
+    <joint name="fridge_main_joint" type="fixed">
+      <origin xyz="0 0 0" rpy="0 0 0" />
+      <parent link="fridge_area" />
+      <child link="fridge_main" />
+    </joint>
+    <link name="fridge_back">
+      <visual>
+        <geometry>
+          <box size="0.036 0.56 1.2" />
+        </geometry>
+      </visual>
+      <collision>
+        <geometry>
+          <box size="0.036 0.56 1.2" />
+        </geometry>
+      </collision>
+    </link>
+    <joint name="fridge_back_joint" type="fixed">
+      <origin xyz="-0.1 0 0.4" rpy="0 0 0" />
+      <parent link="fridge_main" />
+      <child link="fridge_back" />
+    </joint>
+    <link name="fridge_left_side">
+      <visual>
+        <geometry>
+          <box size="0.036 0.5 1.2" />
+        </geometry>
+      </visual>
+      <collision>
+        <geometry>
+          <box size="0.036 0.5 1.2" />
+        </geometry>
+      </collision>
+    </link>
+    <joint name="fridge_left_side_joint" type="fixed">
+      <origin xyz="0.1 -0.25 0.4" rpy="0 0 -1.57" />
+      <parent link="fridge_main" />
+      <child link="fridge_left_side" />
+    </joint>
+        <link name="fridge_right_side">
+      <visual>
+        <geometry>
+          <box size="0.036 0.5 1.2" />
+        </geometry>
+      </visual>
+      <collision>
+        <geometry>
+          <box size="0.036 0.5 1.2" />
+        </geometry>
+      </collision>
+    </link>
+    <joint name="fridge_right_side_joint" type="fixed">
+      <origin xyz="0.1 0.25 0.4" rpy="0 0 -1.57" />
+      <parent link="fridge_main" />
+      <child link="fridge_right_side" />
+    </joint>
+     <link name="fridge_top_side">
+      <visual>
+        <geometry>
+          <box size="0.5 0.535 0.036" />
+        </geometry>
+      </visual>
+      <collision>
+        <geometry>
+         <box size="0.5 0.535 0.036" />
+        </geometry>
+      </collision>
+    </link>
+    <joint name="fridge_top_side_joint" type="fixed">
+      <origin xyz="0.1 0. 1." rpy="0 0 0" />
+      <parent link="fridge_main" />
+      <child link="fridge_top_side" />
+    </joint>
+     <link name="fridge_bottom_side">
+      <visual>
+        <geometry>
+          <box size="0.5 0.535 0.036" />
+        </geometry>
+      </visual>
+      <collision>
+        <geometry>
+         <box size="0.5 0.535 0.036" />
+        </geometry>
+      </collision>
+    </link>
+    <joint name="fridge_bottom_side_joint" type="fixed">
+      <origin xyz="0.1 0. -0.2" rpy="0 0 0" />
+      <parent link="fridge_main" />
+      <child link="fridge_bottom_side" />
+    </joint>
+    <link name="fridge_level1">
+      <visual>
+        <geometry>
+          <box size="0.5 0.535 0.036" />
+        </geometry>
+      </visual>
+      <collision>
+        <geometry>
+         <box size="0.5 0.535 0.036" />
+        </geometry>
+      </collision>
+    </link>
+    <joint name="fridge_level1_joint" type="fixed">
+      <origin xyz="0.1 0. 0.1" rpy="0 0 0" />
+      <parent link="fridge_main" />
+      <child link="fridge_level1" />
+    </joint>
     <joint name="fridge_area_door_top_out_joint" type="revolute">
       <origin xyz="0.39 -0.3 0.5" rpy="0 0 3.14" />
-      <parent link="fridge_area" />
+      <parent link="fridge_main" />
       <child link="fridge_area_door_top_out_fancy" />
       <axis xyz="-1 0 0" />
@@ -360,112 +468,4 @@
       <axis xyz="0 0 -1" />
       <limit effort="1000.0" lower="0.0" upper="1.5708" velocity="1.5708" />
-    </joint>
-    <link name="fridge_main" />
-    <joint name="fridge_main_joint" type="fixed">
-      <origin xyz="0 0 0" rpy="0 0 0" />
-      <parent link="fridge_area" />
-      <child link="fridge_main" />
-    </joint>
-    <link name="fridge_back">
-      <visual>
-        <geometry>
-          <box size="0.036 0.56 1.2" />
-        </geometry>
-      </visual>
-      <collision>
-        <geometry>
-          <box size="0.036 0.56 1.2" />
-        </geometry>
-      </collision>
-    </link>
-    <joint name="fridge_back_joint" type="fixed">
-      <origin xyz="-0.1 0 0.4" rpy="0 0 0" />
-      <parent link="fridge_main" />
-      <child link="fridge_back" />
-    </joint>
-    <link name="fridge_left_side">
-      <visual>
-        <geometry>
-          <box size="0.036 0.5 1.2" />
-        </geometry>
-      </visual>
-      <collision>
-        <geometry>
-          <box size="0.036 0.5 1.2" />
-        </geometry>
-      </collision>
-    </link>
-    <joint name="fridge_left_side_joint" type="fixed">
-      <origin xyz="0.1 -0.25 0.4" rpy="0 0 -1.57" />
-      <parent link="fridge_main" />
-      <child link="fridge_left_side" />
-    </joint>
-        <link name="fridge_right_side">
-      <visual>
-        <geometry>
-          <box size="0.036 0.5 1.2" />
-        </geometry>
-      </visual>
-      <collision>
-        <geometry>
-          <box size="0.036 0.5 1.2" />
-        </geometry>
-      </collision>
-    </link>
-    <joint name="fridge_right_side_joint" type="fixed">
-      <origin xyz="0.1 0.25 0.4" rpy="0 0 -1.57" />
-      <parent link="fridge_main" />
-      <child link="fridge_right_side" />
-    </joint>
-     <link name="fridge_top_side">
-      <visual>
-        <geometry>
-          <box size="0.5 0.535 0.036" />
-        </geometry>
-      </visual>
-      <collision>
-        <geometry>
-         <box size="0.5 0.535 0.036" />
-        </geometry>
-      </collision>
-    </link>
-    <joint name="fridge_top_side_joint" type="fixed">
-      <origin xyz="0.1 0. 1." rpy="0 0 0" />
-      <parent link="fridge_main" />
-      <child link="fridge_top_side" />
-    </joint>
-     <link name="fridge_bottom_side">
-      <visual>
-        <geometry>
-          <box size="0.5 0.535 0.036" />
-        </geometry>
-      </visual>
-      <collision>
-        <geometry>
-         <box size="0.5 0.535 0.036" />
-        </geometry>
-      </collision>
-    </link>
-    <joint name="fridge_bottom_side_joint" type="fixed">
-      <origin xyz="0.1 0. -0.2" rpy="0 0 0" />
-      <parent link="fridge_main" />
-      <child link="fridge_bottom_side" />
-    </joint>
-    <link name="fridge_level1">
-      <visual>
-        <geometry>
-          <box size="0.5 0.535 0.036" />
-        </geometry>
-      </visual>
-      <collision>
-        <geometry>
-         <box size="0.5 0.535 0.036" />
-        </geometry>
-      </collision>
-    </link>
-    <joint name="fridge_level1_joint" type="fixed">
-      <origin xyz="0.1 0. 0.1" rpy="0 0 0" />
-      <parent link="fridge_main" />
-      <child link="fridge_level1" />
     </joint>
     <link name="fridge_area_top_door">
