Commit message: apartment root moved to the left corner.

File: iai_apartment/urdf/apartment.urdf (robot description, URDF)
Before this commit: robot apartment, 11 links, 10 joints
Links:
- added link middle_of_the_room
Joints:
- added joint middle_of_the_room_joint: type fixed, parent apartment_root, child middle_of_the_room, origin xyz=8.85 1.75 0.0 rpy=0 0 0
- joint armchair_joint: parent apartment_root -> middle_of_the_room
- joint bedside_table_joint: parent apartment_root -> middle_of_the_room
- joint coffee_table_joint: parent apartment_root -> middle_of_the_room
- joint sofa_joint: parent apartment_root -> middle_of_the_room
- joint walls_joint: parent apartment_root -> middle_of_the_room
- joint wardrobe_joint: parent apartment_root -> middle_of_the_room
- joint windows_joint: parent apartment_root -> middle_of_the_room

Commit message: floor has been brought back down to the ground.

File: iai_apartment/urdf/apartment.urdf (robot description, URDF)
Before this commit: robot apartment, 12 links, 11 joints
Joints:
- joint armchair_joint: origin xyz=7.9688 -0.3791 0.2000 rpy=0 0 1.9199 -> xyz=7.9688 -0.3791 0.0 rpy=0 0 1.9199
- joint bedside_table_joint: origin xyz=7.2110 0.1296 0.2000 rpy=0 0 0 -> xyz=7.2110 0.1296 0.0 rpy=0 0 0
- joint coffee_table_joint: origin xyz=7.8034 1.02957 0.2000 rpy=0 0 1.5708 -> xyz=7.8034 1.02957 0.0 rpy=0 0 1.5708
- joint sofa_joint: origin xyz=8.1986 2.4096 0.2000 rpy=0 0 0 -> xyz=8.1986 2.4096 0.0 rpy=0 0 0
- joint walls_joint: origin (none) -> xyz=0 0 -0.2 rpy=0 0 0
- joint wardrobe_joint: origin xyz=9.7082 -0.6331 0.2000 rpy=0 0 0 -> xyz=9.7082 -0.6331 0.0 rpy=0 0 0
- joint windows_joint: origin (none) -> xyz=0 0 -0.2 rpy=0 0 0

Commit message: added decomposed meshes

File: iai_apartment/urdf/apartment.urdf (robot description, URDF)
Before this commit: robot apartment, 12 links, 11 joints
Links:
- link armchair: geometry collision mesh filename=package://iai_apartment/meshes/collision/armchair.obj; visual mesh filename=package://iai_apartment/meshes/visual/armchair.dae
- link sofa: geometry collision mesh filename=package://iai_apartment/meshes/collision/sofa.obj; visual mesh filename=package://iai_apartment/meshes/visual/sofa.dae
- link walls: geometry collision mesh filename=package://iai_apartment/meshes/collision/walls.obj; visual mesh filename=package://iai_apartment/meshes/visual/walls.dae
- link windows: geometry collision mesh filename=package://iai_apartment/meshes/collision/windows.obj; visual mesh filename=package://iai_apartment/meshes/visual/windows.dae
Joints:
- joint wardrobe_door_left_joint: axis 0 0 1 -> 0 0 -1; limit lower=-1.5708 upper=0.0 effort=1000.0 velocity=1.5708 -> lower=0.0 upper=1.5708 effort=1000.0 velocity=1.5708

Commit message: Collision screen for walls are added.

File: iai_apartment/urdf/apartment.urdf (robot description, URDF)
Before this commit: robot apartment, 12 links, 11 joints
Links:
- added link wall_coloksu_wall1; collision box size=3.05 18.95 0.003
- added link wall_coloksu_wall2; collision box size=3.05 4.808 0.003
- added link wall_coloksu_wall3; collision box size=3.05 18.95 0.003
- added link wall_coloksu_wall4; collision box size=3.05 4.808 0.003
- link walls: geometry visual mesh filename=package://iai_apartment/meshes/visual/walls.dae
Joints:
- added joint wall_coloksu_wall1_joint: type fixed, parent middle_of_the_room, child wall_coloksu_wall1, origin xyz=0.6 -1.615 1.53 rpy=0 0 -1.57
- added joint wall_coloksu_wall2_joint: type fixed, parent middle_of_the_room, child wall_coloksu_wall2, origin xyz=-8.855 0.782 1.53 rpy=0 0 3.14
- added joint wall_coloksu_wall3_joint: type fixed, parent middle_of_the_room, child wall_coloksu_wall3, origin xyz=0.6 3.180 1.53 rpy=0 0 1.57
- added joint wall_coloksu_wall4_joint: type fixed, parent middle_of_the_room, child wall_coloksu_wall4, origin xyz=10.069 0.782 1.53 rpy=0 0 0

Commit message: reverted urdf

File: iai_apartment/urdf/apartment.urdf (robot description, URDF)
Before this commit: robot apartment, 12 links, 11 joints
Links:
- link armchair: geometry collision mesh filename=package://iai_apartment/meshes/collision/armchair.stl; visual mesh filename=package://iai_apartment/meshes/visual/armchair.dae
- link sofa: geometry collision mesh filename=package://iai_apartment/meshes/collision/sofa.stl; visual mesh filename=package://iai_apartment/meshes/visual/sofa.dae
- link walls: geometry collision mesh filename=package://iai_apartment/meshes/collision/walls.stl; visual mesh filename=package://iai_apartment/meshes/visual/walls.dae
- link windows: geometry collision mesh filename=package://iai_apartment/meshes/collision/windows.stl; visual mesh filename=package://iai_apartment/meshes/visual/windows.dae
Joints:
- joint wardrobe_door_left_joint: axis 0 0 -1 -> 0 0 1; limit lower=0.0 upper=1.5708 effort=1000.0 velocity=1.5708 -> lower=-1.5708 upper=0.0 effort=1000.0 velocity=1.5708

Commit message: merged with master and run magic script

File: iai_apartment/urdf/apartment.urdf (robot description, URDF)
Before this commit: robot apartment, 16 links, 15 joints
Links:
- link armchair: geometry collision mesh filename=package://iai_apartment/meshes/collision/armchair.obj; visual mesh filename=package://iai_apartment/meshes/visual/armchair.dae
- link sofa: geometry collision mesh filename=package://iai_apartment/meshes/collision/sofa.obj; visual mesh filename=package://iai_apartment/meshes/visual/sofa.dae
- link windows: geometry collision mesh filename=package://iai_apartment/meshes/collision/windows.obj; visual mesh filename=package://iai_apartment/meshes/visual/windows.dae
Joints:
- joint wardrobe_door_left_joint: axis 0 0 1 -> 0 0 -1; limit lower=-1.5708 upper=0.0 effort=1000.0 velocity=1.5708 -> lower=0.0 upper=1.5708 effort=1000.0 velocity=1.5708

Commit message: [apartment] removed collision mesh of windows, there's a wall box instead now

File: iai_apartment/urdf/apartment.urdf (robot description, URDF)
Before this commit: robot apartment, 16 links, 15 joints
Links:
- link windows: geometry visual mesh filename=package://iai_apartment/meshes/visual/windows.dae

Commit message: Fix issues #103

File: iai_apartment/urdf/apartment.urdf (robot description, URDF)
Before this commit: robot apartment, 16 links, 15 joints
Links:
- added link wardrobe_door_left_handle; collision box size=0.014486 0.015082 0.13; collision box size=0.033556 0.015082 0.014587
- added link wardrobe_door_right_handle; collision box size=0.014486 0.015082 0.13; collision box size=0.033556 0.015082 0.014587
- link wardrobe_door_left: geometry collision box size=0.012967 0.495438 1.64844; visual mesh filename=package://iai_apartment/meshes/visual/wardrobe_door_left.dae
- link wardrobe_door_right: geometry collision box size=0.012967 0.495438 1.64844; visual mesh filename=package://iai_apartment/meshes/visual/wardrobe_door_right.d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
Joints:
- added joint wardrobe_door_left_handle_joint: type fixed, parent wardrobe_door_left, child wardrobe_door_left_handle, origin xyz=-0.032089 -0.460513 0.973703 rpy=0 0 0
- added joint wardrobe_door_right_handle_joint: type fixed, parent wardrobe_door_right, child wardrobe_door_right_handle, origin xyz=-0.032089 0.460513 0.973703 rpy=0 0 0
