Commit message: Fix issues #106

File: iai_apartment/urdf/apartment.urdf (robot description, URDF)
Before this commit: robot apartment, 18 links, 17 joints
Links:
- removed link middle_of_the_room
- added link cabinet1; collision mesh filename=package://iai_apartment/meshes/cabinet01/IAICabinet1W60.obj; visual mesh filename=package://iai_apartment/meshes/cabinet01/IAICabinet1W60.dae
- added link cabinet10; collision mesh filename=package://iai_apartment/meshes/cabinet10/IAIKitchenCabinet9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; visual mesh filename=package://iai_apartment/meshes/cabinet10/IAIKitchenCabinet9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
- added link cabinet10_drawer_bottom; collision mesh filename=package://iai_apartment/meshes/cabinet10/IAIKitchenDrawerW4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; visual mesh filename=package://iai_apartment/meshes/cabinet10/IAIKitchenDrawerW4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
- added link cabinet10_drawer_middle; collision mesh filename=package://iai_apartment/meshes/cabinet10/IAIKitchenDrawerW4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; visual mesh filename=package://iai_apartment/meshes/cabinet10/IAIKitchenDrawerW4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
- added link cabinet10_drawer_top; collision mesh filename=package://iai_apartment/meshes/cabinet10/IAIKitchenDrawerW4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; visual mesh filename=package://iai_apartment/meshes/cabinet10/IAIKitchenDrawerW4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
- added link cabinet11; collision mesh filename=package://iai_apartment/meshes/cabinet11/IAIKitchenCabinet1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; visual mesh filename=package://iai_apartment/meshes/cabinet11/IAIKitchenCabinet1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
- added link cabinet11_drawer_bottom; collision mesh filename=package://iai_apartment/meshes/cabinet11/IAIKitchenDrawerW9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; visual mesh filename=package://iai_apartment/meshes/cabinet11/IAIKitchenDrawerW9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
- added link cabinet11_drawer_middle; collision mesh filename=package://iai_apartment/meshes/cabinet11/IAIKitchenDrawerW9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; visual mesh filename=package://iai_apartment/meshes/cabinet11/IAIKitchenDrawerW9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
- added link cabinet11_drawer_top; collision mesh filename=package://iai_apartment/meshes/cabinet11/IAIKitchenDrawerW9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; visual mesh filename=package://iai_apartment/meshes/cabinet11/IAIKitchenDrawerW9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
- added link cabinet1_coloksu_level4; collision box size=0.534 0.568 0.003; visual box size=0.534 0.568 0.003
- added link cabinet1_coloksu_level5; collision box size=0.534 0.568 0.02; visual box size=0.534 0.568 0.02
- added link cabinet1_door_top_left; collision mesh filename=package://iai_apartment/meshes/cabinet01/IAIDoorW60H80.obj; visual mesh filename=package://iai_apartment/meshes/cabinet01/IAIDoorW60H80.dae
- added link cabinet1_drawer_bottom; collision mesh filename=package://iai_apartment/meshes/cabinet01/IAIDrawerW60H53.obj; visual mesh filename=package://iai_apartment/meshes/cabinet01/IAIDrawerW60H53.dae
- added link cabinet1_drawer_middle; collision mesh filename=package://iai_apartment/meshes/cabinet01/IAIDrawerW60H26.obj; visual mesh filename=package://iai_apartment/meshes/cabinet01/IAIDrawerW60H26.dae
- added link cabinet2; collision mesh filename=package://iai_apartment/meshes/cabinet02/IAICabinet2W40H57.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; visual mesh filename=package://iai_apartment/meshes/cabinet02/IAICabinet2W40H57.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
- added link cabinet2_door_left; collision mesh filename=package://iai_apartment/meshes/cabinet02/IAIDoorW40H212.obj; visual mesh filename=package://iai_apartment/meshes/cabinet02/IAIDoorW40H212.dae
- added link cabinet2_door_out_fancy
- added link cabinet2_drawer_big; collision mesh filename=package://iai_apartment/meshes/cabinet02/IAIDrawerW40H22.obj; visual mesh filename=package://iai_apartment/meshes/cabinet02/IAIDrawerW40H22.dae
- added link cabinet2_drawer_small; collision mesh filename=package://iai_apartment/meshes/cabinet02/IAIDrawerW40H10.obj; visual mesh filename=package://iai_apartment/meshes/cabinet02/IAIDrawerW40H10.dae
- added link cabinet3; collision mesh filename=package://iai_apartment/meshes/cabinet03/IAICabinet3W60.obj; visual mesh filename=package://iai_apartment/meshes/cabinet03/IAICabinet3W60.dae
- added link cabinet3_door_bottom_left; collision mesh filename=package://iai_apartment/meshes/cabinet03/IAIDoorW60H80.obj; visual mesh filename=package://iai_apartment/meshes/cabinet03/IAIDoorW60H80.dae
- added link cabinet3_door_bottom_out_fancy
- added link cabinet3_door_top_left; collision mesh filename=package://iai_apartment/meshes/cabinet03/IAIDoorW60H133.obj; visual mesh filename=package://iai_apartment/meshes/cabinet03/IAIDoorW60H133.dae
- added link cabinet3_door_top_out_fancy
- added link cabinet4; collision mesh filename=package://iai_apartment/meshes/cabinet04/IAIKitchenCabinet4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; visual mesh filename=package://iai_apartment/meshes/cabinet04/IAIKitchenCabinet4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
- added link cabinet4_door_bottom; collision mesh filename=package://iai_apartment/meshes/cabinet04/IAIDoor2W100H40.obj; visual mesh filename=package://iai_apartment/meshes/cabinet04/IAIDoor2W100H40.dae
- added link cabinet4_door_top; collision mesh filename=package://iai_apartment/meshes/cabinet04/IAIDoor1W100H40.obj; visual mesh filename=package://iai_apartment/meshes/cabinet04/IAIDoor1W100H40.dae
- added link cabinet5; collision mesh filename=package://iai_apartment/meshes/cabinet05/IAIKitchenCabinet5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; visual mesh filename=package://iai_apartment/meshes/cabinet05/IAIKitchenCabinet5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
- added link cabinet5_drawer_bottom; collision mesh filename=package://iai_apartment/meshes/cabinet05/IAIKitchenDrawerW6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; visual mesh filename=package://iai_apartment/meshes/cabinet05/IAIKitchenDrawerW6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
- added link cabinet5_drawer_middle; collision mesh filename=package://iai_apartment/meshes/cabinet05/IAIKitchenDrawerW6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; visual mesh filename=package://iai_apartment/meshes/cabinet05/IAIKitchenDrawerW6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
- added link cabinet5_drawer_top; collision mesh filename=package://iai_apartment/meshes/cabinet05/IAIKitchenDrawerW6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; visual mesh filename=package://iai_apartment/meshes/cabinet05/IAIKitchenDrawerW6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
- added link cabinet6; collision mesh filename=package://iai_apartment/meshes/cabinet06/IAIKitchenCabinet6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; visual mesh filename=package://iai_apartment/meshes/cabinet06/IAIKitchenCabinet6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
- added link cabinet6_drawer_bottom; collision mesh filename=package://iai_apartment/meshes/cabinet06/IAIKitchenDrawerW4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; visual mesh filename=package://iai_apartment/meshes/cabinet06/IAIKitchenDrawerW4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
- added link cabinet6_drawer_middle; collision mesh filename=package://iai_apartment/meshes/cabinet06/IAIKitchenDrawerW4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; visual mesh filename=package://iai_apartment/meshes/cabinet06/IAIKitchenDrawerW4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
- added link cabinet6_drawer_top; collision mesh filename=package://iai_apartment/meshes/cabinet06/IAIKitchenDrawerW4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; visual mesh filename=package://iai_apartment/meshes/cabinet06/IAIKitchenDrawerW4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
- added link cabinet7; collision mesh filename=package://iai_apartment/meshes/cabinet07/IAIKitchenCabinet7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; visual mesh filename=package://iai_apartment/meshes/cabinet07/IAIKitchenCabinet7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
- added link cabinet7_door_bottom_left; collision mesh filename=package://iai_apartment/meshes/cabinet07/IAIKitchenDoorW60H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; visual mesh filename=package://iai_apartment/meshes/cabinet07/IAIKitchenDoorW60H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
- added link cabinet8; collision mesh filename=package://iai_apartment/meshes/cabinet08/IAIKitchenCabinet8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; visual mesh filename=package://iai_apartment/meshes/cabinet08/IAIKitchenCabinet8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
- added link cabinet8_drawer_bottom; collision mesh filename=package://iai_apartment/meshes/cabinet08/IAIKitchenDrawerW6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; visual mesh filename=package://iai_apartment/meshes/cabinet08/IAIKitchenDrawerW6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
- added link cabinet8_drawer_middle; collision mesh filename=package://iai_apartment/meshes/cabinet08/IAIKitchenDrawerW5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; visual mesh filename=package://iai_apartment/meshes/cabinet08/IAIKitchenDrawerW5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
- added link cabinet9; collision mesh filename=package://iai_apartment/meshes/cabinet09/IAIKitchenCabinet9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; visual mesh filename=package://iai_apartment/meshes/cabinet09/IAIKitchenCabinet9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
- added link cabinet9_drawer_bottom; collision mesh filename=package://iai_apartment/meshes/cabinet09/IAIKitchenDrawerW6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; visual mesh filename=package://iai_apartment/meshes/cabinet09/IAIKitchenDrawerW6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
- added link cabinet9_drawer_middle; collision mesh filename=package://iai_apartment/meshes/cabinet09/IAIKitchenDrawerW6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; visual mesh filename=package://iai_apartment/meshes/cabinet09/IAIKitchenDrawerW6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
- added link cabinet9_drawer_top; collision mesh filename=package://iai_apartment/meshes/cabinet09/IAIKitchenDrawerW6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; visual mesh filename=package://iai_apartment/meshes/cabinet09/IAIKitchenDrawerW6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
- added link coffe_machine; collision box size=0.58 0.32 0.41; visual box size=0.58 0.33 0.41
- added link cooktop; collision mesh filename=package://iai_apartment/meshes/cooktop/IAIKitchenCookTop.obj; visual mesh filename=package://iai_apartment/meshes/cooktop/IAIKitchenCookTop.dae
- added link countertop; collision mesh filename=package://iai_apartment/meshes/countertop/IAIKitchenPartW10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; visual mesh filename=package://iai_apartment/meshes/countertop/IAIKitchenPartW10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
- added link dishwasher_drawer_middle; collision mesh filename=package://iai_apartment/meshes/cabinet07/dishwasher_drawer_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; visual mesh filename=package://iai_apartment/meshes/cabinet07/dishwasher_drawer_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
- added link furnitures_root
- added link handle_cab10_b; collision mesh filename=package://iai_apartment/meshes/handles/handle_horizontal.obj; visual mesh filename=package://iai_apartment/meshes/handles/handle_horizontal.dae
- added link handle_cab10_m; collision mesh filename=package://iai_apartment/meshes/handles/handle_horizontal.obj; visual mesh filename=package://iai_apartment/meshes/handles/handle_horizontal.dae
- added link handle_cab10_t; collision mesh filename=package://iai_apartment/meshes/handles/handle_horizontal.obj; visual mesh filename=package://iai_apartment/meshes/handles/handle_horizontal.dae
- added link handle_cab11_b; collision mesh filename=package://iai_apartment/meshes/handles/handle_horizontal.obj; visual mesh filename=package://iai_apartment/meshes/handles/handle_horizontal.dae
- added link handle_cab11_m; collision mesh filename=package://iai_apartment/meshes/handles/handle_horizontal.obj; visual mesh filename=package://iai_apartment/meshes/handles/handle_horizontal.dae
- added link handle_cab11_t; collision mesh filename=package://iai_apartment/meshes/handles/handle_horizontal.obj; visual mesh filename=package://iai_apartment/meshes/handles/handle_horizontal.dae
- added link handle_cab1_drawer_bottom; collision mesh filename=package://iai_apartment/meshes/handles/handle_horizontal.obj; visual mesh filename=package://iai_apartment/meshes/handles/handle_horizontal.dae
- added link handle_cab1_drawer_mid; collision mesh filename=package://iai_apartment/meshes/handles/handle_horizontal.obj; visual mesh filename=package://iai_apartment/meshes/handles/handle_horizontal.dae
- added link handle_cab1_top_door; collision mesh filename=package://iai_apartment/meshes/handles/handle_horizontal.obj; visual mesh filename=package://iai_apartment/meshes/handles/handle_horizontal.dae
- added link handle_cab2_door; collision mesh filename=package://iai_apartment/meshes/handles/handle_horizontal.obj; visual mesh filename=package://iai_apartment/meshes/handles/handle_horizontal.dae
- added link handle_cab3_door_bottom; collision mesh filename=package://iai_apartment/meshes/handles/handle_horizontal.obj; visual mesh filename=package://iai_apartment/meshes/handles/handle_horizontal.dae
- added link handle_cab3_door_top; collision mesh filename=package://iai_apartment/meshes/handles/handle_horizontal.obj; visual mesh filename=package://iai_apartment/meshes/handles/handle_horizontal.dae
- added link handle_cab4_door_bottom; collision mesh filename=package://iai_apartment/meshes/handles/handle_horizontal.obj; visual mesh filename=package://iai_apartment/meshes/handles/handle_horizontal.dae
- added link handle_cab5_b; collision mesh filename=package://iai_apartment/meshes/handles/handle_horizontal.obj; visual mesh filename=package://iai_apartment/meshes/handles/handle_horizontal.dae
- added link handle_cab5_m; collision mesh filename=package://iai_apartment/meshes/handles/handle_horizontal.obj; visual mesh filename=package://iai_apartment/meshes/handles/handle_horizontal.dae
- added link handle_cab5_t; collision mesh filename=package://iai_apartment/meshes/handles/handle_horizontal.obj; visual mesh filename=package://iai_apartment/meshes/handles/handle_horizontal.dae
- added link handle_cab6_b; collision mesh filename=package://iai_apartment/meshes/handles/handle_horizontal.obj; visual mesh filename=package://iai_apartment/meshes/handles/handle_horizontal.dae
- added link handle_cab6_m; collision mesh filename=package://iai_apartment/meshes/handles/handle_horizontal.obj; visual mesh filename=package://iai_apartment/meshes/handles/handle_horizontal.dae
- added link handle_cab6_t; collision mesh filename=package://iai_apartment/meshes/handles/handle_horizontal.obj; visual mesh filename=package://iai_apartment/meshes/handles/handle_horizontal.dae
- added link handle_cab7; collision mesh filename=package://iai_apartment/meshes/handles/handle_horizontal.obj; visual mesh filename=package://iai_apartment/meshes/handles/handle_horizontal.dae
- added link handle_cab7_middle; collision box size=0.015 0.325 0.021; visual box size=0.015 0.325 0.021
- added link handle_cab8; collision mesh filename=package://iai_apartment/meshes/handles/handle_horizontal.obj; visual mesh filename=package://iai_apartment/meshes/handles/handle_horizontal.dae
- added link handle_cab9_b; collision mesh filename=package://iai_apartment/meshes/handles/handle_horizontal.obj; visual mesh filename=package://iai_apartment/meshes/handles/handle_horizontal.dae
- added link handle_cab9_m; collision mesh filename=package://iai_apartment/meshes/handles/handle_horizontal.obj; visual mesh filename=package://iai_apartment/meshes/handles/handle_horizontal.dae
- added link handle_cab9_t; collision mesh filename=package://iai_apartment/meshes/handles/handle_horizontal.obj; visual mesh filename=package://iai_apartment/meshes/handles/handle_horizontal.dae
- added link hotplate1
- added link hotplate2
- added link hotplate3
- added link hotplate4
- added link island_back; collision mesh filename=package://iai_apartment/meshes/IAIKitchenPartW314H90/IAIKit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; visual mesh filename=package://iai_apartment/meshes/IAIKitchenPartW314H90/IAIKit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
- added link island_countertop; collision mesh filename=package://iai_apartment/meshes/island/IAIKitchenIslandAreaT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; visual mesh filename=package://iai_apartment/meshes/island/IAIKitchenIslandAreaT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
- added link island_waterfall_left; collision mesh filename=package://iai_apartment/meshes/IAIKitchenVisiblePartIslandU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; visual mesh filename=package://iai_apartment/meshes/IAIKitchenVisiblePartIslandU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
- added link island_waterfall_right; collision mesh filename=package://iai_apartment/meshes/IAIKitchenVisiblePartIslandU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; visual mesh filename=package://iai_apartment/meshes/IAIKitchenVisiblePartIslandU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
- added link kitchen_root
- added link oven; collision box size=0.58 0.58 0.59; visual mesh filename=package://iai_apartment/meshes/cabinet01/oven.dae
- added link side_A
- added link side_A_left; collision mesh filename=package://iai_apartment/meshes/IAIKitchenPartW58H223/IAIKit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; visual mesh filename=package://iai_apartment/meshes/IAIKitchenPartW58H223/IAIKit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
- added link side_A_rb; collision mesh filename=package://iai_apartment/meshes/IAIKitchenVisiblePartUnderSi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; visual mesh filename=package://iai_apartment/meshes/IAIKitchenVisiblePartUnderSi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
- added link side_A_rt; collision mesh filename=package://iai_apartment/meshes/IAIKitchenVisiblePartUppersi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; visual mesh filename=package://iai_apartment/meshes/IAIKitchenVisiblePartUppersi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
- added link side_B
- added link sink; collision mesh filename=package://iai_apartment/meshes/sink/IAIKitchenSink.obj; visual mesh filename=package://iai_apartment/meshes/sink/IAIKitchenSink.dae
- added link tap_body; collision mesh filename=package://iai_apartment/meshes/tap/IAIKitchenWaterTapBody.o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; visual mesh filename=package://iai_apartment/meshes/tap/IAIKitchenWaterTapBody.d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
- added link tap_handle; collision mesh filename=package://iai_apartment/meshes/tap/IAIKitchenWaterTapHandle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; visual mesh filename=package://iai_apartment/meshes/tap/IAIKitchenWaterTapHandle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
- added link tap_handle_open
- added link useless_underbar_a; collision mesh filename=package://iai_apartment/meshes/floor_socket_side_a/IAIKitch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; visual mesh filename=package://iai_apartment/meshes/floor_socket_side_a/IAIKitch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
- added link useless_underbar_b; collision mesh filename=package://iai_apartment/meshes/floor_socket_side_b/IAIKitch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; visual mesh filename=package://iai_apartment/meshes/floor_socket_side_b/IAIKitch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
Joints:
- removed joint middle_of_the_room_joint
- added joint cabinet10_drawer_bottom_joint: type prismatic, parent cabinet10, child cabinet10_drawer_bottom, origin xyz=0.03 0.0 -0.279 rpy=0 0 3.14, axis -1 0 0, limit lower=0.0 upper=0.45 effort=1000.0 velocity=0.5
- added joint cabinet10_drawer_middle_joint: type prismatic, parent cabinet10, child cabinet10_drawer_middle, origin xyz=0.031 0.0 0.104 rpy=0 0 3.14, axis -1 0 0, limit lower=0.0 upper=0.45 effort=1000.0 velocity=0.5
- added joint cabinet10_drawer_top_joint: type prismatic, parent cabinet10, child cabinet10_drawer_top, origin xyz=0.033 0.0 0.326 rpy=0 0 3.14, axis -1 0 0, limit lower=0.0 upper=0.45 effort=1000.0 velocity=0.5
- added joint cabinet10_joint: type fixed, parent side_B, child cabinet10, origin xyz=0.333 2.204 0.394
- added joint cabinet11_drawer_bottom_joint: type prismatic, parent cabinet11, child cabinet11_drawer_bottom, origin xyz=0.045 0.0 -0.286 rpy=0 0 3.14, axis -1 0 0, limit lower=0.0 upper=0.45 effort=1000.0 velocity=0.5
- added joint cabinet11_drawer_middle_joint: type prismatic, parent cabinet11, child cabinet11_drawer_middle, origin xyz=0.027 0.0 0.106 rpy=0 0 3.14, axis -1 0 0, limit lower=0.0 upper=0.45 effort=1000.0 velocity=0.5
- added joint cabinet11_drawer_top_joint: type prismatic, parent cabinet11, child cabinet11_drawer_top, origin xyz=0.03 0.0 0.326 rpy=0 0 3.14, axis -1 0 0, limit lower=0.0 upper=0.45 effort=1000.0 velocity=0.5
- added joint cabinet11_joint: type fixed, parent side_B, child cabinet11, origin xyz=0.333 2.855 0.394
- added joint cabinet1_coloksu_level4_joint: type fixed, parent cabinet1, child cabinet1_coloksu_level4, origin xyz=-0.172 0.005 0.281
- added joint cabinet1_coloksu_level5_joint: type fixed, parent cabinet1, child cabinet1_coloksu_level5, origin xyz=-0.172 0.005 0.56
- added joint cabinet1_door_top_left_joint: type revolute, parent cabinet1, child cabinet1_door_top_left, origin xyz=0.103 -0.3 0.32 rpy=0 0 3.14, axis 0 0 -1, limit lower=0.0 upper=1.5708 effort=1000.0 velocity=1.5708
- added joint cabinet1_drawer_bottom_joint: type prismatic, parent cabinet1, child cabinet1_drawer_bottom, origin xyz=-0.094 0.0 -0.95 rpy=0 0 3.14, axis -1 0 0, limit lower=0.0 upper=0.45 effort=1000.0 velocity=0.5
- added joint cabinet1_drawer_middle_joint: type prismatic, parent cabinet1, child cabinet1_drawer_middle, origin xyz=-0.117 0.0 -0.43 rpy=0 0 3.14, axis -1 0 0, limit lower=0.0 upper=0.45 effort=1000.0 velocity=0.5
- added joint cabinet1_joint: type fixed, parent side_A, child cabinet1, origin xyz=0.01 0.01 1.02
- added joint cabinet2_door_left_joint: type revolute, parent cabinet2_door_out_fancy, child cabinet2_door_left, axis 0 0 -1, limit lower=0.0 upper=1.5708 effort=1000.0 velocity=1.5708
- added joint cabinet2_door_out_joint: type prismatic, parent cabinet2, child cabinet2_door_out_fancy, origin xyz=0.277 -0.19 0.0 rpy=0 0 3.14, axis -1 0 0, limit lower=0.0 upper=0.02 effort=1.0 velocity=1.5708, mimic joint=cabinet2_door_left_joint multiplier=0.01
- added joint cabinet2_drawer_big_joint: type prismatic, parent cabinet2, child cabinet2_drawer_big, origin xyz=0.04 0.0 -0.12 rpy=0 0 3.14, axis -1 0 0, limit lower=0.0 upper=0.45 effort=500.0 velocity=0.5
- added joint cabinet2_drawer_small_joint: type prismatic, parent cabinet2, child cabinet2_drawer_small, origin xyz=-0.01 0.0 0.17 rpy=0 0 3.14, axis -1 0 0, limit lower=0.0 upper=0.45 effort=500.0 velocity=0.5
- added joint cabinet2_joint: type fixed, parent side_A, child cabinet2, origin xyz=-0.163 0.51 0.975
- added joint cabinet3_door_bottom_left_joint: type revolute, parent cabinet3_door_bottom_out_fancy, child cabinet3_door_bottom_left, axis 0 0 -1, limit lower=0.0 upper=1.5708 effort=1000.0 velocity=1.5708
- added joint cabinet3_door_bottom_out_joint: type prismatic, parent cabinet3, child cabinet3_door_bottom_out_fancy, origin xyz=0.39 -0.3 -0.5 rpy=0 0 3.14, axis -1 0 0, limit lower=0.0 upper=0.02 effort=1.0 velocity=1.5708, mimic joint=cabinet3_door_bottom_left_joint multiplier=0.01
- added joint cabinet3_door_top_left_joint: type revolute, parent cabinet3_door_top_out_fancy, child cabinet3_door_top_left, axis 0 0 -1, limit lower=0.0 upper=1.5708 effort=1000.0 velocity=1.5708
- added joint cabinet3_door_top_out_joint: type prismatic, parent cabinet3, child cabinet3_door_top_out_fancy, origin xyz=0.39 -0.3 0.5 rpy=0 0 3.14, axis -1 0 0, limit lower=0.0 upper=0.02 effort=1.0 velocity=1.5708, mimic joint=cabinet3_door_top_left_joint multiplier=0.01
- added joint cabinet3_joint: type fixed, parent side_A, child cabinet3, origin xyz=-0.273 1.022 1.07
- added joint cabinet4_door_bottom_bottom_joint: type revolute, parent cabinet4_door_top, child cabinet4_door_bottom, origin xyz=0.0 0.0 -0.4 rpy=0 0 0, axis 0 -1 0, limit lower=0.0 upper=1.5708 effort=1000.0 velocity=1.5708, mimic joint=cabinet4_door_top_top_joint multiplier=1.2
- added joint cabinet4_door_top_top_joint: type revolute, parent cabinet4, child cabinet4_door_top, origin xyz=0.07 0 0.42 rpy=0 0 3.14, axis 0 1 0, limit lower=0 upper=2.0 effort=1000.0 velocity=1.5708
- added joint cabinet4_joint: type fixed, parent side_A, child cabinet4, origin xyz=-0.175 1.825 1.72
- added joint cabinet5_drawer_bottom_joint: type prismatic, parent cabinet5, child cabinet5_drawer_bottom, origin xyz=0.037 0.0 -0.28 rpy=0 0 3.14, axis -1 0 0, limit lower=0.0 upper=0.45 effort=1000.0 velocity=0.5
- added joint cabinet5_drawer_middle_joint: type prismatic, parent cabinet5, child cabinet5_drawer_middle, origin xyz=0.027 0.0 0.107 rpy=0 0 3.14, axis -1 0 0, limit lower=0.0 upper=0.45 effort=1000.0 velocity=0.5
- added joint cabinet5_drawer_top_joint: type prismatic, parent cabinet5, child cabinet5_drawer_top, origin xyz=0.03 0.0 0.327 rpy=0 0 3.14, axis -1 0 0, limit lower=0.0 upper=0.45 effort=1000.0 velocity=0.5
- added joint cabinet5_joint: type fixed, parent side_A, child cabinet5, origin xyz=-0.121 1.625 0.4
- added joint cabinet6_drawer_bottom_joint: type prismatic, parent cabinet6, child cabinet6_drawer_bottom, origin xyz=0.047 0.0 -0.28 rpy=0 0 3.14, axis -1 0 0, limit lower=0.0 upper=0.45 effort=1000.0 velocity=0.5
- added joint cabinet6_drawer_middle_joint: type prismatic, parent cabinet6, child cabinet6_drawer_middle, origin xyz=0.03 0.0 0.105 rpy=0 0 3.14, axis -1 0 0, limit lower=0.0 upper=0.45 effort=1000.0 velocity=0.5
- added joint cabinet6_drawer_top_joint: type prismatic, parent cabinet6, child cabinet6_drawer_top, origin xyz=0.033 -0.0125 0.328 rpy=0 0 3.14, axis -1 0 0, limit lower=0.0 upper=0.45 effort=1000.0 velocity=0.5
- added joint cabinet6_joint: type fixed, parent side_A, child cabinet6, origin xyz=-0.121 2.127 0.4
- added joint cabinet7_door_bottom_left_joint: type revolute, parent cabinet7, child cabinet7_door_bottom_left, origin xyz=0.372 0 -0.45 rpy=0 0 3.14, axis 0 -1 0, limit lower=0.0 upper=1.5708 effort=1000.0 velocity=1.5708
- added joint cabinet7_joint: type fixed, parent side_B, child cabinet7, origin xyz=0.2 0.501 0.47
- added joint cabinet8_drawer_bottom_joint: type prismatic, parent cabinet8, child cabinet8_drawer_bottom, origin xyz=0.114 0.0 0.105 rpy=0 0 3.14, axis -1 0 0, limit lower=0.0 upper=0.45 effort=1000.0 velocity=0.5
- added joint cabinet8_drawer_middle_joint: type prismatic, parent cabinet8, child cabinet8_drawer_middle, origin xyz=0.05 0.0 0.48 rpy=0 0 3.14, axis -1 0 0, limit lower=0.0 upper=0.40 effort=1000.0 velocity=0.5
- added joint cabinet8_joint: type fixed, parent side_B, child cabinet8, origin xyz=0.256 1.102 0.006
- added joint cabinet9_drawer_bottom_joint: type prismatic, parent cabinet9, child cabinet9_drawer_bottom, origin xyz=0.036 0.0 -0.281 rpy=0 0 3.14, axis -1 0 0, limit lower=0.0 upper=0.45 effort=1000.0 velocity=0.5
- added joint cabinet9_drawer_middle_joint: type prismatic, parent cabinet9, child cabinet9_drawer_middle, origin xyz=0.027 0.0 0.106 rpy=0 0 3.14, axis -1 0 0, limit lower=0.0 upper=0.45 effort=1000.0 velocity=0.5
- added joint cabinet9_drawer_top_joint: type prismatic, parent cabinet9, child cabinet9_drawer_top, origin xyz=0.03 0.0 0.327 rpy=0 0 3.14, axis -1 0 0, limit lower=0.0 upper=0.45 effort=1000.0 velocity=0.5
- added joint cabinet9_joint: type fixed, parent side_B, child cabinet9, origin xyz=0.333 1.703 0.394
- added joint coffe_machine_joint: type fixed, parent countertop, child coffe_machine, origin xyz=0 0.3 0.2
- added joint cooktop_joint: type fixed, parent island_countertop, child cooktop, origin xyz=0.130 1.074 0.023
- added joint countertop_joint: type fixed, parent cabinet5, child countertop, origin xyz=-0.027 0.21 0.423
- added joint dishwasher_drawer_middle_joint: type prismatic, parent cabinet7, child dishwasher_drawer_middle, origin xyz=-0.065 0.03 0.08 rpy=0 0 3.14, axis -1 0  0, limit lower=0.0 upper=0.45 effort=1000.0 velocity=0.5
- added joint frame_A_joint: type fixed, parent kitchen_root, child side_A, origin xyz=0.49 0.696 0.080
- added joint frame_B_joint: type fixed, parent kitchen_root, child side_B, origin xyz=2.91 3.7 0.11 rpy=0 0 3.14
- added joint furnitures_base: type fixed, parent apartment_root, child furnitures_root, origin xyz=8.85 1.75 0.0
- added joint handle_cab10_bott_joint: type fixed, parent cabinet10_drawer_bottom, child handle_cab10_b, origin xyz=-0.245 0 0.245 rpy=1.57 0 0
- added joint handle_cab10_mid_joint: type fixed, parent cabinet10_drawer_middle, child handle_cab10_m, origin xyz=-0.245 0 0.13 rpy=1.57 0 0
- added joint handle_cab10_top_joint: type fixed, parent cabinet10_drawer_top, child handle_cab10_t, origin xyz=-0.243 0 0.05 rpy=1.57 0 0
- added joint handle_cab11_bott_joint: type fixed, parent cabinet11_drawer_bottom, child handle_cab11_b, origin xyz=-0.228 0 0.245 rpy=1.57 0 0
- added joint handle_cab11_mid_joint: type fixed, parent cabinet11_drawer_middle, child handle_cab11_m, origin xyz=-0.245 0 0.13 rpy=1.57 0 0
- added joint handle_cab11_top_joint: type fixed, parent cabinet11_drawer_top, child handle_cab11_t, origin xyz=-0.243 0 0.05 rpy=1.57 0 0
- added joint handle_cab1_drawer_bottom_joint: type fixed, parent cabinet1_drawer_bottom, child handle_cab1_drawer_bottom, origin xyz=-0.237 0.0 0.35 rpy=1.57 0 0
- added joint handle_cab1_drawer_mid_joint: type fixed, parent cabinet1_drawer_middle, child handle_cab1_drawer_mid, origin xyz=-0.26 0.0 0.11 rpy=1.57 0 0
- added joint handle_cab1_top_door_joint: type fixed, parent cabinet1_door_top_left, child handle_cab1_top_door, origin xyz=-0.055 -0.5 0.0 rpy=1.57 0 0
- added joint handle_cab2_drawer_bottom_joint: type fixed, parent cabinet2_door_left, child handle_cab2_door, origin xyz=-0.040 -0.29 0.05 rpy=1.57 0 0
- added joint handle_cab3_door_bottom_joint: type fixed, parent cabinet3_door_bottom_left, child handle_cab3_door_bottom, origin xyz=-0.036 -0.45 0.1 rpy=1.57 0 0
- added joint handle_cab3_door_top_joint: type fixed, parent cabinet3_door_top_left, child handle_cab3_door_top, origin xyz=-0.036 -0.45 -0.65 rpy=1.57 0 0
- added joint handle_cab4_door_bottom_joint: type fixed, parent cabinet4_door_bottom, child handle_cab4_door_bottom, origin xyz=-0.055 0 -0.35 rpy=1.57 0 0
- added joint handle_cab5_bott_joint: type fixed, parent cabinet5_drawer_bottom, child handle_cab5_b, origin xyz=-0.235 0 0.245 rpy=1.57 0 0
- added joint handle_cab5_mid_joint: type fixed, parent cabinet5_drawer_middle, child handle_cab5_m, origin xyz=-0.245 0 0.13 rpy=1.57 0 0
- added joint handle_cab5_top_joint: type fixed, parent cabinet5_drawer_top, child handle_cab5_t, origin xyz=-0.245 0 0.05 rpy=1.57 0 0
- added joint handle_cab6_bott_joint: type fixed, parent cabinet6_drawer_bottom, child handle_cab6_b, origin xyz=-0.227 0 0.245 rpy=1.57 0 0
- added joint handle_cab6_mid_joint: type fixed, parent cabinet6_drawer_middle, child handle_cab6_m, origin xyz=-0.245 0 0.13 rpy=1.57 0 0
- added joint handle_cab6_top_joint: type fixed, parent cabinet6_drawer_top, child handle_cab6_t, origin xyz=-0.238 0 0.05 rpy=1.57 0 0
- added joint handle_cab7_drawer_middle_joint: type fixed, parent dishwasher_drawer_middle, child handle_cab7_middle, origin xyz=-0.315 0 0.068 rpy=1.57 0 0
- added joint handle_cab7_top_joint: type fixed, parent cabinet7_door_bottom_left, child handle_cab7, origin xyz=-0.06 0 0.74 rpy=1.57 0 0
- added joint handle_cab8_top_joint: type fixed, parent cabinet8_drawer_bottom, child handle_cab8, origin xyz=-0.238 0 0.65 rpy=1.57 0 0
- added joint handle_cab9_bott_joint: type fixed, parent cabinet9_drawer_bottom, child handle_cab9_b, origin xyz=-0.24 0 0.245 rpy=1.57 0 0
- added joint handle_cab9_mid_joint: type fixed, parent cabinet9_drawer_middle, child handle_cab9_m, origin xyz=-0.245 0 0.13 rpy=1.57 0 0
- added joint handle_cab9_top_joint: type fixed, parent cabinet9_drawer_top, child handle_cab9_t, origin xyz=-0.245 0 0.05 rpy=1.57 0 0
- added joint hotplate1_joint: type fixed, parent cooktop, child hotplate1, origin xyz=0.1069 -0.16199 0.005
- added joint hotplate2_joint: type fixed, parent cooktop, child hotplate2, origin xyz=0.066902 0.13801 0.0055
- added joint hotplate3_joint: type fixed, parent cooktop, child hotplate3, origin xyz=-0.155778 0.138013 0.0055
- added joint hotplate4_joint: type fixed, parent cooktop, child hotplate4, origin xyz=-0.115778 -0.161987 0.005333
- added joint island_back_joint: type fixed, parent side_B, child island_back, origin xyz=-0.026 1.754 0.353 rpy=0 1.57 0
- added joint island_countertop_joint: type fixed, parent side_B, child island_countertop, origin xyz=0.13 1.786 0.807
- added joint island_waterfall_left_joint: type fixed, parent side_B, child island_waterfall_left, origin xyz=0.285 0.191 0.354 rpy=1.57 0 1.57
- added joint island_waterfall_right_joint: type fixed, parent side_B, child island_waterfall_right, origin xyz=0.285 3.315 0.354 rpy=1.57 0 1.57
- added joint kitchen_base: type fixed, parent apartment_root, child kitchen_root, origin xyz=-0.03 0.75 0.005
- added joint oven_joint: type fixed, parent cabinet1, child oven, origin xyz=-0.175 0.0 -0.025 rpy=0 0 0
- added joint side_A_left_joint: type fixed, parent side_A, child side_A_left, origin xyz=-0.16 -0.296 1.030 rpy=0 0 1.57
- added joint side_A_right_bott_joint: type fixed, parent side_A, child side_A_rb, origin xyz=-0.159 2.338 0.361 rpy=1.57 0 1.57
- added joint side_A_right_top_joint: type fixed, parent side_A, child side_A_rt, origin xyz=-0.262 2.336 1.74 rpy=0 0 1.57
- added joint sink_joint: type fixed, parent island_countertop, child sink, origin xyz=0.198 -0.698 -0.038
- added joint socket_a_joint: type fixed, parent side_A, child useless_underbar_a, origin xyz=0.095 1.02 -0.03
- added joint socket_b_joint: type fixed, parent side_B, child useless_underbar_b, origin xyz=0.552 1.755 -0.045
- added joint tap_handle_hot_cold_joint: type revolute, parent tap_handle_open, child tap_handle, origin rpy=0 0.5 0, axis 1 0 0, limit lower=-0.5 upper=0 effort=1000.0 velocity=1.5708
- added joint tap_handle_open_joint: type revolute, parent tap_body, child tap_handle_open, origin xyz=0.001233 0.038489 -0.055395, axis 0 1 0, limit lower=-1.5708 upper=1.5708 effort=1000.0 velocity=1.5708
- added joint tap_joint: type revolute, parent sink, child tap_body, origin xyz=-0.228 -0.003 0.164, axis 0 0 1, limit lower=-1.5708 upper=1.5708 effort=1000.0 velocity=1.5708
- joint armchair_joint: parent middle_of_the_room -> furnitures_root
- joint bedside_table_joint: parent middle_of_the_room -> furnitures_root
- joint coffee_table_joint: parent middle_of_the_room -> furnitures_root
- joint sofa_joint: parent middle_of_the_room -> furnitures_root
- joint wall_coloksu_wall1_joint: parent middle_of_the_room -> furnitures_root
- joint wall_coloksu_wall2_joint: parent middle_of_the_room -> furnitures_root
- joint wall_coloksu_wall3_joint: parent middle_of_the_room -> furnitures_root
- joint wall_coloksu_wall4_joint: parent middle_of_the_room -> furnitures_root
- joint walls_joint: parent middle_of_the_room -> furnitures_root
- joint wardrobe_joint: parent middle_of_the_room -> furnitures_root
- joint windows_joint: parent middle_of_the_room -> furnitures_root
