Commit message: Revert to commit a55768516bbfc2139f62eaff3a703e43b11a6f6d

File: iai_apartment/urdf/apartment.urdf (robot description, URDF)
Before this commit: robot apartment, 112 links, 111 joints
Links:
- removed link cabinet1
- removed link cabinet10
- removed link cabinet10_drawer_bottom
- removed link cabinet10_drawer_middle
- removed link cabinet10_drawer_top
- removed link cabinet11
- removed link cabinet11_drawer_bottom
- removed link cabinet11_drawer_middle
- removed link cabinet11_drawer_top
- removed link cabinet1_coloksu_level4
- removed link cabinet1_coloksu_level5
- removed link cabinet1_door_top_left
- removed link cabinet1_drawer_bottom
- removed link cabinet1_drawer_middle
- removed link cabinet2
- removed link cabinet2_door_left
- removed link cabinet2_door_out_fancy
- removed link cabinet2_drawer_big
- removed link cabinet2_drawer_small
- removed link cabinet3
- removed link cabinet3_door_bottom_left
- removed link cabinet3_door_bottom_out_fancy
- removed link cabinet3_door_top_left
- removed link cabinet3_door_top_out_fancy
- removed link cabinet4
- removed link cabinet4_door_bottom
- removed link cabinet4_door_top
- removed link cabinet5
- removed link cabinet5_drawer_bottom
- removed link cabinet5_drawer_middle
- removed link cabinet5_drawer_top
- removed link cabinet6
- removed link cabinet6_drawer_bottom
- removed link cabinet6_drawer_middle
- removed link cabinet6_drawer_top
- removed link cabinet7
- removed link cabinet7_door_bottom_left
- removed link cabinet8
- removed link cabinet8_drawer_bottom
- removed link cabinet8_drawer_middle
- removed link cabinet9
- removed link cabinet9_drawer_bottom
- removed link cabinet9_drawer_middle
- removed link cabinet9_drawer_top
- removed link coffe_machine
- removed link cooktop
- removed link countertop
- removed link dishwasher_drawer_middle
- removed link furnitures_root
- removed link handle_cab10_b
- removed link handle_cab10_m
- removed link handle_cab10_t
- removed link handle_cab11_b
- removed link handle_cab11_m
- removed link handle_cab11_t
- removed link handle_cab1_drawer_bottom
- removed link handle_cab1_drawer_mid
- removed link handle_cab1_top_door
- removed link handle_cab2_door
- removed link handle_cab3_door_bottom
- removed link handle_cab3_door_top
- removed link handle_cab4_door_bottom
- removed link handle_cab5_b
- removed link handle_cab5_m
- removed link handle_cab5_t
- removed link handle_cab6_b
- removed link handle_cab6_m
- removed link handle_cab6_t
- removed link handle_cab7
- removed link handle_cab7_middle
- removed link handle_cab8
- removed link handle_cab9_b
- removed link handle_cab9_m
- removed link handle_cab9_t
- removed link hotplate1
- removed link hotplate2
- removed link hotplate3
- removed link hotplate4
- removed link island_back
- removed link island_countertop
- removed link island_waterfall_left
- removed link island_waterfall_right
- removed link kitchen_root
- removed link oven
- removed link side_A
- removed link side_A_left
- removed link side_A_rb
- removed link side_A_rt
- removed link side_B
- removed link sink
- removed link tap_body
- removed link tap_handle
- removed link tap_handle_open
- removed link useless_underbar_a
- removed link useless_underbar_b
- added link middle_of_the_room
Joints:
- removed joint cabinet10_drawer_bottom_joint
- removed joint cabinet10_drawer_middle_joint
- removed joint cabinet10_drawer_top_joint
- removed joint cabinet10_joint
- removed joint cabinet11_drawer_bottom_joint
- removed joint cabinet11_drawer_middle_joint
- removed joint cabinet11_drawer_top_joint
- removed joint cabinet11_joint
- removed joint cabinet1_coloksu_level4_joint
- removed joint cabinet1_coloksu_level5_joint
- removed joint cabinet1_door_top_left_joint
- removed joint cabinet1_drawer_bottom_joint
- removed joint cabinet1_drawer_middle_joint
- removed joint cabinet1_joint
- removed joint cabinet2_door_left_joint
- removed joint cabinet2_door_out_joint
- removed joint cabinet2_drawer_big_joint
- removed joint cabinet2_drawer_small_joint
- removed joint cabinet2_joint
- removed joint cabinet3_door_bottom_left_joint
- removed joint cabinet3_door_bottom_out_joint
- removed joint cabinet3_door_top_left_joint
- removed joint cabinet3_door_top_out_joint
- removed joint cabinet3_joint
- removed joint cabinet4_door_bottom_bottom_joint
- removed joint cabinet4_door_top_top_joint
- removed joint cabinet4_joint
- removed joint cabinet5_drawer_bottom_joint
- removed joint cabinet5_drawer_middle_joint
- removed joint cabinet5_drawer_top_joint
- removed joint cabinet5_joint
- removed joint cabinet6_drawer_bottom_joint
- removed joint cabinet6_drawer_middle_joint
- removed joint cabinet6_drawer_top_joint
- removed joint cabinet6_joint
- removed joint cabinet7_door_bottom_left_joint
- removed joint cabinet7_joint
- removed joint cabinet8_drawer_bottom_joint
- removed joint cabinet8_drawer_middle_joint
- removed joint cabinet8_joint
- removed joint cabinet9_drawer_bottom_joint
- removed joint cabinet9_drawer_middle_joint
- removed joint cabinet9_drawer_top_joint
- removed joint cabinet9_joint
- removed joint coffe_machine_joint
- removed joint cooktop_joint
- removed joint countertop_joint
- removed joint dishwasher_drawer_middle_joint
- removed joint frame_A_joint
- removed joint frame_B_joint
- removed joint furnitures_base
- removed joint handle_cab10_bott_joint
- removed joint handle_cab10_mid_joint
- removed joint handle_cab10_top_joint
- removed joint handle_cab11_bott_joint
- removed joint handle_cab11_mid_joint
- removed joint handle_cab11_top_joint
- removed joint handle_cab1_drawer_bottom_joint
- removed joint handle_cab1_drawer_mid_joint
- removed joint handle_cab1_top_door_joint
- removed joint handle_cab2_drawer_bottom_joint
- removed joint handle_cab3_door_bottom_joint
- removed joint handle_cab3_door_top_joint
- removed joint handle_cab4_door_bottom_joint
- removed joint handle_cab5_bott_joint
- removed joint handle_cab5_mid_joint
- removed joint handle_cab5_top_joint
- removed joint handle_cab6_bott_joint
- removed joint handle_cab6_mid_joint
- removed joint handle_cab6_top_joint
- removed joint handle_cab7_drawer_middle_joint
- removed joint handle_cab7_top_joint
- removed joint handle_cab8_top_joint
- removed joint handle_cab9_bott_joint
- removed joint handle_cab9_mid_joint
- removed joint handle_cab9_top_joint
- removed joint hotplate1_joint
- removed joint hotplate2_joint
- removed joint hotplate3_joint
- removed joint hotplate4_joint
- removed joint island_back_joint
- removed joint island_countertop_joint
- removed joint island_waterfall_left_joint
- removed joint island_waterfall_right_joint
- removed joint kitchen_base
- removed joint oven_joint
- removed joint side_A_left_joint
- removed joint side_A_right_bott_joint
- removed joint side_A_right_top_joint
- removed joint sink_joint
- removed joint socket_a_joint
- removed joint socket_b_joint
- removed joint tap_handle_hot_cold_joint
- removed joint tap_handle_open_joint
- removed joint tap_joint
- added joint middle_of_the_room_joint: type fixed, parent apartment_root, child middle_of_the_room, origin xyz=8.85 1.75 0.0 rpy=0 0 0
- joint armchair_joint: parent furnitures_root -> middle_of_the_room
- joint bedside_table_joint: parent furnitures_root -> middle_of_the_room
- joint coffee_table_joint: parent furnitures_root -> middle_of_the_room
- joint sofa_joint: parent furnitures_root -> middle_of_the_room
- joint wall_coloksu_wall1_joint: parent furnitures_root -> middle_of_the_room
- joint wall_coloksu_wall2_joint: parent furnitures_root -> middle_of_the_room
- joint wall_coloksu_wall3_joint: parent furnitures_root -> middle_of_the_room
- joint wall_coloksu_wall4_joint: parent furnitures_root -> middle_of_the_room
- joint walls_joint: parent furnitures_root -> middle_of_the_room
- joint wardrobe_joint: parent furnitures_root -> middle_of_the_room
- joint windows_joint: parent furnitures_root -> middle_of_the_room

Commit message: Add new kitchen cabinet to URDF model
Copied the files and XACRO code from cabinet 3
and renamed everything to cabinet 12. Also moved
the cabinet to the left of the kitchen.

File: iai_apartment/urdf/apartment.urdf (robot description, URDF)
Before this commit: robot apartment, 112 links, 111 joints
Links:
- added link cabinet12; collision mesh filename=package://iai_apartment/meshes/cabinet12/IAICabinet12W60.obj; visual mesh filename=package://iai_apartment/meshes/cabinet12/IAICabinet12W60.dae
- added link cabinet12_door_bottom_left; collision mesh filename=package://iai_apartment/meshes/cabinet12/IAIDoorW60H80.obj; visual mesh filename=package://iai_apartment/meshes/cabinet12/IAIDoorW60H80.dae
- added link cabinet12_door_bottom_out_fancy
- added link cabinet12_door_top_left; collision mesh filename=package://iai_apartment/meshes/cabinet12/IAIDoorW60H133.obj; visual mesh filename=package://iai_apartment/meshes/cabinet12/IAIDoorW60H133.dae
- added link cabinet12_door_top_out_fancy
Joints:
- added joint cabinet12_door_bottom_left_joint: type revolute, parent cabinet12_door_bottom_out_fancy, child cabinet12_door_bottom_left, axis 0 0 -1, limit lower=0.0 upper=1.5708 effort=1000.0 velocity=1.5708
- added joint cabinet12_door_bottom_out_joint: type prismatic, parent cabinet12, child cabinet12_door_bottom_out_fancy, origin xyz=0.39 -0.3 -0.5 rpy=0 0 3.14, axis -1 0 0, limit lower=0.0 upper=0.02 effort=1.0 velocity=1.5708, mimic joint=cabinet12_door_bottom_left_joint multiplier=0.01
- added joint cabinet12_door_top_left_joint: type revolute, parent cabinet12_door_top_out_fancy, child cabinet12_door_top_left, axis 0 0 -1, limit lower=0.0 upper=1.5708 effort=1000.0 velocity=1.5708
- added joint cabinet12_door_top_out_joint: type prismatic, parent cabinet12, child cabinet12_door_top_out_fancy, origin xyz=0.39 -0.3 0.5 rpy=0 0 3.14, axis -1 0 0, limit lower=0.0 upper=0.02 effort=1.0 velocity=1.5708, mimic joint=cabinet12_door_top_left_joint multiplier=0.01
- added joint cabinet12_joint: type fixed, parent side_A, child cabinet12, origin xyz=-0.273 -0.5855 1.07
- joint side_A_left_joint: origin xyz=-0.16 -0.296 1.030 rpy=0 0 1.57 -> xyz=-0.16 -0.896 1.030 rpy=0 0 1.57

File: iai_apartment/urdf/kitchen.xacro (robot description, xacro)
@@ -23,5 +23,5 @@
     <link name="side_B" />
     <!-- - - - - - - - - - - - - Cabinets side A - - - - - - - - - -->
-    <!-- Cabinet1 -->
+    <!-- Cabinet 1 -->
     <joint name="cabinet1_joint" type="fixed">
       <origin xyz="0.01 0.01 1.02" />
@@ -222,5 +222,5 @@
       </collision>
     </link>
-    <!-- Cabinet2 -->
+    <!-- Cabinet 2 -->
     <joint name="cabinet2_joint" type="fixed">
       <origin xyz="-0.163 0.51 0.975" />
@@ -328,5 +328,5 @@
       </collision>
     </link>
-    <!-- Cabinet3 -->
+    <!-- Cabinet 3 -->
     <joint name="cabinet3_joint" type="fixed">
       <origin xyz="-0.273 1.022 1.07" />
@@ -438,5 +438,5 @@
       </collision>
     </link>
-    <!-- Cabinet4 -->
+    <!-- Cabinet 4 -->
     <joint name="cabinet4_joint" type="fixed">
       <origin xyz="-0.175 1.825 1.72" />
@@ -516,5 +516,5 @@
       </collision>
     </link>
-    <!-- Cabinet5 -->
+    <!-- Cabinet 5 -->
     <joint name="cabinet5_joint" type="fixed">
       <origin xyz="-0.121 1.625 0.4" />
@@ -648,5 +648,5 @@
       </collision>
     </link>
-    <!-- Cabinet6 -->
+    <!-- Cabinet 6 -->
     <joint name="cabinet6_joint" type="fixed">
       <origin xyz="-0.121 2.127 0.4" />
@@ -777,4 +777,80 @@
         <geometry>
           <mesh filename="package://iai_apartment/meshes/handles/handle_horizontal.obj" />
+        </geometry>
+      </collision>
+    </link>
+    <!-- Cabinet 12 -->
+    <joint name="cabinet12_joint" type="fixed">
+      <origin xyz="-0.273 -0.5855 1.07" />
+      <parent link="side_A" />
+      <child link="cabinet12" />
+    </joint>
+    <link name="cabinet12">
+      <visual>
+        <geometry>
+          <mesh filename="package://iai_apartment/meshes/cabinet12/IAICabinet12W60.dae" />
+        </geometry>
+      </visual>
+      <collision>
+        <geometry>
+          <mesh filename="package://iai_apartment/meshes/cabinet12/IAICabinet12W60.obj" />
+        </geometry>
+      </collision>
+    </link>
+    <joint name="cabinet12_door_top_out_joint" type="prismatic">
+      <origin xyz="0.39 -0.3 0.5" rpy="0 0 3.14" />
+      <parent link="cabinet12" />
+      <child link="cabinet12_door_top_out_fancy" />
+      <axis xyz="-1 0 0" />
+      <limit effort="1.0" lower="0.0" upper="0.02" velocity="1.5708" />
+      <mimic joint="cabinet12_door_top_left_joint" multiplier="0.01" />
+    </joint>
+    <link name="cabinet12_door_top_out_fancy" />
+    <joint name="cabinet12_door_top_left_joint" type="revolute">
+      <parent link="cabinet12_door_top_out_fancy" />
+      <child link="cabinet12_door_top_left" />
+      <axis xyz="0 0 -1" />
+      <limit effort="1000.0" lower="0.0" upper="1.5708" velocity="1.5708" />
+    </joint>
+    <link name="cabinet12_door_top_left">
+      <visual>
+        <origin xyz="0.001 -0.3 -0.1" rpy="0 0 3.14" />
+        <geometry>
+          <mesh filename="package://iai_apartment/meshes/cabinet12/IAIDoorW60H133.dae" />
+        </geometry>
+      </visual>
+      <collision>
+        <origin xyz="0.001 -0.3 -0.1" rpy="0 0 3.14" />
+        <geometry>
+          <mesh filename="package://iai_apartment/meshes/cabinet12/IAIDoorW60H133.obj" />
+        </geometry>
+      </collision>
+    </link>
+    <joint name="cabinet12_door_bottom_out_joint" type="prismatic">
+      <origin xyz="0.39 -0.3 -0.5" rpy="0 0 3.14" />
+      <parent link="cabinet12" />
+      <child link="cabinet12_door_bottom_out_fancy" />
+      <axis xyz="-1 0 0" />
+      <limit effort="1.0" lower="0.0" upper="0.02" velocity="1.5708" />
+      <mimic joint="cabinet12_door_bottom_left_joint" multiplier="0.01" />
+    </joint>
+    <link name="cabinet12_door_bottom_out_fancy" />
+    <joint name="cabinet12_door_bottom_left_joint" type="revolute">
+      <parent link="cabinet12_door_bottom_out_fancy" />
+      <child link="cabinet12_door_bottom_left" />
+      <axis xyz="0 0 -1" />
+      <limit effort="1000.0" lower="0.0" upper="1.5708" velocity="1.5708" />
+    </joint>
+    <link name="cabinet12_door_bottom_left">
+      <visual>
+        <origin xyz="0.001 -0.3 -0.165" rpy="0 0 3.14" />
+        <geometry>
+          <mesh filename="package://iai_apartment/meshes/cabinet12/IAIDoorW60H80.dae" />
+        </geometry>
+      </visual>
+      <collision>
+        <origin xyz="0.001 -0.3 -0.165" rpy="0 0 3.14" />
+        <geometry>
+          <mesh filename="package://iai_apartment/meshes/cabinet12/IAIDoorW60H80.obj" />
         </geometry>
       </collision>
@@ -956,5 +1032,5 @@
       </collision>
     </link>
-    <!-- Cabinet9 -->
+    <!-- Cabinet 9 -->
     <joint name="cabinet9_joint" type="fixed">
       <origin xyz="0.333 1.703 0.394" />
@@ -1610,5 +1686,5 @@
     <!-- side A left panel -->
     <joint name="side_A_left_joint" type="fixed">
-      <origin xyz="-0.16 -0.296 1.030" rpy="0 0 1.57" />
+      <origin xyz="-0.16 -0.896 1.030" rpy="0 0 1.57" />
       <parent link="side_A" />
       <child link="side_A_left" />

Commit message: Adjust joint limit

File: iai_apartment/urdf/apartment.urdf (robot description, URDF)
Before this commit: robot apartment, 117 links, 116 joints
Joints:
- joint cabinet3_door_top_out_joint: limit lower=0.0 upper=0.02 effort=1.0 velocity=1.5708 -> lower=0.0 upper=1.5708 effort=1.0 velocity=1.5708

File: iai_apartment/urdf/kitchen.xacro (robot description, xacro)
@@ -351,5 +351,5 @@
       <child link="cabinet3_door_top_out_fancy" />
       <axis xyz="-1 0 0" />
-      <limit effort="1.0" lower="0.0" upper="0.02" velocity="1.5708" />
+      <limit effort="1.0" lower="0.0" upper="1.5708" velocity="1.5708" />
       <mimic joint="cabinet3_door_top_left_joint" multiplier="0.01" />
     </joint>

Commit message: Change door joint to revolute

File: iai_apartment/urdf/apartment.urdf (robot description, URDF)
Before this commit: robot apartment, 117 links, 116 joints
Joints:
- joint cabinet3_door_top_out_joint: type prismatic -> revolute

File: iai_apartment/urdf/kitchen.xacro (robot description, xacro)
@@ -346,5 +346,5 @@
       </collision>
     </link>
-    <joint name="cabinet3_door_top_out_joint" type="prismatic">
+    <joint name="cabinet3_door_top_out_joint" type="revolute">
       <origin xyz="0.39 -0.3 0.5" rpy="0 0 3.14" />
       <parent link="cabinet3" />

Commit message: added table to apartment lab

File: iai_apartment/urdf/apartment.urdf (robot description, URDF)
Before this commit: robot apartment, 117 links, 116 joints
Links:
- added link table_area_main, mass 1; collision mesh filename=package://iai_apartment/meshes/misc/big_table_1.obj; visual mesh filename=package://iai_apartment/meshes/misc/big_table_1.dae
Joints:
- added joint table_area_main_joint: type fixed, parent apartment_root, child table_area_main, origin xyz=5 4 0 rpy=0 0 1.57
